File: cok-001/cok-001.kicad_sch (KiCad schematic)
At the start: 112 parts, among them J2501 HDMI_A, J3209 ATA Power, J3221 ATA0 for BD, J3301 USB_A_Stacked, J3302 USB_A_Stacked, J3401 Conn_01x22_Pin, U1101 ADT7461A0002RMZR, U1201 Y0_XDR0, U1202 Y0_XDR1, U1301 Y1_XDR0, U1302 Y1_XDR1, U2101 ADT7461A0002RMZR, U2105 TC7WP3125FK, U2108 ICS651MLFT, U2403 L7805, U2407 MM1593DFBEG, U3302 BU9869W, U3802 AS6C1616, U3803 AS6C1616, U6005 NCP511SN33T1G, U6006 NCP511SN18T1, U6009 NCP511SN33T1G, U7301 CXD9208GP

Commit message: new footprints and symbols
Parts:
- removed C2104: 0.01u, Capacitor_SMD:C_0402_1005Metric, symbol Device:C
- added C2102, C2125: XX, Capacitor_SMD:C_0402_1005Metric, symbol Device:C
- added C2109: 8p, Capacitor_SMD:C_0402_1005Metric, symbol Device:C
- added C2112: 9p, Capacitor_SMD:C_0402_1005Metric, symbol Device:C
- added C7347, C7348, C7349, C7350: 0.01u, Capacitor_SMD:C_0402_1005Metric, symbol Device:C
- added C7354: 100p, Capacitor_SMD:C_0402_1005Metric, symbol Device:C
- added Q2401: DTC144E, Package_TO_SOT_SMD:SOT-323_SC-70, symbol Transistor_BJT:DTC144E
- added Q2402: SI2303BDS, Package_TO_SOT_SMD:SOT-23, symbol Transistor_FET:TP0610T
- added R2103, R2104, R2117: 43,2, Resistor_SMD:R_0402_1005Metric, symbol Device:R_US
- added R2107: 0, Resistor_SMD:R_0603_1608Metric, symbol Device:R_US
- added R2109: 39, Resistor_SMD:R_0402_1005Metric, symbol Device:R_US
- added R2408: 150k, Resistor_SMD:R_0402_1005Metric, symbol Device:R_US
- added R7314: 22, Resistor_SMD:R_0402_1005Metric, symbol Device:R_US
- added RN7301, RN7302, RN7303, RN7304, RN7306, RN7307, RN7308, RN7309, RN7311: 56, Resistor_SMD:R_Array_Convex_4x0402, symbol Device:R_Pack04
- added TP7301, TP7302, TP7303, TP7304, TP7305, TP7306, TP7307, TP7308, TP7309, TP7310, TP7311: TestPoint, TestPoint:TestPoint_Pad_1.0x1.0mm, symbol Connector:TestPoint
- added U2402: L7809, Package_TO_SOT_SMD:TO-252-2, symbol Regulator_Linear:L7809
- added U7002, U7003: ~, PS3:BGA-54_7x9_11.8x12.0mm, symbol PS3:K4R271669
- added Y2101: 24.576MHz, Crystal:Crystal_SMD_5032-2Pin_5.0x3.2mm, symbol Device:Crystal
- C2101: value C -> XX
- J2501: footprint (none) -> Connector_FFC-FPC:Hirose_FH12-19S-0.5SH_1x19-1MP_P0.50mm_Horizontal
- J3401: symbol Connector:Conn_01x22_Pin -> PS3:SATA
- R2123: footprint Resistor_SMD:R_0603_1608Metric -> Resistor_SMD:R_0402_1005Metric
Connections:
- net GND: now also C2101.1, J3401.MP (Shield), J3401.P10 (GND), J3401.P11 (Staggered), J3401.P12 (GND), J3401.P4 (GND), J3401.P5 (GND), J3401.P6 (GND), J3401.S1 (GND), J3401.S4 (GND), J3401.S7 (GND), U2102.10 (GND), U2102.15 (GND), U2102.17 (GND), U2102.20 (GND), U2102.22 (GND), U2102.3 (GND), U2102.5 (GND), U2102.8 (GND), U2403.2 (GND), U7301.A1 (TEST_IN_0), U7301.A2 (PLLAVS1), U7301.C11 (Vss), U7301.C12 (Vss), U7301.C3 (TEST_IN_1), U7301.C4 (Vss2), U7301.C5 (Vss2), U7301.D10 (Vss), U7301.D4 (Vss), U7301.D7 (Vss), U7301.E12 (TEST_IN_4), U7301.E4 (Vss2), U7301.E8 (Vss2), U7301.E9 (TEST_IN_3), U7301.F11 (Vss2), U7301.F6 (Vss), U7301.F7 (Vss), U7301.F8 (TEST_IN_2), U7301.G10 (Vss2), U7301.G4 (Vss), U7301.G5 (Vss2), U7301.G6 (Vss), U7301.H10 (Vss), U7301.H5 (TEST_PLL_BP_0), U7301.H6 (Vss2), U7301.J10 (Vss2), U7301.J6 (Vss), U7301.J8 (Vss), U7301.J9 (Vss), U7301.K11 (Vss), U7301.K4 (Vss), U7301.K8 (TEST_PLL_BP_1), U7301.K9 (Vss), U7301.L11 (Vss), U7301.L5 (Vss2), U7301.L6 (Vss), U7301.L7 (Vss2), U7301.L8 (Vss), U7301.M4 (Vss2), U7301.P2 (PLLAVS0), C2102.1, C2109.1, C2112.1, C2125.1, C7347.1, C7348.1, C7349.1, C7350.1, C7354.2, Q2401.2 (E), U2402.2 (GND), U7002.A1 (NC), U7002.A6 (GND), U7002.B3 (GND), U7002.C5 (GND), U7002.D3 (GND), U7002.D5 (GNDA), U7002.E3 (GND), U7002.F5 (GND), U7002.G3 (GND), U7002.H3 (GND), U7002.J6 (GND), U7003.A1 (NC), U7003.A6 (GND), U7003.B3 (GND), U7003.C5 (GND), U7003.D3 (GND), U7003.D5 (GNDA), U7003.E3 (GND), U7003.F5 (GND), U7003.G3 (GND), U7003.H3 (GND), U7003.J6 (GND)
- net RS_MCLK0: now reaches R2181.2, U2108.1 (ICLK)
- net ~{THRRSX_SENS_ALRT}: now reaches U2101.6 (~{ALERT}/~{THERM2})
- net THR_I2C_SDA: now reaches U2101.7 (SDATA)
- net THR_I2C_SCL: now reaches U2101.8 (SCLK)
- net ADAC_MCLK0: now reaches R2179.1, R2181.1
- net RSX_TDN: now reaches R2102.2
- net at U2102.1 (XIN): now also C2109.2, Y2101.1
- net at U2102.14 (VddAud): no longer U2102.23 (VddRef)
- net at U2102.16 (AUDIO): now also R2109.1, R2117.1
- net at U2102.18 (Vdd), U2102.19 (Vdd), U2102.2 (Vdd): now also U2102.7 (Vdd)
- net at U2102.24 (XOUT): now also R2107.2
- net at U2102.4 (54M): now also R2103.2
- net at U2102.9 (53.946M): now also R2104.2
- net at U2105.2 (A1): now also R2117.2
- net at U2403.1 (IN): now also Q2402.3 (D), U2402.1 (IN)
- net RSX_TDP: now reaches R2101.1
- net at U7301.B1 (GPIO33_6): now also TP7307.1
- net at U7301.B2 (GPIO33_5): now also TP7302.1
- net at U7301.B3 (PLLAVD1): now also U7301.D5 (VddC), U7301.D8 (VddC), U7301.E6 (VddC), U7301.F4 (VddC), U7301.G11 (VddC), U7301.G9 (VddC), U7301.H4 (VddC), U7301.H7 (VddC), U7301.J11 (VddC), U7301.J4 (VddC), U7301.K5 (VddC), U7301.L4 (VddC), U7301.N3 (PLLAVD0), C7347.2, C7348.2, C7349.2, C7350.2
- net at U7301.C1 (PCI_AD30): now also RN7301.8 (R1.2)
- net at U7301.C2 (PCI_AD29): now also RN7306.5 (R4.2)
- net at U7301.D1 (PCI_AD26): now also RN7301.6 (R3.2)
- net at U7301.D11 (Vdd): now also U7301.D6 (Vdd), U7301.D9 (Vdd), U7301.E10 (Vdd2), U7301.E11 (Vdd2), U7301.E7 (Vdd), U7301.F10 (Vdd), U7301.G8 (Vdd2), U7301.H11 (Vdd), U7301.H9 (Vdd2), U7301.K10 (Vdd)
- net at U7301.D2 (PCI_AD28): now also RN7301.7 (R2.2)
- net at U7301.D3 (PCI_AD31): now also RN7306.6 (R3.2)
- net at U7301.E1 (PCI_AD25): now also RN7306.8 (R1.2)
- net at U7301.E2 (PCI_AD27): now also RN7306.7 (R2.2)
- net at U7301.E3 (PCI_AD24): now also RN7301.5 (R4.2)
- net at U7301.F1 (PCI_AD20): now also RN7302.7 (R2.2)
- net at U7301.F12 (GPIO15_0): now also TP7306.1
- net at U7301.F2 (PCI_AD22): now also RN7302.8 (R1.2)
- net at U7301.F3 (PCI_AD18): now also RN7302.6 (R3.2)
- net at U7301.G1 (PCI_AD21): now also RN7307.6 (R3.2)
- net at U7301.G12 (GPIO15_1): now also TP7311.1
- net at U7301.G2 (PCI_AD23): now also RN7307.5 (R4.2)
- net at U7301.H1 (PCI_AD15): now also RN7303.8 (R1.2)
- net at U7301.H12 (GPIO15_2): now also TP7305.1
- net at U7301.H2 (PCI_AD16): now also RN7302.5 (R4.2)
- net at U7301.H3 (PCI_AD19): now also RN7307.7 (R2.2)
- net at U7301.J1 (PCI_AD14): now also RN7308.5 (R4.2)
- net at U7301.J12 (GPIO33_0): now also TP7310.1
- net at U7301.J2 (PCI_AD17): now also RN7307.8 (R1.2)
- net at U7301.J3 (PCI_AD6): now also RN7303.7 (R2.2)
- net at U7301.K1 (PCI_AD9): now also RN7303.5 (R4.2)
- net at U7301.K12 (GPIO33_1): now also TP7304.1
- net at U7301.K2 (PCI_AD11): now also RN7303.6 (R3.2)
- net at U7301.K3 (PCI_AD10): now also RN7308.6 (R3.2)
- net at U7301.L1 (PCI_AD3): now also RN7308.8 (R1.2)
- net at U7301.L12 (GPIO33_2): now also TP7309.1
- net at U7301.L2 (PCI_AD7): now also RN7308.7 (R2.2)
- net at U7301.L3 (PCI_AD13): now also RN7304.8 (R1.2)
- net at U7301.M1 (PCI_AD4): now also RN7304.6 (R3.2)
- net at U7301.M10 (~{PCI_RST}): now also R7314.2
- net at U7301.M12 (GPIO33_3): now also TP7303.1
- net at U7301.M2 (PCI_AD2): now also RN7304.7 (R2.2)
- net at U7301.M3 (PCI_AD1): now also RN7309.5 (R4.2)
- net at U7301.N1 (PCI_AD8): now also RN7309.7 (R2.2)
- net at U7301.N12 (GPIO33_4): now also TP7308.1
- net at U7301.N2 (PCI_AD5): now also RN7309.6 (R3.2)
- net at U7301.N7 (~{PCI_CBE2}): now also RN7311.6 (R3.2)
- net at U7301.N8 (~{PCI_GNT}): now also RN7311.8 (R1.2)
- net at U7301.P1 (PCI_AD12): now also RN7309.8 (R1.2)
- net at U7301.P13 (GPIO33_7): now also TP7301.1
- net at U7301.P4 (~{PCI_CBE1}): now also RN7311.5 (R4.2)
- net at U7301.P7 (~{PCI_CBE3}): now also RN7311.7 (R2.2)
- net HDMI_MCLK0: now reaches R2177.1
- new net: Q2402.1 (G), R2408.1
- new net: Q2401.3 (C), R2408.2
- new net: U7002.A2 (VCMOS), U7002.J2 (VCMOS)
- new net: U7002.B5 (VDD), U7002.C3 (VDD), U7002.D6 (VDDA), U7002.E5 (VDD), U7002.F3 (VDD), U7002.G5 (VDD), U7002.H5 (VDD)
- new net: C2112.2, R2107.1, Y2101.2
- new net: C7354.1, R7314.1, RN7304.5 (R4.2)
- new net: J3401.P7 (5Vp), J3401.P8 (5V), J3401.P9 (5V)
- new net: U7003.A2 (VCMOS), U7003.J2 (VCMOS)
- new net: U7003.B5 (VDD), U7003.C3 (VDD), U7003.D6 (VDDA), U7003.E5 (VDD), U7003.F3 (VDD), U7003.G5 (VDD), U7003.H5 (VDD)
- new net RSX_AVCLK0: C2101.2, R2103.1
- new net RSX_AVCLK1: C2102.2, R2104.1
- new net RSX_AVCLK3: C2125.2, R2109.2
Other:
- moved on the sheet: C2103, R2101, R2102, R2123, U2105, U2403

Commit message: flash
Parts:
- added RN2501, RN2502, RN2503: 22, Resistor_SMD:R_Array_Convex_4x0402, symbol Device:R_Pack04
- U3802, U3803: value AS6C1616 -> K9F1G08U0A; symbol Memory_RAM:AS6C1616 -> PS3:K9F1G08
Connections:
- net GND: now also U2502.K3 (GND), U2502.K5 (GND), U2502.K7 (GND), U2502.K9 (GND), U3802.13 (Vss), U3802.36 (Vss), U3803.13 (Vss), U3803.36 (Vss)
- net DQA_A7: now reaches U7002.A7 (DQA7)
- net DQA_A3: now reaches U7002.B1 (DQA3)
- net DQA_A6: now reaches U7002.B2 (DQA6)
- net DQA_A5: now reaches U7002.B6 (DQA5)
- net DQA_A4: now reaches U7002.B7 (DQA4)
- net DQA_A0: now reaches U7002.C1 (DQA0)
- net DQA_A1: now reaches U7002.C2 (DQA1)
- net DQA_A2: now reaches U7002.C6 (DQA2)
- net RQ_A7: now reaches U7002.E2 (RQ7)
- net RQ_A6: now reaches U7002.E6 (RQ6)
- net RQ_A5: now reaches U7002.E7 (RQ5)
- net RQ_A4: now reaches U7002.F1 (RQ4)
- net RQ_A1: now reaches U7002.F2 (RQ1)
- net RQ_A2: now reaches U7002.F6 (RQ2)
- net RQ_A3: now reaches U7002.F7 (RQ3)
- net RQ_A0: now reaches U7002.G1 (RQ0)
- net DQB_A2: now reaches U7002.G2 (DQB2)
- net DQB_A1: now reaches U7002.G6 (DQB1)
- net DQB_A0: now reaches U7002.G7 (DQB0)
- net DQB_A3: now reaches U7002.H1 (DQB3)
- net DQB_A6: now reaches U7002.H2 (DQB6)
- net DQB_A5: now reaches U7002.H6 (DQB5)
- net DQB_A4: now reaches U7002.H7 (DQB4)
- net DQB_A7: now reaches U7002.J7 (DQB7)
- net at U3802.1 (N.C): now also U3802.11 (N.C), U3802.14 (N.C), U3802.2 (N.C), U3802.20 (N.C), U3802.21 (N.C), U3802.23 (N.C), U3802.24 (N.C), U3802.25 (N.C), U3802.26 (N.C), U3802.28 (N.C), U3802.33 (N.C), U3802.35 (N.C), U3802.38 (N.C), U3802.4 (N.C), U3802.40 (N.C), U3802.45 (N.C), U3802.47 (N.C), U3802.48 (N.C), U3802.5 (N.C), U3802.6 (N.C)
- net at U3802.10 (DNU): now also U3802.15 (DNU), U3802.22 (DNU), U3802.27 (DNU), U3802.3 (DNU), U3802.34 (DNU), U3802.39 (DNU), U3802.46 (DNU)
- net SS2_FCLE0: now reaches U3802.16 (CLE)
- net SS2_FALE0: now reaches U3802.17 (ALE)
- net SS2_XFWE0: now reaches U3802.18 (~{WE})
- net SS2_XFWP0: now reaches U3802.19 (~{WP})
- net SS2_FD0_0: now reaches U3802.29 (I/O0)
- net SS2_FD0_1: now reaches U3802.30 (I/O1)
- net SS2_FD0_2: now reaches U3802.31 (I/O2)
- net SS2_FD0_3: now reaches U3802.32 (I/O3)
- net SS2_FD0_4: now reaches U3802.41 (I/O4)
- net SS2_FD0_5: now reaches U3802.42 (I/O5)
- net SS2_FD0_6: now reaches U3802.43 (I/O6)
- net SS2_FD0_7: now reaches U3802.44 (I/O7)
- net SS2_XFRB0: now reaches U3802.7 (R/~{B})
- net SS2_XFRE0: now reaches U3802.8 (~{RE})
- net SS2_XFCE0: now reaches U3802.9 (~{CE})
- net at U3803.1 (N.C): now also U3803.11 (N.C), U3803.14 (N.C), U3803.2 (N.C), U3803.20 (N.C), U3803.21 (N.C), U3803.23 (N.C), U3803.24 (N.C), U3803.25 (N.C), U3803.26 (N.C), U3803.28 (N.C), U3803.33 (N.C), U3803.35 (N.C), U3803.38 (N.C), U3803.4 (N.C), U3803.40 (N.C), U3803.45 (N.C), U3803.47 (N.C), U3803.48 (N.C), U3803.5 (N.C), U3803.6 (N.C)
- net at U3803.10 (DNU): now also U3803.15 (DNU), U3803.22 (DNU), U3803.27 (DNU), U3803.3 (DNU), U3803.34 (DNU), U3803.39 (DNU), U3803.46 (DNU)
- net SS2_FCLE1: now reaches U3803.16 (CLE)
- net SS2_FALE1: now reaches U3803.17 (ALE)
- net SS2_XFWE1: now reaches U3803.18 (~{WE})
- net SS2_XFWP1: now reaches U3803.19 (~{WP})
- net SS2_FD1_0: now reaches U3803.29 (I/O0)
- net SS2_FD1_1: now reaches U3803.30 (I/O1)
- net SS2_FD1_2: now reaches U3803.31 (I/O2)
- net SS2_FD1_3: now reaches U3803.32 (I/O3)
- net SS2_FD1_4: now reaches U3803.41 (I/O4)
- net SS2_FD1_5: now reaches U3803.42 (I/O5)
- net SS2_FD1_6: now reaches U3803.43 (I/O6)
- net SS2_FD1_7: now reaches U3803.44 (I/O7)
- net SS2_XFRB1: now reaches U3803.7 (R/~{B})
- net SS2_XFRE1: now reaches U3803.8 (~{RE})
- net SS2_XFCE1: now reaches U3803.9 (~{CE})
- net at U2502.G1 (SII0_D35): now also RN2501.3 (R3.1)
- net at U2502.H1 (SII0_D34): now also RN2503.3 (R3.1)
- net at U2502.H2 (SII0_D33): now also RN2503.1 (R1.1)
- net at U2502.J1 (SII0_D32): now also RN2501.2 (R2.1)
- net at U2502.J2 (SII0_D31): now also RN2501.4 (R4.1)
- net at U2502.K2 (SII0_D29): now also RN2503.4 (R4.1)
- net at U2502.K4 (SII0_D20): now also RN2502.4 (R4.1)
- net at U2502.L2 (SII0_D27): now also RN2501.1 (R1.1)
- net at U2502.L3 (SII0_D23): now also RN2502.3 (R3.1)
- net at U2502.L4 (SII0_D21): now also RN2503.2 (R2.1)
- net at U2502.L5 (SII0_D18): now also RN2502.1 (R1.1)
- net at U2502.L6 (SII0_D16): now also RN2502.2 (R2.1)
- net DQA_B7: now reaches U7003.A7 (DQA7)
- net DQA_B3: now reaches U7003.B1 (DQA3)
- net DQA_B6: now reaches U7003.B2 (DQA6)
- net DQA_B5: now reaches U7003.B6 (DQA5)
- net DQA_B4: now reaches U7003.B7 (DQA4)
- net DQA_B0: now reaches U7003.C1 (DQA0)
- net DQA_B1: now reaches U7003.C2 (DQA1)
- net DQA_B2: now reaches U7003.C6 (DQA2)
- net RQ_B7: now reaches U7003.E2 (RQ7)
- net RQ_B6: now reaches U7003.E6 (RQ6)
- net RQ_B5: now reaches U7003.E7 (RQ5)
- net RQ_B4: now reaches U7003.F1 (RQ4)
- net RQ_B1: now reaches U7003.F2 (RQ1)
- net RQ_B2: now reaches U7003.F6 (RQ2)
- net RQ_B3: now reaches U7003.F7 (RQ3)
- net RQ_B0: now reaches U7003.G1 (RQ0)
- net DQB_B2: now reaches U7003.G2 (DQB2)
- net DQB_B1: now reaches U7003.G6 (DQB1)
- net DQB_B0: now reaches U7003.G7 (DQB0)
- net DQB_B3: now reaches U7003.H1 (DQB3)
- net DQB_B6: now reaches U7003.H2 (DQB6)
- net DQB_B5: now reaches U7003.H6 (DQB5)
- net DQB_B4: now reaches U7003.H7 (DQB4)
- net DQB_B7: now reaches U7003.J7 (DQB7)
Other:
- moved on the sheet: U7003

Commit message: ncp511 that i ended up scrapping
Parts:
- added C3823, C3824, C3825, C3826: 0.1u, Capacitor_SMD:C_0402_1005Metric, symbol Device:C
- added F6001: Fuse, Fuse:Fuse_1206_3216Metric, symbol Device:Fuse
- added F6002: Fuse, Fuse:Fuse_2920_7451Metric, symbol Device:Fuse
- added R3813, R3815: 0, Resistor_SMD:R_0402_1005Metric, symbol Device:R_US
- added R3840, R3841: 2200, Resistor_SMD:R_0402_1005Metric, symbol Device:R_US
- added U6008, U6011, U6019: NCP511SN18T1, Package_SO:TSOP-5_1.65x3.05mm_P0.95mm, symbol Regulator_Linear:MIC5219-3.3YM5
- added U6013, U6014, U6020, U6021, U6022: ~, Package_SO:SOP-8_3.9x4.9mm_P1.27mm, symbol PS3:MM159X
Connections:
- net GND: now also U6005.2 (GND), U6006.2 (GND), U6009.2 (GND), C3823.2, C3824.2, C3825.2, C3826.2, U6008.2 (GND), U6011.2 (GND), U6013.2 (NC), U6013.3 (GND), U6013.6 (SUB), U6013.7 (SUB), U6014.2 (NC), U6014.3 (GND), U6014.6 (SUB), U6014.7 (SUB), U6019.2 (GND), U6020.2 (NC), U6020.3 (GND), U6020.6 (SUB), U6020.7 (SUB), U6021.2 (NC), U6021.3 (GND), U6021.6 (SUB), U6021.7 (SUB), U6022.2 (NC), U6022.3 (GND), U6022.6 (SUB), U6022.7 (SUB)
- net SS2_XFRB0: now also R3841.1
- net SS2_XFRB1: now also R3840.1
- net SS2_XFWP0: now also R3813.1
- net SS2_XFWP1: now also R3815.1
- net at U6005.1 (IN): now also U6006.1 (IN), U6009.1 (IN)
- net at U3802.12 (Vcc): now also U3802.37 (Vcc), U3803.12 (Vcc), U3803.37 (Vcc), C3823.1, C3824.1, C3825.1, C3826.1, R3813.2, R3815.2, R3840.2, R3841.2
- new net: F6001.1, U6008.1 (IN), U6019.1 (IN)
- new net: U6011.1 (IN), U6013.8 (Vin), U6014.8 (Vin), U6021.8 (Vin)
Other:
- moved on the sheet: U3803, U6005, U6006, U6009

Commit message: starship
Parts:
- added C1, C5070: 0.001u, Capacitor_SMD:C_0402_1005Metric, symbol Device:C
- added C4025, C4026, C4027, C4028: 15p, Capacitor_SMD:C_0402_1005Metric, symbol Device:C
- added C4067: 0.01u, Capacitor_SMD:C_0402_1005Metric, symbol Device:C
- added C4068: 0.1u, Capacitor_SMD:C_0402_1005Metric, symbol Device:C
- added C4069: 4.7u, Capacitor_SMD:C_0402_1005Metric, symbol Device:C
- added C5153: 100p, Capacitor_SMD:C_0402_1005Metric, symbol Device:C
- added D4007, D4008, D4009: RB751, symbol Device:D
- added J4001: Conn_01x03_Pin, symbol Connector:Conn_01x03_Pin
- added J4003: Conn_01x02_Pin, Connector_JST:JST_ZH_B2B-ZR-SM4-TF_1x02-1MP_P1.50mm_Vertical, symbol Connector:Conn_01x02_Pin
- added J4009: Conn_01x30_Socket, Connector_FFC-FPC:TE_3-1734839-0_1x30-1MP_P0.5mm_Horizontal, symbol Connector:Conn_01x30_Socket
- added J4010: Conn_01x10_Socket, symbol Connector:Conn_01x10_Socket
- added Q4014: DTC143ZUA, Package_TO_SOT_SMD:SOT-323_SC-70, symbol Transistor_BJT:DTC144E
- added R1, R7312, R7313: 56, Resistor_SMD:R_0402_1005Metric, symbol Device:R_US
- added R3812, R3814: 0, Resistor_SMD:R_0402_1005Metric, symbol Device:R_US
- added R3830, R3831, R3832, R3833, R3834, R3835, R3836, R3837, R5048, R5070, R5097, R5098, R5183: 10k, Resistor_SMD:R_0402_1005Metric, symbol Device:R_US
- added R4002, R4030, R4031: 33, Resistor_SMD:R_0402_1005Metric, symbol Device:R_US
- added R4003, R4004, R4006, R4007, R4008, R4106: 47, Resistor_SMD:R_0402_1005Metric, symbol Device:R_US
- added R4025, R4026, R4027, R4028, R4043, R4104, R4105: 22, Resistor_SMD:R_0402_1005Metric, symbol Device:R_US
- added R4041: 2200, Resistor_SMD:R_0402_1005Metric, symbol Device:R_US
- added R4042: 1M, Resistor_SMD:R_0402_1005Metric, symbol Device:R_US
- added R4044: 1k, Resistor_SMD:R_0402_1005Metric, symbol Device:R_US
- added R4049, R7302, R7303, R7304, R7305, R7306, R7307, R7308, R7309: 4700, Resistor_SMD:R_0402_1005Metric, symbol Device:R_US
- added R4128: 1k, Resistor_SMD:R_0603_1608Metric, symbol Device:R_US
- added R5072: 270, Resistor_SMD:R_0402_1005Metric, symbol Device:R_US
- added R5103: 330, Resistor_SMD:R_0402_1005Metric, symbol Device:R_US
- added TP40005, TP4001, TP4002, TP4003, TP4004, TP4005, TP4006, TP4007, TP4008, TP4009, TP4016, TP4020, TP4021, TP4022, TP4034, TP4035, TP4036, TP4040, TP4044, TP4046, TP4075, TP4080, TP4081, TP4082, TP4083, TP4089, TP4090, TP4093, TP4096, TP4097, TP4105, TP9401, TP9402: TestPoint, symbol Connector:TestPoint
- added U3801: ~, PS3:Starship2, symbol PS3:CXD43
- added U4002: ~, PS3:SYSCON, symbol PS3:CXR71
- added U5002, U5003: ~, Package_SO:QSOP-28_3.9x9.9mm_P0.635mm, symbol PS3:ICS9218
- added U5004: ~, Package_SO:QSOP-28_3.9x9.9mm_P0.635mm, symbol PS3:ICS9214
- added U5005: ~, Package_SO:VSSOP-8_2.3x2mm_P0.5mm, symbol PS3:TC7WB66FK
- added Y4001: Crystal, Crystal:Crystal_SMD_FOX_FQ7050-2Pin_7.0x5.0mm, symbol Device:Crystal
- added Y4002: Crystal, Crystal:Crystal_SMD_5032-4Pin_5.0x3.2mm, symbol Device:Crystal
- R1106, R1107, R2101, R2102: footprint Resistor_SMD:R_0603_1608Metric -> Resistor_SMD:R_0402_1005Metric
Connections:
- net GND: now also C1.1, C4025.2, C4026.2, C4027.2, C4028.2, C4067.2, C4068.2, C4069.2, C5070.1, C5153.2, J4003.2 (Pin_2), J4009.12 (Pin_12), J4009.29 (Pin_29), J4009.9 (Pin_9), Q4014.2 (E), R3830.2, R3831.2, R3832.2, R3833.2, R3834.2, R3835.2, R3836.2, R3837.2, R5072.1, R5103.1, R5183.1, U3801.D11 (GND), U3801.D4 (GND), U3801.F6 (GND), U3801.F7 (GND), U3801.F8 (GND), U3801.F9 (GND), U3801.G6 (GND), U3801.G7 (GND), U3801.G8 (GND), U3801.G9 (GND), U3801.H2 (GNDP), U3801.H6 (GND), U3801.H7 (GND), U3801.H8 (GND), U3801.H9 (GND), U3801.J6 (GND), U3801.J7 (GND), U3801.J8 (GND), U3801.J9 (GND), U3801.L11 (GND), U3801.L4 (GND), U4002.C15 (VSSep), U4002.E1 (Vss), U4002.G10 (Vss), U4002.G7 (Vss), U4002.G8 (Vss), U4002.L1 (Vss), U4002.R6 (Vss), U4002.T3 (Vss), U4002.T6 (Vss), U5002.16 (GND), U5002.17 (GND), U5002.2 (AGND), U5002.20 (GND), U5002.23 (GND), U5002.26 (GND), U5002.27 (GND), U5002.4 (AGND), U5002.8 (GND), U5003.16 (GND), U5003.17 (GND), U5003.2 (AGND), U5003.20 (GND), U5003.23 (GND), U5003.26 (GND), U5003.27 (GND), U5003.4 (AGND), U5003.8 (GND), U5004.18 (GND), U5004.2 (AGND), U5004.21 (GND), U5004.25 (GND), U5004.4 (AGND), U5004.8 (GND), U5005.4 (GND)
- net SS2_FALE0: now also U3801.L9 (FALE0)
- net SS2_FALE1: now also U3801.L5 (FALE1)
- net SS2_FCLE0: now also U3801.M9 (FCLE0)
- net SS2_FCLE1: now also U3801.M4 (FCLE1)
- net SS2_FD0_0: now also U3801.M14 (FD00)
- net SS2_FD0_1: now also U3801.M13 (FD01)
- net SS2_FD0_2: now also U3801.N13 (FD02)
- net SS2_FD0_3: now also U3801.P13 (FD03)
- net SS2_FD0_4: now also U3801.P12 (FD04)
- net SS2_FD0_5: now also U3801.P11 (FD05)
- net SS2_FD0_6: now also U3801.P10 (FD06)
- net SS2_FD0_7: now also U3801.P9 (FD07)
- net SS2_FD1_0: now also U3801.P7 (FD10)
- net SS2_FD1_1: now also U3801.P6 (FD11)
- net SS2_FD1_2: now also U3801.P5 (FD12)
- net SS2_FD1_3: now also U3801.P4 (FD13)
- net SS2_FD1_4: now also U3801.P3 (FD14)
- net SS2_FD1_5: now also U3801.P2 (FD15)
- net SS2_FD1_6: now also U3801.P1 (FD16)
- net SS2_FD1_7: now also U3801.M2 (FD17)
- net SS2_XFCE0: now also U3801.M8 (XFCE0)
- net SS2_XFCE1: now also U3801.L3 (XFCE1)
- net SS2_XFRB0: now also U3801.M7 (XFRB0)
- net SS2_XFRB1: now also U3801.L2 (XFRB1)
- net SS2_XFRE0: now also U3801.P8 (XFRE0)
- net SS2_XFRE1: now also U3801.M3 (XFRE1)
- net SS2_XFWE0: now also U3801.M10 (XFWE0)
- net SS2_XFWE1: now also U3801.M5 (XFWE1)
- net SS2_XFWP0: now also R3812.2, U3801.M11 (XFWP0); no longer R3813.1, U3802.19 (~{WP})
- net SS2_XFWP1: now also R3814.1, U3801.M6 (XFWP1); no longer R3815.1, U3803.19 (~{WP})
- net SB_PCI_AD25: now reaches RN7306.1 (R1.1)
- net SB_PCI_AD27: now reaches RN7306.2 (R2.1)
- net SB_PCI_AD31: now reaches RN7306.3 (R3.1)
- net SB_PCI_AD29: now reaches RN7306.4 (R4.1)
- net at R2450.2: now also C2456.2; no longer C2456.1
- net ~{SB_PCI_GNT1}: now reaches RN7311.1 (R1.1)
- net ~{SB_PCI_CBE3}: now reaches RN7311.2 (R2.1)
- net ~{SB_PCI_CBE2}: now reaches RN7311.3 (R3.1)
- net ~{SB_PCI_CBE1}: now reaches RN7311.4 (R4.1)
- net SB_PCI_AD22: now reaches RN7302.1 (R1.1)
- net SB_PCI_AD20: now reaches RN7302.2 (R2.1)
- net SB_PCI_AD18: now reaches RN7302.3 (R3.1)
- net SB_PCI_AD16: now reaches RN7302.4 (R4.1)
- net at BZ4001.1 (+): now also Q4014.3 (C), R4128.1
- net at BZ4001.2 (-): now also R4128.2
- net SB_PCI_AD17: now reaches RN7307.1 (R1.1)
- net SB_PCI_AD19: now reaches RN7307.2 (R2.1)
- net SB_PCI_AD21: now reaches RN7307.3 (R3.1)
- net SB_PCI_AD23: now reaches RN7307.4 (R4.1)
- net at RN7307.8 (R1.2), U7301.J2 (PCI_AD17): now also U7301.G3 (PCI_IDSEL)
- net SB_PCI_AD30: now reaches RN7301.1 (R1.1)
- net SB_PCI_AD28: now reaches RN7301.2 (R2.1)
- net SB_PCI_AD26: now reaches RN7301.3 (R3.1)
- net SB_PCI_AD24: now reaches RN7301.4 (R4.1)
- net at U7301.M5 (~{PCI_STOP}): now also R7305.2
- net at U7301.M6 (PCI_PAR): now also R7312.2
- net at U7301.M7 (~{PCI_TADY}): now also R7303.2
- net at U7301.M8 (~{PCI_CBE0}): now also R7313.2
- net at U7301.M9 (~{PCI_FRAME}): now also R7302.2
- net at U7301.N4 (PCI_AD0): now also R1.2
- net at U7301.N5 (~{PCI_SERR}): now also R7308.2
- net at U7301.N6 (~{PCI_DEVSEL}): now also R7306.2
- net at U7301.P5 (~{PCI_PERR}): now also R7307.2
- net at U7301.P6 (~{PCI_IADY}): now also R7304.2
- net at U7301.P8 (~{PCI_REQ}): now also R7309.2
- net SB_PCI_AD15: now reaches RN7303.1 (R1.1)
- net SB_PCI_AD6: now reaches RN7303.2 (R2.1)
- net SB_PCI_AD11: now reaches RN7303.3 (R3.1)
- net SB_PCI_AD9: now reaches RN7303.4 (R4.1)
- net SB_PCI_AD13: now reaches RN7304.1 (R1.1)
- net SB_PCI_AD2: now reaches RN7304.2 (R2.1)
- net SB_PCI_AD4: now reaches RN7304.3 (R3.1)
- net SB_PCI_AD3: now reaches RN7308.1 (R1.1)
- net SB_PCI_AD7: now reaches RN7308.2 (R2.1)
- net SB_PCI_AD10: now reaches RN7308.3 (R3.1)
- net SB_PCI_AD14: now reaches RN7308.4 (R4.1)
- net SB_PCI_AD12: now reaches RN7309.1 (R1.1)
- net SB_PCI_AD8: now reaches RN7309.2 (R2.1)
- net SB_PCI_AD5: now reaches RN7309.3 (R3.1)
- net SB_PCI_AD1: now reaches RN7309.4 (R4.1)
- new net: C4067.1, C4068.1, C4069.1, D4008.1 (K), D4009.1 (K), U4002.F11 (Vddbat)
- new net: R3834.1, U3801.F13 (ID4)
- new net: TP9402.1, U4002.P16 (UART0_TXD)
- new net: TP9401.1, U4002.P15 (UART0_RXD)
- new net: R3837.1, U3801.G14 (ID7)
- new net: R4041.1, R4042.1, U4002.T4 (XTAL)
- new net: C4025.1, R4042.2, U4002.T5 (EXTAL), Y4001.2
- new net: R7302.1, R7303.1, R7304.1, R7305.1, R7306.1, R7307.1, R7308.1, R7309.1
- new net: TP4001.1, U4002.L7 (JNTRST)
- new net: R4026.2, U4002.D1 (SEL0_I2C_SCL)
- new net: J4009.8 (Pin_8), TP4090.1
- new net: R3831.1, U3801.D14 (ID1)
- new net: R4105.1, U4002.A10 (SEL2_I2C_SCL)
- new net: R4004.1, U4002.A8 (SB_SPI_CLK)
- new net: D4009.2 (A), R4044.2, R4049.2, U4002.B1 (AvRef1), U4002.F10 (Vdd3), U4002.F6 (Vdd3), U4002.F7 (AVdd), U4002.F8 (Vdd3), U4002.G11 (VDDep), U4002.H10 (Vdd3), U4002.J6 (Vdd3), U4002.L6 (VddF), U4002.R5 (AVDUO)
- new net: R4104.1, U4002.B10 (SEL2_I2C_SDA)
- new net: TP4093.1, U4002.B11 (PK0)
- new net: C4028.1, U4002.B16 (OSCOUT), Y4002.2
- new net: TP4089.1, U4002.B3 (PJ3)
- new net: R4003.1, U4002.B8 (SB_SPI_DO)
- new net: R4002.1, U4002.B9 (~{SB_SPI_CS})
- new net: R4025.2, U4002.C1 (SEL0_I2C_SDA)
- new net: C4027.1, U4002.C16 (OSCIN), Y4002.1
- new net: U4002.C2 (AvRef2), U4002.G6 (AVss)
- new net: TP4075.1, U4002.D12 (PF2)
- new net: R4043.1, U4002.D15 (32KIN)
- new net: R4043.2, R4044.1, U4002.D16 (32KOUT)
- new net: TP4096.1, U4002.E10 (~{MUL_CHKSTP_OUT})
- new net: TP4046.1, U4002.E13 (PF1)
- new net: U4002.E15 (PP3), U4002.E16 (SKB)
- new net: R4049.1, U4002.F15 (PP0), U4002.F16 (CSB)
- new net: U4002.G15 (PP2), U4002.G16 (DI)
- new net: TP4097.1, U4002.G4 (HDMI_RST1)
- new net: U4002.H15 (PP1), U4002.H16 (DO)
- new net: U4002.H7 (DVdd), U4002.J10 (DVdd), U4002.J7 (DVdd), U4002.K10 (DVdd), U4002.L10 (DVdd), U4002.L11 (DVdd), U4002.R7 (DVdd)
- new net: U4002.J15 (WCB), U4002.K15 (PI6)
- new net: U4002.J16 (RBB), U4002.K16 (PI7)
- new net: U4002.K11 (VssF), U4002.K6 (VssF)
- new net: TP4002.1, U4002.K7 (JTDI)
- new net: TP4005.1, U4002.K8 (JTCK)
- new net: TP4004.1, U4002.K9 (JTDO)
- new net: TP4006.1, U4002.L8 (JRTCK)
- new net: TP4003.1, U4002.L9 (JTMS)
- new net: R4006.1, U4002.M2 (~{BE_SPI_CS})
- new net: TP4044.1, U4002.M8 (FANPWM1)
- new net: Q4014.1 (B), U4002.M9 (BUZZER)
- new net: R4008.1, U4002.N1 (BE_SPI_CLK)
- new net: R4007.1, U4002.N2 (BE_SPI_DO)
- new net: R4106.1, U4002.P2 (~{BE_RESET})
- new net: J4009.17 (Pin_17), U4002.R10 (RMC_IN)
- new net: R4027.2, U4002.R15 (SEL1_I2C_SDA)
- new net: R4028.2, U4002.R16 (SEL1_I2C_SCL)
- new net: TP4020.1, U4002.R9 (PQ1)
- new net: TP4021.1, U4002.T10 (PQ4)
- new net: TP4022.1, U4002.T11 (PQ5)
- new net: TP4040.1, U4002.T7 (XXTAL0)
- new net: R4031.2, U4002.T8 (SEL2_I2C_SCL)
- new net: R4030.2, U4002.T9 (SEL2_I2C_SDA)
- new net: R3830.1, U3801.D13 (ID0)
- new net: R3832.1, U3801.E13 (ID2)
- new net: R3833.1, U3801.E14 (ID3)
- new net: R3835.1, U3801.F14 (ID5)
- new net: R3836.1, U3801.G13 (ID6)
- new net: C4026.1, R4041.2, Y4001.1
- new net: R3812.1, R3813.1, U3802.19 (~{WP})
- new net: J4009.7 (Pin_7), TP4009.1
- new net: R3814.2, R3815.1, U3803.19 (~{WP})
- new net: R5072.2, U5003.3 (ISET)
- new net: C5070.2, R5097.2, R5098.2, U5004.7 (VDD2.5)
- new net: J4009.10 (Pin_10), TP4080.1
- new net: C1.2, R5048.1, R5070.1, U5003.7 (VDD2.5)
- new net: J4009.13 (Pin_13), TP4082.1
- new net: R5070.2, U5003.14 (~{BYPASS})
- new net: J4009.6 (Pin_6), TP4034.1
- new net: J4009.4 (Pin_4), TP4036.1
- new net: J4009.11 (Pin_11), TP4081.1
- new net: J4009.14 (Pin_14), TP4083.1
- new net: J4009.16 (Pin_16), TP4105.1
- new net: J4009.2 (Pin_2), TP4007.1
- new net: J4009.3 (Pin_3), TP4008.1
- new net: J4009.5 (Pin_5), TP4035.1
- new net: R5183.2, U5004.12 (ID0)
- new net: R5097.1, U5004.13 (ID1)
- new net: R5098.1, U5004.14 (~{BYPASS})
- new net: D4007.1 (K), D4008.2 (A)
- new net: D4007.2 (A), J4003.1 (Pin_1), TP40005.1
- new net: R5103.2, U5004.3 (ISET)
- new net DISC_IN_MECHA: U4002.F5 (DISC_IN_MECHA)
- new net EJECT_MECHA: U4002.E4 (EJECT_MECHA)
- new net HDMI_I2C_SCL: R4028.1
- new net HDMI_I2C_SDA: R4027.1
- new net MK_I2C_SCL: R4026.1, U5005.5 (A2)
- new net MK_I2C_SDA: R4025.1, U5005.1 (A1)
- new net SB_PCI_AD0: R1.1
- new net SB_PCI_PAR: R7312.1
- new net SW_AVCG: TP4016.1, U4002.G5 (PO5)
- new net XCG_EN: C5153.1, R5048.2, U5002.11 (EN), U5003.11 (EN), U5004.11 (EN)
- new net XCG_I2C_SCL: U5002.9 (SCL), U5003.9 (SCL), U5004.9 (SCL), U5005.6 (B2)
- new net XCG_I2C_SDA: U5002.10 (SDA), U5003.10 (SDA), U5004.10 (SDA), U5005.2 (B1)
- new net XDR_RQ_RST: U4002.D4 (~{XDR_FET_RST})
- new net ~{HDMI0_RST}: U4002.F4 (HDMI_RST0)
- new net ~{SB_PCI_CBE0}: R7313.1
- no-connect marks 5 -> 30
Other:
- moved on the sheet: BZ4001, C2456, C3823, C3824, C3825, C3826, C6116, C6117, C6118, C6217, C6218, C7354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
