File: cok-001/cok-001.kicad_sch (KiCad schematic)
At the start: 220 parts, among them J3209 ATA Power, J3221 ATA0 for BD, J3301 USB_A_Stacked, J3302 USB_A_Stacked, J3401 Conn_01x22_Pin, J4001 Conn_01x03_Pin, J4003 Conn_01x02_Pin, J4009 Conn_01x30_Socket, J4010 Conn_01x10_Socket, Q2401 DTC144E, Q2402 SI2303BDS, Q4014 DTC143ZUA, U2101 ADT7461A0002RMZR, U2105 TC7WP3125FK, U2108 ICS651MLFT, U2402 L7809, U2403 L7805, U2407 MM1593DFBEG, U3302 BU9869W, U6005 NCP511SN33T1G, U6006 NCP511SN18T1, U6008 NCP511SN18T1, U6009 NCP511SN33T1G, U6011 NCP511SN18T1, U6019 NCP511SN18T1, Y2101 24.576MHz, Y4001 Crystal, Y4002 Crystal

Commit message: wip eegs
Parts:
- removed RN7001, RN7002, RN7003, RN7004, RN7005, RN7006: R_Pack08, Resistor_SMD:R_Cat16-8, symbol Device:R_Pack08
- removed U7002, U7003: ~, PS3:BGA-54_7x9_11.8x12.0mm, symbol PS3:K4R271669
- TP9401, TP9402: footprint TestPoint:TestPoint_Pad_1.0x1.0mm -> TestPoint:TestPoint_Pad_D1.5mm
Connections:
- net at U4002.B16 (OSCOUT): now also C4028.1, Y4002.2
- net at U4002.C16 (OSCIN): now also C4027.1, Y4002.1
Other:
- added sheet PS2 EEGS (eegs.kicad_sch)

Commit message: eegs dc
Parts:
- added F6302: 5A, Fuse:Fuse_1206_3216Metric, symbol Device:Fuse
- added L6302: 1uH, Inductor_SMD:L_TDK_SLF6028, symbol Device:L
Connections:
- net at U4002.B16 (OSCOUT): now also C4028.1, Y4002.2
- net at U4002.C16 (OSCIN): now also C4027.1, Y4002.1
- new net: F6302.2, L6302.1
Other:
- added sheet DC-DC Converters (dcdc.kicad_sch)
Changed lines of the file:
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@@
 	(wire
 		(pts
+			(xy 982.98 24.13) (xy 990.6 24.13)
+		)
+		(stroke
+			(width 0)
+			(type default)
+		)
+	)
+	(wire
+		(pts
 			(xy 1010.92 171.45) (xy 1000.76 171.45)
 		)
@@
 	)
 	(symbol
+		(lib_id "Device:Fuse")
+		(at 979.17 24.13 90)
+		(unit 1)
+		(exclude_from_sim no)
+		(in_bom yes)
+		(on_board yes)
+		(dnp no)
+		(fields_autoplaced yes)
+		(property "Reference" "F6302"
+			(at 979.17 17.78 90)
+			(effects
+				(font
+					(size 1.27 1.27)
+				)
+			)
+		)
+		(property "Value" "5A"
+			(at 979.17 20.32 90)
+			(effects
+				(font
+					(size 1.27 1.27)
+				)
+			)
+		)
+		(property "Footprint" "Fuse:Fuse_1206_3216Metric"
+			(at 979.17 25.908 90)
+			(effects
+				(font
+					(size 1.27 1.27)
+				)
+				(hide yes)
+			)
+		)
+		(property "Datasheet" "~"
+			(at 979.17 24.13 0)
+			(effects
+				(font
+					(size 1.27 1.27)
+				)
+				(hide yes)
+			)
+		)
+		(property "Description" "Fuse"
+			(at 979.17 24.13 0)
+			(effects
+				(font
+					(size 1.27 1.27)
+				)
+				(hide yes)
+			)
+		)
+		(pin "2"
+		)
+		(pin "1"
+		)
+		(instances
+			(project ""
+				(path "/976eb78d-8215-4cc0-9d72-f9d535c7970b"
+					(reference "F6302")
+					(unit 1)
+				)
+			)
+		)
+	)
+	(symbol
 		(lib_id "Device:C")
 		(at 148.59 397.51 0)
@@
 	)
 	(symbol
+		(lib_id "Device:L")
+		(at 994.41 24.13 90)
+		(unit 1)
+		(exclude_from_sim no)
+		(in_bom yes)
+		(on_board yes)
+		(dnp no)
+		(fields_autoplaced yes)
+		(property "Reference" "L6302"
+			(at 994.41 19.05 90)
+			(effects
+				(font
+					(size 1.27 1.27)
+				)
+			)
+		)
+		(property "Value" "1uH"
+			(at 994.41 21.59 90)
+			(effects
+				(font
+					(size 1.27 1.27)
+				)
+			)
+		)
+		(property "Footprint" "Inductor_SMD:L_TDK_SLF6028"
+			(at 994.41 24.13 0)
+			(effects
+				(font
+					(size 1.27 1.27)
+				)
+				(hide yes)
+			)
+		)
+		(property "Datasheet" "~"
+			(at 994.41 24.13 0)
+			(effects
+				(font
+					(size 1.27 1.27)
+				)
+				(hide yes)
+			)
+		)
+		(property "Description" "Inductor"
+			(at 994.41 24.13 0)
+			(effects
+				(font
+					(size 1.27 1.27)
+				)
+				(hide yes)
+			)
+		)
+		(pin "1"
+		)
+		(pin "2"
+		)
+		(instances
+			(project ""
+				(path "/976eb78d-8215-4cc0-9d72-f9d535c7970b"
+					(reference "L6302")
+					(unit 1)
+				)
+			)
+		)
+	)
+	(symbol
 		(lib_id "Connector:TestPoint")
 		(at 247.65 114.3 0)
@@
 				)
 			)
+		)
+	)
+	(sheet
+		(at 209.55 13.97)
+		(size 24.13 15.24)
+		(fields_autoplaced yes)
+		(stroke
+			(width 0.1524)
+			(type solid)
+		)
+		(fill
+			(color 0 0 0 0.0000)
+		)
+		(property "Sheetname" "DC-DC Converters"
+			(at 209.55 13.2584 0)
+			(effects
+				(font
+					(size 1.27 1.27)
+				)
+				(justify left bottom)
+			)
+		)
+		(property "Sheetfile" "dcdc.kicad_sch"
+			(at 209.55 29.7946 0)
+			(effects
+				(font
+					(size 1.27 1.27)
+				)
+				(justify left top)
+			)
+		)
+		(instances
+			(project "cok-001"
+				(path "/976eb78d-8215-4cc0-9d72-f9d535c7970b"
+					(page "63")
+				)
+			)

Commit message: add some stupid n channel mosfet
Parts:
- removed BZ4001: Buzzer, Buzzer_Beeper:Buzzer_TDK_PS1240P02BT_D12.2mm_H6.5mm, symbol Device:Buzzer
- removed C4025, C4026, C4027, C4028: 15p, Capacitor_SMD:C_0402_1005Metric, symbol Device:C
- removed C4067: 0.01u, Capacitor_SMD:C_0402_1005Metric, symbol Device:C
- removed C4068: 0.1u, Capacitor_SMD:C_0402_1005Metric, symbol Device:C
- removed C4069: 4.7u, Capacitor_SMD:C_0402_1005Metric, symbol Device:C
- removed D4007, D4008, D4009: RB751, Diode_SMD:D_SOD-923, symbol Device:D
- removed F6001: Fuse, Fuse:Fuse_1206_3216Metric, symbol Device:Fuse
- removed F6002: Fuse, Fuse:Fuse_2920_7451Metric, symbol Device:Fuse
- removed J4001: Conn_01x03_Pin, symbol Connector:Conn_01x03_Pin
- removed J4003: Conn_01x02_Pin, Connector_JST:JST_ZH_B2B-ZR-SM4-TF_1x02-1MP_P1.50mm_Vertical, symbol Connector:Conn_01x02_Pin
- removed J4009: Conn_01x30_Socket, Connector_FFC-FPC:TE_3-1734839-0_1x30-1MP_P0.5mm_Horizontal, symbol Connector:Conn_01x30_Socket
- removed J4010: Conn_01x10_Socket, symbol Connector:Conn_01x10_Socket
- removed Q4014: DTC143ZUA, Package_TO_SOT_SMD:SOT-323_SC-70, symbol Transistor_BJT:DTC144E
- removed R4002, R4030, R4031: 33, Resistor_SMD:R_0402_1005Metric, symbol Device:R_US
- removed R4003, R4004, R4006, R4007, R4008, R4106: 47, Resistor_SMD:R_0402_1005Metric, symbol Device:R_US
- removed R4025, R4026, R4027, R4028, R4043, R4104, R4105: 22, Resistor_SMD:R_0402_1005Metric, symbol Device:R_US
- removed R4041: 2200, Resistor_SMD:R_0402_1005Metric, symbol Device:R_US
- removed R4042: 1M, Resistor_SMD:R_0402_1005Metric, symbol Device:R_US
- removed R4044: 1k, Resistor_SMD:R_0402_1005Metric, symbol Device:R_US
- removed R4049: 4700, Resistor_SMD:R_0402_1005Metric, symbol Device:R_US
- removed R4128: 1k, Resistor_SMD:R_0603_1608Metric, symbol Device:R_US
- removed TP40005, TP4001, TP4002, TP4003, TP4004, TP4005, TP4006, TP4007, TP4008, TP4009, TP4016, TP4020, TP4021, TP4022, TP4034, TP4035, TP4036, TP4040, TP4044, TP4046, TP4075, TP4080, TP4081, TP4082, TP4083, TP4089, TP4090, TP4093, TP4096, TP4097, TP4105: TestPoint, TestPoint:TestPoint_Pad_1.0x1.0mm, symbol Connector:TestPoint
- removed TP9401, TP9402: TestPoint, TestPoint:TestPoint_Pad_D1.5mm, symbol Connector:TestPoint
- removed U4002: ~, PS3:SYSCON, symbol PS3:CXR71
- removed U6008, U6011, U6019: NCP511SN18T1, Package_SO:TSOP-5_1.65x3.05mm_P0.95mm, symbol Regulator_Linear:MIC5219-3.3YM5
- removed U6013, U6014, U6020, U6021, U6022: ~, Package_SO:SOP-8_3.9x4.9mm_P1.27mm, symbol PS3:MM159X
- removed Y4001: Crystal, Crystal:Crystal_SMD_FOX_FQ7050-2Pin_7.0x5.0mm, symbol Device:Crystal
- removed Y4002: Crystal, Crystal:Crystal_SMD_5032-4Pin_5.0x3.2mm, symbol Device:Crystal
- added H10, H11, H7, H8, H9: MountingHole_Pad, MountingHole:MountingHole_4.3mm_M4_Pad_Via, symbol Mechanical:MountingHole_Pad
- added H12: MountingHole_Pad, MountingHole:MountingHole_4.3x6.2mm_M4_Pad_Via, symbol Mechanical:MountingHole_Pad
- H1, H2, H3, H4, H5, H6: footprint MountingHole:MountingHole_4.3mm_M4_DIN965_Pad -> MountingHole:MountingHole_4.3mm_M4_Pad_Via
Connections:
- net GND: now also H10.1, H11.1, H12.1, H7.1, H8.1, H9.1
- no-connect marks 19 -> 10
Other:
- added sheet Ethernet (ethernet.kicad_sch)
- added sheet Power Management (powermgmt.kicad_sch)
- added sheet Syscon (syscon.kicad_sch)
- moved on the sheet: C3246, C3247, C6116, C6117, C6118, C6217, C6218, J3209, R3297

Commit message: ethernet
Parts:
- L3301, L3302, L3401, L3402: value L_Iron_Coupled_Small -> L_Iron_Coupled_Small_1243
Changed lines of the file:
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@@
 		(dnp no)
 		(property "Reference" "L3401"
-			(at 915.67 694.69 0)
+			(at 915.67 704.215 0)
 			(effects
 				(font
@@
 			)
 		)
-		(property "Value" "L_Iron_Coupled_Small"
-			(at 915.67 697.23 0)
+		(property "Value" "L_Iron_Coupled_Small_1243"
+			(at 915.67 697.865 0)
 			(effects
 				(font
@@
 			)
 		)
-		(property "Value" "L_Iron_Coupled_Small"
+		(property "Value" "L_Iron_Coupled_Small_1243"
 			(at 915.67 704.85 0)
 			(effects
@@
 		(dnp no)
 		(property "Reference" "L3301"
-			(at 236.22 67.31 0)
+			(at 236.22 57.785 0)
 			(effects
 				(font
@@
 			)
 		)
-		(property "Value" "L_Iron_Coupled_Small"
-			(at 236.22 64.77 0)
+		(property "Value" "L_Iron_Coupled_Small_1243"
+			(at 236.22 64.135 0)
 			(effects
 				(font
@@
 		(dnp no)
 		(property "Reference" "L3302"
-			(at 236.22 72.39 0)
+			(at 236.22 62.865 0)
 			(effects
 				(font
@@
 			)
 		)
-		(property "Value" "L_Iron_Coupled_Small"
-			(at 236.22 69.85 0)
+		(property "Value" "L_Iron_Coupled_Small_1243"
+			(at 236.22 69.215 0)
 			(effects
 				(font

Commit message: av
Parts:
- removed C2451: 470p 50V, Resistor_SMD:R_0402_1005Metric, symbol Device:C
- removed C2453, C2455: 220u 4V, Capacitor_SMD:CP_Elec_6.3x4.5, symbol Device:C_Polarized_US
- removed C2454, C2457, C2458: 1000u 4V, Capacitor_SMD:CP_Elec_8x6.9, symbol Device:C_Polarized_US
- removed C2456: 0.1u 16V, Capacitor_SMD:C_0603_1608Metric, symbol Device:C
- removed Q2401: DTC144E, Package_TO_SOT_SMD:SOT-323_SC-70, symbol Transistor_BJT:DTC144E
- removed Q2402: SI2303BDS, Package_TO_SOT_SMD:SOT-23, symbol Transistor_FET:TP0610T
- removed R2408: 150k, Resistor_SMD:R_0402_1005Metric, symbol Device:R_US
- removed R2447, R2448, R2449, R2450, R2451, R2452: 75, Resistor_SMD:R_0603_1608Metric, symbol Device:R_US
- removed U2402: L7809, Package_TO_SOT_SMD:TO-252-2, symbol Regulator_Linear:L7809
- removed U2403: L7805, Package_TO_SOT_SMD:TO-252-2, symbol Regulator_Linear:L7805
- removed U2406: ~, Package_QFP:TQFP-100_14x14mm_P0.5mm, symbol PS3:CXM4024
- removed U2407: MM1593DFBEG, Package_SO:SOP-8_3.9x4.9mm_P1.27mm, symbol PS3:MM159X
Connections:
- net HDMI_MCLK0 renamed HDMI_MCLKO0
Other:
- added sheet AV Out (av.kicad_sch)

Commit message: row c and d
Other:
- added sheet Shouthbridge (southbridge.kicad_sch)
Changed lines of the file:
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@@
+	)
+	(sheet
+		(at 364.49 13.97)
+		(size 22.86 15.24)
+		(fields_autoplaced yes)
+		(stroke
+			(width 0.1524)
+			(type solid)
+		)
+		(fill
+			(color 0 0 0 0.0000)
+		)
+		(property "Sheetname" "Shouthbridge"
+			(at 364.49 13.2584 0)
+			(effects
+				(font
+					(size 1.27 1.27)
+				)
+				(justify left bottom)
+			)
+		)
+		(property "Sheetfile" "southbridge.kicad_sch"
+			(at 364.49 29.7946 0)
+			(effects
+				(font
+					(size 1.27 1.27)
+				)
+				(justify left top)
+			)
+		)
+		(instances
+			(project "cok-001"
+				(path "/976eb78d-8215-4cc0-9d72-f9d535c7970b"
+					(page "13")
+				)
+			)
+		)
 	)
 	(sheet

Commit message: sata
Parts:
- removed C3412, C3413, C3414, C3415: 0.01u, Capacitor_SMD:C_0402_1005Metric, symbol Device:C
- removed J3401: Conn_01x22_Pin, PS3:SATA, symbol PS3:SATA
- removed L3401, L3402: L_Iron_Coupled_Small_1243, Inductor_SMD:L_CommonModeChoke_Coilcraft_0805USB, symbol Device:L_Iron_Coupled_Small_1243
- removed U3401: ~, Package_QFP:LQFP-64_10x10mm_P0.5mm, symbol PS3:88SA8040C0
- C2271: footprint Resistor_SMD:R_0402_1005Metric -> Capacitor_SMD:C_0402_1005Metric
- renumbered C1 to C5064
Other:
- added sheet SATA (sata.kicad_sch)

Commit message: southbridge
Parts:
- removed C3301, C3309, C3311, C3313, C3314, C3316, C3328: 0.1u, Capacitor_SMD:C_0402_1005Metric, symbol Device:C
- removed J3301, J3302: USB_A_Stacked, PS3:USB_A_Vertical, symbol Connector:USB_A_Stacked
- removed L3301, L3302: L_Iron_Coupled_Small_1243, Inductor_SMD:L_CommonModeChoke_Coilcraft_0805USB, symbol Device:L_Iron_Coupled_Small_1243
- removed R3328, R3329: 0, Resistor_SMD:R_0603_1608Metric, symbol Device:R_US
- removed R3360, R3361, R3362, R3363, R3364, R3365, R3366, R3367: 0, Resistor_SMD:R_0402_1005Metric, symbol Device:R_US
- removed TP9505, TP9506, TP9507, TP9508, TP9509, TP9510, TP9511, TP9512, TP9520, TP9522, TP9527, TP9529: TestPoint, TestPoint:TestPoint_Pad_1.0x1.0mm, symbol Connector:TestPoint
- removed U3302: BU9869W, Package_SO:SSOP-8_2.95x2.8mm_P0.65mm, symbol Memory_EEPROM:93CxxA
- removed U3303, U3304: ~, Package_SO:SOIC-8_3.9x4.9mm_P1.27mm, symbol PS3:BD6517F
- removed U3305: ~, Package_QFP:LQFP-64_10x10mm_P0.5mm, symbol PS3:GL852
- U6005, U6006, U6009: footprint Package_SO:TSOP-5_1.65x3.05mm_P0.95mm -> Package_TO_SOT_SMD:SOT-23-5
Connections:
- no-connect marks 10 -> 3
Other:
- added sheet USB (usb.kicad_sch)
