File: cok-001/cok-001.kicad_sch (KiCad schematic)
At the start: 72 parts, among them J3209 ATA Power, J3221 ATA0 for BD, U2101 ADT7461A0002RMZR, U2105 TC7WP3125FK, U2108 ICS651MLFT, U6005 NCP511SN33T1G, U6006 NCP511SN18T1, U6009 NCP511SN33T1G, Y2101 24.576MHz

Commit message: L
Other:
- sheet Shouthbridge renamed Southbridge
Changed lines of the file:
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@@
 			(color 0 0 0 0.0000)
 		)
-		(property "Sheetname" "Shouthbridge"
+		(property "Sheetname" "Southbridge"
 			(at 364.49 13.2584 0)
 			(effects
@@
 			(project "cok-001"
 				(path "/976eb78d-8215-4cc0-9d72-f9d535c7970b"
-					(page "13")
+					(page "30")
 				)
 			)

Commit message: seperate out
Parts:
- removed C2101, C2102, C2125: XX, Capacitor_SMD:C_0402_1005Metric, symbol Device:C
- removed C2103: 0.001u 50V, Capacitor_SMD:C_0402_1005Metric, symbol Device:C
- removed C2108: 0.1u 10V, Capacitor_SMD:C_0402_1005Metric, symbol Device:C
- removed C2109: 8p, Capacitor_SMD:C_0402_1005Metric, symbol Device:C
- removed C2112: 9p, Capacitor_SMD:C_0402_1005Metric, symbol Device:C
- removed C2271: 0.01u 25V, Capacitor_SMD:C_0402_1005Metric, symbol Device:C
- removed C2272: 100p, Capacitor_SMD:C_0402_1005Metric, symbol Device:C
- removed C3246: 47u 25V, Capacitor_Tantalum_SMD:CP_EIA-3528-15_AVX-H, symbol Device:C_Polarized_US
- removed C3247: 47u 25V, Capacitor_Tantalum_SMD:CP_EIA-7132-28_AVX-C, symbol Device:C_Polarized_US
- removed D3208: LED_Dual_AAKK, Package_TO_SOT_SMD:SC-82AA, symbol Device:LED_Dual_AAKK
- removed F6302: 5A, Fuse:Fuse_1206_3216Metric, symbol Device:Fuse
- removed J3209: ATA Power, Connector_JST:JST_PH_B4B-PH-SM4-TB_1x04-1MP_P2.00mm_Vertical, symbol Connector:Conn_01x04_Socket
- removed J3221: ATA0 for BD, PS3:Hirose_FH12-60S, symbol Connector:Conn_01x60_Pin
- removed L6302: 1uH, Inductor_SMD:L_TDK_SLF6028, symbol Device:L
- removed R2101, R2102: 100, Resistor_SMD:R_0402_1005Metric, symbol Device:R_US
- removed R2103, R2104, R2117: 43,2, Resistor_SMD:R_0402_1005Metric, symbol Device:R_US
- removed R2106: 10k, Resistor_SMD:R_0402_1005Metric, symbol Device:R_US
- removed R2107: 0, Resistor_SMD:R_0603_1608Metric, symbol Device:R_US
- removed R2109: 39, Resistor_SMD:R_0402_1005Metric, symbol Device:R_US
- removed R2123, R2177, R2179: 33, Resistor_SMD:R_0402_1005Metric, symbol Device:R_US
- removed R2181: R, Resistor_SMD:R_0402_1005Metric, symbol Device:R_US
- removed R3211, R3225, R3226, R3227: 0, Resistor_SMD:R_0402_1005Metric, symbol Device:R_US
- removed R3297: 0, Resistor_SMD:R_0805_2012Metric, symbol Device:R_US
- removed U2101: ADT7461A0002RMZR, Package_SO:MSOP-8_3x3mm_P0.65mm, symbol PS3:ADT7461A
- removed U2102: ~, Package_SO:SSOP-24_3.9x8.7mm_P0.635mm, symbol PS3:ICS422A
- removed U2105: TC7WP3125FK, Package_SO:VSSOP-8_2.3x2mm_P0.5mm, symbol PS3:TC7WP3125FK
- removed U2108: ICS651MLFT, Package_SO:SOIC-8_3.9x4.9mm_P1.27mm, symbol PS3:ICS651
- removed Y2101: 24.576MHz, Crystal:Crystal_SMD_5032-2Pin_5.0x3.2mm, symbol Device:Crystal
Connections:
- no-connect marks 3 -> 0
Other:
- added sheet External (external.kicad_sch)
- added sheet RSX Setting (rsxsetting.kicad_sch)
- added sheet SB MISC (sbmisc.kicad_sch)
- added sheet VRM for RSX (rsxvrm.kicad_sch)
- moved on the sheet: C5064, C5070, C5153, C6116, C6117, C6118, C6217, C6218, H1, H10, H11, H12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

Commit message: update to 9
Changed lines of the file:
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@@
 (kicad_sch
-	(version 20231120)
+	(version 20250114)
 	(generator "eeschema")
-	(generator_version "8.0")
+	(generator_version "9.0")
 	(paper "A4")
 	(junction
@@
 		(at 363.22 15.24)
 		(size 25.4 15.24)
+		(exclude_from_sim no)
+		(in_bom yes)
+		(on_board yes)
+		(dnp no)
 		(fields_autoplaced yes)
 		(stroke
@@
 		(at 76.2 15.24)
 		(size 25.4 15.24)
+		(exclude_from_sim no)
+		(in_bom yes)
+		(on_board yes)
+		(dnp no)
 		(fields_autoplaced yes)
 		(stroke
@@
 		(at 15.24 38.1)
 		(size 22.86 15.24)
+		(exclude_from_sim no)
+		(in_bom yes)
+		(on_board yes)
+		(dnp no)
 		(fields_autoplaced yes)
 		(stroke
@@
 		(at 332.74 15.24)
 		(size 25.4 15.24)
+		(exclude_from_sim no)
+		(in_bom yes)
+		(on_board yes)
+		(dnp no)
 		(fields_autoplaced yes)
 		(stroke
@@
 		(at 302.26 38.1)
 		(size 27.94 15.24)
+		(exclude_from_sim no)
+		(in_bom yes)
+		(on_board yes)
+		(dnp no)
 		(fields_autoplaced yes)
 		(stroke
@@
 		(at 110.49 15.24)
 		(size 26.67 15.24)
+		(exclude_from_sim no)
+		(in_bom yes)
+		(on_board yes)
+		(dnp no)
 		(fields_autoplaced yes)
 		(stroke
@@
 		(at 144.78 15.24)
 		(size 25.4 15.24)
+		(exclude_from_sim no)
+		(in_bom yes)
+		(on_board yes)
+		(dnp no)
 		(fields_autoplaced yes)
 		(stroke
@@
 		(at 209.55 15.24)
 		(size 24.13 15.24)
+		(exclude_from_sim no)
+		(in_bom yes)
+		(on_board yes)
+		(dnp no)
 		(fields_autoplaced yes)
 		(stroke
@@
 		(at 177.8 15.24)
 		(size 25.4 15.24)
+		(exclude_from_sim no)
+		(in_bom yes)
+		(on_board yes)
+		(dnp no)
 		(fields_autoplaced yes)
 		(stroke
@@
 		(at 419.1 15.24)
 		(size 25.4 15.24)
+		(exclude_from_sim no)
+		(in_bom yes)
+		(on_board yes)
+		(dnp no)
 		(fields_autoplaced yes)
 		(stroke
@@
 		(at 269.24 15.24)
 		(size 25.4 15.24)
+		(exclude_from_sim no)
+		(in_bom yes)
+		(on_board yes)
+		(dnp no)
 		(fields_autoplaced yes)
 		(stroke
@@
 		(at 238.76 15.24)
 		(size 25.4 15.24)
+		(exclude_from_sim no)
+		(in_bom yes)
+		(on_board yes)
+		(dnp no)
 		(fields_autoplaced yes)
 		(stroke
@@
 		(at 45.72 15.24)
 		(size 22.86 15.24)
+		(exclude_from_sim no)
+		(in_bom yes)
+		(on_board yes)
+		(dnp no)
 		(fields_autoplaced yes)
 		(stroke
@@
 		(at 302.26 15.24)
 		(size 25.4 15.24)
+		(exclude_from_sim no)
+		(in_bom yes)
+		(on_board yes)
+		(dnp no)
 		(fields_autoplaced yes)
 		(stroke
@@
 		(at 332.74 38.1)
 		(size 25.4 15.24)
+		(exclude_from_sim no)
+		(in_bom yes)
+		(on_board yes)
+		(dnp no)
 		(fields_autoplaced yes)
 		(stroke
@@
 		(at 15.24 15.24)
 		(size 22.86 15.24)
+		(exclude_from_sim no)
+		(in_bom yes)
+		(on_board yes)
+		(dnp no)
 		(fields_autoplaced yes)
 		(stroke
@@
 		(at 363.22 38.1)
 		(size 25.4 15.24)
+		(exclude_from_sim no)
+		(in_bom yes)
+		(on_board yes)
+		(dnp no)
 		(fields_autoplaced yes)
 		(stroke
@@
 		(at 391.16 15.24)
 		(size 25.4 15.24)
+		(exclude_from_sim no)
+		(in_bom yes)
+		(on_board yes)
+		(dnp no)
 		(fields_autoplaced yes)
 		(stroke
@@
 		)
 	)
+	(embedded_fonts no)
 )

Commit message: another ics
Parts:
- removed C5064, C5070: 0.001u, Capacitor_SMD:C_0402_1005Metric, symbol Device:C
- removed C5153: 100p, Capacitor_SMD:C_0402_1005Metric, symbol Device:C
- removed R5048, R5070, R5097, R5098, R5183: 10k, Resistor_SMD:R_0402_1005Metric, symbol Device:R_US
- removed R5072: 270, Resistor_SMD:R_0402_1005Metric, symbol Device:R_US
- removed R5103: 330, Resistor_SMD:R_0402_1005Metric, symbol Device:R_US
- removed U5002, U5003: ~, Package_SO:QSOP-28_3.9x9.9mm_P0.635mm, symbol PS3:ICS9218
- removed U5004: ~, Package_SO:QSOP-28_3.9x9.9mm_P0.635mm, symbol PS3:ICS9214
Other:
- added sheet XCG Clock (xcgclock.kicad_sch)

Commit message: footprints
Parts:
- removed U5005: ~, Package_SO:VSSOP-8_2.3x2mm_P0.5mm, symbol PS3:TC7WB66FK
Changed lines of the file:
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@@
-		)
-	)
-	(global_label "XCG_I2C_SCL"
-		(shape output)
-		(at 53.34 149.86 0)
-		(fields_autoplaced yes)
-		(effects
-			(font
-				(size 1.27 1.27)
-			)
-			(justify left)
-		)
-		(property "Intersheetrefs" "${INTERSHEET_REFS}"
-			(at 68.6018 149.86 0)
-			(effects
-				(font
-					(size 1.27 1.27)
-				)
-				(justify left)
-				(hide yes)
-			)
-		)
-	)
-	(global_label "MK_I2C_SCL"
-		(shape output)
-		(at 53.34 152.4 0)
-		(fields_autoplaced yes)
-		(effects
-			(font
-				(size 1.27 1.27)
-			)
-			(justify left)
-		)
-		(property "Intersheetrefs" "${INTERSHEET_REFS}"
-			(at 67.5737 152.4 0)
-			(effects
-				(font
-					(size 1.27 1.27)
-				)
-				(justify left)
-				(hide yes)
-			)
-		)
-	)
-	(global_label "XCG_I2C_SDA"
-		(shape output)
-		(at 38.1 147.32 180)
-		(fields_autoplaced yes)
-		(effects
-			(font
-				(size 1.27 1.27)
-			)
-			(justify right)
-		)
-		(property "Intersheetrefs" "${INTERSHEET_REFS}"
-			(at 22.7777 147.32 0)
-			(effects
-				(font
-					(size 1.27 1.27)
-				)
-				(justify right)
-				(hide yes)
-			)
-		)
-	)
-	(global_label "MK_I2C_SDA"
-		(shape output)
-		(at 38.1 144.78 180)
-		(fields_autoplaced yes)
-		(effects
-			(font
-				(size 1.27 1.27)
-			)
-			(justify right)
-		)
-		(property "Intersheetrefs" "${INTERSHEET_REFS}"
-			(at 23.8058 144.78 0)
-			(effects
-				(font
-					(size 1.27 1.27)
-				)
-				(justify right)
-				(hide yes)
-			)
 		)
 	)
@@
 	)
 	(symbol
-		(lib_id "power:GND")
-		(at 38.1 152.4 0)
-		(unit 1)
-		(exclude_from_sim no)
-		(in_bom yes)
-		(on_board yes)
-		(dnp no)
-		(fields_autoplaced yes)
-		(property "Reference" "#PWR0140"
-			(at 38.1 158.75 0)
-			(effects
-				(font
-					(size 1.27 1.27)
-				)
-				(hide yes)
-			)
-		)
-		(property "Value" "GND"
-			(at 38.1 157.48 0)
-			(effects
-				(font
-					(size 1.27 1.27)
-				)
-			)
-		)
-		(property "Footprint" ""
-			(at 38.1 152.4 0)
-			(effects
-				(font
-					(size 1.27 1.27)
-				)
-				(hide yes)
-			)
-		)
-		(property "Datasheet" ""
-			(at 38.1 152.4 0)
-			(effects
-				(font
-					(size 1.27 1.27)
-				)
-				(hide yes)
-			)
-		)
-		(property "Description" "Power symbol creates a global label with name \"GND\" , ground"
-			(at 38.1 152.4 0)
-			(effects
-				(font
-					(size 1.27 1.27)
-				)
-				(hide yes)
-			)
-		)
-		(pin "1"
-		)
-		(instances
-			(project "cok-001"
-				(path "/976eb78d-8215-4cc0-9d72-f9d535c7970b"
-					(reference "#PWR0140")
-					(unit 1)
-				)
-			)
-		)
-	)
-	(symbol
 		(lib_id "Regulator_Linear:MIC5219-3.3YM5")
 		(at 306.07 177.8 0)
@@
 				(path "/976eb78d-8215-4cc0-9d72-f9d535c7970b"
 					(reference "#PWR0178")
-					(unit 1)
-				)
-			)
-		)
-	)
-	(symbol
-		(lib_id "PS3:TC7WB66FK")
-		(at 45.72 142.24 0)
-		(unit 1)
-		(exclude_from_sim no)
-		(in_bom yes)
-		(on_board yes)
-		(dnp no)
-		(fields_autoplaced yes)
-		(property "Reference" "U5005"
-			(at 45.72 139.7 0)
-			(effects
-				(font
-					(size 1.27 1.27)
-				)
-			)
-		)
-		(property "Value" "~"
-			(at 45.72 142.24 0)
-			(effects
-				(font
-					(size 1.27 1.27)
-				)
-			)
-		)
-		(property "Footprint" "Package_SO:VSSOP-8_2.3x2mm_P0.5mm"
-			(at 45.72 142.24 0)
-			(effects
-				(font
-					(size 1.27 1.27)
-				)
-				(hide yes)
-			)
-		)
-		(property "Datasheet" ""
-			(at 45.72 142.24 0)
-			(effects
-				(font
-					(size 1.27 1.27)
-				)
-				(hide yes)
-			)
-		)
-		(property "Description" ""
-			(at 45.72 142.24 0)
-			(effects
-				(font
-					(size 1.27 1.27)
-				)
-				(hide yes)
-			)
-		)
-		(pin "3"
-		)
-		(pin "2"
-		)
-		(pin "1"
-		)
-		(pin "7"
-		)
-		(pin "4"
-		)
-		(pin "5"
-		)
-		(pin "6"
-		)
-		(pin "8"
-		)
-		(instances
-			(project ""
-				(path "/976eb78d-8215-4cc0-9d72-f9d535c7970b"
-					(reference "U5005")
 					(unit 1)
 				)
@@
 			(project "cok-001"
 				(path "/976eb78d-8215-4cc0-9d72-f9d535c7970b"
-					(page "20")
-				)
-			)
+					(page "50")
+				)
+			)

Commit message: cpu file
Other:
- added sheet CPU (cpu.kicad_sch)
Changed lines of the file:
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@@
+	)
+	(sheet
+		(at 76.2 38.1)
+		(size 25.4 15.24)
+		(exclude_from_sim no)
+		(in_bom yes)
+		(on_board yes)
+		(dnp no)
+		(fields_autoplaced yes)
+		(stroke
+			(width 0.1524)
+			(type solid)
+		)
+		(fill
+			(color 0 0 0 0.0000)
+		)
+		(property "Sheetname" "CPU"
+			(at 76.2 37.3884 0)
+			(effects
+				(font
+					(size 1.27 1.27)
+				)
+				(justify left bottom)
+			)
+		)
+		(property "Sheetfile" "cpu.kicad_sch"
+			(at 76.2 53.9246 0)
+			(effects
+				(font
+					(size 1.27 1.27)
+				)
+				(justify left top)
+			)
+		)
+		(instances
+			(project "cok-001"
+				(path "/976eb78d-8215-4cc0-9d72-f9d535c7970b"
+					(page "10")
+				)
+			)
+		)
 	)
 	(sheet

Commit message: new sheets
Other:
- added sheet Wireless Board (wireless.kicad_sch)
Changed lines of the file:
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@@
 			(project "cok-001"
 				(path "/976eb78d-8215-4cc0-9d72-f9d535c7970b"
-					(page "18")
-				)
-			)
-		)
-	)
-	(sheet
-		(at 110.49 15.24)
-		(size 26.67 15.24)
+					(page "62")
+				)
+			)
+		)
+	)
+	(sheet
+		(at 109.22 15.24)
+		(size 27.94 15.24)
 		(exclude_from_sim no)
 		(in_bom yes)
@@
 		)
 		(property "Sheetname" "Starship2"
-			(at 110.49 14.5284 0)
+			(at 109.22 14.5284 0)
 			(effects
 				(font
@@
 		)
 		(property "Sheetfile" "starship.kicad_sch"
-			(at 110.49 31.0646 0)
+			(at 109.22 31.0646 0)
 			(effects
 				(font
@@
 				)
 			)
+		)
+	)
+	(sheet
+		(at 109.22 38.1)
+		(size 27.94 15.24)
+		(exclude_from_sim no)
+		(in_bom yes)
+		(on_board yes)
+		(dnp no)
+		(fields_autoplaced yes)
+		(stroke
+			(width 0.1524)
+			(type solid)
+		)
+		(fill
+			(color 0 0 0 0.0000)
+		)
+		(property "Sheetname" "Wireless Board"
+			(at 109.22 37.3884 0)
+			(effects
+				(font
+					(size 1.27 1.27)
+				)
+				(justify left bottom)
+			)
+		)
+		(property "Sheetfile" "wireless.kicad_sch"
+			(at 109.22 53.9246 0)
+			(effects
+				(font
+					(size 1.27 1.27)
+				)
+				(justify left top)
+			)
+		)
+		(instances
+			(project "cok-001"
+				(path "/976eb78d-8215-4cc0-9d72-f9d535c7970b"
+					(page "37")
+				)
+			)

Commit message: power
Other:
- added sheet VRM for BE (bevrm.kicad_sch)
Changed lines of the file:
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@@
+	)
+	(sheet
+		(at 144.78 38.1)
+		(size 25.4 15.24)
+		(exclude_from_sim no)
+		(in_bom yes)
+		(on_board yes)
+		(dnp no)
+		(fields_autoplaced yes)
+		(stroke
+			(width 0.1524)
+			(type solid)
+		)
+		(fill
+			(color 0 0 0 0.0000)
+		)
+		(property "Sheetname" "VRM for BE"
+			(at 144.78 37.3884 0)
+			(effects
+				(font
+					(size 1.27 1.27)
+				)
+				(justify left bottom)
+			)
+		)
+		(property "Sheetfile" "bevrm.kicad_sch"
+			(at 144.78 53.9246 0)
+			(effects
+				(font
+					(size 1.27 1.27)
+				)
+				(justify left top)
+			)
+		)
+		(instances
+			(project "cok-001"
+				(path "/976eb78d-8215-4cc0-9d72-f9d535c7970b"
+					(page "61")
+				)
+			)
+		)
 	)
 	(sheet
