File: cok-001/southbridge.kicad_sch (KiCad schematic)
At the start: 1 part, among them U3001 CXD29

Commit message: southbridge
Parts:
- removed U3001: CXD29, PS3:SouthBridge, symbol PS3:CXD29
- added TP3001, TP3004, TP3008, TP3009, TP3010, TP3011: TestPoint, TestPoint:TestPoint_Pad_1.0x1.0mm, symbol Connector:TestPoint
- added U3001: CXD2973GB, PS3:SouthBridge, symbol PS3:CXD2973GB
Connections:
- new net: TP3010.1, U3001.D3 (PIO2)
- new net: U3001.F17 (VDD33), U3001.F18 (VDD33)
- new net: U3001.F21 (VDD33), U3001.F22 (VDD33)
- new net: U3001.F30 (VA), U3001.F31 (VA)
- new net: U3001.F33 (DDRDQ4), U3001.F34 (DDRDQ0), U3001.F35 (VDD18), U3001.F36 (DDRDQ5), U3001.F37 (DDRVREF)
- new net: U3001.B25 (VA), U3001.B27 (VA), U3001.B29 (VA), U3001.B31 (VA)
- new net: U3001.A25 (VA), U3001.A27 (VA), U3001.A29 (VA), U3001.A31 (VA)
- new net: TP3004.1, U3001.A5 (~{SIORTSZ0})
- new net: TP3001.1, U3001.C5 (~{SIOCTSZ0})
- new net: TP3008.1, U3001.D31 (USB0DA)
- new net: TP3009.1, U3001.C31 (USB0DP)
- new net: U3001.D33 (VDD18), U3001.D34 (VDD18), U3001.D35 (VDD18), U3001.D36 (VDD18), U3001.D37 (VDD18)
- new net: TP3011.1, U3001.D4 (PIO1)
- new net: U3001.E10 (VDD33), U3001.E11 (VDD33)
- new net: U3001.E19 (ATA0CLK), U3001.E20 (ATA1CLK)
- new net: U3001.E38 (VDD18), U3001.E39 (VDD18)
- new net GND: U3001.A1 (GND), U3001.A2 (GND), U3001.A33 (GND), U3001.A35 (GND), U3001.A37 (GND), U3001.A38 (GND), U3001.B1 (GND), U3001.B2 (GND), U3001.B33 (GND), U3001.B35 (GND), U3001.B37 (GND), U3001.B38 (GND), U3001.B39 (GND), U3001.C26 (GA), U3001.C28 (GA), U3001.C30 (GA), U3001.C32 (GA), U3001.C33 (GND), U3001.C34 (GND), U3001.C35 (GND), U3001.C36 (GND), U3001.C37 (GND), U3001.C38 (GND), U3001.C39 (GND), U3001.D26 (GA), U3001.D28 (GA), U3001.D30 (GA), U3001.D32 (GA), U3001.D9 (GND), U3001.E12 (GND), U3001.E13 (GND), U3001.E32 (GND), U3001.E33 (GND), U3001.E34 (GND), U3001.E35 (GND), U3001.E36 (GND), U3001.E37 (GND), U3001.E6 (GND), U3001.E8 (GND), U3001.E9 (GND), U3001.F15 (GND), U3001.F16 (GND), U3001.F19 (GND), U3001.F20 (GND), U3001.F23 (GND), U3001.F24 (GND), U3001.F25 (GA), U3001.F26 (GA), U3001.F27 (GA), U3001.F28 (GA), U3001.F29 (GA), U3001.F32 (GND), U3001.F6 (GND)
- new net SB_ATA1_DD0: U3001.C14 (ATA1DD0)
- new net SB_ATA1_DD1: U3001.A15 (ATA1DD1)
- new net SB_ATA1_DD10: U3001.D17 (ATA1DD10)
- new net SB_ATA1_DD11: U3001.B17 (ATA1DD11)
- new net SB_ATA1_DD12: U3001.D16 (ATA1DD12)
- new net SB_ATA1_DD13: U3001.D15 (ATA1DD13)
- new net SB_ATA1_DD14: U3001.B15 (ATA1DD14)
- new net SB_ATA1_DD15: U3001.D14 (ATA1DD15)
- new net SB_ATA1_DD2: U3001.C15 (ATA1DD2)
- new net SB_ATA1_DD3: U3001.C16 (ATA1DD3)
- new net SB_ATA1_DD4: U3001.A17 (ATA1DD4)
- new net SB_ATA1_DD5: U3001.C17 (ATA1DD5)
- new net SB_ATA1_DD6: U3001.C18 (ATA1DD6)
- new net SB_ATA1_DD7: U3001.A19 (ATA1DD7)
- new net SB_ATA1_DD8: U3001.B19 (ATA1DD8)
- new net SB_ATA1_DD9: U3001.D18 (ATA1DD9)
- new net SB_USB1_DM: U3001.D29 (USB1DM)
- new net SB_USB1_DP: U3001.C29 (USB1DP)
- new net SB_USB2_DM: U3001.D27 (USB2DM)
- new net SB_USB2_DP: U3001.C27 (USB2DP)
- new net SB_USB3_DM: U3001.D25 (USB3DM)
- new net SB_USB3_DP: U3001.C25 (USB3DP)

Commit message: L
Parts:
- added unit 11 of U3001
- added unit 13 of U3001
- added unit 10 of U3001
- added unit 14 of U3001
- added unit 12 of U3001
Connections:
- new net SB_EBUS_ADDR0: U3001.J4 (EBUSADDR0)
- new net SB_EBUS_ADDR1: U3001.J1 (EBUSADDR1)
- new net SB_EBUS_ADDR17: U3001.L3 (EBUSADDR17)
- new net SB_EBUS_ADDR2: U3001.J2 (EBUSADDR2)
- new net SB_EBUS_ADDR3: U3001.J3 (EBUSADDR3)
- new net SB_EBUS_ADDR4: U3001.K3 (EBUSADDR4)
- new net SB_EBUS_ADDR5: U3001.K4 (EBUSADDR5)
- new net SB_EBUS_ADDR6: U3001.L1 (EBUSADDR6)
- new net SB_EBUS_ADDR7: U3001.L2 (EBUSADDR7)

Commit message: aj
Parts:
- added TP3005: TestPoint, TestPoint:TestPoint_Pad_1.0x1.0mm, symbol Connector:TestPoint
- added unit 34 of U3001
- added unit 36 of U3001
- added unit 28 of U3001
- added unit 23 of U3001
- added unit 32 of U3001
- added unit 25 of U3001
- added unit 29 of U3001
- added unit 22 of U3001
- added unit 27 of U3001
- added unit 21 of U3001
- added unit 20 of U3001
- added unit 31 of U3001
- added unit 18 of U3001
- added unit 33 of U3001
- added unit 30 of U3001
- added unit 16 of U3001
Connections:
- net GND: now also U3001.G25 (GA), U3001.G26 (GA), U3001.G27 (GA), U3001.G28 (GND), U3001.G32 (GND), U3001.G38 (GND), U3001.G39 (GND), U3001.H10 (GND), U3001.H11 (GND), U3001.H19 (GND), U3001.H35 (GND), U3001.J10 (GND), U3001.J11 (GND), U3001.J12 (GND), U3001.J13 (GND), U3001.J14 (GND), U3001.J15 (GND), U3001.J23 (GA), U3001.J24 (GA), U3001.J25 (GA), U3001.J26 (GA), U3001.J27 (GA), U3001.J28 (GA), U3001.J29 (GA), U3001.J30 (GA), U3001.J31 (GA), U3001.J35 (GND), U3001.J6 (GND), U3001.J9 (GND), U3001.K31 (GND), U3001.K32 (GND), U3001.K6 (GND), U3001.K8 (TESTIN6), U3001.K9 (GND), U3001.L11 (GND), U3001.L12 (GND), U3001.L13 (GND), U3001.L14 (GND), U3001.L15 (GND), U3001.L23 (GA), U3001.L24 (GA), U3001.L25 (GA), U3001.L26 (GA), U3001.L27 (GA), U3001.L28 (GA), U3001.L29 (GA), U3001.L30 (GA), U3001.L31 (GND), U3001.L32 (GND), U3001.L38 (GND), U3001.L39 (GND), U3001.L8 (TESTIN5), U3001.M11 (GND), U3001.M31 (GND), U3001.M35 (GND), U3001.M8 (TESTIN4), U3001.N13 (GND), U3001.N14 (GND), U3001.N16 (GND), U3001.N18 (GND), U3001.N20 (GND), U3001.N22 (GND), U3001.N24 (GND), U3001.N26 (GND), U3001.N28 (GND), U3001.N29 (GND), U3001.N31 (GND), U3001.N35 (GND), U3001.N6 (GND), U3001.AA13 (GND), U3001.AA14 (GND), U3001.AA16 (GND), U3001.AA18 (GND), U3001.AA20 (GND), U3001.AA22 (GND), U3001.AA24 (GND), U3001.AA26 (GND), U3001.AA28 (GND), U3001.AA29 (GND), U3001.AA31 (GND), U3001.AA35 (GND), U3001.AA6 (GND), U3001.AB11 (GND), U3001.AB13 (GND), U3001.AB15 (GND), U3001.AB17 (GND), U3001.AB19 (GND), U3001.AB21 (GND), U3001.AB23 (GND), U3001.AB25 (GND), U3001.AB27 (GND), U3001.AB29 (GND), U3001.AB31 (GND), U3001.AB32 (GND), U3001.AB6 (GND), U3001.AB9 (GND), U3001.AC1 (GND), U3001.AC11 (GND), U3001.AC14 (GND), U3001.AC16 (GND), U3001.AC18 (GND), U3001.AC2 (GND), U3001.AC20 (GND), U3001.AC22 (GND), U3001.AC24 (GND), U3001.AC26 (GND), U3001.AC28 (GND), U3001.AC29 (GND), U3001.AC3 (GND), U3001.AC31 (GND), U3001.AC32 (GND), U3001.AC38 (GND), U3001.AC39 (GND), U3001.AC4 (GND), U3001.AC5 (GND), U3001.AC6 (GND), U3001.AC7 (GND), U3001.AC8 (GND), U3001.AC9 (GND), U3001.AD11 (GND), U3001.AD15 (GND), U3001.AD17 (GND), U3001.AD19 (GND), U3001.AD21 (GND), U3001.AD23 (GND), U3001.AD25 (GND), U3001.AD27 (GND), U3001.AD29 (GND), U3001.AD31 (GND), U3001.AD35 (GND), U3001.AD8 (GND), U3001.AD9 (GND), U3001.AE11 (GND), U3001.AE14 (GND), U3001.AE16 (GND), U3001.AE18 (GND), U3001.AE20 (GND), U3001.AE22 (GND), U3001.AE24 (GND), U3001.AE26 (GND), U3001.AE28 (GND), U3001.AE29 (GND), U3001.AE31 (GND), U3001.AE35 (GND), U3001.AE8 (GND), U3001.AE9 (GND), U3001.AF10 (GND), U3001.AF15 (GND), U3001.AF17 (GND), U3001.AF19 (GND), U3001.AF21 (GND), U3001.AF23 (GND), U3001.AF25 (GND), U3001.AF27 (GND), U3001.AF29 (GND), U3001.AF31 (GND), U3001.AF32 (GND), U3001.AF5 (GND), U3001.AF9 (GND), U3001.AG10 (GND), U3001.AG14 (GND), U3001.AG16 (GND), U3001.AG18 (GND), U3001.AG20 (GND), U3001.AG22 (GND), U3001.AG24 (GND), U3001.AG26 (GND), U3001.AG28 (GND), U3001.AG29 (GND), U3001.AG31 (GND), U3001.AG32 (GND), U3001.AG38 (GND), U3001.AG39 (GND), U3001.AG5 (GND), U3001.AG9 (GND), U3001.AH29 (GND), U3001.AH31 (GND), U3001.AH35 (GND), U3001.AH8 (GND), U3001.AH9 (GND), U3001.AJ17 (GND), U3001.AJ18 (GND), U3001.AJ19 (GND), U3001.AJ20 (GND), U3001.AJ21 (GND), U3001.AJ27 (GND), U3001.AJ28 (GND), U3001.AJ29 (GND), U3001.AJ31 (GND), U3001.AJ35 (GND), U3001.AJ8 (GND), U3001.AJ9 (GND), U3001.P15 (GND), U3001.P17 (GND), U3001.P19 (GND), U3001.P21 (GND), U3001.P23 (GND), U3001.P25 (GND), U3001.P27 (GND), U3001.P29 (GND), U3001.P31 (GND), U3001.P32 (GND), U3001.P6 (GND), U3001.R14 (GND), U3001.R16 (GND), U3001.R18 (GND), U3001.R20 (GND), U3001.R22 (GND), U3001.R24 (GND), U3001.R26 (GND), U3001.R28 (GND), U3001.R29 (GND), U3001.R31 (GND), U3001.R32 (GND), U3001.R38 (GND), U3001.R39 (GND), U3001.T13 (GND), U3001.T15 (GND), U3001.T17 (GND), U3001.T19 (GND), U3001.T21 (GND), U3001.T23 (GND), U3001.T25 (GND), U3001.T27 (GND), U3001.T29 (GND), U3001.T31 (GND), U3001.T35 (GND), U3001.U13 (GND), U3001.U14 (GND), U3001.U16 (GND), U3001.U18 (GND), U3001.U20 (GND), U3001.U22 (GND), U3001.U24 (GND), U3001.U26 (GND), U3001.U28 (GND), U3001.U29 (GND), U3001.U31 (GND), U3001.U35 (GND), U3001.U6 (GND), U3001.V15 (GND), U3001.V17 (GND), U3001.V19 (GND), U3001.V21 (GND), U3001.V23 (GND), U3001.V25 (GND), U3001.V27 (GND), U3001.V29 (GND), U3001.V31 (GND), U3001.V32 (GND), U3001.V6 (GND), U3001.W14 (GND), U3001.W16 (GND), U3001.W18 (GND), U3001.W20 (GND), U3001.W22 (GND), U3001.W24 (GND), U3001.W26 (GND), U3001.W28 (GND), U3001.W29 (GND), U3001.W31 (GND), U3001.W32 (GND), U3001.W38 (GND), U3001.W39 (GND), U3001.Y13 (GND), U3001.Y15 (GND), U3001.Y17 (GND), U3001.Y19 (GND), U3001.Y21 (GND), U3001.Y23 (GND), U3001.Y25 (GND), U3001.Y27 (GND), U3001.Y29 (GND), U3001.Y31 (GND), U3001.Y35 (GND)
- net SB_EBUS_ADDR10: now also U3001.R1 (EBUSADDR10)
- net SB_EBUS_ADDR11: now also U3001.R2 (EBUSADDR11)
- net SB_EBUS_ADDR12: now also U3001.R3 (EBUSADDR12)
- net SB_EBUS_ADDR13: now also U3001.R4 (EBUSADDR13)
- net SB_EBUS_ADDR14: now also U3001.T3 (EBUSADDR14)
- net SB_EBUS_ADDR15: now also U3001.T4 (EBUSADDR15)
- net SB_EBUS_ADDR16: now also U3001.U4 (EBUSADDR16)
- net SB_EBUS_ADDR8: now also U3001.P3 (EBUSADDR8)
- net SB_EBUS_ADDR9: now also U3001.P4 (EBUSADDR9)
- net +3.3V_SB_VDDIO: now reaches U3001.K10 (VDD33)
- net +3.3V_SB_VDDIO: now also U3001.E10 (VDD33), U3001.E11 (VDD33), U3001.F14 (VDD33), U3001.F17 (VDD33), U3001.F18 (VDD33), U3001.F21 (VDD33), U3001.F22 (VDD33), U3001.G29 (VDD33), U3001.G6 (VDD33), U3001.H12 (VDD33), U3001.H13 (VDD33), U3001.H14 (VDD33), U3001.H28 (VDD33), U3001.H6 (VDD33), U3001.H8 (VDD33), U3001.H9 (VDD33), U3001.K11 (VDD33), U3001.K12 (VDD33), U3001.K13 (VDD33), U3001.K14 (VDD33), U3001.K15 (VDD33), U3001.K16 (TSB13), U3001.L10 (VDD33), U3001.L6 (VDD33), U3001.M12 (VDD33), U3001.M13 (VDD33), U3001.M14 (VDD33), U3001.M15 (VDD33), U3001.M6 (VDD33), U3001.AB10 (VDD33), U3001.AB12 (VDD33), U3001.AH27 (VDD33), U3001.AH28 (VDD33), U3001.P13 (VDD33), U3001.R13 (VDD33), U3001.R6 (VDD33), U3001.T6 (VDD33), U3001.V13 (VDD33), U3001.W13 (VDD33), U3001.W6 (VDD33), U3001.Y6 (VDD33)
- net at U3001.K23 (VA): now also U3001.K24 (VA), U3001.K25 (VA), U3001.K26 (VA), U3001.K27 (VA), U3001.K28 (VA), U3001.K29 (VA), U3001.K30 (VA)
- net SB_GBE_TXD4: now reaches U3001.F10 (GBETXD4)
- net SB_GBE_TXD2: now reaches U3001.F11 (GBETXD2)
- net SB_GBE_TXD0: now reaches U3001.F12 (GBETXD0)
- net SB_GBE_TXD6: now reaches U3001.F9 (GBETXD6)
- net SB_GBE_TXD5: now reaches U3001.G10 (GBETXD5)
- net SB_GBE_TXD3: now reaches U3001.G11 (GBETXD3)
- net SB_GBE_TXD1: now reaches U3001.G12 (GBETXD1)
- net SB_GBE_TXD7: now reaches U3001.G9 (GBETXD7)
- net SB_GBE_RXD4: now reaches U3001.B11 (GBERXD4)
- net SB_GBE_TXCLK: now reaches U3001.B13 (GBETX_CLK)
- net SB_ATA0_DD13: now reaches U3001.B21 (ATA0DD13)
- net SB_ATA0_DD10: now reaches U3001.B23 (ATA0DD10)
- net SB_SIO0_TXD: now reaches U3001.B5 (SIOTXD0)
- net SB_GBE_PHYINT: now reaches U3001.B7 (GBEPHY_INT)
- net SB_GBE_CRS: now reaches U3001.B9 (GBECRS)
- net SB_GBE_RXD3: now reaches U3001.A11 (GBERXD3)
- net SB_GBE_MDIO: now reaches U3001.A13 (GBEMDIO)
- net SB_ATA0_DD2: now reaches U3001.A21 (ATA0DD2)
- net SB_ATA0_DD5: now reaches U3001.A23 (ATA0DD5)
- net SB_GBE_CLK: now reaches U3001.A7 (GBECLK)
- net SB_GBE_RXER: now reaches U3001.A9 (GBERX_ER)
- net at U3001.M23 (VA): now also U3001.M24 (VA), U3001.M25 (VA), U3001.M26 (VA), U3001.M27 (VA), U3001.M28 (VA), U3001.M29 (VA)
- net ~{SB_EBUS_SWE}: now reaches U3001.M4 (~{EBUSSWEZ})
- net SB_EBUS_DATA0: now reaches U3001.M5 (EBUSDATA0)
- net SB_EBUS_DATA8: now reaches U3001.M7 (EBUSDATA8)
- net SB_ATA1_DA1: now reaches U3001.H15 (ATA1DA1)
- net SB_ATA1_INTRQ: now reaches U3001.H16 (ATA1INTRQ)
- net ~{SB_ATA1_DIOW}: now reaches U3001.H17 (~{ATA1DIOW})
- net ~{SB_ATA1_RESET}: now reaches U3001.H18 (~{ATA1RESET})
- net ~{SB_ATA0_CS0}: now reaches U3001.H20 (~{ATA0CS0})
- net SB_ATA0_DA1: now reaches U3001.H21 (ATA0DA1)
- net SB_ATA0_INTRQ: now reaches U3001.H22 (ATA0INTRQ)
- net ~{SB_ATA0_DIOW}: now reaches U3001.H23 (~{ATA0DIOW})
- net ~{SB_ATA0_RESET}: now reaches U3001.H24 (~{ATA0RESET})
- net SB_USB_CLK: now reaches U3001.H27 (USBCLK)
- net ~{SB_EBUS_CE0}: now reaches U3001.H5 (~{EBUSCEZ0})
- net at U3001.H7 (~{EBUSCEZ1}): now also TP3005.1
- net SB_GBE_RXDV: now reaches U3001.D10 (GBERX_DV)
- net SB_GBE_RXD6: now reaches U3001.D11 (GBERXD6)
- net SB_GBE_RXD2: now reaches U3001.D12 (GBERXD2)
- net SB_GBE_RXD0: now reaches U3001.D13 (GBERXD0)
- net SB_ATA0_DD15: now reaches U3001.D19 (ATA0DD15)
- net SB_ATA0_DD14: now reaches U3001.D20 (ATA0DD14)
- net SB_ATA0_DD12: now reaches U3001.D21 (ATA0DD12)
- net SB_ATA0_DD11: now reaches U3001.D22 (ATA0DD11)
- net SB_ATA0_DD9: now reaches U3001.D23 (ATA0DD9)
- net SB_ATA0_DD8: now reaches U3001.D24 (ATA0DD8)
- net PIO0: now reaches U3001.D5 (PIO0)
- net SB_GBE_ETOMOD: now reaches U3001.D7 (GBEETOMOD)
- net SB_GBE_RVRX: now reaches U3001.D8 (GBERV_RX)
- net SB_GBE_RXD7: now reaches U3001.C10 (GBERXD7)
- net SB_GBE_RXD5: now reaches U3001.C11 (GBERXD5)
- net SB_GBE_RXD1: now reaches U3001.C12 (GBERXD1)
- net SB_GBE_RXCLK: now reaches U3001.C13 (GBERX_CLK)
- net SB_ATA0_DD0: now reaches U3001.C19 (ATA0DD0)
- net SB_ATA0_DD1: now reaches U3001.C20 (ATA0DD1)
- net SB_ATA0_DD3: now reaches U3001.C21 (ATA0DD3)
- net SB_ATA0_DD4: now reaches U3001.C22 (ATA0DD4)
- net SB_ATA0_DD6: now reaches U3001.C23 (ATA0DD6)
- net SB_ATA0_DD7: now reaches U3001.C24 (ATA0DD7)
- net SB_SIO0_RXD: now reaches U3001.C6 (SIORXD0)
- net SB_GBE_RVTX: now reaches U3001.C8 (GBERV_TX)
- net SB_GBE_COL: now reaches U3001.C9 (GBECOL)
- net ~{SB_EBUS_CE2}: now reaches U3001.J5 (~{EBUSCEZ2})
- net SB_TESTIN7: now reaches U3001.J8 (TESTIN7)
- net ~{SB_EBUS_IOR}: now reaches U3001.N3 (~{EBUSIORZ})
- net SB_EBUS_DATA1: now reaches U3001.N5 (EBUSDATA1)
- net SB_EBUS_DATA9: now reaches U3001.N7 (EBUSDATA9)
- net ~{SB_EBUS_OE}: now reaches U3001.L5 (~{EBUSOEZ})
- net ~{SB_EBUS_RESET}: now reaches U3001.E1 (PIO7)
- net MECHA_INT: now reaches U3001.E2 (PIO6)
- net ~{SS2_INT}: now reaches U3001.E3 (PIO5)
- net ~{MC_DET}: now reaches U3001.E4 (PIO4)
- new net: U3001.AH10 (VDDC), U3001.AH11 (VDDC), U3001.AH12 (VDDC), U3001.AH13 (VDDC), U3001.AH14 (VDDC), U3001.AH15 (VDDC), U3001.AH16 (VDDC), U3001.AH17 (VDDC), U3001.AH18 (VDDC)
- new net: U3001.AH19 (VDD33), U3001.AH20 (VDD33), U3001.AH21 (VDD33)
- new net: U3001.AJ10 (VDDC), U3001.AJ11 (VDDC), U3001.AJ12 (VDDC), U3001.AJ13 (VDDC), U3001.AJ14 (VDDC), U3001.AJ15 (VDDC), U3001.AJ16 (VDDC)
- new net: U3001.AG11 (VDDC), U3001.AG12 (VDDC), U3001.AG13 (VDDC)
- new net SB_EBUS_DATA10: U3001.P7 (EBUSDATA10)
- new net SB_EBUS_DATA11: U3001.R7 (EBUSDATA11)
- new net SB_EBUS_DATA12: U3001.T7 (EBUSDATA12)
- new net SB_EBUS_DATA14: U3001.V7 (EBUSDATA14)
- new net SB_EBUS_DATA15: U3001.W7 (EBUSDATA15)
- new net SB_EBUS_DATA2: U3001.P5 (EBUSDATA2)
- new net SB_EBUS_DATA3: U3001.R5 (EBUSDATA3)
- new net SB_EBUS_DATA4: U3001.T5 (EBUSDATA4)
- new net SB_EBUS_DATA5: U3001.U5 (EBUSDATA5)
- new net SB_EBUS_DATA6: U3001.V5 (EBUSDATA6)
- new net SB_EBUS_DATA7: U3001.W5 (EBUSDATA7)
- no-connect marks 0 -> 63
Other:
- moved on the sheet: TP3001, TP3004, TP3008, TP3009, TP3010, TP3011, U3001A, U3001B, U3001C, U3001D, U3001E, U3001F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

Commit message: bridge sif
Parts:
- added unit 37 of U3001
- added unit 42 of U3001
- added unit 38 of U3001
- added unit 39 of U3001
Connections:
- net +3.3V_SB_VDDIO: now also U3001.AK19 (VDD33), U3001.AK20 (VDD33), U3001.AM22 (VDD33), U3001.AM23 (VDD33), U3001.AM30 (VDD33), U3001.AM31 (VDD33)
- net GND: now also U3001.AK15 (GND), U3001.AK16 (GND), U3001.AK3 (GND), U3001.AK31 (GND), U3001.AK32 (GND), U3001.AL14 (GND), U3001.AL15 (GND), U3001.AL16 (GND), U3001.AL17 (GND), U3001.AL18 (GND), U3001.AL19 (GND), U3001.AL20 (GND), U3001.AL27 (GND), U3001.AL28 (GND), U3001.AL29 (GND), U3001.AL30 (GND), U3001.AL31 (GND), U3001.AL32 (GND), U3001.AL38 (GND), U3001.AL39 (GND), U3001.AL5 (GND), U3001.AM18 (GND), U3001.AM19 (GND), U3001.AM20 (GND), U3001.AM21 (GND), U3001.AM24 (GND), U3001.AM25 (GND), U3001.AM28 (GND), U3001.AM29 (GND), U3001.AM35 (GND)
- new net: U3001.AK10 (VDDC), U3001.AK11 (VDDC), U3001.AK12 (VDDC), U3001.AK13 (VDDC), U3001.AK14 (VDDC), U3001.AK7 (VDDC), U3001.AK8 (VDDC), U3001.AK9 (VDDC)
- new net: U3001.AL10 (VDDC), U3001.AL11 (VDDC), U3001.AL12 (VDDC), U3001.AL13 (VDDC), U3001.AL9 (VDDC)
- new net: U3001.AM10 (VDDC), U3001.AM11 (VDDC), U3001.AM12 (VDDC), U3001.AM9 (VDDC)
- new net: U3001.AM3 (VDDR), U3001.AM4 (VDDR), U3001.AM5 (VDDR), U3001.AM6 (VDDR), U3001.AM7 (VDDR), U3001.AM8 (VDDR)
Other:
- moved on the sheet: U3001G, U3001H, U3001J
