File: cok-001/southbridge.kicad_sch (KiCad schematic)
At the start: 8 parts, among them U3001 CXD2973GB

Commit message: sb
Connections:
- net +1.2V_SB_VDDC: now also U3001.AR2 (DVD), U3001.AT13 (VDDA12), U3001.AU13 (VDDA12)
- net GND: now also U3001.AR1 (DVS)
- net +1.5V_SB_RC_VDDA: now reaches U3001.AK8 (VDDA15)
- net +1.5V_SB_RC_VDDA: now also U3001.AL8 (VDDA15)
- net ~{SB_PCI_CBE0_SB}: now reaches U3001.AP19 (~{PCICBE0})
- net ~{SB_PCI_CBE2_SB}: now reaches U3001.AP20 (~{PCICBE2})
- net ~{SB_PCI_PME}: now reaches U3001.AP21 (~{PCIPMEMZ})
- net ~{SB_PCI_REQ0_SB}: now reaches U3001.AP22 (~{PCIREQ0})
- net ~{SB_PCI_REQ2}: now reaches U3001.AP23 (~{PCIREQ2})
- net ~{SB_PCI_GNT0_SB}: now reaches U3001.AP24 (~{PCIGNT0})
- net SB_PCI_CLK: now reaches U3001.AP28 (PCICLKI)
- net ~{SB_PCI_RST_SB}: now reaches U3001.AP29 (PCIRSTZ)
- net ~{SB_PCI_INTD_SB}: now reaches U3001.AP30 (PCIINTDZ)
- net ~{SB_PCI_INTB_SB}: now reaches U3001.AP31 (PCIINTBZ)
- net ~{SB_PCI_STOP_SB}: now reaches U3001.AV25 (~{PCISTOPZ})
- net SB_CHKSTP_IN: now reaches U3001.AV3 (CHECKSTOP_IN)
- net SB_SPI_DI: now reaches U3001.AV5 (SYSCSSPIDO)
- net ~{SB_SPI_CS}: now reaches U3001.AV7 (~{SYSCSSPCIS})
- net ~{SB_PCI_PERR_SB}: now reaches U3001.AW25 (~{PCIPERRZ})
- net BE_RX4_RXN1: now reaches U3001.AL6 (IOIFTXDN1)
- net BE_RX4_RXP1: now reaches U3001.AL7 (IOIFTXDP1)
- net SB_PLL_GNDA: now reaches U3001.AU1 (AVS)
- net SB_PEX0_REFCLKP: now reaches U3001.AU17 (PEXREFCLKP)
- net SB_PLL_VDDA: now reaches U3001.AU2 (AVD)
- net SB_PCI_PAR_SB: now reaches U3001.AU24 (PCIPAR)
- net ~{SB_PCI_DEVSEL_SB}: now reaches U3001.AU25 (~{PCIDEVSELZ})
- net ~{SB_PCI_IRDY_SB}: now reaches U3001.AU26 (~{PCIIRDYZ})
- net SB_TRG_OUT: now reaches U3001.AU3 (TRIGGER_OUT)
- net SB_CHKSTP_OUT: now reaches U3001.AU4 (CHECKSTOP_OUT)
- net ~{SB_CGRST}: now reaches U3001.AU5 (~{CGRSTZ})
- net ~{SB_INT}: now reaches U3001.AU6 (SYSCSINT)
- net SB_PLLBYPASS: now reaches U3001.AR4 (PLLBYPASS)
- net SB_TRG_IN: now reaches U3001.AR5 (TRIGGER_IN)
- net ~{SB_RESET}: now reaches U3001.AR6 (~{SYSRSTZ})
- net SB_SPI_CLK: now reaches U3001.AR7 (SZSCSSPICLK)
- net SB_PEX0_REFCLKN: now reaches U3001.AT17 (PEXREFCLKN)
- net ~{SB_PCI_SERR_SB}: now reaches U3001.AT24 (~{PCISERRZ})
- net ~{SB_PCI_TRDY_SB}: now reaches U3001.AT25 (~{PCITRDYZ})
- net ~{SB_PCI_FRAME_SB}: now reaches U3001.AT26 (~{PCIFRAMEZ})
- net SB_SYSCLK: now reaches U3001.AT3 (SYSCLK)
- no-connect marks 151 -> 157

Commit message: sb gnd
Connections:
- net 1.8_SB_VDD is gone; now on net GND: U3001.AA30 (VDD18), U3001.AA32 (VDD18), U3001.AA33 (DDRDQ36), U3001.AA34 (DDRDQ32), U3001.AA36 (DDRA1), U3001.AA37 (DDRCK0), U3001.AA38 (VDD18), U3001.AA39 (VDD18), U3001.AB30 (VDD18), U3001.AB33 (DDRDQ37), U3001.AB34 (DDRDQ33), U3001.AB35 (VDD18), U3001.AB36 (DDRDM4), U3001.AB37 (DDRCKZ0), U3001.AC30 (VDD18), U3001.AC33 (DDRDQSZ4), U3001.AC34 (DDRDQS4), U3001.AC35 (VDD18), U3001.AC36 (DDRDQ38), U3001.AC37 (DDRA0), U3001.AD30 (VDD18), U3001.AD32 (VDD18), U3001.AD33 (DDRDQ34), U3001.AD34 (DDRDQ39), U3001.AD36 (DDRDQ35), U3001.AD37 (DDRA10), U3001.AE30 (VDD18), U3001.AE32 (VDD18), U3001.AE33 (DDRDQ44), U3001.AE34 (DDRDQ40), U3001.AE36 (DDRDQ41), U3001.AE37 (DDRBA1), U3001.AE38 (VDD18), U3001.AE39 (VDD18), U3001.AF30 (VDD18), U3001.AF33 (DDRDQ45), U3001.AF34 (DDRDM5), U3001.AF35 (VDD18), U3001.AF36 (DDRDQSZ5), U3001.AF37 (DDRDQS5), U3001.AG30 (VDD18), U3001.AG33 (DDRDQ46), U3001.AG34 (DDRDQ42), U3001.AG35 (VDD18), U3001.AG36 (DDRDQ47), U3001.AG37 (DDRBA0), U3001.AH30 (VDD18), U3001.AH32 (VDD18), U3001.AH33 (DDRDQ43), U3001.AH34 (DDRDQ52), U3001.AH36 (DDRDQ48), U3001.AH37 (~{DDRRASZ}), U3001.AJ30 (VDD18), U3001.AJ32 (VDD18), U3001.AJ33 (DDRDQ53), U3001.AJ34 (DDRDQ49), U3001.AJ36 (DDRDM6), U3001.AJ37 (~{DDRWEZ}), U3001.AJ38 (VDD18), U3001.AJ39 (VDD18), U3001.AK30 (VDD18), U3001.AK33 (DDRDQSZ6), U3001.AK34 (DDRDQS6), U3001.AK35 (VDD18), U3001.AK36 (~{DDRCASZ}), U3001.AK37 (~{DDRCSZ_0}), U3001.AL33 (DDRDQ54), U3001.AL34 (DDRDQ50), U3001.AL35 (VDD18), U3001.AL36 (DDRDQ55), U3001.AL37 (DDRCSZ_1), U3001.AM32 (VDD18), U3001.AM33 (DDRDQ51), U3001.AM34 (DDRDQ60), U3001.AM36 (DDRDQ56), U3001.AM37 (DDRA13), U3001.AN32 (VDD18), U3001.AN33 (DDRDQ61), U3001.AN34 (DDRDQ57), U3001.AN36 (DDRDM7), U3001.AN37 (DDRCK2), U3001.AN38 (VDD18), U3001.AN39 (VDD18), U3001.AP33 (DDRDQSZ7), U3001.AP34 (DDRDQS7), U3001.AP35 (VDD18), U3001.AP36 (DDRDQ62), U3001.AP37 (DDRCKZ2), U3001.AR33 (DDRDQ58), U3001.AR34 (DDRDQ63), U3001.AR35 (VDD18), U3001.AR36 (DDRDQ59), U3001.AR37 (VDD18), U3001.AU34 (VDD18), U3001.AU35 (VDD18), U3001.AU36 (VDD18), U3001.AU37 (VDD18), U3001.AU38 (VDD18), U3001.AU39 (VDD18), U3001.D33 (VDD18), U3001.D34 (VDD18), U3001.D35 (VDD18), U3001.D36 (VDD18), U3001.D37 (VDD18), U3001.E38 (VDD18), U3001.E39 (VDD18), U3001.F33 (DDRDQ4), U3001.F34 (DDRDQ0), U3001.F35 (VDD18), U3001.F36 (DDRDQ5), U3001.F37 (DDRVREF), U3001.G33 (DDRDQ1), U3001.G34 (DDRDM0), U3001.G35 (VDD18), U3001.G36 (DDRDQSZ0), U3001.G37 (DDRDQS0), U3001.H32 (VDD18), U3001.H33 (DDRDQ6), U3001.H34 (DDRDQ2), U3001.H36 (DDRDQ7), U3001.H37 (DDRCK1), U3001.J32 (VDD18), U3001.J33 (DDRDQ3), U3001.J34 (DDRDQ12), U3001.J36 (DDRDQ8), U3001.J37 (DDRCKZ1), U3001.J38 (VDD18), U3001.J39 (VDD18), U3001.K33 (DDRDQ13), U3001.K34 (DDRDQ9), U3001.K35 (VDD18), U3001.K36 (DDRDM1), U3001.K37 (DDRCK3), U3001.L33 (DDRDQSZ1), U3001.L34 (DDRDQS1), U3001.L35 (VDD18), U3001.L36 (DDRMCKE), U3001.L37 (DDRCKZ3), U3001.M30 (VDD18), U3001.M32 (VDD18), U3001.M33 (DDRDQ14), U3001.M34 (DDRDQ10), U3001.M36 (DDRDQ15), U3001.M37 (DDRA12), U3001.N30 (VDD18), U3001.N32 (VDD18), U3001.N33 (DDRDQ11), U3001.N34 (DDRDQ20), U3001.N36 (DDRDQ16), U3001.N37 (DDRA11), U3001.N38 (VDD18), U3001.N39 (VDD18), U3001.P30 (VDD18), U3001.P33 (DDRDQ21), U3001.P34 (DDRDQ17), U3001.P35 (VDD18), U3001.P36 (DDRDM2), U3001.P37 (DDRA9), U3001.R33 (DDRDQSZ2), U3001.R34 (DDRDQS2), U3001.R35 (VDD18), U3001.R36 (DDRDQ22), U3001.R37 (DDRA7), U3001.T30 (VDD18), U3001.T32 (VDD18), U3001.T33 (DDRDQ18), U3001.T34 (DDRDQ23), U3001.T36 (DDRDQ19), U3001.T37 (DDRA8), U3001.U30 (VDD18), U3001.U32 (VDD18), U3001.U33 (DDRDQ28), U3001.U34 (DDRDQ24), U3001.U36 (DDRDQ25), U3001.U37 (DDRA5), U3001.U38 (VDD18), U3001.U39 (VDD18), U3001.V30 (VDD18), U3001.V33 (DDRDQ29), U3001.V34 (DDRDM3), U3001.V35 (VDD18), U3001.V36 (DDRDQSZ3), U3001.V37 (DDRDQS3), U3001.W30 (VDD18), U3001.W33 (DDRDQ30), U3001.W34 (DDRDQ26), U3001.W35 (VDD18), U3001.W36 (DDRA6), U3001.W37 (DDRA4), U3001.Y30 (VDD18), U3001.Y32 (VDD18), U3001.Y33 (DDRDQ31), U3001.Y34 (DDRDQ27), U3001.Y36 (DDRA3), U3001.Y37 (DDRA2)
- net GND: now also U3001.R30 (VDD18)
