File: cok-001/starship.kicad_sch (KiCad schematic)
At the start: 60 parts, among them U3802 K9F1G08U0A, U3803 K9F1G08U0A

Commit message: add some stupid n channel mosfet
Parts:
- TP9321, TP9322, TP9323, TP9324, TP9326, TP9327, TP9328, TP9329, TP9330, TP9331, TP9332, TP9333, TP9334, TP9335, TP9336, TP9337, TP9338, TP9339, TP9340, TP9341, TP9342, TP9343, TP9344, TP9345, TP9346: footprint (none) -> TestPoint:TestPoint_Pad_D1.5mm
Changed lines of the file:
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@@
 			)
 		)
-		(property "Footprint" ""
+		(property "Footprint" "TestPoint:TestPoint_Pad_D1.5mm"
 			(at 33.02 78.74 0)
 			(effects
@@
 			)
 		)
-		(property "Footprint" ""
+		(property "Footprint" "TestPoint:TestPoint_Pad_D1.5mm"
 			(at 33.02 60.96 0)
 			(effects
@@
 			)
 		)
-		(property "Footprint" ""
+		(property "Footprint" "TestPoint:TestPoint_Pad_D1.5mm"
 			(at 33.02 99.06 0)
 			(effects
@@
 			)
 		)
-		(property "Footprint" ""
+		(property "Footprint" "TestPoint:TestPoint_Pad_D1.5mm"
 			(at 57.15 185.42 0)
 			(effects
@@
 			)
 		)
-		(property "Footprint" ""
+		(property "Footprint" "TestPoint:TestPoint_Pad_D1.5mm"
 			(at 33.02 119.38 0)
 			(effects
@@
 			)
 		)
-		(property "Footprint" ""
+		(property "Footprint" "TestPoint:TestPoint_Pad_D1.5mm"
 			(at 33.02 137.16 0)
 			(effects
@@
 			)
 		)
-		(property "Footprint" ""
+		(property "Footprint" "TestPoint:TestPoint_Pad_D1.5mm"
 			(at 33.02 127 0)
 			(effects
@@
 			)
 		)
-		(property "Footprint" ""
+		(property "Footprint" "TestPoint:TestPoint_Pad_D1.5mm"
 			(at 33.02 134.62 0)
 			(effects
@@
 			)
 		)
-		(property "Footprint" ""
+		(property "Footprint" "TestPoint:TestPoint_Pad_D1.5mm"
 			(at 33.02 86.36 0)
 			(effects
@@
 			)
 		)
-		(property "Footprint" ""
+		(property "Footprint" "TestPoint:TestPoint_Pad_D1.5mm"
 			(at 33.02 58.42 0)
 			(effects
@@
 			)
 		)
-		(property "Footprint" ""
+		(property "Footprint" "TestPoint:TestPoint_Pad_D1.5mm"
 			(at 33.02 76.2 0)
 			(effects
@@
 			)
 		)
-		(property "Footprint" ""
+		(property "Footprint" "TestPoint:TestPoint_Pad_D1.5mm"
 			(at 33.02 93.98 0)
 			(effects
@@
 			)
 		)
-		(property "Footprint" ""
+		(property "Footprint" "TestPoint:TestPoint_Pad_D1.5mm"
 			(at 85.09 185.42 0)
 			(effects
@@
 			)
 		)
-		(property "Footprint" ""
+		(property "Footprint" "TestPoint:TestPoint_Pad_D1.5mm"
 			(at 33.02 106.68 0)
 			(effects
@@
 			)
 		)
-		(property "Footprint" ""
+		(property "Footprint" "TestPoint:TestPoint_Pad_D1.5mm"
 			(at 62.23 185.42 0)
 			(effects
@@
 			)
 		)
-		(property "Footprint" ""
+		(property "Footprint" "TestPoint:TestPoint_Pad_D1.5mm"
 			(at 33.02 121.92 0)
 			(effects
@@
 			)
 		)
-		(property "Footprint" ""
+		(property "Footprint" "TestPoint:TestPoint_Pad_D1.5mm"
 			(at 33.02 81.28 0)
 			(effects
@@
 			)
 		)
-		(property "Footprint" ""
+		(property "Footprint" "TestPoint:TestPoint_Pad_D1.5mm"
 			(at 33.02 116.84 0)
 			(effects
@@
 			)
 		)
-		(property "Footprint" ""
+		(property "Footprint" "TestPoint:TestPoint_Pad_D1.5mm"
 			(at 33.02 104.14 0)
 			(effects
@@
 			)
 		)
-		(property "Footprint" ""
+		(property "Footprint" "TestPoint:TestPoint_Pad_D1.5mm"
 			(at 77.47 185.42 0)
 			(effects
@@
 			)
 		)
-		(property "Footprint" ""
+		(property "Footprint" "TestPoint:TestPoint_Pad_D1.5mm"
 			(at 33.02 55.88 0)
 			(effects
@@
 			)
 		)
-		(property "Footprint" ""
+		(property "Footprint" "TestPoint:TestPoint_Pad_D1.5mm"
 			(at 33.02 48.26 0)
 			(effects
@@
 			)
 		)
-		(property "Footprint" ""
+		(property "Footprint" "TestPoint:TestPoint_Pad_D1.5mm"
 			(at 33.02 88.9 0)
 			(effects
@@
 			)
 		)
-		(property "Footprint" ""
+		(property "Footprint" "TestPoint:TestPoint_Pad_D1.5mm"
 			(at 90.17 185.42 0)
 			(effects
@@
 			)
 		)
-		(property "Footprint" ""
+		(property "Footprint" "TestPoint:TestPoint_Pad_D1.5mm"
 			(at 33.02 129.54 0)
 			(effects

Commit message: southbridge
Changed lines of the file:
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@@
 		(pin "F1"
 		)
-		(pin "IA2"
+		(pin "B13"
 		)
 		(pin "J8"

Commit message: aj
Parts:
- added R3801, R3807, R3808: 10k, Resistor_SMD:R_0402_1005Metric, symbol Device:R_US
- added R3802: 22, Resistor_SMD:R_0402_1005Metric, symbol Device:R_US
- added R3838, R3839: 0, Resistor_SMD:R_0402_1005Metric, symbol Device:R_US
- added TP9303, TP9304, TP9305, TP9306, TP9307, TP9308, TP9309, TP9310: TestPoint, TestPoint:TestPoint_Pad_D1.5mm, symbol Connector:TestPoint
Connections:
- net +3V3SB: now also R3801.2, R3807.2, R3808.2
- net ~{SB_EBUS_OE}: now reaches U3801.A2 (XHOE)
- net ~{SB_EBUS_OE}: now also TP9305.1
- net ~{SB_EBUS_SWE}: now reaches U3801.A7 (XHWE)
- net ~{SB_EBUS_SWE}: now also TP9304.1
- net ~{SB_EBUS_CE0}: now reaches U3801.B1 (XHCE0)
- net ~{SB_EBUS_CE0}: now also TP9307.1
- net ~{SB_EBUS_IOR}: now reaches U3801.B12 (XHBE)
- net ~{SB_EBUS_IOR}: now also TP9303.1
- net at U3801.B6 (XHRST): now also R3801.1, R3838.2, R3839.2
- net ~{SB_EBUS_ACK}: now reaches U3801.C1 (HRDY)
- net ~{SB_EBUS_ACK}: now also TP9308.1
- net ~{SB_EBUS_CE2}: now reaches U3801.C2 (XHCE1)
- net ~{SB_EBUS_CE2}: now also TP9306.1
- net at U3801.D1 (BRDY): now also R3802.2
- net ~{SS2_INT}: now reaches U3801.D2 (XINT)
- net ~{SS2_INT}: now also R3808.1, TP9310.1
- net SE_EBUS_DATA0 renamed SB_EBUS_DATA0
- net SE_EBUS_DATA1 renamed SB_EBUS_DATA1
- net SE_EBUS_DATA10 renamed SB_EBUS_DATA10
- net SE_EBUS_DATA11 renamed SB_EBUS_DATA11
- net SE_EBUS_DATA12 renamed SB_EBUS_DATA12
- net SE_EBUS_DATA13 renamed SB_EBUS_DATA13
- net SE_EBUS_DATA14 renamed SB_EBUS_DATA14
- net SE_EBUS_DATA15 renamed SB_EBUS_DATA15
- net SE_EBUS_DATA2 renamed SB_EBUS_DATA2
- net SE_EBUS_DATA3 renamed SB_EBUS_DATA3
- net SE_EBUS_DATA4 renamed SB_EBUS_DATA4
- net SE_EBUS_DATA5 renamed SB_EBUS_DATA5
- net SE_EBUS_DATA6 renamed SB_EBUS_DATA6
- net SE_EBUS_DATA7 renamed SB_EBUS_DATA7
- net SE_EBUS_DATA8 renamed SB_EBUS_DATA8
- net SE_EBUS_DATA9 renamed SB_EBUS_DATA9
- new net SS2_BRDY: R3802.1, R3807.1, TP9309.1
- new net ~{SB_EBUS_RESET}: R3838.1
- new net ~{SS2_RESET}: R3839.1
