File: cok-001/powermgmt.kicad_sch (KiCad schematic)
At the start: 29 parts, among them J6004 +12V_MAIN, J6005 +5V_EVER, Q6002 FDQ7238AS, U6003 MB39A, U6008 NCP511SN18T1, U6011 NCP511, U6012 MM3141, U6014 MM1591, U6019 NCP511SN18T1, U6021 MM1591, U6022 MM1593

Commit message: ethernet
Parts:
- TP6060, TP6063: footprint (none) -> TestPoint:TestPoint_Pad_1.0x1.0mm
Changed lines of the file:
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@@
 			)
 		)
-		(property "Footprint" ""
+		(property "Footprint" "TestPoint:TestPoint_Pad_1.0x1.0mm"
 			(at 218.44 22.86 0)
 			(effects
@@
 			)
 		)
-		(property "Footprint" ""
+		(property "Footprint" "TestPoint:TestPoint_Pad_1.0x1.0mm"
 			(at 218.44 46.99 0)
 			(effects

Commit message: sata
Parts:
- J6004: footprint (none) -> Connector:Banana_Jack_2Pin
- J6005: footprint (none) -> Connector_JST:JST_PH_B5B-PH-SM4-TB_1x05-1MP_P2.00mm_Vertical
Connections:
- net at J6005.1 (Pin_1): now also J6005.2 (Pin_2)
Changed lines of the file:
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@@
 	(wire
 		(pts
+			(xy 31.75 25.4) (xy 31.75 27.94)
+		)
+		(stroke
+			(width 0)
+			(type default)
+		)
+	)
+	(wire
+		(pts
 			(xy 189.23 151.13) (xy 189.23 148.59)
 		)
@@
 			)
 		)
-		(property "Footprint" ""
+		(property "Footprint" "Connector:Banana_Jack_2Pin"
 			(at 26.67 53.34 0)
 			(effects
@@
 			)
 		)
-		(property "Footprint" ""
+		(property "Footprint" "Connector_JST:JST_PH_B5B-PH-SM4-TB_1x05-1MP_P2.00mm_Vertical"
 			(at 26.67 30.48 0)
 			(effects

Commit message: southbridge
Parts:
- U6008, U6019: footprint Package_SO:TSOP-5_1.65x3.05mm_P0.95mm -> Package_TO_SOT_SMD:SOT-23-5
Changed lines of the file:
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@@
 			)
 		)
-		(property "Footprint" "Package_SO:TSOP-5_1.65x3.05mm_P0.95mm"
+		(property "Footprint" "Package_TO_SOT_SMD:SOT-23-5"
 			(at 257.81 55.245 0)
 			(effects
@@
 			)
 		)
-		(property "Footprint" "Package_SO:TSOP-5_1.65x3.05mm_P0.95mm"
+		(property "Footprint" "Package_TO_SOT_SMD:SOT-23-5"
 			(at 257.81 83.185 0)
 			(effects

Commit message: sc
Parts:
- added C6010: 22u 16V, Capacitor_SMD:C_1210_3225Metric, symbol Device:C
- added C6021, C6025: 0.1u 16V, Capacitor_SMD:C_0603_1608Metric, symbol Device:C
- added C6027: 4.7u 10V, Capacitor_SMD:C_0805_2012Metric, symbol Device:C
- added L6001: 2uH, Inductor_SMD:L_TDK_SLF6028, symbol Device:L
- added L6004: 5.6uH, Inductor_SMD:L_TDK_SLF10145, symbol Device:L
- added Q6001: FDQ7238AS, Package_SO:SO-14_3.9x8.65mm_P1.27mm, symbol PS3:FDQ7238AS
- added R6030: 10, Resistor_SMD:R_0603_1608Metric, symbol Device:R_US
- added R6031: XX, Resistor_SMD:R_0402_1005Metric, symbol Device:R_US
Connections:
- net GND: now also U6003.20 (PGND2), C6010.2, C6021.2, C6027.2, Q6001.5 (D), Q6001.6, Q6001.7
- net at U6003.16 (CB2): now also C6025.2
- net at U6003.17 (OUT1-2): now also R6030.2
- net at U6003.18 (VS2): now also C6025.1, L6004.1, Q6001.10, Q6001.11, Q6001.12, Q6001.13, Q6001.14, Q6001.8, Q6001.9
- net at U6003.19 (OUT2-2): now also Q6001.4 (G)
- net at U6003.21 (PWRGOOD): now also R6031.2
- net at U6003.22 (VB): now also C6027.1, R6031.1
- new net: C6010.1, C6021.1, L6001.2, Q6001.1 (S), Q6001.2 (S)
- new net: Q6001.3 (S), R6030.1

Commit message: seperate out
Parts:
- added C6029: 330u, Capacitor_Tantalum_SMD:CP_EIA-6032-20_AVX-F, symbol Device:C_Polarized_US
- U6014, U6020, U6021, U6022: footprint Package_SO:SOP-8_3.9x4.9mm_P1.27mm -> Package_SO:SSOP-8_3.9x5.05mm_P1.27mm
Connections:
- net GND: now also C6029.2
- net at L6004.2: now also C6029.1
Changed lines of the file:
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@@
 	(wire
 		(pts
+			(xy 115.57 176.53) (xy 120.65 176.53)
+		)
+		(stroke
+			(width 0)
+			(type default)
+		)
+	)
+	(wire
+		(pts
 			(xy 167.64 128.27) (xy 173.99 128.27)
 		)
@@
 			)
 		)
-		(property "Footprint" "Package_SO:SOP-8_3.9x4.9mm_P1.27mm"
+		(property "Footprint" "Package_SO:SSOP-8_3.9x5.05mm_P1.27mm"
 			(at 181.61 96.52 0)
 			(effects
@@
 	(symbol
 		(lib_id "power:GND")
+		(at 120.65 184.15 0)
+		(unit 1)
+		(exclude_from_sim no)
+		(in_bom yes)
+		(on_board yes)
+		(dnp no)
+		(fields_autoplaced yes)
+		(property "Reference" "#PWR068"
+			(at 120.65 190.5 0)
+			(effects
+				(font
+					(size 1.27 1.27)
+				)
+				(hide yes)
+			)
+		)
+		(property "Value" "GND"
+			(at 120.65 189.23 0)
+			(effects
+				(font
+					(size 1.27 1.27)
+				)
+			)
+		)
+		(property "Footprint" ""
+			(at 120.65 184.15 0)
+			(effects
+				(font
+					(size 1.27 1.27)
+				)
+				(hide yes)
+			)
+		)
+		(property "Datasheet" ""
+			(at 120.65 184.15 0)
+			(effects
+				(font
+					(size 1.27 1.27)
+				)
+				(hide yes)
+			)
+		)
+		(property "Description" "Power symbol creates a global label with name \"GND\" , ground"
+			(at 120.65 184.15 0)
+			(effects
+				(font
+					(size 1.27 1.27)
+				)
+				(hide yes)
+			)
+		)
+		(pin "1"
+		)
+		(instances
+			(project "cok-001"
+				(path "/976eb78d-8215-4cc0-9d72-f9d535c7970b/be970d6c-aeec-4303-8a86-89c9df8950fa"
+					(reference "#PWR068")
+					(unit 1)
+				)
+			)
+		)
+	)
+	(symbol
+		(lib_id "power:GND")
 		(at 265.43 71.12 0)
 		(mirror y)
@@
 			)
 		)
-		(property "Footprint" "Package_SO:SOP-8_3.9x4.9mm_P1.27mm"
+		(property "Footprint" "Package_SO:SSOP-8_3.9x5.05mm_P1.27mm"
 			(at 181.61 119.38 0)
 			(effects
@@
 			)
 		)
-		(property "Footprint" "Package_SO:SOP-8_3.9x4.9mm_P1.27mm"
+		(property "Footprint" "Package_SO:SSOP-8_3.9x5.05mm_P1.27mm"
 			(at 259.08 30.48 0)
 			(effects
@@
 			)
 		)
-		(property "Footprint" "Package_SO:SOP-8_3.9x4.9mm_P1.27mm"
+		(property "Footprint" "Package_SO:SSOP-8_3.9x5.05mm_P1.27mm"
 			(at 181.61 142.24 0)
 			(effects
@@
 					(unit 1)
 				)
+			)
+		)
+	)
+	(symbol
+		(lib_id "Device:C_Polarized_US")
+		(at 120.65 180.34 0)
+		(unit 1)
+		(exclude_from_sim no)
+		(in_bom yes)
+		(on_board yes)
+		(dnp no)
+		(fields_autoplaced yes)
+		(property "Reference" "C6029"
+			(at 124.46 178.4349 0)
+			(effects
+				(font
+					(size 1.27 1.27)
+				)
+				(justify left)
+			)
+		)
+		(property "Value" "330u"
+			(at 124.46 180.9749 0)
+			(effects
+				(font
+					(size 1.27 1.27)
+				)
+				(justify left)
+			)
+		)
+		(property "Footprint" "Capacitor_Tantalum_SMD:CP_EIA-6032-20_AVX-F"
+			(at 120.65 180.34 0)
+			(effects
+				(font
+					(size 1.27 1.27)
+				)
+				(hide yes)
+			)
+		)
+		(property "Datasheet" "~"
+			(at 120.65 180.34 0)
+			(effects
+				(font
+					(size 1.27 1.27)
+				)
+				(hide yes)
+			)
+		)
+		(property "Description" "Polarized capacitor, US symbol"
+			(at 120.65 180.34 0)
+			(effects
+				(font
+					(size 1.27 1.27)
+				)
+				(hide yes)
+			)
+		)
+		(pin "2"
+		)
+		(pin "1"
+		)
+		(instances
+			(project ""
+				(path "/976eb78d-8215-4cc0-9d72-f9d535c7970b/be970d6c-aeec-4303-8a86-89c9df8950fa"
+					(reference "C6029")
+					(unit 1)
+				)

Commit message: update to 9
Changed lines of the file:
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@@
 (kicad_sch
-	(version 20231120)
+	(version 20250114)
 	(generator "eeschema")
-	(generator_version "8.0")
+	(generator_version "9.0")
 	(paper "A4")
 	(junction

Commit message: footprints
Parts:
- added C6041: 25V, Capacitor_SMD:C_1210_3225Metric, symbol Device:C
- added FB6001: 0uH, Inductor_SMD:L_0603_1608Metric, symbol Device:FerriteBead_Small
- added Q1: SI3493, Package_SO:TSOP-6_1.65x3.05mm_P0.95mm, symbol Transistor_FET:PMN48XP
- added Q6003: DTC144E, Package_TO_SOT_SMD:SOT-323_SC-70, symbol Transistor_BJT:DTC144E
- added R6045, R6047: 100k, Resistor_SMD:R_0603_1608Metric, symbol Device:R_US
- added R6523: 390, Resistor_SMD:R_0603_1608Metric, symbol Device:R_US
- added U6013: MM1562, Package_SO:SSOP-8_3.9x5.05mm_P1.27mm, symbol PS3:MM159X
- F6001: value Fuse -> 5A
Connections:
- net GND: now also C6041.2, Q6003.2 (E), R6523.1, U6013.2 (NC), U6013.3 (GND), U6013.6 (SUB), U6013.7 (SUB)
- net SW_4_B: now also Q6003.1 (B)
- net +1.8V_SB_PERI: now reaches U6014.1 (Vout)
- net +3.3V_MISC: now reaches U6014.8 (Vin)
- net +3.3V_MISC: now also C6029.1, L6004.2, U6008.1 (IN), U6011.1 (Vin), U6012.1 (Vin), U6019.1 (IN), U6021.8 (Vin), Q1.4 (S), R6047.2, U6013.8 (Vin)
- net +1.5V_BRIDGE: now reaches U6021.1 (Vout)
- net +12V_MAIN: now reaches J6004.1 (Pin_1)
- net +12V_MAIN: now also F6001.1
- net +3.3V_MK_VDD: now reaches U6020.1 (Vout)
- net +5V_MISC: now reaches U6020.8 (Vin)
- net +5V_MISC: now also U6022.8 (Vin)
- net +3.3V_BRIDGE: now reaches U6022.1 (Vout)
- net +1.5V_AVCG_VDDIO: now reaches U6019.5 (OUT)
- net at F6001.2: now also L6002.1
- net at U6008.5 (OUT): now also FB6001.1
- net +5V_EVER: now reaches J6005.1 (Pin_1), J6005.2 (Pin_2)
- new net: Q6003.3 (C), R6045.1, R6047.1
- new net: C6041.1, Q1.3 (G), R6045.2
- new net +1.8V_RSX_PLL_VDD: FB6001.2
- new net +2.5V_LREG_XCG_500_MEM: U6013.1 (Vout)
- new net +3.3V_SB_VDDIO: Q1.1 (D), Q1.2 (D), Q1.5 (D), Q1.6 (D), R6523.2
- new net SW_1_B: U6013.5 (Cont)
Other:
- moved on the sheet: C6029, F6001, F6002, J6004, L6002, L6004, U6014, U6021, U6022

Commit message: power
Parts:
- added PS6001: 2A, Fuse:Fuse_1210_3225Metric, symbol Device:Fuse
- added Q6009: UMH2NTN, Package_TO_SOT_SMD:SOT-363_SC-70-6, symbol Transistor_BJT:UMH3N
- added Q6010: SI4943, Package_SO:SOIC-8_3.9x4.9mm_P1.27mm, symbol Transistor_FET:IRF7324
- added TH6001: Fuse, Fuse:Fuse_1210_3225Metric, symbol Device:Fuse
- renumbered Q1 to Q6004, F6002 to TH6002
Connections:
- net +12V_MAIN: now also PS6001.1
- net GND: now also Q6009.1 (E1), Q6009.4 (E2)
- net at L6001.1: now also PS6001.2
- net ACDC_STBY: now reaches J6005.5 (Pin_5)
- net at TH6002.2: now also Q6010.1 (S1)
- new net: Q6010.3 (S2), TH6001.2
- new net +12V_BD: Q6010.7 (D1), Q6010.8 (D1)
- new net +5V_BD: Q6010.5 (D2), Q6010.6 (D2)
- new net SW_ATA: Q6009.2 (B1), Q6009.5 (B2)
Other:
- moved on the sheet: TH6002
