File: cok-001/powermgmt.kicad_sch (KiCad schematic)
At the start: 123 parts, among them J6004 +12V_MAIN, J6005 +5V_EVER, Q6001 FDQ7238AS, Q6002 FDQ7238AS, Q6003 DTC144E, Q6004 SI3493, Q6006 UMH2NTN, Q6007 SI3493, Q6008 SI3493, Q6009 UMH2NTN, Q6010 SI4943, Q6012 Si3460DV, U6003 MB39A, U6004 PST3642UL, U6005 NCP511SN33T1G, U6006 NCP511SN18T1, U6007 TPS73101DBV, U6008 NCP511SN18T1, U6009 NCP511SN33T1G, U6011 NCP511, U6012 MM3141, U6013 MM1562, U6014 MM1591, U6017 BD3521, U6019 NCP511SN18T1, U6020 MM1593DFBEG, U6021 MM1591, U6022 MM1593, U6023 PST3642UL

Commit message: rdy
Parts:
- R6045, R6524, R6525: footprint Resistor_SMD:R_0603_1608Metric -> Resistor_SMD:R_0402_1005Metric
Changed lines of the file:
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@@
 			)
 		)
-		(property "Footprint" "Resistor_SMD:R_0603_1608Metric"
+		(property "Footprint" "Resistor_SMD:R_0402_1005Metric"
 			(at 241.554 257.556 90)
 			(effects
@@
 			)
 		)
-		(property "Footprint" "Resistor_SMD:R_0603_1608Metric"
+		(property "Footprint" "Resistor_SMD:R_0402_1005Metric"
 			(at 135.636 124.206 90)
 			(effects
@@
 			)
 		)
-		(property "Footprint" "Resistor_SMD:R_0603_1608Metric"
+		(property "Footprint" "Resistor_SMD:R_0402_1005Metric"
 			(at 241.554 234.696 90)
 			(effects
