File: cok-001/hdmi.kicad_sch (KiCad schematic)
At the start: 60 parts, among them J2501 HDMI_A, Q2502 DTA144E, Q2504 DTA144E, Q2507 DTC144E

Commit message: ethernet
Parts:
- L2501, L2502, L2503, L2504: value L_Iron_Coupled_Small -> L_Iron_Coupled_Small_1243
Changed lines of the file:
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@@
 		(dnp no)
 		(property "Reference" "L2501"
-			(at 334.01 92.71 0)
+			(at 334.01 102.235 0)
 			(effects
 				(font
@@
 			)
 		)
-		(property "Value" "L_Iron_Coupled_Small"
-			(at 334.01 95.25 0)
+		(property "Value" "L_Iron_Coupled_Small_1243"
+			(at 334.01 95.885 0)
 			(effects
 				(font
@@
 		(dnp no)
 		(property "Reference" "L2502"
-			(at 322.58 97.79 0)
+			(at 322.58 107.315 0)
 			(effects
 				(font
@@
 			)
 		)
-		(property "Value" "L_Iron_Coupled_Small"
-			(at 322.58 100.33 0)
+		(property "Value" "L_Iron_Coupled_Small_1243"
+			(at 322.58 100.965 0)
 			(effects
 				(font
@@
 		(dnp no)
 		(property "Reference" "L2503"
-			(at 334.01 102.87 0)
+			(at 334.01 112.395 0)
 			(effects
 				(font
@@
 			)
 		)
-		(property "Value" "L_Iron_Coupled_Small"
-			(at 334.01 105.41 0)
+		(property "Value" "L_Iron_Coupled_Small_1243"
+			(at 334.01 106.045 0)
 			(effects
 				(font
@@
 		(dnp no)
 		(property "Reference" "L2504"
-			(at 322.58 107.95 0)
+			(at 322.58 117.475 0)
 			(effects
 				(font
@@
 			)
 		)
-		(property "Value" "L_Iron_Coupled_Small"
-			(at 322.58 110.49 0)
+		(property "Value" "L_Iron_Coupled_Small_1243"
+			(at 322.58 111.125 0)
 			(effects
 				(font

Commit message: sata
Parts:
- added C2517, C2518, C2520, C2522: 0.1u 10V, Capacitor_SMD:C_0402_1005Metric, symbol Device:C
- added C2519, C2521, C2523: 0.001u 10V, Capacitor_SMD:C_0402_1005Metric, symbol Device:C
Connections:
- net GND: now also C2517.2, C2518.2, C2519.1, C2520.2, C2521.1, C2522.2, C2523.1
- net at U2502.K3: now also C2517.1
- net at U2502.K5: now also U2502.K7, U2502.K9, C2518.1, C2519.2, C2520.1, C2521.2, C2522.1, C2523.2

Commit message: southbridge
Parts:
- D251, D252, D253, D254, D255, D256, D257, D258: footprint Diode_SMD:D_SOD-923 -> Diode_SMD:D_SOD-523
Changed lines of the file:
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@@
 			)
 		)
-		(property "Footprint" "Diode_SMD:D_SOD-923"
+		(property "Footprint" "Diode_SMD:D_SOD-523"
 			(at 282.575 147.32 0)
 			(effects
@@
 			)
 		)
-		(property "Footprint" "Diode_SMD:D_SOD-923"
+		(property "Footprint" "Diode_SMD:D_SOD-523"
 			(at 311.785 147.32 0)
 			(effects
@@
 			)
 		)
-		(property "Footprint" "Diode_SMD:D_SOD-923"
+		(property "Footprint" "Diode_SMD:D_SOD-523"
 			(at 287.655 147.32 0)
 			(effects
@@
 			)
 		)
-		(property "Footprint" "Diode_SMD:D_SOD-923"
+		(property "Footprint" "Diode_SMD:D_SOD-523"
 			(at 316.865 147.32 0)
 			(effects
@@
 			)
 		)
-		(property "Footprint" "Diode_SMD:D_SOD-923"
+		(property "Footprint" "Diode_SMD:D_SOD-523"
 			(at 292.735 147.32 0)
 			(effects
@@
 			)
 		)
-		(property "Footprint" "Diode_SMD:D_SOD-923"
+		(property "Footprint" "Diode_SMD:D_SOD-523"
 			(at 321.945 147.32 0)
 			(effects
@@
 			)
 		)
-		(property "Footprint" "Diode_SMD:D_SOD-923"
+		(property "Footprint" "Diode_SMD:D_SOD-523"
 			(at 306.705 147.32 0)
 			(effects
@@
 			)
 		)
-		(property "Footprint" "Diode_SMD:D_SOD-923"
+		(property "Footprint" "Diode_SMD:D_SOD-523"
 			(at 277.495 147.32 0)
 			(effects

Commit message: aj
Parts:
- added RN2504, RN2505, RN2506, RN2507, RN2508, RN2509: 22, Resistor_SMD:R_Array_Convex_4x0402, symbol Device:R_Pack04
Connections:
- net RSX_VO29: now reaches RN2503.5 (R4.2)
- net RSX_VO34: now reaches RN2503.6 (R3.2)
- net RSX_VO21: now reaches RN2503.7 (R2.2)
- net RSX_VO33: now reaches RN2503.8 (R1.2)
- net RSX_VO20: now reaches RN2502.5 (R4.2)
- net RSX_VO23: now reaches RN2502.6 (R3.2)
- net RSX_VO16: now reaches RN2502.7 (R2.2)
- net RSX_VO18: now reaches RN2502.8 (R1.2)
- net at U2502.K10 (SII0_D0): now also RN2504.1 (R1.1)
- net at U2502.K11 (SII0_D1): now also RN2504.3 (R3.1)
- net at U2502.K12 (SII0_D2): now also RN2509.1 (R1.1)
- net at U2502.K8 (SII0_D11): now also RN2505.4 (R4.1)
- net at U2502.L10 (SII0_D7): now also RN2505.1 (R1.1)
- net at U2502.L11 (SII0_D5): now also RN2504.4 (R4.1)
- net at U2502.L12 (SII0_D3): now also RN2509.2 (R2.1)
- net at U2502.L7 (SII0_D14): now also RN2504.2 (R2.1)
- net at U2502.L8 (SII0_D12): now also RN2505.2 (R2.1)
- net at U2502.L9 (SII0_D9): now also RN2505.3 (R3.1)
- net at U2502.M10 (SII0_D8): now also RN2507.1 (R1.1)
- net at U2502.M11 (SII0_D6): now also RN2509.4 (R4.1)
- net at U2502.M12 (SII0_D4): now also RN2509.3 (R3.1)
- net at U2502.M3 (SII0_D24): now also RN2508.4 (R4.1)
- net at U2502.M4 (SII0_D22): now also RN2508.3 (R3.1)
- net at U2502.M5 (SII0_D19): now also RN2508.2 (R2.1)
- net at U2502.M6 (SII0_D17): now also RN2508.1 (R1.1)
- net at U2502.M7 (SII0_D15): now also RN2507.4 (R4.1)
- net at U2502.M8 (SII0_D13): now also RN2507.3 (R3.1)
- net at U2502.M9 (SII0_D10): now also RN2507.2 (R2.1)
- net RSX_VO31: now reaches RN2501.5 (R4.2)
- net RSX_VO35: now reaches RN2501.6 (R3.2)
- net RSX_VO32: now reaches RN2501.7 (R2.2)
- net RSX_VO27: now reaches RN2501.8 (R1.2)

Commit message: hd sb
Connections:
- net RSX_VO0: now also RN2504.8 (R1.2)
- net RSX_VO1: now also RN2504.6 (R3.2)
- net RSX_VO10: now also RN2507.7 (R2.2)
- net RSX_VO11: now also RN2505.5 (R4.2)
- net RSX_VO12: now also RN2505.7 (R2.2)
- net RSX_VO13: now also RN2507.6 (R3.2)
- net RSX_VO14: now also RN2504.7 (R2.2)
- net RSX_VO15: now also RN2507.5 (R4.2)
- net RSX_VO17: now also RN2508.8 (R1.2)
- net RSX_VO19: now also RN2508.7 (R2.2)
- net RSX_VO2: now also RN2509.8 (R1.2)
- net RSX_VO22: now also RN2508.6 (R3.2)
- net RSX_VO24: now also RN2508.5 (R4.2)
- net RSX_VO25: now also RN2506.8 (R1.2)
- net RSX_VO26: now also RN2506.7 (R2.2)
- net RSX_VO28: now also RN2506.6 (R3.2)
- net RSX_VO3: now also RN2509.7 (R2.2)
- net RSX_VO30: now also RN2506.5 (R4.2)
- net RSX_VO4: now also RN2509.6 (R3.2)
- net RSX_VO5: now also RN2504.5 (R4.2)
- net RSX_VO6: now also RN2509.5 (R4.2)
- net RSX_VO7: now also RN2505.8 (R1.2)
- net RSX_VO8: now also RN2507.8 (R1.2)
- net RSX_VO9: now also RN2505.6 (R3.2)
- net at U2502.K1 (SII0_D30): now also RN2506.4 (R4.1)
- net at U2502.L1 (SII0_D28): now also RN2506.3 (R3.1)
- net at U2502.M1 (SII0_D26): now also RN2506.2 (R2.1)
- net at U2502.M2 (SII0_D25): now also RN2506.1 (R1.1)
Other:
- moved on the sheet: R2501, R2502, R2503, R2505, R2506, R2507, R2510, R2511, R2512, R2513, R2514, R2515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

Commit message: seperate out
Parts:
- added C2525, C2528: 0.1u 10V, Capacitor_SMD:C_0402_1005Metric, symbol Device:C
- added C2586, C2587: 10p 50V, Capacitor_SMD:C_0402_1005Metric, symbol Device:C
- added U2501: ~, Package_SO:VSSOP-8_2.3x2mm_P0.5mm, symbol PS3:TC7WP3125FK
Connections:
- net GND: now also U2502.A4 (GND), C2525.2, C2528.2, C2586.2, C2587.2, U2501.4 (GND), U2501.5 (~{OE})
- net at U2502.E10 (HDMI): now also U2501.3 (A2)
- new net: C2528.1, C2587.1, U2501.1 (VccA)
- new net: C2525.1, C2586.1, U2501.8 (VccB)
- new net RS_SPDO0: U2501.2 (A1)
- new net RS_SPDO0_33: U2501.7 (B1)
- new net ~{HDMI_INT}: U2501.6 (B2)

Commit message: update to 9
Changed lines of the file:
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@@
 (kicad_sch
-	(version 20231120)
+	(version 20250114)
 	(generator "eeschema")
-	(generator_version "8.0")
+	(generator_version "9.0")
 	(paper "A4")
 	(junction

Commit message: hdmi diodes
Parts:
- added R2524: 698, Resistor_SMD:R_0603_1608Metric, symbol Device:R_US
- D251, D252, D253, D254, D255, D256, D257, D258: footprint Diode_SMD:D_SOD-523 -> Diode_SMD:D_SOD-923
Connections:
- net at U2502.A12: now also R2524.2
Changed lines of the file:
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@@
 	(wire
 		(pts
+			(xy 200.66 139.7) (xy 200.66 107.95)
+		)
+		(stroke
+			(width 0)
+			(type default)
+		)
+	)
+	(wire
+		(pts
 			(xy 339.09 135.89) (xy 335.28 135.89)
 		)
@@
 		)
 	)
+	(wire
+		(pts
+			(xy 200.66 107.95) (xy 194.31 107.95)
+		)
+		(stroke
+			(width 0)
+			(type default)
+		)
+	)
 	(bus
 		(pts
@@
 			)
 		)
-		(property "Footprint" "Diode_SMD:D_SOD-523"
+		(property "Footprint" "Diode_SMD:D_SOD-923"
 			(at 282.575 147.32 0)
 			(effects
@@
 			)
 		)
-		(property "Footprint" "Diode_SMD:D_SOD-523"
+		(property "Footprint" "Diode_SMD:D_SOD-923"
 			(at 311.785 147.32 0)
 			(effects
@@
 	)
 	(symbol
+		(lib_id "Device:R_US")
+		(at 200.66 143.51 0)
+		(mirror x)
+		(unit 1)
+		(exclude_from_sim no)
+		(in_bom yes)
+		(on_board yes)
+		(dnp no)
+		(property "Reference" "R2524"
+			(at 208.28 144.272 0)
+			(effects
+				(font
+					(size 1.27 1.27)
+				)
+				(justify right)
+			)
+		)
+		(property "Value" "698"
+			(at 204.724 146.304 0)
+			(effects
+				(font
+					(size 1.27 1.27)
+				)
+				(justify right)
+			)
+		)
+		(property "Footprint" "Resistor_SMD:R_0603_1608Metric"
+			(at 201.676 143.256 90)
+			(effects
+				(font
+					(size 1.27 1.27)
+				)
+				(hide yes)
+			)
+		)
+		(property "Datasheet" "~"
+			(at 200.66 143.51 0)
+			(effects
+				(font
+					(size 1.27 1.27)
+				)
+				(hide yes)
+			)
+		)
+		(property "Description" "Resistor, US symbol"
+			(at 200.66 143.51 0)
+			(effects
+				(font
+					(size 1.27 1.27)
+				)
+				(hide yes)
+			)
+		)
+		(pin "2"
+		)
+		(pin "1"
+		)
+		(instances
+			(project "cok-001"
+				(path "/976eb78d-8215-4cc0-9d72-f9d535c7970b/0c5bdaa3-92f7-4616-b4f9-a5dd748f69e5"
+					(reference "R2524")
+					(unit 1)
+				)
+			)
+		)
+	)
+	(symbol
 		(lib_id "Device:R_Pack04")
 		(at 139.7 165.1 0)
@@
 			)
 		)
-		(property "Footprint" "Diode_SMD:D_SOD-523"
+		(property "Footprint" "Diode_SMD:D_SOD-923"
 			(at 287.655 147.32 0)
 			(effects
@@
 			)
 		)
-		(property "Footprint" "Diode_SMD:D_SOD-523"
+		(property "Footprint" "Diode_SMD:D_SOD-923"
 			(at 316.865 147.32 0)
 			(effects
@@
 			)
 		)
-		(property "Footprint" "Diode_SMD:D_SOD-523"
+		(property "Footprint" "Diode_SMD:D_SOD-923"
 			(at 292.735 147.32 0)
 			(effects
@@
 			)
 		)
-		(property "Footprint" "Diode_SMD:D_SOD-523"
+		(property "Footprint" "Diode_SMD:D_SOD-923"
 			(at 321.945 147.32 0)
 			(effects
@@
 			)
 		)
-		(property "Footprint" "Diode_SMD:D_SOD-523"
+		(property "Footprint" "Diode_SMD:D_SOD-923"
 			(at 306.705 147.32 0)
 			(effects
@@
 			)
 		)
-		(property "Footprint" "Diode_SMD:D_SOD-523"
+		(property "Footprint" "Diode_SMD:D_SOD-923"
 			(at 277.495 147.32 0)
 			(effects
