File: cok-001/hdmi.kicad_sch (KiCad schematic)
At the start: 79 parts, among them J2501 HDMI_A, Q2502 DTA144E, Q2504 DTA144E, Q2507 DTC144E

Commit message: fix 1 rsx pin
Connections:
- net RSX_VO0: now also RN2504.5 (R4.2); no longer RN2504.8 (R1.2)
- net RSX_VO1: now also RN2504.7 (R2.2); no longer RN2504.6 (R3.2)
- net RSX_VO11: now also RN2505.8 (R1.2); no longer RN2505.5 (R4.2)
- net RSX_VO12: now also RN2505.6 (R3.2); no longer RN2505.7 (R2.2)
- net RSX_VO14: now also RN2504.6 (R3.2); no longer RN2504.7 (R2.2)
- net RSX_VO16: now also RN2502.6 (R3.2); no longer RN2502.7 (R2.2)
- net RSX_VO18: now also RN2502.5 (R4.2); no longer RN2502.8 (R1.2)
- net RSX_VO20: now also RN2502.8 (R1.2); no longer RN2502.5 (R4.2)
- net RSX_VO23: now also RN2502.7 (R2.2); no longer RN2502.6 (R3.2)
- net RSX_VO5: now also RN2504.8 (R1.2); no longer RN2504.5 (R4.2)
- net RSX_VO7: now also RN2505.5 (R4.2); no longer RN2505.8 (R1.2)
- net RSX_VO9: now also RN2505.7 (R2.2); no longer RN2505.6 (R3.2)
- net at RN2505.1 (R1.1): now also U2502.K8 (SII0_D11); no longer U2502.L10 (SII0_D7)
- net at RN2505.2 (R2.1): now also U2502.L9 (SII0_D9); no longer U2502.L8 (SII0_D12)
- net at RN2505.3 (R3.1): now also U2502.L8 (SII0_D12); no longer U2502.L9 (SII0_D9)
- net at RN2505.4 (R4.1): now also U2502.L10 (SII0_D7); no longer U2502.K8 (SII0_D11)
- net at RN2502.1 (R1.1): now also U2502.K4 (SII0_D20); no longer U2502.L5 (SII0_D18)
- net at RN2502.2 (R2.1): now also U2502.L3 (SII0_D23); no longer U2502.L6 (SII0_D16)
- net at RN2502.3 (R3.1): now also U2502.L6 (SII0_D16); no longer U2502.L3 (SII0_D23)
- net at RN2502.4 (R4.1): now also U2502.L5 (SII0_D18); no longer U2502.K4 (SII0_D20)
- net at U2502.K10 (SII0_D0): now also RN2504.4 (R4.1); no longer RN2504.1 (R1.1)
- net at U2502.K11 (SII0_D1): now also RN2504.2 (R2.1); no longer RN2504.3 (R3.1)
- net at U2502.L11 (SII0_D5): no longer RN2504.4 (R4.1)
- net at U2502.L7 (SII0_D14): now also RN2504.3 (R3.1); no longer RN2504.2 (R2.1)
Other:
- moved on the sheet: RN2502, RN2504, RN2505
Changed lines of the file:
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@@
 	(wire
 		(pts
-			(xy 149.86 185.42) (xy 124.46 185.42)
+			(xy 149.86 185.42) (xy 127 185.42)
 		)
 		(stroke
@@
 	(symbol
 		(lib_id "Device:R_Pack04")
-		(at 151.13 196.85 0)
-		(mirror x)
+		(at 148.59 196.85 180)
 		(unit 1)
 		(exclude_from_sim no)
@@
 		(dnp no)
 		(property "Reference" "RN2505"
-			(at 156.21 198.1201 0)
+			(at 143.51 198.1201 0)
 			(effects
 				(font
@@
 		)
 		(property "Value" "22"
-			(at 156.21 195.5801 0)
+			(at 143.51 195.5801 0)
 			(effects
 				(font
@@
 		)
 		(property "Footprint" "Resistor_SMD:R_Array_Convex_4x0402"
-			(at 158.115 196.85 90)
+			(at 141.605 196.85 90)
 			(effects
 				(font
@@
 		)
 		(property "Datasheet" "~"
-			(at 151.13 196.85 0)
+			(at 148.59 196.85 0)
 			(effects
 				(font
@@
 		)
 		(property "Description" "4 resistor network, parallel topology"
-			(at 151.13 196.85 0)
+			(at 148.59 196.85 0)
 			(effects
 				(font
@@
 	(symbol
 		(lib_id "Device:R_Pack04")
-		(at 139.7 165.1 0)
-		(mirror x)
+		(at 137.16 165.1 180)
 		(unit 1)
 		(exclude_from_sim no)
@@
 		(dnp no)
 		(property "Reference" "RN2502"
-			(at 144.78 166.3701 0)
+			(at 132.08 166.3701 0)
 			(effects
 				(font
@@
 		)
 		(property "Value" "22"
-			(at 144.78 163.8301 0)
+			(at 132.08 163.8301 0)
 			(effects
 				(font
@@
 		)
 		(property "Footprint" "Resistor_SMD:R_Array_Convex_4x0402"
-			(at 146.685 165.1 90)
+			(at 130.175 165.1 90)
 			(effects
 				(font
@@
 		)
 		(property "Datasheet" "~"
-			(at 139.7 165.1 0)
+			(at 137.16 165.1 0)
 			(effects
 				(font
@@
 		)
 		(property "Description" "4 resistor network, parallel topology"
-			(at 139.7 165.1 0)
+			(at 137.16 165.1 0)
 			(effects
 				(font
@@
 	(symbol
 		(lib_id "Device:R_Pack04")
-		(at 121.92 190.5 0)
-		(mirror x)
+		(at 119.38 190.5 180)
 		(unit 1)
 		(exclude_from_sim no)
@@
 		(dnp no)
 		(property "Reference" "RN2504"
-			(at 127 191.7701 0)
+			(at 114.3 191.7701 0)
 			(effects
 				(font
@@
 		)
 		(property "Value" "22"
-			(at 127 189.2301 0)
+			(at 114.3 189.2301 0)
 			(effects
 				(font
@@
 		)
 		(property "Footprint" "Resistor_SMD:R_Array_Convex_4x0402"
-			(at 128.905 190.5 90)
+			(at 112.395 190.5 90)
 			(effects
 				(font
@@
 		)
 		(property "Datasheet" "~"
-			(at 121.92 190.5 0)
+			(at 119.38 190.5 0)
 			(effects
 				(font
@@
 		)
 		(property "Description" "4 resistor network, parallel topology"
-			(at 121.92 190.5 0)
+			(at 119.38 190.5 0)
 			(effects
 				(font
