File: cok-001/hdmi.kicad_sch (KiCad schematic)
At the start: 79 parts, among them J2501 HDMI_A, Q2502 DTA144E, Q2504 DTA144E, Q2507 DTC144E

Commit message: update 10
Parts:
- U2501, U2502: value ~ -> (none)
