File: cok-001/cpu.kicad_sch (KiCad schematic)
At the start: 1 part

Commit message: power in
Connections:
- net GND: now also IC1001.A13 (GND), IC1001.A15 (GND), IC1001.A17 (GND), IC1001.A19 (GND), IC1001.A21 (GND), IC1001.A23 (GND), IC1001.A25 (GND), IC1001.A27 (GND), IC1001.A29 (GND), IC1001.A31 (GND), IC1001.A33 (GND), IC1001.AL19 (GND), IC1001.AL21 (GND), IC1001.AL23 (GND), IC1001.AL25 (GND), IC1001.AL27 (GND), IC1001.AM20 (GND), IC1001.AM22 (GND), IC1001.AM24 (GND), IC1001.AM26 (GND), IC1001.AM28 (GND), IC1001.B12 (GND), IC1001.B14 (GND), IC1001.B16 (GND), IC1001.B18 (GND), IC1001.B20 (GND), IC1001.B22 (GND), IC1001.B24 (GND), IC1001.B30 (GND), IC1001.B32 (GND), IC1001.C13 (GND), IC1001.C15 (GND), IC1001.C17 (GND), IC1001.C19 (GND), IC1001.C21 (GND), IC1001.C23 (GND), IC1001.C25 (GND), IC1001.C27 (GND), IC1001.C29 (GND), IC1001.C31 (GND), IC1001.C33 (GND), IC1001.D14 (GND), IC1001.D16 (GND), IC1001.D18 (GND), IC1001.D20 (GND), IC1001.D22 (GND), IC1001.D24 (GND), IC1001.D26 (GND), IC1001.D28 (GND), IC1001.D30 (GND), IC1001.D32 (GND), IC1001.E13 (GND), IC1001.E15 (GND), IC1001.E17 (GND), IC1001.E19 (GND), IC1001.E21 (GND), IC1001.E23 (GND), IC1001.E25 (GND), IC1001.E27 (GND), IC1001.E29 (GND), IC1001.E31 (GND), IC1001.F12 (GND), IC1001.F14 (GND), IC1001.F16 (GND), IC1001.F18 (GND), IC1001.F20 (GND), IC1001.F22 (GND), IC1001.F24 (GND), IC1001.F26 (GND), IC1001.F28 (GND), IC1001.F30 (GND), IC1001.G13 (GND), IC1001.G15 (GND), IC1001.G17 (GND), IC1001.G19 (GND), IC1001.G21 (GND), IC1001.G23 (GND), IC1001.G25 (GND), IC1001.G27 (GND), IC1001.G29 (GND), IC1001.G31 (GND), IC1001.H12 (GND), IC1001.H14 (GND), IC1001.H16 (GND), IC1001.H18 (GND), IC1001.H20 (GND), IC1001.H22 (GND), IC1001.H24 (GND), IC1001.H26 (GND), IC1001.H28 (GND), IC1001.H30 (GND), IC1001.J13 (GND), IC1001.J15 (GND), IC1001.J17 (GND), IC1001.J19 (GND), IC1001.J21 (GND), IC1001.J23 (GND), IC1001.J25 (GND), IC1001.J27 (GND), IC1001.J29 (GND), IC1001.J31 (GND), IC1001.K10 (GND), IC1001.K12 (GND), IC1001.K14 (GND), IC1001.K16 (GND), IC1001.K18 (GND), IC1001.K20 (GND), IC1001.K22 (GND), IC1001.K24 (GND), IC1001.K26 (GND), IC1001.K28 (GND), IC1001.L11 (GND), IC1001.L13 (GND), IC1001.L15 (GND), IC1001.L17 (GND), IC1001.L19 (GND), IC1001.L21 (GND), IC1001.L23 (GND), IC1001.L25 (GND), IC1001.L27 (GND), IC1001.L29 (GND)
- net Y0_XDR0_DQ0: now also IC1001.D2 (Y0_DQ1_6)
- net Y0_XDR0_DQ10: now also IC1001.B2 (Y0_DQ1_5)
- net Y0_XDR0_DQ12: now also IC1001.D3 (Y0_DQ1_4)
- net Y0_XDR0_DQ14: now also IC1001.B4 (Y0_DQ0_6)
- net Y0_XDR0_DQ2: now also IC1001.B5 (Y0_DQ0_4)
- net Y0_XDR0_DQ4: now also IC1001.D4 (Y0_DQ0_0)
- net Y0_XDR0_DQ6: now also IC1001.B3 (Y0_DQ1_2)
- net Y0_XDR0_DQ8: now also IC1001.D5 (Y0_DQ0_5)
- net Y0_XDR0_DQN0: now also IC1001.C2 (Y0_DQ1N_6)
- net Y0_XDR0_DQN10: now also IC1001.A2 (Y0_DQ1N_5)
- net Y0_XDR0_DQN12: now also IC1001.C3 (Y0_DQ1N_4)
- net Y0_XDR0_DQN14: now also IC1001.A4 (Y0_DQ0N_6)
- net Y0_XDR0_DQN2: now also IC1001.A5 (Y0_DQ0N_4)
- net Y0_XDR0_DQN4: now also IC1001.C4 (Y0_DQ0N_0)
- net Y0_XDR0_DQN6: now also IC1001.A3 (Y0_DQ1N_2)
- net Y0_XDR0_DQN8: now also IC1001.C5 (Y0_DQ0N_5)
- net Y0_XDR1_DQ14: now also IC1001.B8 (Y0_DQ0_1)
- net Y0_XDR1_DQN14: now also IC1001.A8 (Y0_DQ0N_1)
- net +1.0V_BE_VDDC: now reaches IC1001.B15 (VDD)
- net +1.0V_BE_VDDC: now also IC1001.A12 (VDD), IC1001.A14 (VDD), IC1001.A16 (VDD), IC1001.A18 (VDD), IC1001.A20 (VDD), IC1001.A22 (VDD), IC1001.A24 (VDD), IC1001.A26 (VDD), IC1001.A28 (VDD), IC1001.AL10 (VDD), IC1001.AL12 (VDD), IC1001.AL14 (VDD), IC1001.AL18 (VDD), IC1001.AL20 (VDD), IC1001.AL22 (VDD), IC1001.AL24 (VDD), IC1001.AL26 (VDD), IC1001.AL28 (VDD), IC1001.AM19 (VDD), IC1001.AM21 (VDD), IC1001.AM23 (VDD), IC1001.AM25 (VDD), IC1001.AM27 (VDD), IC1001.B17 (VDD), IC1001.B19 (VDD), IC1001.B21 (VDD), IC1001.B23 (VDD), IC1001.B25 (VDD), IC1001.B27 (VDD), IC1001.B29 (VDD), IC1001.C12 (VDD), IC1001.C14 (VDD), IC1001.C16 (VDD), IC1001.C18 (VDD), IC1001.C20 (VDD), IC1001.C22 (VDD), IC1001.C24 (VDD), IC1001.C26 (VDD), IC1001.C28 (VDD), IC1001.D13 (VDD), IC1001.D15 (VDD), IC1001.D17 (VDD), IC1001.D19 (VDD), IC1001.D21 (VDD), IC1001.D23 (VDD), IC1001.D25 (VDD), IC1001.D27 (VDD), IC1001.D29 (VDD), IC1001.D31 (VDD), IC1001.D33 (VDD), IC1001.E12 (VDD), IC1001.E14 (VDD), IC1001.E16 (VDD), IC1001.E18 (VDD), IC1001.E20 (VDD), IC1001.E22 (VDD), IC1001.E24 (VDD), IC1001.E26 (VDD), IC1001.E28 (VDD), IC1001.E30 (VDD), IC1001.E32 (VDD), IC1001.F13 (VDD), IC1001.F15 (VDD), IC1001.F17 (VDD), IC1001.F19 (VDD), IC1001.F21 (VDD), IC1001.F23 (VDD), IC1001.F25 (VDD), IC1001.F27 (VDD), IC1001.F29 (VDD), IC1001.F31 (VDD), IC1001.F33 (VDD), IC1001.G12 (VDD), IC1001.G14 (VDD), IC1001.G16 (VDD), IC1001.G18 (VDD), IC1001.G20 (VDD), IC1001.G22 (VDD), IC1001.G24 (VDD), IC1001.G26 (VDD), IC1001.G28 (VDD), IC1001.G30 (VDD), IC1001.G32 (VDD), IC1001.H13 (VDD), IC1001.H15 (VDD), IC1001.H17 (VDD), IC1001.H19 (VDD), IC1001.H21 (VDD), IC1001.H23 (VDD), IC1001.H25 (VDD), IC1001.H27 (VDD), IC1001.H29 (VDD), IC1001.H31 (VDD), IC1001.H33 (VDD), IC1001.J12 (VDD), IC1001.J14 (VDD), IC1001.J16 (VDD), IC1001.J18 (VDD), IC1001.J20 (VDD), IC1001.J22 (VDD), IC1001.J24 (VDD), IC1001.J26 (VDD), IC1001.J28 (VDD), IC1001.J30 (VDD), IC1001.J32 (VDD), IC1001.K11 (VDD), IC1001.K13 (VDD), IC1001.K15 (VDD), IC1001.K17 (VDD), IC1001.K19 (VDD), IC1001.K21 (VDD), IC1001.K23 (VDD), IC1001.K25 (VDD), IC1001.K27 (VDD), IC1001.K29 (VDD), IC1001.K31 (VDD), IC1001.L10 (VDD), IC1001.L12 (VDD), IC1001.L14 (VDD), IC1001.L16 (VDD), IC1001.L18 (VDD), IC1001.L20 (VDD), IC1001.L22 (VDD), IC1001.L24 (VDD), IC1001.L26 (VDD), IC1001.L28 (VDD), IC1001.L30 (VDD), IC1001.L32 (VDD), IC1001.M11 (VDD)

Commit message: pcb update
Parts:
- added R1011: 100, Resistor_SMD:R_0402_1005Metric, symbol Device:R_US
Connections:
- net GND: now also IC1001.AG11 (GND), IC1001.AG31 (GND), IC1001.AG37 (GND), IC1001.AG8 (GND), IC1001.AH10 (GND), IC1001.AH32 (GND), IC1001.AJ11 (GND), IC1001.AJ31 (GND), IC1001.AJ34 (GND), IC1001.AJ5 (GND), IC1001.AJ8 (GND), IC1001.AK10 (GND), IC1001.AK32 (GND), IC1001.AK37 (GND), IC1001.AK4 (GND), IC1001.AK6 (GND), IC1001.AK7 (GND), IC1001.AU1 (GND), IC1001.AU10 (GND), IC1001.AU13 (GND), IC1001.AU22 (GND), IC1001.AU23 (GND), IC1001.AU28 (GND), IC1001.AU29 (GND), IC1001.AU3 (GND), IC1001.AU32 (GND), IC1001.AU33 (GND), IC1001.AU5 (GND), IC1001.AU6 (GND), IC1001.AU9 (GND), IC1001.AV34 (GND), IC1001.AV37 (GND), IC1001.AW1 (GND), IC1001.AW11 (YC_SCAN_IN), IC1001.AW15 (PLL_NC), IC1001.AW34 (GND), IC1001.AW37 (GND), IC1001.BA35 (GND), IC1001.BA36 (GND), IC1001.BA38 (GND), IC1001.BA41 (GND), IC1001.P10 (GND), IC1001.P32 (GND), IC1001.T10 (GND), IC1001.T32 (GND), IC1001.T5 (GND), R1011.1
- net Y1_XDR0_DQ11: now also IC1001.AY2 (Y1_DQ2_4)
- net Y1_XDR0_DQN1: now also IC1001.AW2 (Y1_DQ2N_1)
- net Y1_XDR0_DQN11: now also IC1001.BA2 (Y1_DQ2N_4)
- net Y1_XDR0_DQN13: now also IC1001.AW3 (Y1_DQ2N_5)
- net Y1_XDR0_DQN5: now also IC1001.AW4 (Y1_DQ2N_0)
- net Y1_XDR0_DQN9: now also IC1001.AW5 (Y1_DQ3N_4)
- net Y1_XDR1_DQN11: now also IC1001.AW7 (Y1_DQ2N_3)
- net Y1_XDR1_DQN3: now also IC1001.AW9 (Y1_DQ3N_3)
- net Y1_XDR1_DQN7: now also IC1001.AW8 (Y1_DQ3N_1)
- net BE_TX6_TXP4: now reaches IC1001.BA30 (TX6_TXP4)
- net BE_TX6_TXP0: now reaches IC1001.BA32 (TX6_TXP0)
- net BE_TMS: now reaches IC1001.AW12 (TMS)
- net BE_TDI: now reaches IC1001.AW13 (TDI)
- net BE_TDO: now reaches IC1001.AW14 (TDO)
- net at IC1001.AW18 (PLL_CTL0): now also R1011.2
- net BE_INT: now reaches IC1001.AW19 (ATTENTION)
- net BE_TX6_TXP7: now reaches IC1001.AW29 (TX6_TXP7)
- net BE_TX6_TXP6: now reaches IC1001.AW30 (TX6_TXP6)
- net BE_TX6_TXP2: now reaches IC1001.AW32 (TX6_TXP2)
- net BE_TX6_TXN7: now reaches IC1001.AV29 (TX6_TXN7)
- net BE_TX6_TXN6: now reaches IC1001.AV30 (TX6_TXN6)
- net BE_TX6_TXN2: now reaches IC1001.AV32 (TX6_TXN2)
- no-connect marks 2 -> 10
