File: cok-001/cpu.kicad_sch (KiCad schematic)
At the start: 5 parts

Commit message: cpu pins
Connections:
- net +1.0V_BE_VDDC: now also U1001.E12 (VDD), U1001.E14 (VDD), U1001.E16 (VDD), U1001.E18 (VDD), U1001.E20 (VDD), U1001.E22 (VDD), U1001.E24 (VDD), U1001.E26 (VDD), U1001.E28 (VDD), U1001.E30 (VDD), U1001.E32 (VDD); no longer U1001.AL10 (VDD), U1001.AL12 (VDD), U1001.AL14 (VDD), U1001.AL18 (VDD), U1001.AL20 (VDD), U1001.AL22 (VDD), U1001.AL24 (VDD), U1001.AL26 (VDD), U1001.AL28 (VDD), U1001.AM19 (VDD), U1001.AM21 (VDD), U1001.AM23 (VDD), U1001.AM25 (VDD), U1001.AM27 (VDD), U1001.M11 (VDD)
- net +1.5V_BE_RC_VDDA: no longer U1001.AP29 (RX4_VDDA), U1001.AP30 (TX6_VDDA), U1001.AP34 (RX3_VDDA), U1001.E34 (TX0_VDDA), U1001.F34 (RX0_VDDA)
- net +1.5V_BE_YC_VDDA: now also U1001.AN10 (NC_OPEN51), U1001.AN11 (NC_OPEN52), U1001.AN12 (NC_OPEN53), U1001.AN13 (NC_OPEN54), U1001.AN14 (NC_OPEN55), U1001.AN15 (PLL_NC), U1001.AN16 (PLL_NC), U1001.AN17 (PLL_NC), U1001.AN18 (PLL_NC), U1001.AN19 (NC_OPEN56), U1001.AN20 (NC_OPEN57), U1001.AN21 (NC_OPEN58), U1001.AN22 (NC_OPEN59), U1001.AN23 (NC_OPEN60), U1001.AN24 (NC_OPEN61), U1001.AN25 (NC_OPEN62), U1001.AN26 (NC_OPEN63), U1001.AN27 (NC_OPEN64), U1001.AN28 (NC_OPEN65), U1001.AN29 (NC_OPEN66), U1001.AN30 (NC_OPEN67), U1001.AN31 (NC_OPEN68), U1001.AN32 (NC_OPEN69), U1001.AN33 (NC_OPEN26), U1001.AN35 (GND), U1001.AN36 (GND), U1001.AN9 (NC_OPEN01)
- net GND: now also U1001.E11 (VDDE), U1001.F1 (GND), U1001.F11 (YC_SCAN_CLK4), U1001.F3 (GND), U1001.F32 (GND), U1001.F5 (GND), U1001.G11 (YC_SCAN_CLK3), U1001.G2 (GND), U1001.G4 (GND), U1001.G6 (GND), U1001.H1 (GND), U1001.H10 (GND), U1001.H11 (YC_SCAN_CLK2), U1001.H3 (GND), U1001.H5 (GND), U1001.H7 (GND), U1001.H9 (Y0_DQ0_GNDA), U1001.J10 (YC_SCAN_CLK0), U1001.J11 (YC_SCAN_CLK1), U1001.J33 (NC_OPEN50), U1001.J4 (GND), U1001.J6 (GND), U1001.J9 (NC_OPEN25), U1001.K3 (GND), U1001.K33 (NC_OPEN49), U1001.K5 (GND), U1001.K8 (Y0_DQ1_GNDA), U1001.K9 (NC_OPEN24), U1001.L2 (GND), U1001.L31 (GND), U1001.L33 (NC_OPEN48), U1001.L34 (TX1_GNDA), U1001.L4 (GND), U1001.L6 (GND), U1001.L9 (NC_OPEN23); no longer U1001.AL19 (GND), U1001.AL21 (GND), U1001.AL25 (GND), U1001.AL27 (GND), U1001.AM20 (GND), U1001.AM22 (GND), U1001.AM24 (GND), U1001.AM26 (GND), U1001.AM28 (GND), U1001.AN35 (GND), U1001.AN36 (GND), U1001.AN38 (GND), U1001.AP27 (GND), U1001.AP32 (GND), U1001.AP37 (GND), U1001.AR34 (GND), U1001.AR37 (GND)
- net at U1001.V10 (GND): now also U1001.V32 (GND), U1001.V37 (GND)
- net at U1001.V11 (VDD): now also U1001.V31 (VDD)
- net BE_VDDS2: now reaches U1001.D11 (VDDS2)
- net at U1001.AL1 (GND): now also U1001.AL15 (GND), U1001.AL19 (GND), U1001.AL21 (GND), U1001.AL23 (GND), U1001.AL25 (GND), U1001.AL27 (GND), U1001.AL29 (GND), U1001.AL3 (GND), U1001.AL31 (GND), U1001.AL33 (NC_OPEN28), U1001.AL34 (GND), U1001.AL37 (GND), U1001.AL5 (GND), U1001.AL6 (GND), U1001.AN1 (GND), U1001.AN3 (GND), U1001.AN38 (GND), U1001.AN5 (GND), U1001.AP10 (GND), U1001.AP11 (YC_SCAN_EN), U1001.AP12 (YC_TREF), U1001.AP14 (PLL_NC), U1001.AP15 (PLL_NC), U1001.AP18 (PLL_NC), U1001.AP27 (GND), U1001.AP32 (GND), U1001.AP37 (GND), U1001.AP4 (GND), U1001.AP6 (GND), U1001.AP7 (GND), U1001.AP9 (Y1_DQ3_GNDA), U1001.AR14 (PLL_NC), U1001.AR15 (PLL_NC), U1001.AR16 (PLL_NC), U1001.AR17 (PLL_NC), U1001.AR18 (PLL_NC), U1001.AR25 (RC_TEST_MODE_ST), U1001.AR3 (GND), U1001.AR34 (GND), U1001.AR37 (GND), U1001.AR5 (GND)
- net BE_Y1_RQ0: now reaches U1001.AL2 (Y1_RQ0)
- net at U1001.AL30 (VDD): now also U1001.AL10 (VDD), U1001.AL12 (VDD), U1001.AL18 (VDD), U1001.AL20 (VDD), U1001.AL22 (VDD), U1001.AL24 (VDD), U1001.AL26 (VDD), U1001.AL28 (VDD), U1001.AL32 (VDD)
- net BE_Y1_RQ1: now reaches U1001.AL4 (Y1_RQ1)
- net at U1001.AT11 (GND): now also U1001.AT12 (GND), U1001.AT19 (GND), U1001.AT2 (GND), U1001.AT20 (GND), U1001.AT21 (GND), U1001.AT24 (GND), U1001.AT25 (GND), U1001.AT4 (GND), U1001.AT6 (GND)
- net BE_Y0_RQ_VREF: now reaches U1001.H6 (Y0_RQ_VREF)
- net BE_Y0_RQ_CTM: now reaches U1001.J1 (Y0_RQ_CTMP)
- net BE_Y0_RQ_CTMN: now reaches U1001.J2 (Y0_RQ_CTMN)
- net BE_RC_VOLGND0: now reaches U1001.J34 (RC_VOLGND0)
- net BE_RC_VOLREF0: now reaches U1001.J36 (RC_VOLREF0)
- net BE_RC_RLOAD0: now reaches U1001.J39 (RC_RLOAD0)
- net BE_Y0_DQC_ROLREF: now reaches U1001.J7 (Y0_DQC_ROLREF)
- net BE_Y1_RQ_CTM: now reaches U1001.AP1 (Y1_RQ_CTMP)
- net ~{BE_SPI_CS}: now reaches U1001.AP13 (~{SPI_EN_B})
- net BE_PLL_VDDA: now reaches U1001.AP16 (PLL_VDDA)
- net BE_SYS_CONF2: now reaches U1001.AP19 (SYS_CONFIG2)
- net BE_Y1_RQ_CTMN: now reaches U1001.AP2 (Y1_RQ_CTMN)
- net BE_SYS_CONF0: now reaches U1001.AP20 (SYS_CONFIG0)
- net BE_TBEN: now reaches U1001.AP22 (TBEN)
- net BE_THR_ALRT: now reaches U1001.AP23 (THERMAL_OVERLOAD_B)
- net BE_TRG_IN: now reaches U1001.AP24 (TRIGGER_IN)
- net BE_Y1_RQ7: now reaches U1001.AP3 (Y1_RQ7)
- net BE_Y1_RQ8: now reaches U1001.AP5 (Y1_RQ8)
- net BE_SYS_CONF1: now reaches U1001.AR19 (SYS_CONFIG1)
- net BE_SYS_CONF3: now reaches U1001.AR20 (SYS_CONFIG3)
- net BE_TRG_OUT: now reaches U1001.AR24 (TRIGGER_OUT)
- net BE_RX4_RXP1: now reaches U1001.AR26 (RX4_RXP1)
- net BE_RX4_RXP3: now reaches U1001.AR27 (RX4_RXP3)
- net BE_RX4_RXP5: now reaches U1001.AR28 (RX4_RXP5)
- net BE_RX4_RXP7: now reaches U1001.AR29 (RX4_RXP7)
- net BE_TX6_TXN5: now reaches U1001.AR30 (TX6_TXN5)
- net BE_TX6_TXN3: now reaches U1001.AR31 (TX6_TXN3)
- net BE_TX6_TXN1: now reaches U1001.AR32 (TX6_TXN1)
- net at U1001.M10 (GND): now also U1001.M3 (GND), U1001.M32 (GND), U1001.M5 (GND), U1001.M7 (GND)
- net at U1001.M31 (VDD): now also U1001.M11 (VDD)
- net BE_Y0_RQ_CFMN: now reaches U1001.K1 (Y0_RQ_CFMN)
- net BE_Y0_RQ_CFM: now reaches U1001.K2 (Y0_RQ_CFMP)
- net BE_Y0_RQ9: now reaches U1001.K4 (Y0_RQ9)
- net BE_Y0_RQ_SCK: now reaches U1001.K6 (Y0_RQ_SCK)
- net BE_Y0_DQC_VOLGND: now reaches U1001.K7 (Y0_DQC_VOLGND)
- net BE_Y0_RQ10: now reaches U1001.L1 (Y0_RQ10)
- net BE_Y0_RQ11: now reaches U1001.L3 (Y0_RQ11)
- net BE_Y0_RQ_CMD: now reaches U1001.L5 (Y0_RQ_CMD)
- net BE_Y0_DQC_VOLREF: now reaches U1001.L7 (Y0_DQC_VOLREF)
- net at U1001.Y11 (VDD): now also U1001.Y31 (VDD)
- net BE_Y1_RQ3: now reaches U1001.AM1 (Y1_RQ3)
- net at U1001.AM10 (GND): now also U1001.AM12 (GND), U1001.AM14 (GND), U1001.AM16 (PLL_NC), U1001.AM17 (PLL_NC), U1001.AM18 (GND), U1001.AM2 (GND), U1001.AM20 (GND), U1001.AM22 (GND), U1001.AM24 (GND), U1001.AM26 (GND), U1001.AM28 (GND), U1001.AM30 (GND), U1001.AM32 (GND), U1001.AM4 (GND), U1001.AM6 (GND), U1001.AM8 (Y1_DQ2_GNDA), U1001.AM9 (NC_OPEN02)
- net at U1001.AM11 (VDD): now also U1001.AM13 (VDD), U1001.AM15 (VDD), U1001.AM19 (VDD), U1001.AM21 (VDD), U1001.AM23 (VDD), U1001.AM25 (VDD), U1001.AM27 (VDD), U1001.AM29 (VDD), U1001.AM31 (VDD)
- net BE_Y1_RQ5: now reaches U1001.AM3 (Y1_RQ5)
- net BE_Y1_RQ2: now reaches U1001.AM5 (Y1_RQ2)
- net BE_Y1_DQC_VOLGND: now reaches U1001.AM7 (Y1_DQC_VOLGND)
- net BE_Y1_RQ4: now reaches U1001.AN2 (Y1_RQ4)
- net BE_Y1_RQ6: now reaches U1001.AN4 (Y1_RQ6)
- net BE_Y1_RQ_VREF: now reaches U1001.AN6 (Y1_RQ_VREF)
- net BE_Y1_DQC_ROLREF: now reaches U1001.AN7 (Y1_DQC_ROLREF)
- no-connect marks 53 -> 48

Commit message: lanes
Connections:
- net Y1_XDR0_DQ0: now also U1001.AJ6 (Y1_DQ1_6)
- net Y1_XDR0_DQ10: now also U1001.AJ3 (Y1_DQ1_7)
- net Y1_XDR0_DQ12: now also U1001.AH7 (Y1_DQ1N_4)
- net Y1_XDR0_DQ14: now also U1001.AH3 (Y1_DQ1_5)
- net Y1_XDR0_DQ2: now also U1001.AG3 (Y1_DQ0_6)
- net Y1_XDR0_DQ4: now also U1001.AG6 (Y1_DQ1_2)
- net Y1_XDR0_DQ6: now also U1001.AH1 (Y1_DQ0_3)
- net Y1_XDR0_DQN0: now also U1001.AJ7 (Y1_DQ1N_6)
- net Y1_XDR0_DQN10: now also U1001.AJ4 (Y1_DQ1N_7)
- net Y1_XDR0_DQN12: now also U1001.AH8 (YC_VDDIO)
- net Y1_XDR0_DQN14: now also U1001.AH4 (Y1_DQ1N_5)
- net Y1_XDR0_DQN2: now also U1001.AG4 (Y1_DQ0N_6)
- net Y1_XDR0_DQN4: now also U1001.AG7 (Y1_DQ1N_2)
- net Y1_XDR0_DQN6: now also U1001.AH2 (Y1_DQ0N_3)
- net BE_Y1_DQ0_RLOAD: now reaches U1001.AA1 (Y1_DQ0_RLOAD)
- net BE_RX2_RXP7: now reaches U1001.AA35 (RX2_RXP7)
- net BE_RX2_RXN7: now reaches U1001.AA36 (RX2_RXN7)
- net BE_TX2_TXN7: now reaches U1001.AA38 (TX2_TXN7)
- net BE_TX2_TXP7: now reaches U1001.AA39 (TX2_TXP7)
- net BE_TX3_TXN7: now reaches U1001.AJ38 (TX3_TXN7)
- net BE_TX3_TXP7: now reaches U1001.AJ39 (TX3_TXP7)
- net BE_TX3_TXCLKN: now reaches U1001.AG38 (TX3_TXCLKN)
- net BE_TX3_TXCLKP: now reaches U1001.AG39 (TX3_TXCLKP)
- net BE_Y1_DQC_VOLREF: now reaches U1001.AL7 (Y1_DQC_VOLREF)
- net BE_RX2_RXP3: now reaches U1001.AC35 (RX2_RXP3)
- net BE_RX2_RXN3: now reaches U1001.AC36 (RX2_RXN3)
- net BE_RX2_RXCLKP: now reaches U1001.AC38 (RX2_RXCLKP)
- net BE_RX2_RXCLKN: now reaches U1001.AC39 (RX2_RXCLKN)
- net BE_Y0_DQ2_RLOAD: now reaches U1001.M4 (Y0_DQ2_RLOAD)
- net BE_TX2_TXN3: now reaches U1001.W35 (TX2_TXN3)
- net BE_TX2_TXP3: now reaches U1001.W36 (TX2_TXP3)
- net BE_TX2_TXCLKN: now reaches U1001.W38 (TX2_TXCLKN)
- net BE_TX2_TXCLKP: now reaches U1001.W39 (TX2_TXCLKP)
- net BE_TX3_TXN5: now reaches U1001.AH35 (TX3_TXN5)
- net BE_TX3_TXP5: now reaches U1001.AH36 (TX3_TX5)
- net BE_TX3_TXN6: now reaches U1001.AH38 (TX3_TXN6)
- net BE_TX3_TXP6: now reaches U1001.AH39 (TX3_TXP6)
- net BE_TX3_TXN4: now reaches U1001.AH40 (TX3_TXN4)
- net BE_TX3_TXP4: now reaches U1001.AH41 (TX3_TXP4)
- no-connect marks 48 -> 54
