File: cok-001/cpu.kicad_sch (KiCad schematic)
At the start: 5 parts

Commit message: update 10
Parts:
- U1001: value ~ -> (none)
Connections:
- net +1.0V_BE_VDDC: now also U1001.C12 (VDD)
- net +1.2V_MC2_VDDIO: now also U1001.H8 (Y0_DQ0_VDDA), U1001.J8 (Y0_DQ1_VDDA), U1001.L8 (Y0_RQ_VDDA)
- net +1.2V_YC_RC_VDDIO: now also U1001.A40 (RC_VDDIO), U1001.E37 (RC_VDDIO), U1001.H37 (RC_VDDIO), U1001.J37 (RC_VDDIO), U1001.J38 (RC_ROLREF0)
- net GND: now also U1001.AL1 (GND), U1001.AL15 (GND), U1001.AL19 (GND), U1001.AL21 (GND), U1001.AL23 (GND), U1001.AL25 (GND), U1001.AL27 (GND), U1001.AL29 (GND), U1001.AL3 (GND), U1001.AL31 (GND), U1001.AL33 (NC_OPEN28), U1001.AL34 (GND), U1001.AL37 (GND), U1001.AL5 (GND), U1001.AL6 (GND), U1001.AN1 (GND), U1001.AN3 (GND), U1001.AN38 (GND), U1001.AN5 (GND), U1001.AP10 (GND), U1001.AP11 (YC_SCAN_EN), U1001.AP12 (YC_TREF), U1001.AP14 (PLL_NC), U1001.AP15 (PLL_NC), U1001.AP18 (PLL_NC), U1001.AP27 (GND), U1001.AP32 (GND), U1001.AP37 (GND), U1001.AP4 (GND), U1001.AP6 (GND), U1001.AP7 (GND), U1001.AP9 (Y1_DQ3_GNDA), U1001.AR14 (PLL_NC), U1001.AR15 (PLL_NC), U1001.AR16 (PLL_NC), U1001.AR17 (PLL_NC), U1001.AR18 (PLL_NC), U1001.AR25 (RC_TEST_MODE_ST), U1001.AR3 (GND), U1001.AR34 (GND), U1001.AR37 (GND), U1001.AR5 (GND), U1001.C1 (GND), U1001.D1 (GND)
- no-connect marks 57 -> 59
