File: cok-001/dcdc.kicad_sch (KiCad schematic)
At the start: 5 parts, among them U6303 BD3520FVM-TR, U6304 BD3504FVM-TR, U6305 BD3520FVM-TR, U6602 BD3504FVM-TR

Commit message: add some stupid n channel mosfet
Parts:
- added R6619, R6621, R6622, R6623: 10k, Resistor_SMD:R_0402_1005Metric, symbol Device:R_US
- added U6600: MM3143, Package_SO:TSOP-5_1.65x3.05mm_P0.95mm, symbol PS3:NCP511
- added U6604: XX, Package_SO:TSOP-5_1.65x3.05mm_P0.95mm, symbol PS3:NCP511
- added U6605: MM1573, Package_SO:TSOP-5_1.65x3.05mm_P0.95mm, symbol PS3:NCP511
- U6601: value ~ -> NCP511
Connections:
- net GND: now also R6619.1, R6621.1, R6622.1, R6623.1, U6600.2 (GND), U6604.2 (GND), U6605.2 (GND)
- net SW_3: now reaches U6305.3 (EN)
- net +5V_MISC: now reaches U6305.4 (VCC)
- net +5V_MISC: now also U6303.4 (VCC), U6304.4 (VCC), U6602.4 (VCC), U6600.1 (Vin), U6605.1 (Vin)
- net SW_1.2: now reaches U6602.3 (EN)
- net SW_1.2: now also R6623.2
- net SW2.5: now reaches U6601.3 (Enable)
- net SW2.5: now also R6619.2
- net SW_8_A: now reaches U6304.3 (EN)
- net SW_6: now reaches U6303.3 (EN)
- new net SW3.1: R6622.2, U6600.3 (Enable)
- new net SW3.3: R6621.2, U6605.3 (Enable)
Other:
- moved on the sheet: U6303, U6304, U6305, U6601, U6602

Commit message: av
Parts:
- added C6310, C6316: 100p 50V, Capacitor_SMD:C_0402_1005Metric, symbol Device:C
- added C6355, C6356: 10u 6.3V, Capacitor_SMD:C_0805_2012Metric, symbol Device:C
- added C6358, C6359: 0.1u 10V, Capacitor_SMD:C_0402_1005Metric, symbol Device:C
- added C6362: 1u 10V, Capacitor_SMD:C_0603_1608Metric, symbol Device:C
- added C6365: 0.022u 16V, Capacitor_SMD:C_0402_1005Metric, symbol Device:C
- added FB6302: FerriteBead_Small, symbol Device:FerriteBead_Small
- added Q6308, Q6309: IRF7607PBF, Package_SO:SOP-8_3.9x4.9mm_P1.27mm, symbol Transistor_FET:IRF7607PBF
- added R6355: 220, Resistor_SMD:R_0402_1005Metric, symbol Device:R_US
- added TP9648, TP9655: TestPoint, symbol Connector:TestPoint
Connections:
- net +5V_MISC: now also C6362.1
- net GND: now also C6310.2, C6316.2, C6355.2, C6356.2, C6358.1, C6359.1, C6362.2, C6365.2
- net SW_3: now also C6310.1
- net SW_8_A: now also C6316.1
- net at U6305.1 (NACS): now also C6359.2
- net +1.2V_SB_VDDC: now reaches U6305.6 (VS)
- net +1.2V_SB_VDDC: now also FB6302.2, Q6309.5 (D), Q6309.6 (D), Q6309.7 (D), Q6309.8 (D), TP9648.1
- net at U6305.7 (G): now also Q6309.4 (G), R6355.2
- net at U6304.1 (NACS): now also C6358.2
- net +1.5V_YC_RC_VDDA: now reaches U6304.6 (VS)
- net +1.5V_YC_RC_VDDA: now also Q6308.5 (D), Q6308.6 (D), Q6308.7 (D), Q6308.8 (D), TP9655.1
- net at U6304.7 (G): now also Q6308.4 (G)
- new net: C6365.1, R6355.1
- new net: C6355.1, Q6308.1 (S), Q6308.2 (S), Q6308.3 (S)
- new net: C6356.1, Q6309.1 (S), Q6309.2 (S), Q6309.3 (S)
- new net +1.2V_SB_VDDA: FB6302.1

Commit message: sata
Parts:
- FB6302: footprint (none) -> Resistor_SMD:R_0603_1608Metric
- TP9648, TP9655: footprint (none) -> TestPoint:TestPoint_Pad_1.0x1.0mm
Changed lines of the file:
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@@
 			)
 		)
-		(property "Footprint" ""
+		(property "Footprint" "TestPoint:TestPoint_Pad_1.0x1.0mm"
 			(at 187.96 165.1 0)
 			(effects
@@
 			)
 		)
-		(property "Footprint" ""
+		(property "Footprint" "Resistor_SMD:R_0603_1608Metric"
 			(at 175.26 193.802 90)
 			(effects
@@
 			)
 		)
-		(property "Footprint" ""
+		(property "Footprint" "TestPoint:TestPoint_Pad_1.0x1.0mm"
 			(at 180.34 191.77 0)
 			(effects

Commit message: southbridge
Parts:
- Q6308, Q6309: footprint Package_SO:SOP-8_3.9x4.9mm_P1.27mm -> Package_SO:MSOP-8_3x3mm_P0.65mm
Changed lines of the file:
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@@
 			)
 		)
-		(property "Footprint" "Package_SO:SOP-8_3.9x4.9mm_P1.27mm"
+		(property "Footprint" "Package_SO:MSOP-8_3x3mm_P0.65mm"
 			(at 170.18 161.925 0)
 			(effects
@@
 			)
 		)
-		(property "Footprint" "Package_SO:SOP-8_3.9x4.9mm_P1.27mm"
+		(property "Footprint" "Package_SO:MSOP-8_3x3mm_P0.65mm"
 			(at 168.91 188.595 0)
 			(effects

Commit message: seperate out
Parts:
- added C6320, C6322: 22u 16V, Capacitor_SMD:C_1210_3225Metric, symbol Device:C
- added F6302, F6303: 5A, Fuse:Fuse_1206_3216Metric, symbol Device:Fuse
- added L6302: 1uH, Inductor_SMD:L_TDK_SLF6028, symbol Device:L
- added L6306: 1.4uH, Inductor_SMD:L_TDK_SLF12555, symbol Device:L
- added Q6303, Q6307: SI4336, Package_SO:SSOP-8_3.9x5.05mm_P1.27mm, symbol Transistor_FET:IRF7606PBF
- added Q6305: SI4392, Package_SO:SSOP-8_3.9x5.05mm_P1.27mm, symbol Transistor_FET:IRF7606PBF
- added Q6310, Q6600: SUD40N02, Package_TO_SOT_SMD:TO-252-2, symbol Device:Q_NMOS_Depletion_GDS
- added R6368: 0, Resistor_SMD:R_0402_1005Metric, symbol Device:R_US
- added R6605: 3300, Resistor_SMD:R_0402_1005Metric, symbol Device:R_US
- added R6608: 180, Resistor_SMD:R_0402_1005Metric, symbol Device:R_US
- Q6308: footprint Package_SO:MSOP-8_3x3mm_P0.65mm -> Package_SO:SSOP-8_3.9x5.05mm_P1.27mm
- Q6309: value IRF7607PBF -> SI4866DY; footprint Package_SO:MSOP-8_3x3mm_P0.65mm -> Package_SO:SSOP-8_3.9x5.05mm_P1.27mm
Connections:
- net +1.2V_SB_VDDC: now also C6356.1
- net GND: now also C6320.2, C6322.2, Q6303.1 (S), Q6303.2 (S), Q6303.3 (S), Q6307.1 (S), Q6307.2 (S), Q6307.3 (S)
- net +1.2V_EEGS_VDD: now reaches U6602.6 (VS)
- net at U6602.7 (G): now also Q6600.1 (G)
- net at U6602.8 (VD): now also R6605.1
- net at C6355.1, Q6308.1 (S), Q6308.2 (S)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: now also F6303.2
- net +1.7V_MISC: now reaches Q6309.1 (S), Q6309.2 (S), Q6309.3 (S)
- net +1.7V_MISC: now also F6303.1, Q6310.2 (D), R6368.2; no longer C6356.1
- net at U6303.7 (G): now also Q6310.1 (G)
- net at U6303.8 (VD): now also R6368.1
- new net: F6302.2, L6302.1
- new net: C6320.1, C6322.1, L6302.2, Q6305.5 (D), Q6305.6 (D), Q6305.7 (D), Q6305.8 (D)
- new net: Q6600.2 (D), R6608.2
- new net: L6306.1, Q6303.5 (D), Q6303.6 (D), Q6303.7 (D), Q6303.8 (D), Q6305.1 (S), Q6305.2 (S), Q6305.3 (S), Q6307.5 (D), Q6307.6 (D), Q6307.7 (D), Q6307.8 (D)
- new net: R6605.2, R6608.1
- new net +12V_MAIN: F6302.1
Other:
- moved on the sheet: C6356

Commit message: update to 9
Changed lines of the file:
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@@
 (kicad_sch
-	(version 20231120)
+	(version 20250114)
 	(generator "eeschema")
-	(generator_version "8.0")
+	(generator_version "9.0")
 	(paper "A4")
 	(junction

Commit message: footprints
Parts:
- added F6304: 5A, Fuse:Fuse_1206_3216Metric, symbol Device:Fuse
- added L6303: 1uH, Inductor_SMD:L_TDK_SLF6028, symbol Device:L
- added Q6301: FDQ7238AS, Package_SO:SO-14_3.9x8.65mm_P1.27mm, symbol PS3:FDQ7238AS
- added Q6311: UMH2NTN, Package_TO_SOT_SMD:SOT-363_SC-70-6, symbol Transistor_BJT:MUN5213DW1
- added R6304, R6309: 10k, Resistor_SMD:R_0402_1005Metric, symbol Device:R_US
- added U6603, U6606: MM1561, Package_SO:SSOP-8_3.9x5.05mm_P1.27mm, symbol PS3:MM159X
- added U6607: MM1662, Package_SO:SSOP-8_3.9x5.05mm_P1.27mm, symbol PS3:MM159X
Connections:
- net +1.2V_EEGS_VDD: now also Q6600.3 (S)
- net GND: now also Q6301.5 (D), Q6301.6, Q6301.7, Q6311.1 (E1), Q6311.4 (E2), U6603.2 (NC), U6603.3 (GND), U6603.6 (SUB), U6603.7 (SUB), U6606.2 (NC), U6606.3 (GND), U6606.6 (SUB), U6606.7 (SUB), U6607.2 (NC), U6607.3 (GND), U6607.6 (SUB), U6607.7 (SUB)
- net +3.1V_EEGS_AVDA: now reaches U6600.5 (Vout)
- net +3.3V_MISC: now reaches U6601.1 (Vin)
- net +3.3V_MISC: now also U6604.1 (Vin), R6309.2, U6603.8 (Vin), U6606.8 (Vin), U6607.8 (Vin)
- net +2.5V_EEGS_PLLVDD1: now reaches U6601.5 (Vout)
- net +1.8V_RDRAM_VCMOS: now reaches U6604.5 (Vout)
- net +1.2V_YC_RC_VDDIO: now reaches Q6310.3 (S)
- net +1.2V_YC_RC_VDDIO: now also U6303.6 (VS)
- net +3.3V_DRCG_VDD: now reaches U6605.5 (Vout)
- new net: Q6311.3 (C2), R6309.1
- new net: L6303.2, Q6301.1 (S), Q6301.2 (S)
- new net: Q6301.10, Q6301.11, Q6301.12, Q6301.13, Q6301.14, Q6301.8, Q6301.9
- new net: Q6311.6 (C1), R6304.1
- new net: F6304.2, L6303.1
- new net +1.5V_EEGS_VDD0: U6606.1 (Vout)
- new net +1.8V_EEGS_VDDIO: U6603.1 (Vout)
- new net +2.5V_RDRAM_VDD: U6607.1 (Vout)
- new net +3.3V_EVER: R6304.2
- new net +5V_EVER: F6304.1
Other:
- moved on the sheet: R6622, U6600, U6604

Commit message: pcb update
Parts:
- added Q6302, Q6306: SI4336, Package_SO:SSOP-8_3.9x5.05mm_P1.27mm, symbol Transistor_FET:IRF7606PBF
- added Q6304: SI4392, Package_SO:SSOP-8_3.9x5.05mm_P1.27mm, symbol Transistor_FET:IRF7606PBF
Connections:
- new net: Q6302.5 (D), Q6302.6 (D), Q6302.7 (D), Q6302.8 (D), Q6304.1 (S), Q6304.2 (S), Q6304.3 (S), Q6306.5 (D), Q6306.6 (D), Q6306.7 (D), Q6306.8 (D)
- new net: Q6304.5 (D), Q6304.6 (D), Q6304.7 (D), Q6304.8 (D)
- new net: Q6302.1 (S), Q6302.2 (S), Q6302.3 (S)
- new net: Q6302.4 (G), Q6306.4 (G)
- new net: Q6306.1 (S), Q6306.2 (S), Q6306.3 (S)
