File: cok-001/dcdc.kicad_sch (KiCad schematic)
At the start: 52 parts, among them Q6301 FDQ7238AS, Q6302 SI4336, Q6303 SI4336, Q6304 SI4392, Q6305 SI4392, Q6306 SI4336, Q6307 SI4336, Q6308 IRF7607PBF, Q6309 SI4866DY, Q6310 SUD40N02, Q6311 UMH2NTN, Q6600 SUD40N02, U6303 BD3520FVM-TR, U6304 BD3504FVM-TR, U6305 BD3520FVM-TR, U6600 MM3143, U6601 NCP511, U6602 BD3504FVM-TR, U6603 MM1561, U6604 XX, U6605 MM1573, U6606 MM1561, U6607 MM1662

Commit message: switching regulator
Parts:
- added U6301: SN105233DBTR, Package_SO:TSSOP-30_4.4x7.8mm_P0.5mm, symbol PS3:TPS5120
Changed lines of the file:
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@@
+	)
+	(symbol
+		(lib_id "PS3:TPS5120")
+		(at -30.48 130.81 0)
+		(unit 1)
+		(exclude_from_sim no)
+		(in_bom yes)
+		(on_board yes)
+		(dnp no)
+		(fields_autoplaced yes)
+		(property "Reference" "U6301"
+			(at -30.48 130.81 0)
+			(effects
+				(font
+					(size 1.27 1.27)
+				)
+			)
+		)
+		(property "Value" "SN105233DBTR"
+			(at -30.48 133.35 0)
+			(effects
+				(font
+					(size 1.27 1.27)
+				)
+			)
+		)
+		(property "Footprint" "Package_SO:TSSOP-30_4.4x7.8mm_P0.5mm"
+			(at -30.48 130.81 0)
+			(effects
+				(font
+					(size 1.27 1.27)
+				)
+				(hide yes)
+			)
+		)
+		(property "Datasheet" ""
+			(at -30.48 130.81 0)
+			(effects
+				(font
+					(size 1.27 1.27)
+				)
+				(hide yes)
+			)
+		)
+		(property "Description" ""
+			(at -30.48 130.81 0)
+			(effects
+				(font
+					(size 1.27 1.27)
+				)
+				(hide yes)
+			)
+		)
+		(pin "12"
+		)
+		(pin "28"
+		)
+		(pin "24"
+		)
+		(pin "9"
+		)
+		(pin "11"
+		)
+		(pin "17"
+		)
+		(pin "7"
+		)
+		(pin "30"
+		)
+		(pin "29"
+		)
+		(pin "10"
+		)
+		(pin "27"
+		)
+		(pin "14"
+		)
+		(pin "21"
+		)
+		(pin "5"
+		)
+		(pin "1"
+		)
+		(pin "25"
+		)
+		(pin "15"
+		)
+		(pin "6"
+		)
+		(pin "26"
+		)
+		(pin "22"
+		)
+		(pin "18"
+		)
+		(pin "4"
+		)
+		(pin "19"
+		)
+		(pin "16"
+		)
+		(pin "20"
+		)
+		(pin "13"
+		)
+		(pin "23"
+		)
+		(pin "3"
+		)
+		(pin "8"
+		)
+		(pin "2"
+		)
+		(instances
+			(project ""
+				(path "/976eb78d-8215-4cc0-9d72-f9d535c7970b/7ae61751-b28b-4bb2-bf4e-5615938a2f1e"
+					(reference "U6301")
+					(unit 1)
+				)
+			)
+		)
 	)
 	(symbol

Commit message: temp sensor and clock
Parts:
- added L6305: 1.4uH, Inductor_SMD:L_TDK_SLF12555, symbol Device:L
Connections:
- net at Q6302.5 (D), Q6302.6 (D), Q6302.7 (D)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: now also L6305.1
Changed lines of the file:
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@@
 	)
 	(junction
+		(at -3.81 76.2)
+		(diameter 0)
+		(color 0 0 0 0)
+	)
+	(junction
 		(at 166.37 138.43)
 		(diameter 0)
@@
 	(wire
 		(pts
+			(xy -3.81 76.2) (xy 1.27 76.2)
+		)
+		(stroke
+			(width 0)
+			(type default)
+		)
+	)
+	(wire
+		(pts
 			(xy 66.04 106.68) (xy 67.31 106.68)
 		)
@@
 					(unit 1)
 				)
+			)
+		)
+	)
+	(symbol
+		(lib_id "Device:L")
+		(at 5.08 76.2 90)
+		(unit 1)
+		(exclude_from_sim no)
+		(in_bom yes)
+		(on_board yes)
+		(dnp no)
+		(fields_autoplaced yes)
+		(property "Reference" "L6305"
+			(at 5.08 71.12 90)
+			(effects
+				(font
+					(size 1.27 1.27)
+				)
+			)
+		)
+		(property "Value" "1.4uH"
+			(at 5.08 73.66 90)
+			(effects
+				(font
+					(size 1.27 1.27)
+				)
+			)
+		)
+		(property "Footprint" "Inductor_SMD:L_TDK_SLF12555"
+			(at 5.08 76.2 0)
+			(effects
+				(font
+					(size 1.27 1.27)
+				)
+				(hide yes)
+			)
+		)
+		(property "Datasheet" "~"
+			(at 5.08 76.2 0)
+			(effects
+				(font
+					(size 1.27 1.27)
+				)
+				(hide yes)
+			)
+		)
+		(property "Description" "Inductor"
+			(at 5.08 76.2 0)
+			(effects
+				(font
+					(size 1.27 1.27)
+				)
+				(hide yes)
+			)
+		)
+		(pin "1"
+		)
+		(pin "2"
+		)
+		(instances
+			(project "cok-001"
+				(path "/976eb78d-8215-4cc0-9d72-f9d535c7970b/7ae61751-b28b-4bb2-bf4e-5615938a2f1e"
+					(reference "L6305")
+					(unit 1)
+				)

Commit message: powea
Parts:
- added U6302: TPS51117, Package_SO:TSSOP-14_4.4x5mm_P0.65mm, symbol PS3:TPS51117
Connections:
- net GND: now also U6302.7 (GND)
Changed lines of the file:
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@@
+	)
+	(symbol
+		(lib_id "PS3:TPS51117")
+		(at 59.69 -1.27 0)
+		(unit 1)
+		(exclude_from_sim no)
+		(in_bom yes)
+		(on_board yes)
+		(dnp no)
+		(fields_autoplaced yes)
+		(property "Reference" "U6302"
+			(at 59.69 -5.08 0)
+			(effects
+				(font
+					(size 1.27 1.27)
+				)
+			)
+		)
+		(property "Value" "TPS51117"
+			(at 59.69 -2.54 0)
+			(effects
+				(font
+					(size 1.27 1.27)
+				)
+			)
+		)
+		(property "Footprint" "Package_SO:TSSOP-14_4.4x5mm_P0.65mm"
+			(at 59.69 -1.27 0)
+			(effects
+				(font
+					(size 1.27 1.27)
+				)
+				(hide yes)
+			)
+		)
+		(property "Datasheet" ""
+			(at 59.69 -1.27 0)
+			(effects
+				(font
+					(size 1.27 1.27)
+				)
+				(hide yes)
+			)
+		)
+		(property "Description" ""
+			(at 59.69 -1.27 0)
+			(effects
+				(font
+					(size 1.27 1.27)
+				)
+				(hide yes)
+			)
+		)
+		(pin "11"
+		)
+		(pin "14"
+		)
+		(pin "4"
+		)
+		(pin "3"
+		)
+		(pin "13"
+		)
+		(pin "9"
+		)
+		(pin "7"
+		)
+		(pin "2"
+		)
+		(pin "10"
+		)
+		(pin "12"
+		)
+		(pin "1"
+		)
+		(pin "8"
+		)
+		(pin "6"
+		)
+		(pin "5"
+		)
+		(instances
+			(project ""
+				(path "/976eb78d-8215-4cc0-9d72-f9d535c7970b/7ae61751-b28b-4bb2-bf4e-5615938a2f1e"
+					(reference "U6302")
+					(unit 1)
+				)
+			)
+		)
 	)
 	(symbol
@@
 					(unit 1)
 				)
+			)
+		)
+	)
+	(symbol
+		(lib_id "power:GND")
+		(at 49.53 16.51 0)
+		(unit 1)
+		(exclude_from_sim no)
+		(in_bom yes)
+		(on_board yes)
+		(dnp no)
+		(fields_autoplaced yes)
+		(property "Reference" "#PWR0326"
+			(at 49.53 22.86 0)
+			(effects
+				(font
+					(size 1.27 1.27)
+				)
+				(hide yes)
+			)
+		)
+		(property "Value" "GND"
+			(at 49.53 21.59 0)
+			(effects
+				(font
+					(size 1.27 1.27)
+				)
+			)
+		)
+		(property "Footprint" ""
+			(at 49.53 16.51 0)
+			(effects
+				(font
+					(size 1.27 1.27)
+				)
+				(hide yes)
+			)
+		)
+		(property "Datasheet" ""
+			(at 49.53 16.51 0)
+			(effects
+				(font
+					(size 1.27 1.27)
+				)
+				(hide yes)
+			)
+		)
+		(property "Description" "Power symbol creates a global label with name \"GND\" , ground"
+			(at 49.53 16.51 0)
+			(effects
+				(font
+					(size 1.27 1.27)
+				)
+				(hide yes)
+			)
+		)
+		(pin "1"
+		)
+		(instances
+			(project "cok-001"
+				(path "/976eb78d-8215-4cc0-9d72-f9d535c7970b/7ae61751-b28b-4bb2-bf4e-5615938a2f1e"
+					(reference "#PWR0326")
+					(unit 1)
+				)

Commit message: msop
Parts:
- U6303, U6304, U6305, U6602: footprint Package_SO:MSOP-8_3x3mm_P0.65mm -> PS3:MSOP-8_2.9x4mm_P0.65mm
Changed lines of the file:
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@@
 			)
 		)
-		(property "Footprint" "Package_SO:MSOP-8_3x3mm_P0.65mm"
+		(property "Footprint" "PS3:MSOP-8_2.9x4mm_P0.65mm"
 			(at 127 184.15 0)
 			(effects
@@
 			)
 		)
-		(property "Footprint" "Package_SO:MSOP-8_3x3mm_P0.65mm"
+		(property "Footprint" "PS3:MSOP-8_2.9x4mm_P0.65mm"
 			(at 125.73 105.41 0)
 			(effects
@@
 			)
 		)
-		(property "Footprint" "Package_SO:MSOP-8_3x3mm_P0.65mm"
+		(property "Footprint" "PS3:MSOP-8_2.9x4mm_P0.65mm"
 			(at 128.27 157.48 0)
 			(effects
@@
 			)
 		)
-		(property "Footprint" "Package_SO:MSOP-8_3x3mm_P0.65mm"
+		(property "Footprint" "PS3:MSOP-8_2.9x4mm_P0.65mm"
 			(at 127 130.81 0)
 			(effects
