File: cok-001/av.kicad_sch (KiCad schematic)
At the start: 26 parts, among them Q2401 DTC144E, Q2402 SI2303BDS, U2402 L7809, U2403 L7805

Commit message: sata
Parts:
- C2444, C2452, C2459, C2461: footprint Resistor_SMD:R_0805_2012Metric -> Capacitor_SMD:C_0805_2012Metric
- C2451, C2460: footprint Resistor_SMD:R_0402_1005Metric -> Capacitor_SMD:C_0402_1005Metric
Changed lines of the file:
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@@
 			)
 		)
-		(property "Footprint" "Resistor_SMD:R_0402_1005Metric"
+		(property "Footprint" "Capacitor_SMD:C_0402_1005Metric"
 			(at 228.2952 95.25 0)
 			(effects
@@
 			)
 		)
-		(property "Footprint" "Resistor_SMD:R_0402_1005Metric"
+		(property "Footprint" "Capacitor_SMD:C_0402_1005Metric"
 			(at 276.5552 95.25 0)
 			(effects
@@
 			)
 		)
-		(property "Footprint" "Resistor_SMD:R_0805_2012Metric"
+		(property "Footprint" "Capacitor_SMD:C_0805_2012Metric"
 			(at 250.4948 95.25 0)
 			(effects
@@
 			)
 		)
-		(property "Footprint" "Resistor_SMD:R_0805_2012Metric"
+		(property "Footprint" "Capacitor_SMD:C_0805_2012Metric"
 			(at 202.2348 95.25 0)
 			(effects
@@
 			)
 		)
-		(property "Footprint" "Resistor_SMD:R_0805_2012Metric"
+		(property "Footprint" "Capacitor_SMD:C_0805_2012Metric"
 			(at 234.6452 87.63 0)
 			(effects
@@
 			)
 		)
-		(property "Footprint" "Resistor_SMD:R_0805_2012Metric"
+		(property "Footprint" "Capacitor_SMD:C_0805_2012Metric"
 			(at 282.9052 87.63 0)
 			(effects

Commit message: seperate out
Parts:
- added C2404, C2405, C2411: 2.2u 25V, Capacitor_Tantalum_SMD:CP_EIA-3216-10_Kemet-I, symbol Device:C_Polarized_US
- added C2406, C2407, C2408: 0.1u 16V, Capacitor_SMD:C_0603_1608Metric, symbol Device:C
- added C2409: 0.1u 10V, Capacitor_SMD:C_0402_1005Metric, symbol Device:C
- added C2410: 2.2u 25V, Capacitor_Tantalum_SMD:CP_EIA-3528-12_Kemet-T, symbol Device:C_Polarized_US
- added R2429, R2430: 2200, Resistor_SMD:R_0402_1005Metric, symbol Device:R_US
- added TP2404, TP2407, TP2408, TP2409, TP2410: TestPoint, TestPoint:TestPoint_Pad_1.0x1.0mm, symbol Connector:TestPoint
- U2402: value L7809 -> MC78M09
- U2403: value L7805 -> MC78M05
- U2407, U2408: footprint Package_SO:SOP-8_3.9x4.9mm_P1.27mm -> Package_SO:SSOP-8_3.9x5.05mm_P1.27mm
Connections:
- net GND: now also U2406.1 (AVS), U2406.12 (GND_YCCVBS), U2406.14 (AGND1), U2406.22 (VSS), U2406.25 (AVS), U2406.28 (AVS), U2406.29 (VSS), U2406.3 (TESTIN), U2406.33 (VSS), U2406.4 (TESTSEL), U2406.43 (VSS), U2406.56 (VSS), U2406.6 (AGND2), U2406.71 (VSS), U2406.8 (GND_RGB), U2406.82 (VSS), U2406.94 (VSS), U2406.95 (VSSP), U2406.97 (AVS), C2404.2, C2405.2, C2406.2, C2407.2, C2408.2, C2409.2, C2410.2, C2411.2
- net at Q2402.3 (D), U2402.1 (IN), U2403.1 (IN): now also C2404.1, C2405.1, C2406.1, C2407.1
- net at U2403.3 (OUT): now also C2409.1, C2410.1
- net at U2406.10 (AVCC2): now also U2406.16 (AVCC1)
- net at U2406.100 (AVD): now also U2406.24 (AVD), U2406.27 (AVD), U2406.98 (AVD), R2429.2, R2430.2
- net at U2406.17 (S2): now also TP2410.1
- net at U2406.18 (DL3): now also TP2409.1
- net at U2406.19 (DL2): now also TP2408.1
- net at U2406.20 (DL1): now also TP2407.1
- net at U2406.21 (DVD): now also U2406.42 (DVD), U2406.51 (DVD), U2406.60 (DVD), U2406.70 (DVD), U2406.81 (DVD), U2406.88 (DVD), U2406.96 (DVDP)
- net at U2406.34 (FLDD): now also TP2404.1
- net DVE_I2C_SCL: now reaches U2406.35 (SCL)
- net DVE_I2C_SCL: now also R2430.1
- net DVE_I2C_SDA: now reaches U2406.36 (SDA)
- net DVE_I2C_SDA: now also R2429.1
- net at U2402.3 (OUT): now also C2408.1, C2411.1

Commit message: update to 9
Parts:
- added RN2401, RN2402, RN2403, RN2404, RN2405, RN2406, RN2407, RN2408, RN2409: 22, Resistor_SMD:R_Array_Convex_4x0402, symbol Device:R_Pack04
Connections:
- net at U2406.37 (R11): now also RN2401.8 (R1.2)
- net at U2406.38 (R10): now also RN2402.5 (R4.2)
- net at U2406.39 (R9): now also RN2402.6 (R3.2)
- net at U2406.40 (R8): now also RN2401.7 (R2.2)
- net at U2406.41 (R7): now also RN2402.7 (R2.2)
- net at U2406.44 (R6): now also RN2401.6 (R3.2)
- net at U2406.45 (R5): now also RN2402.8 (R1.2)
- net at U2406.46 (R4): now also RN2401.5 (R4.2)
- net at U2406.47 (R3): now also RN2404.5 (R4.2)
- net at U2406.48 (R2): now also RN2403.8 (R1.2)
- net at U2406.49 (R1): now also RN2403.7 (R2.2)
- net at U2406.50 (R0): now also RN2403.6 (R3.2)
- net at U2406.52 (G11): now also RN2404.6 (R3.2)
- net at U2406.53 (G10): now also RN2403.5 (R4.2)
- net at U2406.54 (G9): now also RN2404.7 (R2.2)
- net at U2406.55 (G8): now also RN2404.8 (R1.2)
- net at U2406.57 (G7): now also RN2405.8 (R1.2)
- net at U2406.59 (G5): now also RN2405.7 (R2.2)
- net at U2406.62 (G3): now also RN2405.6 (R3.2)
- net at U2406.64 (G1): now also RN2405.5 (R4.2)
- net at U2406.67 (B10): now also RN2407.8 (R1.2)
- net at U2406.69 (B8): now also RN2407.7 (R2.2)
- net at U2406.73 (B6): now also RN2407.6 (R3.2)
- net at U2406.75 (B4): now also RN2407.5 (R4.2)

Commit message: footprints
Parts:
- added FL2401, FL2402, FL2403: Filter_EMI_LCL, Filter:Filter_Mini-Circuits_FV1206-7, symbol Device:Filter_EMI_LCL
- added J2401: Conn_01x12_MountingPin, PS3:AVOUT, symbol Connector_Generic_MountingPin:Conn_01x12_MountingPin
- added R2471, R2473, R2474, R2475, R2476, R2477: 0, Resistor_SMD:R_0603_1608Metric, symbol Device:R_US
- added TP9203, TP9204, TP9205, TP9206, TP9207, TP9208, TP9209, TP9210, TP9211: TestPoint, TestPoint:TestPoint_Pad_D1.5mm, symbol Connector:TestPoint
Connections:
- net GND: now also FL2401.2, FL2402.2, FL2403.2, J2401.10 (Pin_10), J2401.5 (Pin_5), J2401.MP (MountPin)
- new net: FL2403.3, J2401.4 (Pin_4), TP9206.1
- new net: J2401.6 (Pin_6), R2473.2, TP9207.1
- new net: FL2401.3, J2401.1 (Pin_1), TP9203.1
- new net: J2401.9 (Pin_9), R2476.2, TP9210.1
- new net: J2401.3 (Pin_3), R2471.2, TP9205.1
- new net: J2401.8 (Pin_8), R2475.2, TP9209.1
- new net: FL2402.3, J2401.2 (Pin_2), TP9204.1
- new net: J2401.11 (Pin_11), R2477.2, TP9211.1
- new net: J2401.7 (Pin_7), R2474.2, TP9208.1
- new net GNDA: J2401.12 (Pin_12)

Commit message: rgb
Parts:
- J2401: value Conn_01x12_MountingPin -> AV OUT
Connections:
- net at FL2403.1: now also C2455.2
- net at C2458.2: now also R2475.1
- net at C2453.2: now also FL2402.1
- net at R2473.1: now also C2456.1
- net at C2457.2: now also R2474.1
- net at FL2401.1: now also C2454.2
Other:
- moved on the sheet: R2471
Changed lines of the file:
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@@
 	(wire
 		(pts
+			(xy 142.24 80.01) (xy 157.48 80.01)
+		)
+		(stroke
+			(width 0)
+			(type default)
+		)
+	)
+	(wire
+		(pts
 			(xy 86.36 104.14) (xy 86.36 111.76)
 		)
@@
 	(wire
 		(pts
+			(xy 191.77 29.21) (xy 162.56 29.21)
+		)
+		(stroke
+			(width 0)
+			(type default)
+		)
+	)
+	(wire
+		(pts
 			(xy 27.94 80.01) (xy 5.08 80.01)
 		)
@@
 	(wire
 		(pts
+			(xy 160.02 74.93) (xy 160.02 22.86)
+		)
+		(stroke
+			(width 0)
+			(type default)
+		)
+	)
+	(wire
+		(pts
 			(xy 251.46 87.63) (xy 251.46 80.01)
 		)
@@
 	(wire
 		(pts
+			(xy 142.24 74.93) (xy 160.02 74.93)
+		)
+		(stroke
+			(width 0)
+			(type default)
+		)
+	)
+	(wire
+		(pts
 			(xy 227.33 129.54) (xy 242.57 129.54)
 		)
@@
 	(wire
 		(pts
+			(xy 160.02 22.86) (xy 177.8 22.86)
+		)
+		(stroke
+			(width 0)
+			(type default)
+		)
+	)
+	(wire
+		(pts
 			(xy 11.43 54.61) (xy 11.43 52.07)
 		)
@@
 	(wire
 		(pts
+			(xy 170.18 45.72) (xy 193.04 45.72)
+		)
+		(stroke
+			(width 0)
+			(type default)
+		)
+	)
+	(wire
+		(pts
 			(xy 12.7 3.81) (xy 34.29 3.81)
 		)
@@
 	(wire
 		(pts
+			(xy 170.18 69.85) (xy 170.18 45.72)
+		)
+		(stroke
+			(width 0)
+			(type default)
+		)
+	)
+	(wire
+		(pts
 			(xy 2.54 74.93) (xy 2.54 85.09)
 		)
@@
 	(wire
 		(pts
+			(xy 172.72 64.77) (xy 172.72 43.18)
+		)
+		(stroke
+			(width 0)
+			(type default)
+		)
+	)
+	(wire
+		(pts
 			(xy 54.61 22.86) (xy 54.61 15.24)
 		)
@@
 	(wire
 		(pts
+			(xy 157.48 80.01) (xy 157.48 20.32)
+		)
+		(stroke
+			(width 0)
+			(type default)
+		)
+	)
+	(wire
+		(pts
 			(xy 210.82 38.1) (xy 223.52 38.1)
 		)
@@
 	(wire
 		(pts
-			(xy 187.96 43.18) (xy 187.96 24.13)
+			(xy 187.96 35.56) (xy 187.96 24.13)
 		)
 		(stroke
@@
 	(wire
 		(pts
+			(xy 157.48 20.32) (xy 191.77 20.32)
+		)
+		(stroke
+			(width 0)
+			(type default)
+		)
+	)
+	(wire
+		(pts
 			(xy 227.33 166.37) (xy 242.57 166.37)
 		)
@@
 	(wire
 		(pts
+			(xy 191.77 27.94) (xy 191.77 29.21)
+		)
+		(stroke
+			(width 0)
+			(type default)
+		)
+	)
+	(wire
+		(pts
 			(xy 46.99 22.86) (xy 46.99 -13.97)
 		)
@@
 	(wire
 		(pts
+			(xy 142.24 85.09) (xy 162.56 85.09)
+		)
+		(stroke
+			(width 0)
+			(type default)
+		)
+	)
+	(wire
+		(pts
 			(xy 59.69 22.86) (xy 59.69 -24.13)
 		)
@@
 	(wire
 		(pts
+			(xy 167.64 48.26) (xy 167.64 59.69)
+		)
+		(stroke
+			(width 0)
+			(type default)
+		)
+	)
+	(wire
+		(pts
 			(xy 109.22 107.95) (xy 109.22 36.83)
 		)
@@
 	(wire
 		(pts
+			(xy 193.04 48.26) (xy 167.64 48.26)
+		)
+		(stroke
+			(width 0)
+			(type default)
+		)
+	)
+	(wire
+		(pts
 			(xy 36.83 1.27) (xy 12.7 1.27)
 		)
@@
 	(wire
 		(pts
+			(xy 167.64 59.69) (xy 142.24 59.69)
+		)
+		(stroke
+			(width 0)
+			(type default)
+		)
+	)
+	(wire
+		(pts
 			(xy 205.74 43.18) (xy 205.74 33.02)
 		)
@@
 	(wire
 		(pts
+			(xy 172.72 43.18) (xy 193.04 43.18)
+		)
+		(stroke
+			(width 0)
+			(type default)
+		)
+	)
+	(wire
+		(pts
 			(xy 212.09 83.82) (xy 212.09 85.09)
 		)
@@
 	(wire
 		(pts
+			(xy 142.24 64.77) (xy 172.72 64.77)
+		)
+		(stroke
+			(width 0)
+			(type default)
+		)
+	)
+	(wire
+		(pts
 			(xy 69.85 -13.97) (xy 72.39 -13.97)
 		)
@@
 	(wire
 		(pts
-			(xy 182.88 43.18) (xy 187.96 43.18)
+			(xy 175.26 35.56) (xy 187.96 35.56)
+		)
+		(stroke
+			(width 0)
+			(type default)
+		)
+	)
+	(wire
+		(pts
+			(xy 162.56 85.09) (xy 162.56 29.21)
+		)
+		(stroke
+			(width 0)
+			(type default)
+		)
+	)
+	(wire
+		(pts
+			(xy 142.24 69.85) (xy 170.18 69.85)
 		)
 		(stroke
@@
 	)
 	(symbol
-		(lib_id "power:GND")
-		(at 185.42 27.94 0)
-		(unit 1)
-		(exclude_from_sim no)
-		(in_bom yes)
-		(on_board yes)
-		(dnp no)
-		(fields_autoplaced yes)
-		(property "Reference" "#PWR0258"
-			(at 185.42 34.29 0)
-			(effects
-				(font
-					(size 1.27 1.27)
-				)
-				(hide yes)
-			)
-		)
-		(property "Value" "GND"
-			(at 185.42 33.02 0)
-			(effects
-				(font
-					(size 1.27 1.27)
-				)
-			)
-		)
-		(property "Footprint" ""
-			(at 185.42 27.94 0)
-			(effects
-				(font
-					(size 1.27 1.27)
-				)
-				(hide yes)
-			)
-		)
-		(property "Datasheet" ""
-			(at 185.42 27.94 0)
-			(effects
-				(font
-					(size 1.27 1.27)
-				)
-				(hide yes)
-			)
-		)
-		(property "Description" "Power symbol creates a global label with name \"GND\" , ground"
-			(at 185.42 27.94 0)
-			(effects
-				(font
-					(size 1.27 1.27)
-				)
-				(hide yes)
-			)
-		)
-		(pin "1"
-		)
-		(instances
-			(project "cok-001"
-				(path "/976eb78d-8215-4cc0-9d72-f9d535c7970b/2ac218b5-28da-4878-811c-803b1ba4c592"
-					(reference "#PWR0258")
-					(unit 1)
-				)
-			)
-		)
-	)
-	(symbol
 		(lib_id "Device:C_Polarized_US")
 		(at 227.33 133.35 0)
@@
 	(symbol
 		(lib_id "Device:R_US")
-		(at 179.07 43.18 90)
+		(at 171.45 35.56 90)
 		(unit 1)
 		(exclude_from_sim no)
@@
 		(dnp no)
 		(property "Reference" "R2471"
-			(at 173.228 41.91 90)
+			(at 165.608 34.29 90)
 			(effects
 				(font
@@
 		)
 		(property "Value" "0"
-			(at 182.626 41.91 90)
+			(at 175.006 34.29 90)
 			(effects
 				(font
@@
 		)
 		(property "Footprint" "Resistor_SMD:R_0603_1608Metric"
-			(at 179.324 42.164 90)
+			(at 171.704 34.544 90)
 			(effects
 				(font
@@
 		)
 		(property "Datasheet" "~"
-			(at 179.07 43.18 0)
+			(at 171.45 35.56 0)
 			(effects
 				(font
@@
 		)
 		(property "Description" "Resistor, US symbol"
-			(at 179.07 43.18 0)
+			(at 171.45 35.56 0)
 			(effects
 				(font
@@
 	(symbol
 		(lib_id "power:GND")
+		(at 185.42 27.94 0)
+		(unit 1)
+		(exclude_from_sim no)
+		(in_bom yes)
+		(on_board yes)
+		(dnp no)
+		(fields_autoplaced yes)
+		(property "Reference" "#PWR0258"
+			(at 185.42 34.29 0)
+			(effects
+				(font
+					(size 1.27 1.27)
+				)
+				(hide yes)
+			)
+		)
+		(property "Value" "GND"
+			(at 185.42 33.02 0)
+			(effects
+				(font
+					(size 1.27 1.27)
+				)
+			)
+		)
+		(property "Footprint" ""
+			(at 185.42 27.94 0)
+			(effects
+				(font
+					(size 1.27 1.27)
+				)
+				(hide yes)
+			)
+		)
+		(property "Datasheet" ""
+			(at 185.42 27.94 0)
+			(effects
+				(font
+					(size 1.27 1.27)
+				)
+				(hide yes)
+			)
+		)
+		(property "Description" "Power symbol creates a global label with name \"GND\" , ground"
+			(at 185.42 27.94 0)
+			(effects
+				(font
+					(size 1.27 1.27)
+				)
+				(hide yes)
+			)
+		)
+		(pin "1"
+		)
+		(instances
+			(project "cok-001"
+				(path "/976eb78d-8215-4cc0-9d72-f9d535c7970b/2ac218b5-28da-4878-811c-803b1ba4c592"
+					(reference "#PWR0258")
+					(unit 1)
+				)
+			)
+		)
+	)
+	(symbol
+		(lib_id "power:GND")
 		(at 242.57 166.37 0)
 		(unit 1)
@@
 			)
 		)
-		(property "Value" "Conn_01x12_MountingPin"
+		(property "Value" "AV OUT"
 			(at 231.14 35.9155 0)
 			(effects

Commit message: pcb update
Parts:
- added R2419, R2420, R2421, R2480: 0, Resistor_SMD:R_0402_1005Metric, symbol Device:R_US
- added U2405: CX4351, Package_SO:SSOP-20_4.4x6.5mm_P0.65mm, symbol PS3:CX4351
Connections:
- new net: R2420.2, U2405.2 (SCLK)
- new net: R2419.2, U2405.1 (SDIN)
- new net: R2421.2, U2405.3 (LACK)
- new net: R2480.2, U2405.4 (MCLK)
- new net ADAC_MCLKO0: R2480.1
- new net RS_BCLKO: R2420.1
- new net RS_LRCKO: R2421.1
- new net RS_SDOUT0: R2419.1

Commit message: cr
Parts:
- added D2401: DAP202UT106, Package_TO_SOT_SMD:SOT-323_SC-70, symbol Device:D_Dual_CommonAnode_KKA
- added Q2403: IMH20T108, Package_TO_SOT_SMD:ROHM_SOT-457_ClockwisePinNumbering, symbol PS3:Q_Dual_NPN_NPN_BRT_No_R2_C1E2B2C2E1B1
- added Q2404: DTA144E, Package_TO_SOT_SMD:SOT-323_SC-70, symbol Transistor_BJT:DTA144E
- added R2415: XX, Resistor_SMD:R_0402_1005Metric, symbol Device:R_US
- added R2416, R2417: 4700, Resistor_SMD:R_0402_1005Metric, symbol Device:R_US
- added R2422: 0, Resistor_SMD:R_0805_2012Metric, symbol Device:R_US
Connections:
- net GND: now also U2405.16 (GND), U2405.6 (GND), Q2403.2 (E2), Q2403.5 (E1), R2415.1, R2416.1, R2417.1
- net at RN2409.5 (R4.2): now also U2406.79 (B0)
- net at RN2409.6 (R3.2): now also U2406.78 (B1)
- net at RN2409.7 (R2.2): now also U2406.77 (B2)
- net at RN2409.8 (R1.2): now also U2406.76 (B3)
- net +3.3V_ANA: now reaches C2452.1, U2407.1 (Vout)
- net +3.3V_ANA: now also R2422.1
- net RSX_GPIO7: now reaches U2405.10 (~{RST})
- net at U2405.5 (VD): now also R2422.2
- net at U2405.7 (DIF1): now also R2415.2
- net at U2405.8 (DIF0): now also R2416.2
- net at U2405.9 (DEM): now also R2417.2
- new net: D2401.3 (A), Q2404.1 (B)
- new net: Q2403.3 (B2), Q2403.6 (B1), Q2404.3 (C)
- no-connect marks 0 -> 3
Other:
- moved on the sheet: RN2409

Commit message: rsx vo
Connections:
- net RSX_VO65: now reaches RN2402.1 (R1.1)
- net RSX_VO67: now reaches RN2402.2 (R2.1)
- net RSX_VO69: now reaches RN2402.3 (R3.1)
- net RSX_VO70: now reaches RN2402.4 (R4.1)
- net RSX_VO56: now reaches RN2404.1 (R1.1)
- net RSX_VO57: now reaches RN2404.2 (R2.1)
- net RSX_VO59: now reaches RN2404.3 (R3.1)
- net RSX_VO63: now reaches RN2404.4 (R4.1)
- net RSX_VO71: now reaches RN2401.1 (R1.1)
- net RSX_VO68: now reaches RN2401.2 (R2.1)
- net RSX_VO66: now reaches RN2401.3 (R3.1)
- net RSX_VO64: now reaches RN2401.4 (R4.1)
- net RSX_VO55: now reaches RN2405.1 (R1.1)
- net RSX_VO53: now reaches RN2405.2 (R2.1)
- net RSX_VO51: now reaches RN2405.3 (R3.1)
- net RSX_VO49: now reaches RN2405.4 (R4.1)
- net RSX_VO62: now reaches RN2403.1 (R1.1)
- net RSX_VO61: now reaches RN2403.2 (R2.1)
- net RSX_VO60: now reaches RN2403.3 (R3.1)
- net RSX_VO58: now reaches RN2403.4 (R4.1)
