File: cok-001/av.kicad_sch (KiCad schematic)
At the start: 81 parts, among them J2401 AV OUT, Q2401 DTC144E, Q2402 SI2303BDS, Q2403 IMH20T108, Q2404 DTA144E, U2402 MC78M09, U2403 MC78M05, U2405 CX4351

Commit message: optical out
Parts:
- added C2469: 100u 10V, Capacitor_SMD:CP_Elec_6.3x5.4, symbol Device:C_Polarized_US
- added R2412: 0, Resistor_SMD:R_0603_1608Metric, symbol Device:R_US
- added U2409: LIGHT TRANSMITTER UNIT, OptoDevice:Vishay_MOLD-3Pin, symbol Interface_Optical:TSOP32S40F
Connections:
- net GND: now also C2469.2, U2409.3 (GND)
- new net: R2412.2, U2409.1 (OUT)
- new net: C2469.1, U2409.2 (Vs)
- new net RS_SPDO0_33: R2412.1
Other:
- moved on the sheet: C2404, C2405, C2406, C2407, C2408, C2409, C2410, C2411, C2444, C2451, C2452, C2459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

Commit message: filters
Parts:
- FL2401, FL2402, FL2403: footprint Filter:Filter_Mini-Circuits_FV1206-7 -> PS3:FL_0805_2012Metric
Changed lines of the file:
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@@
 			)
 		)
-		(property "Footprint" "Filter:Filter_Mini-Circuits_FV1206-7"
+		(property "Footprint" "PS3:FL_0805_2012Metric"
 			(at 284.48 41.91 90)
 			(effects
@@
 			)
 		)
-		(property "Footprint" "Filter:Filter_Mini-Circuits_FV1206-7"
+		(property "Footprint" "PS3:FL_0805_2012Metric"
 			(at 284.48 34.29 90)
 			(effects
@@
 			)
 		)
-		(property "Footprint" "Filter:Filter_Mini-Circuits_FV1206-7"
+		(property "Footprint" "PS3:FL_0805_2012Metric"
 			(at 270.51 36.83 90)
 			(effects

Commit message: av move
Parts:
- added R2403, R2404, R2465, R2466, R2467: 0, Resistor_SMD:R_0402_1005Metric, symbol Device:R_US
Connections:
- net GND: now also U2406.86 (TMODE1), U2406.87 (TMODE0)
- net RSX_VO36: now also RN2409.4 (R4.1)
- net RSX_VO37: now also RN2409.3 (R3.1)
- net RSX_VO38: now also RN2409.2 (R2.1)
- net RSX_VO39: now also RN2409.1 (R1.1)
- net RSX_VO40: now also RN2407.4 (R4.1)
- net RSX_VO41: now also RN2408.1 (R1.1)
- net RSX_VO42: now also RN2407.3 (R3.1)
- net RSX_VO43: now also RN2408.2 (R2.1)
- net RSX_VO44: now also RN2407.2 (R2.1)
- net RSX_VO45: now also RN2408.3 (R3.1)
- net RSX_VO46: now also RN2407.1 (R1.1)
- net RSX_VO47: now also RN2408.4 (R4.1)
- net RSX_VO48: now also RN2406.1 (R1.1)
- net RSX_VO50: now also RN2406.2 (R2.1)
- net RSX_VO52: now also RN2406.4 (R4.1)
- net RSX_VO54: now also RN2406.3 (R3.1)
- net at U2406.58 (G6): now also RN2406.6 (R3.2)
- net at U2406.61 (G4): now also RN2406.5 (R4.2)
- net at U2406.63 (G2): now also RN2406.7 (R2.2)
- net at U2406.65 (G0): now also RN2406.8 (R1.2)
- net at U2406.66 (B11): now also RN2408.5 (R4.2)
- net at U2406.68 (B9): now also RN2408.6 (R3.2)
- net at U2406.72 (B7): now also RN2408.7 (R2.2)
- net at U2406.74 (B5): now also RN2408.8 (R1.2)
- net at U2406.80 (CSYNC): now also R2465.2
- net at U2406.83 (VSYNC): now also R2466.2
- net at U2406.84 (HSYNC): now also R2467.2
- net at U2406.85 (DEN): now also R2403.2
- net at U2406.93 (CLOCK): now also R2404.2
- new net RSX_CLKOUT1: R2404.1
- new net RSX_CSYNCO1: R2465.1
- new net RSX_HSYNCO1: R2467.1
- new net RSX_VO_DE1: R2403.1
- new net RSX_VSYNCO1: R2466.1
Other:
- moved on the sheet: RN2401, RN2402, RN2403, RN2404, RN2405, RN2406, RN2407, RN2408, RN2409

Commit message: voltage symbols
Parts:
- added R2437: 10k, Resistor_SMD:R_0402_1005Metric, symbol Device:R_US
Connections:
- net GND: now also R2437.1
- net +3.3V_EVER: now reaches Q2404.2 (E)
- net at Q2403.4 (C2): now also R2476.1
- net at R2477.1: now also Q2403.1 (C1)
- net AUDIO_MUTE: now reaches D2401.1 (K)
- net AUDIO_MUTE: now also R2437.2
Other:
- moved on the sheet: D2401, Q2403A, Q2403B, Q2404
