File: cok-001/av.kicad_sch (KiCad schematic)
At the start: 90 parts, among them J2401 AV OUT, Q2401 DTC144E, Q2402 SI2303BDS, Q2403 IMH20T108, Q2404 DTA144E, U2402 MC78M09, U2403 MC78M05, U2405 CX4351, U2409 LIGHT TRANSMITTER UNIT

Commit message: update 10
Parts:
- added L2404: 10uH, symbol Device:L
- added R2406: 100k, Resistor_SMD:R_0402_1005Metric, symbol Device:R_US
- U2406, U2407, U2408: value ~ -> (none)
Connections:
- net +5V_ANA: now reaches C2409.1, C2410.1, U2403.3 (OUT)
- net +5V_ANA: now also L2404.1
- net at C2469.1, U2409.2 (Vs): now also L2404.2
- net SW_8_B: now reaches U2407.5 (Cont)
- net SW_8_B: now also Q2401.1 (B), U2408.5 (Cont)
- net at C2408.1, C2411.1, U2402.3 (OUT): now also U2405.17 (VA_H)
- net +12V_MAIN: now reaches Q2402.2 (S)
- net +12V_MAIN: now also R2406.1
- net at Q2401.3 (C), R2408.2: now also R2406.2
Other:
- moved on the sheet: C2469, R2412

Commit message: lf
Parts:
- L2404: footprint (none) -> Inductor_SMD_Wurth:L_Wurth_WE-LQSH-2010
Changed lines of the file:
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@@
 			)
 		)
-		(property "Footprint" ""
+		(property "Footprint" "Inductor_SMD_Wurth:L_Wurth_WE-LQSH-2010"
 			(at 332.74 179.07 0)
 			(hide yes)
