File: cok-001/eegs.kicad_sch (KiCad schematic)
At the start: 9 parts

Commit message: eegs dc
Parts:
- added RN7013: 56, Resistor_SMD:R_Array_Convex_4x0402, symbol Device:R_Pack04
- added TP7001, TP7004, TP7005, TP7006, TP7007, TP7008, TP7009: TestPoint, TestPoint:TestPoint_Pad_1.0x1.0mm, symbol Connector:TestPoint
- renumbered U501 to U7004
Connections:
- net GND: now also U7004.A30 (GNDr), U7004.B30 (GNDr), U7004.B32 (GNDr), U7004.C31 (GNDr), U7004.D31 (GNDr), U7004.E29 (GNDr), U7004.E31 (GNDr), U7004.F28 (GNDr), U7004.F29 (GNDr), U7004.F31 (GNDr), U7004.G28 (GNDr), U7004.G29 (GNDr), U7004.G31 (GNDr), U7004.H29 (GNDr), U7004.H31 (GNDr), U7004.J28 (GNDr), U7004.J29 (GNDr), U7004.J31 (GNDr), U7004.K29 (GNDr), U7004.K31 (GNDr), U7004.L29 (GNDr), U7004.L31 (GNDr), U7004.M29 (GNDr), U7004.M31 (GNDr), U7004.N29 (GNDr), U7004.N31 (GNDr), U7004.P29 (GNDr), U7004.P31 (GNDr), U7004.R29 (GNDr), U7004.R31 (GNDr)
- new net: TP7006.1, U7004.AM27 (PCLK)
- new net: TP7001.1, U7004.C1 (SRXD)
- new net: RN7013.2 (R2.1), U7004.A20 (AD1)
- new net: U7004.A31 (VDDio), U7004.AE28 (VDDio), U7004.AM31 (VDDio), U7004.D29 (VDDio), U7004.P28 (VDDio), U7004.V28 (VDDio)
- new net: U7004.AA3 (VDD), U7004.AC4 (VDD), U7004.AC5 (VDD), U7004.AF4 (VDD), U7004.AH13 (VDD), U7004.AH19 (VDD), U7004.AH22 (VDD), U7004.AH6 (VDD), U7004.AH9 (VDD), U7004.AJ22 (VDD), U7004.AJ3 (VDD), U7004.AJ6 (VDD), U7004.AK12 (VDD), U7004.AK16 (VDD), U7004.AK25 (VDD), U7004.AK28 (VDD), U7004.AL16 (VDD), U7004.AM2 (VDD), U7004.B1 (VDD), U7004.C16 (VDD), U7004.D10 (VDD), U7004.D13 (VDD), U7004.D18 (VDD), U7004.D22 (VDD), U7004.D25 (VDD), U7004.D3 (VDD), U7004.D4 (VDD), U7004.D7 (VDD), U7004.E10 (VDD), U7004.E13 (VDD), U7004.E18 (VDD), U7004.E22 (VDD), U7004.E25 (VDD), U7004.E7 (VDD), U7004.F4 (VDD), U7004.H4 (VDD), U7004.H5 (VDD), U7004.L5 (VDD), U7004.P5 (VDD), U7004.T5 (VDD), U7004.V5 (VDD)
- new net: U7004.AA4 (AVD1), U7004.AF3 (AVD1), U7004.AH23 (AVD0), U7004.AH24 (AVD0), U7004.AH25 (AVD0), U7004.AJ10 (AVD1), U7004.AJ12 (AVD1), U7004.AJ23 (AVD0), U7004.AJ7 (AVD1), U7004.AJ9 (AVD1), U7004.V4 (AVD1), U7004.Y4 (AVD1)
- new net: U7004.AB4 (VDDo), U7004.AB5 (VDDo), U7004.AE4 (VDDo), U7004.AE5 (VDDo), U7004.AG5 (VDDo), U7004.AH11 (VDDo), U7004.AH14 (VDDo), U7004.AH17 (VDDo), U7004.AH27 (VDDo), U7004.AH8 (VDDo), U7004.AJ14 (VDDo), U7004.AJ28 (VDDo), U7004.AJ4 (VDDo), U7004.AK20 (VDDo), U7004.AK23 (VDDo), U7004.AK4 (VDDo), U7004.AL1 (VDDo), U7004.B2 (VDDo), U7004.C12 (VDDo), U7004.C17 (VDDo), U7004.C2 (VDDo), U7004.C28 (VDDo), U7004.D12 (VDDo), U7004.D15 (VDDo), U7004.D17 (VDDo), U7004.D20 (VDDo), U7004.D28 (VDDo), U7004.D5 (VDDo), U7004.E15 (VDDo), U7004.E23 (VDDo), U7004.E5 (VDDo), U7004.E8 (VDDo), U7004.G5 (VDDo), U7004.J4 (VDDo), U7004.M4 (VDDo), U7004.M5 (VDDo), U7004.R4 (VDDo), U7004.Y5 (VDDo)
- new net: U7004.AC28 (VDDr), U7004.AH28 (VDDr), U7004.E28 (VDDr), U7004.L28 (VDDr), U7004.N28 (VDDr), U7004.R28 (VDDr), U7004.T28 (VDDr), U7004.U28 (VDDr), U7004.W28 (VDDr)
- new net: U7004.AD28 (VDDar), U7004.M28 (VDDar)
- new net: U7004.AD4 (AVDA1), U7004.AJ11 (AVDA1), U7004.AJ19 (AVDA0), U7004.AJ20 (AVDA0), U7004.AJ21 (AVDA0), U7004.AJ8 (AVDA1), U7004.W4 (AVDA1)
- new net: TP7005.1, U7004.AK19 (CLKMON)
- new net: TP7004.1, U7004.AK26 (FLDO)
- new net: TP7007.1, U7004.AM12 (PCLK2)
- new net: TP7008.1, U7004.AM29 (ROOut)
- new net: RN7013.3 (R3.1), U7004.B19 (AD0)
- new net: RN7013.1 (R1.1), U7004.B20 (AD2)
- new net: RN7013.4 (R4.1), U7004.C19 (AD3)
- new net: TP7009.1, U7004.C27 (SynClk)
- new net SIF_AD0: RN7013.6 (R3.2)
- new net SIF_AD1: RN7013.7 (R2.2)
- new net SIF_AD2: RN7013.8 (R1.2)
- new net SIF_AD3: RN7013.5 (R4.2)
- no-connect marks 0 -> 74

Commit message: sata
Parts:
- added JL7003, JL7004, JL7005, JL7006: TestPoint, TestPoint:TestPoint_Pad_1.0x1.0mm, symbol Connector:TestPoint
- added R7029, R7030: 47, Resistor_SMD:R_0402_1005Metric, symbol Device:R_US
- added R7031, R7032: 0, Resistor_SMD:R_0603_1608Metric, symbol Device:R_US
- added R7035: XX, Resistor_SMD:R_0603_1608Metric, symbol Device:R_US
- added R7036, R7037: 4700, Resistor_SMD:R_0402_1005Metric, symbol Device:R_US
- renumbered TP7001 to JL7001
Connections:
- net GND: now also U7004.W1 (EEenable), U7004.W2 (GSenable), JL7005.1, R7031.1, R7032.1
- net at U7004.A4 (TIMIN0): now also R7030.2
- net at U7004.B5 (TIMIN1): now also R7029.2
- net at U7004.D1 (~{SRTS}): now also JL7004.1
- net at U7004.D2 (~{SCTS}): now also JL7003.1
- net at U7004.F3 (STXD): now also JL7006.1
- net at U7004.T2 (JTDI): now also R7031.2
- net at U7004.U1 (JTMS): now also R7037.1
- net at U7004.U2 (JTCK): now also R7036.1
- net at U7004.U3 (JTRST): now also R7032.2
- net at U7004.V1 (JTDO): now also R7035.1
- new net: R7035.2, R7036.2, R7037.2

Commit message: bridge sif
Parts:
- added R7041, R7042: 0, Resistor_SMD:R_0603_1608Metric, symbol Device:R_US
- added R7080: 56, Resistor_SMD:R_0402_1005Metric, symbol Device:R_US
- added RN7014, RN7015, RN7016, RN7017, RN7018, RN7019, RN7020, RN7023: 56, Resistor_SMD:R_Array_Convex_4x0402, symbol Device:R_Pack04
- added RN7021: 4700, Resistor_SMD:R_Array_Convex_4x0402, symbol Device:R_Pack04
Connections:
- net GND: now also R7041.2, R7042.2, RN7021.5 (R4.2), RN7021.6 (R3.2); no longer U7004.B27 (CMD)
- net at U7004.A10 (AD23): now also RN7016.3 (R3.1)
- net at U7004.A11 (AD20): now also RN7018.3 (R3.1)
- net at U7004.A12 (AD18): now also RN7018.2 (R2.1)
- net at U7004.A13 (AD17): now also RN7014.1 (R1.1)
- net at U7004.A14 (AD16): now also RN7014.4 (R4.1)
- net at U7004.A15 (AD12): now also RN7019.4 (R4.1)
- net at U7004.A16 (AD8): now also RN7019.3 (R3.1)
- net at U7004.A17 (AD5): now also RN7019.1 (R1.1)
- net at U7004.A18 (AD6): now also RN7017.1 (R1.1)
- net at U7004.A19 (AD4): now also RN7017.4 (R4.1)
- net at U7004.A24 (DREQ1): now also R7080.1
- net at U7004.A25 (DACK): now also RN7023.4 (R4.1)
- net at U7004.A6 (TestClkSw): now also R7041.1
- net at U7004.A8 (AD31): now also RN7020.4 (R4.1)
- net at U7004.A9 (AD26): now also RN7020.3 (R3.1)
- net at U7004.B10 (AD25): now also RN7016.2 (R2.1)
- net at U7004.B11 (AD24): now also RN7016.4 (R4.1)
- net at U7004.B12 (AD28): now also RN7018.1 (R1.1)
- net at U7004.B13 (AD19): now also RN7014.2 (R2.1)
- net at U7004.B14 (AD14): now also RN7015.2 (R2.1)
- net at U7004.B15 (AD15): now also RN7015.3 (R3.1)
- net at U7004.B16 (AD10): now also RN7019.2 (R2.1)
- net at U7004.B18 (AD9): now also RN7017.2 (R2.1)
- net at U7004.B23 (~{WRAC}): now also RN7023.2 (R2.1)
- net at U7004.B24 (DREQ0): now also RN7023.3 (R3.1)
- net at U7004.B25 (TestClock): now also RN7021.1 (R1.1)
- net at U7004.B9 (AD29): now also RN7020.2 (R2.1)
- net at U7004.C10 (AD27): now also RN7016.1 (R1.1)
- net at U7004.C11 (AD21): now also RN7018.4 (R4.1)
- net at U7004.C13 (AD22): now also RN7014.3 (R3.1)
- net at U7004.C14 (AD13): now also RN7015.1 (R1.1)
- net at U7004.C15 (AD11): now also RN7015.4 (R4.1)
- net at U7004.C18 (AD7): now also RN7017.3 (R3.1)
- net at U7004.C21 (~{INTOUT}): now also RN7023.1 (R1.1)
- net at U7004.C25 (TestReset): now also RN7021.2 (R2.1)
- net at U7004.C9 (AD30): now also RN7020.1 (R1.1)
- net at U7004.W3 (GearRatio): now also R7042.1
- new net SIF_AD10: RN7019.7 (R2.2)
- new net SIF_AD11: RN7015.5 (R4.2)
- new net SIF_AD12: RN7019.5 (R4.2)
- new net SIF_AD13: RN7015.8 (R1.2)
- new net SIF_AD14: RN7015.7 (R2.2)
- new net SIF_AD15: RN7015.6 (R3.2)
- new net SIF_AD16: RN7014.5 (R4.2)
- new net SIF_AD17: RN7014.8 (R1.2)
- new net SIF_AD18: RN7018.7 (R2.2)
- new net SIF_AD19: RN7014.7 (R2.2)
- new net SIF_AD20: RN7018.6 (R3.2)
- new net SIF_AD21: RN7018.5 (R4.2)
- new net SIF_AD22: RN7014.6 (R3.2)
- new net SIF_AD23: RN7016.6 (R3.2)
- new net SIF_AD24: RN7016.5 (R4.2)
- new net SIF_AD25: RN7016.7 (R2.2)
- new net SIF_AD26: RN7020.6 (R3.2)
- new net SIF_AD27: RN7016.8 (R1.2)
- new net SIF_AD28: RN7018.8 (R1.2)
- new net SIF_AD29: RN7020.7 (R2.2)
- new net SIF_AD30: RN7020.8 (R1.2)
- new net SIF_AD31: RN7020.5 (R4.2)
- new net SIF_AD4: RN7017.5 (R4.2)
- new net SIF_AD5: RN7019.8 (R1.2)
- new net SIF_AD6: RN7017.8 (R1.2)
- new net SIF_AD7: RN7017.6 (R3.2)
- new net SIF_AD8: RN7019.6 (R3.2)
- new net SIF_AD9: RN7017.7 (R2.2)
- new net SIF_DACK: RN7023.5 (R4.2)
- new net SIF_DREQ0: RN7023.6 (R3.2)
- new net SIF_DREQ1: R7080.2
- new net ~{SIF_WRAC}: RN7023.7 (R2.2)
- new net ~{SINT}: RN7023.8 (R1.2)

Commit message: footprints
Parts:
- added C7286: 10V, Capacitor_SMD:C_0402_1005Metric, symbol Device:C
- added R7073, R7074: XX, Resistor_SMD:R_0402_1005Metric, symbol Device:R_US
- added U7005: LM75B, Package_SO:VSSOP-8_3x3mm_P0.65mm, symbol Sensor_Temperature:LM75B
Connections:
- net GND: now also C7286.2, U7005.4 (GND), U7005.5 (A2), U7005.7 (A0)
- new net: R7073.2, U7005.1 (SDA)
- new net: R7074.2, U7005.2 (SCL)
- new net +3.3V_THERMAL: C7286.1, U7005.6 (A1), U7005.8 (+Vs)
- new net THR_I2C_SCL: R7074.1
- new net THR_I2C_SDA: R7073.1
- no-connect marks 74 -> 75

Commit message: ps2
Parts:
- added R7033: 0, Resistor_SMD:R_0603_1608Metric, symbol Device:R_US
- added R7034: 47, Resistor_SMD:R_0402_1005Metric, symbol Device:R_US
- added R7044, R7045: 1k, Resistor_SMD:R_0603_1608Metric, symbol Device:R_US
Connections:
- net GND: now also U7004.T29 (DQBA8), R7033.1
- net at U7004.A5 (~{INTIN1}): now also R7034.2
- net at U7004.AA1 (CLKGCCG): now also R7033.2
- net CFMN_B: now reaches U7004.AA30 (CFMNB)
- net CFMN_B: now also U7003.D7 (CFMN)
- net CFM_B: now reaches U7004.AA32 (CFMB)
- net CFM_B: now also U7003.C7 (CFM)
- net CTM_B: now reaches U7004.AB30 (CTMB)
- net CTM_B: now also U7003.E1 (CTM)
- net CTMN_B: now reaches U7004.AB32 (CTMNB)
- net CTMN_B: now also U7003.D1 (CTMN)
- net at U7004.AL11 (~{INT}): now also R7034.1
- net at U7004.B4 (~{ERESET}): now also R7044.1
- net CFM_A: now reaches U7004.G30 (CFMA)
- net CFM_A: now also U7002.C7 (CFM)
- net CFMN_A: now reaches U7004.G32 (CFMNA)
- net CFMN_A: now also U7002.D7 (CFMN)
- net CTMN_A: now reaches U7004.H30 (CTMNA)
- net CTMN_A: now also U7002.E1 (CTM)
- net CTM_A: now reaches U7004.H32 (CTMA)
- net CTM_A: now also U7002.D1 (CTMN)
- net at U7004.Y1 (PwrUp): now also R7045.1
- new net PWRUP_EE: R7045.2
- new net ~{EGRST}: R7044.2
- no-connect marks 75 -> 76
Other:
- moved on the sheet: C7286, R7073, R7074, U7002, U7005

Commit message: PCIe
Parts:
- added RN7007, RN7008, RN7009, RN7010, RN7011, RN7012: 22, Resistor_SMD:R_Array_Convex_4x0402, symbol Device:R_Pack04
Connections:
- net at U7004.AB4 (VDDo), U7004.AB5 (VDDo), U7004.AE4 (VDDo)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: now also U7004.E20 (VDDo)
- net at U7004.AK14 (BO6): now also RN7012.7 (R2.2)
- net at U7004.AK15 (BO3): now also RN7009.8 (R1.2)
- net at U7004.AK18 (GO6): now also RN7011.7 (R2.2)
- net at U7004.AK21 (GO2): now also RN7008.7 (R2.2)
- net at U7004.AK24 (RO3): now also RN7007.8 (R1.2)
- net at U7004.AL14 (BO7): now also RN7012.8 (R1.2)
- net at U7004.AL15 (BO4): now also RN7012.5 (R4.2)
- net at U7004.AL18 (GO7): now also RN7011.8 (R1.2)
- net at U7004.AL19 (GO4): now also RN7011.5 (R4.2)
- net at U7004.AL21 (GO3): now also RN7008.8 (R1.2)
- net at U7004.AL22 (GO0): now also RN7008.5 (R4.2)
- net at U7004.AL23 (RO6): now also RN7010.7 (R2.2)
- net at U7004.AL24 (RO4): now also RN7010.5 (R4.2)
- net at U7004.AL25 (RO1): now also RN7007.6 (R3.2)
- net at U7004.AM15 (BO5): now also RN7012.6 (R3.2)
- net at U7004.AM16 (BO2): now also RN7009.7 (R2.2)
- net at U7004.AM17 (BO1): now also RN7009.6 (R3.2)
- net at U7004.AM19 (GO5): now also RN7011.6 (R3.2)
- net at U7004.AM22 (GO1): now also RN7008.6 (R3.2)
- net at U7004.AM23 (RO7): now also RN7010.8 (R1.2)
- net at U7004.AM24 (RO5): now also RN7010.6 (R3.2)
- net at U7004.AM25 (RO2): now also RN7007.7 (R2.2)
- net at U7004.AM26 (RO0): now also RN7007.5 (R4.2)
- new net: RN7009.5 (R4.2), U7004.AM18 (B00)
- new net RSX_VI12: RN7009.4 (R4.1)
- new net RSX_VI13: RN7009.3 (R3.1)
- new net RSX_VI14: RN7009.2 (R2.1)
- new net RSX_VI15: RN7009.1 (R1.1)
- new net RSX_VI16: RN7012.4 (R4.1)
- new net RSX_VI17: RN7012.3 (R3.1)
- new net RSX_VI18: RN7012.2 (R2.1)
- new net RSX_VI19: RN7012.1 (R1.1)
- new net RSX_VI20: RN7008.4 (R4.1)
- new net RSX_VI21: RN7008.3 (R3.1)
- new net RSX_VI22: RN7008.2 (R2.1)
- new net RSX_VI23: RN7008.1 (R1.1)
- new net RSX_VI24: RN7011.4 (R4.1)
- new net RSX_VI25: RN7011.3 (R3.1)
- new net RSX_VI26: RN7011.2 (R2.1)
- new net RSX_VI27: RN7011.1 (R1.1)
- new net RSX_VI28: RN7007.4 (R4.1)
- new net RSX_VI29: RN7007.3 (R3.1)
- new net RSX_VI30: RN7007.2 (R2.1)
- new net RSX_VI31: RN7007.1 (R1.1)
- new net RSX_VI32: RN7010.4 (R4.1)
- new net RSX_VI33: RN7010.3 (R3.1)
- new net RSX_VI34: RN7010.2 (R2.1)
- new net RSX_VI35: RN7010.1 (R1.1)
