File: cok-001/eegs.kicad_sch (KiCad schematic)
At the start: 59 parts, among them U7001 ICS626BGLFT, U7005 LM75B, Y7001 XX

Commit message: update 10
Parts:
- U7002, U7003, U7004: value ~ -> (none)

Commit message: lf
Parts:
- added CL7010: TestPoint, TestPoint:TestPoint_Pad_1.0x1.0mm, symbol Connector:TestPoint
- added R7046, R7058: 22, Resistor_SMD:R_0402_1005Metric, symbol Device:R_US
- added R7075, R7077, R7078: 56, Resistor_SMD:R_0402_1005Metric, symbol Device:R_US
Connections:
- net at U7004.A21 (PGCLK): now also R7058.1
- net at U7004.A7 (~{BREQ}): now also R7078.1
- net at U7004.B6 (~{INTIN0}): now also R7075.1
- net at U7004.B7 (~{BGNT}): now also R7077.1
- net at U7004.B8 (MSCLK): now also R7046.1
- net at U7004.C7 (~{SRST}): now also CL7010.1
- new net MSCLK: R7046.2, R7058.2
- new net ~{BGNT}: R7077.2
- new net ~{BREQ}: R7078.2
- new net ~{SGINT}: R7075.2
