File: cok-001/gpu.kicad_sch (KiCad schematic)
At the start: 0 parts

Commit message: rename symbols
Parts:
- added R2067: 60.4, Resistor_SMD:R_0402_1005Metric, symbol Device:R_US
- added R2068: 39.2, Resistor_SMD:R_0402_1005Metric, symbol Device:R_US
- added R2071: 240, Resistor_SMD:R_0603_1608Metric, symbol Device:R_US
- added U2001: ~, PS3:RSX, symbol PS3:CXD2971GB
Connections:
- new net: R2068.2, U2001.K39 (FBCAL0_PU_GND)
- new net: U2001.D34 (FBVDD), U2001.D35 (FBVDD), U2001.D38 (FBVDD), U2001.D39 (FBVDD), U2001.D40 (FBVDD)
- new net: R2071.1, U2001.L41 (FB_ZQ1)
- new net: U2001.K35 (FBVDD), U2001.K36 (FBVDD)
- new net: U2001.C33 (FBVDD), U2001.C34 (FBVDD), U2001.C36 (FBVDD), U2001.C37 (FBVDD), U2001.C38 (FBVDD), U2001.C39 (FBVDD), U2001.C40 (FBVDD)
- new net: U2001.F35 (FBVDD), U2001.F36 (FBVDD), U2001.F38 (FBVDD), U2001.F39 (FBVDD), U2001.F40 (FBVDD), U2001.F41 (FBVDD)
- new net: U2001.B2 (VDDR), U2001.B4 (VDDR)
- new net: U2001.B34 (FBVDD), U2001.B35 (FBVDD), U2001.B36 (FBVDD), U2001.B37 (FBVDD), U2001.B38 (FBVDD), U2001.B39 (FBVDD), U2001.B40 (FBVDD)
- new net: U2001.A3 (VDDR), U2001.A4 (VDDR), U2001.A5 (VDDR)
- new net: U2001.A34 (FBVDD), U2001.A35 (FBVDD), U2001.A36 (FBVDD), U2001.A37 (FBVDD), U2001.A38 (FBVDD)
- new net: R2067.1, U2001.H32 (FBVDD), U2001.H33 (FBVDD), U2001.H35 (FBVDD), U2001.H38 (FBVDD), U2001.H39 (FBVDD)
- new net: R2067.2, U2001.H40 (FBCAL0_PD_VD)
- new net: U2001.E32 (FBVDD), U2001.E33 (FBVDD), U2001.E36 (FBVDD), U2001.E37 (FBVDD), U2001.E39 (FBVDD)
- new net: U2001.G33 (FBVDD), U2001.G34 (FBVDD), U2001.G36 (FBVDD), U2001.G37 (FBVDD), U2001.G38 (FBVDD), U2001.G39 (FBVDD), U2001.G40 (FBVDD)
- new net BE_TX0_TXCLKN: U2001.K4 (RX0_RXCKN)
- new net BE_TX0_TXCLKP: U2001.K3 (RX0_RXCKP)
- new net BE_TX0_TXN0: U2001.J2 (RX0_RXN0)
- new net BE_TX0_TXN1: U2001.J7 (RX0_RXN1)
- new net BE_TX0_TXN2: U2001.J4 (RX0_RXN2)
- new net BE_TX0_TXN3: U2001.K7 (RX0_RXN3)
- new net BE_TX0_TXN4: U2001.L2 (RX0_RXN4)
- new net BE_TX0_TXN5: U2001.L7 (RX0_RXN5)
- new net BE_TX0_TXN6: U2001.L4 (RX0_RXN6)
- new net BE_TX0_TXN7: U2001.M4 (RX0_RXN7)
- new net BE_TX0_TXP0: U2001.J1 (RX0_RXP0)
- new net BE_TX0_TXP1: U2001.J6 (RX0_RXP1)
- new net BE_TX0_TXP2: U2001.J3 (RX0_RXP2)
- new net BE_TX0_TXP3: U2001.K6 (RX0_RXP3)
- new net BE_TX0_TXP4: U2001.L1 (RX0_RXP4)
- new net BE_TX0_TXP5: U2001.L6 (RX0_RXP5)
- new net BE_TX0_TXP6: U2001.L3 (RX0_RXP6)
- new net BE_TX0_TXP7: U2001.M3 (RX0_RXP7)
- new net GND: R2071.2, U2001.A10 (GND), U2001.A12 (GND), U2001.A14 (GND), U2001.A16 (GND), U2001.A18 (GND), U2001.A20 (GND), U2001.A22 (GND), U2001.A24 (GND), U2001.A26 (GND), U2001.A28 (GND), U2001.A30 (GND), U2001.A6 (GND), U2001.A8 (GND), U2001.B11 (GND), U2001.B13 (GND), U2001.B15 (GND), U2001.B17 (GND), U2001.B19 (GND), U2001.B21 (GND), U2001.B23 (GND), U2001.B25 (GND), U2001.B27 (GND), U2001.B29 (GND), U2001.B5 (GND), U2001.B7 (GND), U2001.B9 (GND), U2001.C10 (GND), U2001.C12 (GND), U2001.C14 (GND), U2001.C16 (GND), U2001.C18 (GND), U2001.C20 (GND), U2001.C22 (GND), U2001.C24 (GND), U2001.C26 (GND), U2001.C28 (GND), U2001.C30 (GND), U2001.C6 (GND), U2001.C8 (GND), U2001.D11 (GND), U2001.D13 (GND), U2001.D15 (GND), U2001.D17 (GND), U2001.D19 (GND), U2001.D21 (GND), U2001.D23 (GND), U2001.D25 (GND), U2001.D27 (GND), U2001.D3 (GND), U2001.D5 (GND), U2001.D7 (GND), U2001.D9 (GND), U2001.E10 (GND), U2001.E12 (GND), U2001.E14 (GND), U2001.E16 (GND), U2001.E18 (GND), U2001.E20 (GND), U2001.E22 (GND), U2001.E24 (GND), U2001.E26 (GND), U2001.E28 (GND), U2001.E30 (GND), U2001.E6 (GND), U2001.E8 (GND), U2001.F11 (GND), U2001.F13 (GND), U2001.F15 (GND), U2001.F17 (GND), U2001.F19 (GND), U2001.F21 (GND), U2001.F23 (GND), U2001.F25 (GND), U2001.F27 (GND), U2001.F29 (GND), U2001.F3 (GND), U2001.F31 (GND), U2001.F33 (GND), U2001.F34 (GND), U2001.F37 (GND), U2001.F5 (GND), U2001.F7 (GND), U2001.F9 (GND), U2001.G10 (GND), U2001.G12 (GND), U2001.G14 (GND), U2001.G16 (GND), U2001.G18 (GND), U2001.G20 (GND), U2001.G22 (GND), U2001.G24 (GND), U2001.G26 (GND), U2001.G28 (GND), U2001.G30 (GND), U2001.G32 (GND), U2001.G35 (GND), U2001.G41 (GND), U2001.H11 (GND), U2001.H13 (GND), U2001.H15 (GND), U2001.H17 (GND), U2001.H19 (GND), U2001.H21 (GND), U2001.H23 (GND), U2001.H25 (GND), U2001.H27 (GND), U2001.H29 (GND), U2001.H3 (GND), U2001.H31 (GND), U2001.H4 (GND), U2001.H5 (GND), U2001.H6 (GND), U2001.H7 (GND), U2001.H9 (GND), U2001.K14 (GND), U2001.K16 (GND), U2001.K18 (GND), U2001.K20 (GND), U2001.K22 (GND), U2001.K24 (GND), U2001.K26 (GND), U2001.K28 (GND), U2001.K34 (GND), U2001.K37 (FB_MF1), U2001.K38 (FB_SEN1), U2001.L35 (GND), U2001.L39 (GND), U2001.L5 (GND), U2001.L8 (GND), U2001.M10 (GND), U2001.M15 (GND), U2001.M17 (GND), U2001.M19 (GND), U2001.M21 (GND), U2001.M23 (GND), U2001.M25 (GND), U2001.M27 (GND), U2001.M30 (GND), U2001.M34 (GND), U2001.M36 (GND), U2001.M5 (GND), U2001.M8 (GND), U2001.P10 (GND), U2001.P15 (GND), U2001.P17 (GND), U2001.P19 (GND), U2001.P21 (GND), U2001.P23 (GND), U2001.P25 (GND), U2001.P27 (GND), U2001.P30 (GND), U2001.P34 (GND), U2001.P37 (GND)
- new net RSX_FB_VDD_VREF2: U2001.E2 (FB_VDDVREF2)
- new net RSX_FB_VREF2: U2001.E1 (FB_VREF2)
- new net RSX_VDDMONI: U2001.B31 (VDDMON)
- new net RSX_VI21: U2001.N36 (VI21)
- new net RSX_VI27: U2001.N37 (VI27)
- new net RSX_VI28: U2001.N39 (VI28)
- new net RSX_VI29: U2001.L36 (VI29)
- new net RSX_VI31: U2001.L37 (VI31)
- new net RSX_VI33: U2001.L38 (VI33)
- new net RSX_VI34: U2001.L40 (VI34)
- new net RSX_VSSMONI: U2001.A31 (VSSMON)
- no-connect marks 0 -> 1

Commit message: rsx vo
Parts:
- added R2061: 240, Resistor_SMD:R_0402_1005Metric, symbol Device:R_US
Connections:
- net GND: now also U2001.AE12 (GND), U2001.AE14 (GND), U2001.AE28 (GND), U2001.AE35 (GND), U2001.AE38 (GND), U2001.AE8 (GND), U2001.AF10 (GND), U2001.AF15 (GND), U2001.AF27 (GND), U2001.AF30 (GND), U2001.AF32 (GND), U2001.AF34 (GND), U2001.AF37 (GND), U2001.AF8 (GND), U2001.D29 (GND), U2001.D31 (GND), U2001.D33 (GND), U2001.G2 (FB_SEN2), R2061.2
- net RSX_VO47: now reaches U2001.AF35 (VO_111)
- net RSX_VO50: now reaches U2001.AF36 (VO_114)
- net RSX_VO48: now reaches U2001.AF38 (VO_112)
- net RSX_VO53: now reaches U2001.AF39 (VO_117)
- net RSX_VO51: now reaches U2001.AF40 (VO_115)
- net at U2001.D10 (VDD): now also U2001.D12 (VDD), U2001.D14 (VDD), U2001.D16 (VDD), U2001.D18 (VDD), U2001.D20 (VDD), U2001.D22 (VDD), U2001.D24 (VDD), U2001.D26 (VDD), U2001.D28 (VDD), U2001.D30 (VDD), U2001.D6 (VDD), U2001.D8 (VDD)
- net at U2001.K13 (VDD): now also U2001.K15 (VDD), U2001.K17 (VDD), U2001.K19 (VDD), U2001.K21 (VDD), U2001.K23 (VDD), U2001.K25 (VDD), U2001.K27 (VDD), U2001.K29 (VDD)
- net RSX_VO54: now reaches U2001.AE37 (VO_118)
- net RSX_VO55: now reaches U2001.AE39 (VO_119)
- net at U2001.P14 (VDD): now also U2001.P16 (VDD), U2001.P18 (VDD), U2001.P20 (VDD), U2001.P22 (VDD), U2001.P24 (VDD), U2001.P26 (VDD), U2001.P28 (VDD)
- net at U2001.C11 (VDD): now also U2001.C13 (VDD), U2001.C15 (VDD), U2001.C17 (VDD), U2001.C19 (VDD), U2001.C21 (VDD), U2001.C23 (VDD), U2001.C25 (VDD), U2001.C27 (VDD), U2001.C29 (VDD), U2001.C31 (VDD), U2001.C7 (VDD), U2001.C9 (VDD)
- net at U2001.M14 (VDD): now also U2001.M16 (VDD), U2001.M18 (VDD), U2001.M20 (VDD), U2001.M22 (VDD), U2001.M24 (VDD), U2001.M26 (VDD), U2001.M28 (VDD)
- net at U2001.F10 (VDD): now also U2001.F12 (VDD), U2001.F14 (VDD), U2001.F16 (VDD), U2001.F18 (VDD), U2001.F20 (VDD), U2001.F22 (VDD), U2001.F24 (VDD), U2001.F26 (VDD), U2001.F28 (VDD), U2001.F30 (VDD), U2001.F6 (VDD), U2001.F8 (VDD)
- net at U2001.B10 (VDD): now also U2001.B12 (VDD), U2001.B14 (VDD), U2001.B16 (VDD), U2001.B18 (VDD), U2001.B20 (VDD), U2001.B22 (VDD), U2001.B24 (VDD), U2001.B26 (VDD), U2001.B28 (VDD), U2001.B30 (VDD), U2001.B6 (VDD), U2001.B8 (VDD)
- net at U2001.A11 (VDD): now also U2001.A13 (VDD), U2001.A15 (VDD), U2001.A17 (VDD), U2001.A19 (VDD), U2001.A21 (VDD), U2001.A23 (VDD), U2001.A25 (VDD), U2001.A27 (VDD), U2001.A29 (VDD), U2001.A7 (VDD), U2001.A9 (VDD)
- net at U2001.E11 (VDD): now also U2001.E13 (VDD), U2001.E15 (VDD), U2001.E17 (VDD), U2001.E19 (VDD), U2001.E21 (VDD), U2001.E23 (VDD), U2001.E25 (VDD), U2001.E27 (VDD), U2001.E29 (VDD), U2001.E31 (VDD), U2001.E7 (VDD), U2001.E9 (VDD)
- net at U2001.H10 (VDD): now also U2001.H12 (VDD), U2001.H14 (VDD), U2001.H16 (VDD), U2001.H18 (VDD), U2001.H20 (VDD), U2001.H22 (VDD), U2001.H24 (VDD), U2001.H26 (VDD), U2001.H28 (VDD), U2001.H30 (VDD)
- net at U2001.G1 (FB_ZQ2): now also R2061.1
- net at U2001.G11 (VDD): now also U2001.G13 (VDD), U2001.G15 (VDD), U2001.G17 (VDD), U2001.G19 (VDD), U2001.G21 (VDD), U2001.G23 (VDD), U2001.G25 (VDD), U2001.G27 (VDD), U2001.G29 (VDD), U2001.G31 (VDD), U2001.G9 (VDD)
- net at U2001.G3 (VDDR): now also U2001.G4 (VDDR), U2001.G5 (VDDR), U2001.G6 (VDDR), U2001.G7 (VDDR), U2001.G8 (VDDR)

Commit message: PCIe
Parts:
- added R2063, R2064, R2065: 22, Resistor_SMD:R_0402_1005Metric, symbol Device:R_US
- added R2070: 39.2, Resistor_SMD:R_0402_1005Metric, symbol Device:R_US
Connections:
- net GND: now also U2001.AL35 (GND), U2001.AL41 (GND), U2001.AL5 (GND), U2001.AP12 (GND), U2001.AP14 (GND), U2001.AP16 (GND), U2001.AP18 (GND), U2001.AP20 (GND), U2001.AP22 (GND), U2001.AP24 (GND), U2001.AP26 (GND), U2001.AP28 (GND), U2001.AP30 (GND), U2001.AP32 (GND), U2001.AR13 (GND), U2001.AR15 (GND), U2001.AR17 (GND), U2001.AR19 (GND), U2001.AR21 (GND), U2001.AR23 (GND), U2001.AR25 (GND), U2001.AR27 (GND), U2001.AR29 (GND), U2001.AR31 (GND), U2001.AR33 (GND), U2001.AR35 (GND), U2001.J35 (GND), U2001.J38 (GND), U2001.J8 (GND), U2001.N12 (GND), U2001.N35 (GND), U2001.N38 (GND), R2070.1
- net BE_TX2_TXP7: now reaches U2001.AF3 (RX2_RXP7)
- net BE_TX2_TXN7: now reaches U2001.AF4 (RX2_RXN7)
- net +1.2V_YC_RC_VDDIO: now reaches U2001.L10 (VDDIORW)
- net +1.2V_YC_RC_VDDIO: now also U2001.AL10 (VDDIORW), U2001.AL8 (VDDIORW), U2001.J5 (VDDIORW), U2001.N5 (VDDIORW), U2001.N8 (VDDIORW)
- net BE_TX2_TXP4: now reaches U2001.AE1 (RX2_RXP4)
- net BE_TX2_TXN4: now reaches U2001.AE2 (RX2_RXN4)
- net BE_TX2_TXP6: now reaches U2001.AE3 (RX2_RXP6)
- net BE_TX2_TXN6: now reaches U2001.AE4 (RX2_RXN6)
- net BE_TX2_TXP5: now reaches U2001.AE6 (RX2_RXP5)
- net BE_TX2_TXN5: now reaches U2001.AE7 (RX2_RXN5)
- net BE_TX1_TXP0: now reaches U2001.T1 (RX1_RXP0)
- net BE_TX1_TXN0: now reaches U2001.T2 (RX1_RXN0)
- net BE_TX1_TXP2: now reaches U2001.T3 (RX1_RXP2)
- net BE_TX1_TXN2: now reaches U2001.T4 (RX1_RXN2)
- net BE_TX1_TXP1: now reaches U2001.T6 (RX1_RXP1)
- net BE_TX1_TXN1: now reaches U2001.T7 (RX1_RXN1)
- net RSX_GPIO6: now reaches U2001.AV14 (GPIO6)
- net RSX_GPIO3: now reaches U2001.AV16 (GPIO3)
- net RSX_GPIO5: now reaches U2001.AY14 (GPIO6)
- net RSX_GPIO4: now reaches U2001.AY15 (GPIO4)
- net RSX_GPIO2: now reaches U2001.AY16 (GPIO2)
- net at U2001.AY18 (LRCKO): now also R2063.2
- net at U2001.AY19 (BCLKO): now also R2064.2
- net at U2001.AY20 (SDOUT1): now also R2065.2
- net RSX_VO_EE0: now reaches U2001.AY22 (DE0)
- net RSX_VO02: now reaches U2001.AY23 (VO_002)
- net RSX_VO04: now reaches U2001.AY24 (VO_004)
- net RSX_VO15: now reaches U2001.AY26 (VO_015)
- net RSX_VO17: now reaches U2001.AY27 (VO_017)
- net RSX_VO22: now reaches U2001.AY28 (VO_022)
- net RSX_VO30: now reaches U2001.AY30 (VO_030)
- net RSX_VO35: now reaches U2001.AY31 (VO_035)
- net RSX_AVCLK0: now reaches U2001.AY32 (AVCLKO)
- net RSX_AVCLK1: now reaches U2001.AY34 (AVCLK1)
- net RSX_FB_VREF4: now reaches U2001.AY35 (FB_VREF4)
- net BE_TX3_TXCLKP: now reaches U2001.AL3 (RX3_RXCKP)
- net RSX_VO_VINTE1: now reaches U2001.AL38 (VINTE1)
- net BE_TX3_TXCLKN: now reaches U2001.AL4 (RX3_RXCKN)
- net RSX_VO_DE1: now reaches U2001.AL40 (DE1)
- net BE_TX3_TXP3: now reaches U2001.AL6 (RX3_RXP3)
- net BE_TX3_TXN3: now reaches U2001.AL7 (RX3_RXN3)
- net BE_RX0_RXN6: now reaches U2001.N1 (TX0_TXN6)
- net +1.2V_RSX_VDDR: now reaches U2001.N10 (VDDR)
- net BE_RX0_RXP6: now reaches U2001.N2 (TX1_TXP6)
- net BE_RX0_RXN4: now reaches U2001.N3 (TX2_TXN4)
- net BE_RX0_RXP4: now reaches U2001.N4 (TX3_TXP4)
- net BE_RX0_RXN5: now reaches U2001.N6 (TX5_TXN5)
- net BE_RX0_RXP5: now reaches U2001.N7 (TX6_TXP5)
- net +1.8V_RSX_FBVDDQ: now reaches U2001.J34 (FBVDD)
- net +1.8V_RSX_FBVDDQ: now also U2001.J36 (FBVDD), U2001.J37 (FBVDD)
- net at U2001.J39 (FBCAL0_TERM_GND): now also R2070.2
- net RSX_GPIO1: now reaches U2001.AW16 (GPIO1)
- net RSX_GPIO0: now reaches U2001.AW17 (GPIO0)
- net RSX_AVCLK2: now reaches U2001.AW33 (AVCLK2)
- new net RS_BCLKO: R2064.1
- new net RS_LRCKO: R2063.1
- new net RS_SDOUT1: R2065.1
- no-connect marks 1 -> 3
