File: cok-001/gpu.kicad_sch (KiCad schematic)
At the start: 9 parts

Commit message: switching regulator
Connections:
- net +1.2V_RSX_VDDR: now also U2001.E3 (VDDR), U2001.E4 (VDDR), U2001.E5 (VDDR), U2001.F4 (VDDR), U2001.G3 (VDDR), U2001.G4 (VDDR), U2001.G5 (VDDR), U2001.G6 (VDDR), U2001.G7 (VDDR), U2001.G8 (VDDR), U2001.M12 (VDDR), U2001.P12 (VDDR), U2001.V12 (VDDR)
- net +1.2V_YC_RC_VDDIO: now also U2001.R10 (VDDIORW), U2001.V5 (VDDIORW), U2001.V8 (VDDIORW)
- net GND: now also U2001.A39 (GND), U2001.H34 (GND), U2001.H36 (GND), U2001.H37 (GND), U2001.M32 (GND), U2001.R12 (GND), U2001.R14 (GND), U2001.R16 (GND), U2001.R18 (GND), U2001.R20 (GND), U2001.R22 (GND), U2001.R24 (GND), U2001.R26 (GND), U2001.R28 (GND), U2001.R35 (GND), U2001.R41 (GND), U2001.R5 (GND), U2001.R8 (GND), U2001.V10 (GND), U2001.V15 (GND), U2001.V19 (GND), U2001.V21 (GND), U2001.V23 (GND), U2001.V27 (GND), U2001.V30 (GND), U2001.V34 (GND), U2001.V37 (GND)
- net BE_RX0_RXN2: now reaches U2001.R1 (TX0_TXN2)
- net at U2001.R15 (VDD): now also U2001.R17 (VDD), U2001.R19 (VDD), U2001.R21 (VDD), U2001.R23 (VDD), U2001.R25 (VDD), U2001.R27 (VDD), U2001.R30 (VDD)
- net BE_RX0_RXP2: now reaches U2001.R2 (TX0_TXP2)
- net BE_RX0_RXN0: now reaches U2001.R3 (TX0_TXN0)
- net RSX_VI12: now reaches U2001.R36 (VI12)
- net RSX_VI14: now reaches U2001.R37 (VI14)
- net RSX_PCLKI: now reaches U2001.R38 (PCLKI)
- net BE_RX0_RXP0: now reaches U2001.R4 (TX0_TXP0)
- net RSX_VI22: now reaches U2001.R40 (VI22)
- net BE_RX0_RXN1: now reaches U2001.R6 (TX0_TXN1)
- net BE_RX0_RXP1: now reaches U2001.R7 (TX0_TXP1)
- net BE_TX1_TXP4: now reaches U2001.V1 (RX1_RXP4)
- net at U2001.V14 (VDD): now also U2001.V18 (VDD), U2001.V20 (VDD), U2001.V22 (VDD), U2001.V24 (VDD), U2001.V28 (VDD), U2001.V32 (GND)
- net BE_TX1_TXN4: now reaches U2001.V2 (RX1_RXN4)
- net BE_TX1_TXP6: now reaches U2001.V3 (RX1_RXP6)
- net BE_TX1_TXN6: now reaches U2001.V4 (RX1_RXN6)
- net BE_TX1_TXP5: now reaches U2001.V6 (RX1_RXP5)
- net BE_TX1_TXN5: now reaches U2001.V7 (RX1_RXN5)
- no-connect marks 3 -> 4

Commit message: ram lines
Connections:
- net BE_RX0_RXCLKN: now reaches U2001.P3 (TX0_TXCKN)
- net BE_RX0_RXCLKP: now reaches U2001.P4 (TX0_TXCKP)
- net BE_RX0_RXN3: now reaches U2001.P6 (TX0_TXN3)
- net BE_RX0_RXP3: now reaches U2001.P7 (TX0_TXP3)
- net BE_RX0_RXN7: now reaches U2001.M6 (TX0_TXN7)
- net BE_RX0_RXP7: now reaches U2001.M7 (TX0_TXP7)
Changed lines of the file:
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@@
+		)
+	)
+	(global_label "BE_RX0_RXP3"
+		(shape output)
+		(at 325.12 27.94 180)
+		(fields_autoplaced yes)
+		(effects
+			(font
+				(size 1.27 1.27)
+			)
+			(justify right)
+		)
+		(property "Intersheetrefs" "${INTERSHEET_REFS}"
+			(at 309.1326 27.94 0)
+			(effects
+				(font
+					(size 1.27 1.27)
+				)
+				(justify right)
+				(hide yes)
+			)
 		)
 	)
@@
 		)
 	)
+	(global_label "BE_RX0_RXN7"
+		(shape output)
+		(at 297.18 25.4 180)
+		(fields_autoplaced yes)
+		(effects
+			(font
+				(size 1.27 1.27)
+			)
+			(justify right)
+		)
+		(property "Intersheetrefs" "${INTERSHEET_REFS}"
+			(at 281.1321 25.4 0)
+			(effects
+				(font
+					(size 1.27 1.27)
+				)
+				(justify right)
+				(hide yes)
+			)
+		)
+	)
 	(global_label "BE_RX0_RXN2"
 		(shape output)
@@
 		)
 	)
+	(global_label "BE_RX0_RXN3"
+		(shape output)
+		(at 325.12 25.4 180)
+		(fields_autoplaced yes)
+		(effects
+			(font
+				(size 1.27 1.27)
+			)
+			(justify right)
+		)
+		(property "Intersheetrefs" "${INTERSHEET_REFS}"
+			(at 309.0721 25.4 0)
+			(effects
+				(font
+					(size 1.27 1.27)
+				)
+				(justify right)
+				(hide yes)
+			)
+		)
+	)
 	(global_label "RSX_VI28"
 		(shape input)
@@
 		)
 	)
+	(global_label "BE_RX0_RXCLKN"
+		(shape output)
+		(at 325.12 17.78 180)
+		(fields_autoplaced yes)
+		(effects
+			(font
+				(size 1.27 1.27)
+			)
+			(justify right)
+		)
+		(property "Intersheetrefs" "${INTERSHEET_REFS}"
+			(at 306.7135 17.78 0)
+			(effects
+				(font
+					(size 1.27 1.27)
+				)
+				(justify right)
+				(hide yes)
+			)
+		)
+	)
 	(global_label "BE_TX2_TXN6"
 		(shape input)
@@
 		)
 	)
+	(global_label "BE_RX0_RXCLKP"
+		(shape output)
+		(at 325.12 20.32 180)
+		(fields_autoplaced yes)
+		(effects
+			(font
+				(size 1.27 1.27)
+			)
+			(justify right)
+		)
+		(property "Intersheetrefs" "${INTERSHEET_REFS}"
+			(at 306.774 20.32 0)
+			(effects
+				(font
+					(size 1.27 1.27)
+				)
+				(justify right)
+				(hide yes)
+			)
+		)
+	)
 	(global_label "RSX_VO69"
 		(shape input)
@@
 			(effects
 				(font
+					(size 1.27 1.27)
+				)
+				(justify right)
+				(hide yes)
+			)
+		)
+	)
+	(global_label "BE_RX0_RXP7"
+		(shape output)
+		(at 297.18 27.94 180)
+		(fields_autoplaced yes)
+		(effects
+			(font
+				(size 1.27 1.27)
+			)
+			(justify right)
+		)
+		(property "Intersheetrefs" "${INTERSHEET_REFS}"
+			(at 281.1926 27.94 0)
+			(effects
+				(font
