File: cok-001/gpu.kicad_sch (KiCad schematic)
At the start: 9 parts

Commit message: rsx pins
Connections:
- net RS_TMS: now reaches U2001.AR14 (JTAG_TMS)
- net TS_TDO: now reaches U2001.AR16 (JTAG_TDO)
- net RS_TDI: now reaches U2001.AT16 (JTAG_TDI)
- net RS_TCK: now reaches U2001.AU13 (JTAG_TCK)
- net ~{RS_TRSTNEG}: now reaches U2001.AU15 (JTAG_TRST_N)
- net RS_LRCKI1: now reaches U2001.AU17 (LRCKI1)
- net RS_SPMCLKI: now reaches U2001.AU19 (SPMCLKI)
- net RSX_VO05: now reaches U2001.AU25 (VO_005)
- net RSX_VO11: now reaches U2001.AU27 (VO_011)
- net RSX_VO18: now reaches U2001.AU29 (VO_018)
- net RSX_VO23: now reaches U2001.AU31 (VO_023)
- no-connect marks 4 -> 9

Commit message: rsx symbol done
Connections:
- net GND: now also R2068.1, U2001.W18 (GND), U2001.W20 (GND), U2001.W22 (GND), U2001.W24 (GND), U2001.W28 (GND), U2001.Y15 (GND), U2001.Y19 (GND), U2001.Y21 (GND), U2001.Y23 (GND), U2001.Y27 (GND)
- net RSX_VO69: now also U2001.AA36 (VO_133)
- net RSX_VO70: now also U2001.Y35 (VO_134)
- net RSX_VO71: now also U2001.AA39 (VO_135)
- net RSX_VI16: now reaches U2001.P35 (VI16)
- net RSX_VI20: now reaches U2001.P36 (VI20)
- net RSX_VI18: now reaches U2001.P38 (VI18)
- net RSX_VI26: now reaches U2001.P39 (VI26)
- net RSX_VI25: now reaches U2001.P40 (VI25)
- net RSX_VI24: now reaches U2001.P41 (VI24)
- net RSX_VI23: now reaches U2001.M35 (VI23)
- net RSX_VI30: now reaches U2001.M38 (VI30)
- net RSX_VI35: now reaches U2001.M39 (VI35)
- net RSX_VI32: now reaches U2001.M40 (VI32)
- net at U2001.Y14 (VDD): now also U2001.Y18 (VDD), U2001.Y20 (VDD), U2001.Y22 (VDD), U2001.Y24 (VDD), U2001.Y28 (VDD)
- net RSX_HSYNCI: now reaches U2001.Y38 (HSYNCI)
- net at U2001.W15 (VDD): now also U2001.W19 (VDD), U2001.W21 (VDD), U2001.W23 (VDD), U2001.W27 (VDD)
- net BE_TX1_TXP7: now reaches U2001.W3 (RX1_RXP7)
- net RSX_HTPLGIN: now reaches U2001.W36 (HTPLGI)
- net RSX_VSYNCI: now reaches U2001.W38 (VSYNCI)
- net BE_TX1_TXN7: now reaches U2001.W4 (RX1_RXN7)
- net BE_RX1_RXN7: now reaches U2001.W6 (TX1_TXN7)
- net BE_RX1_RXP7: now reaches U2001.W7 (TX1_TXP7)
Other:
- moved on the sheet: R2063, R2064, R2065
