File: cok-001/wireless.kicad_sch (KiCad schematic)
At the start: 21 parts, among them J3701 Conn_01x33_MountingPin, Q3701 UMH2NTN

Commit message: lf
Parts:
- TH3701, TH3702: value Thermistor_PTC -> !
- renumbered L3701 to LF3701, L3702 to LF3702, L3703 to LF3703
Changed lines of the file:
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@@
 		(in_pos_files yes)
 		(dnp yes)
-		(property "Reference" "L3703"
+		(property "Reference" "LF3703"
 			(at 182.88 78.105 0)
 			(show_name no)
@@
 			(project "cok-001"
 				(path "/976eb78d-8215-4cc0-9d72-f9d535c7970b/a8d3d0f2-2567-4d70-a367-7d8ff0d1aec4"
-					(reference "L3703")
+					(reference "LF3703")
 					(unit 1)
 				)
@@
 		(in_pos_files yes)
 		(dnp no)
-		(fields_autoplaced yes)
 		(property "Reference" "Q3701"
 			(at 55.88 105.5877 0)
@@
 		)
 		(property "Value" "UMH2NTN"
-			(at 55.88 108.1277 0)
+			(at 57.15 109.22 0)
 			(show_name no)
 			(do_not_autoplace no)
@@
 			)
 		)
-		(property "Value" "Thermistor_PTC"
+		(property "Value" "!"
 			(at 176.8475 29.21 90)
 			(show_name no)
@@
 		(in_pos_files yes)
 		(dnp yes)
-		(property "Reference" "L3701"
+		(property "Reference" "LF3701"
 			(at 182.88 57.785 0)
 			(show_name no)
@@
 			(project "cok-001"
 				(path "/976eb78d-8215-4cc0-9d72-f9d535c7970b/a8d3d0f2-2567-4d70-a367-7d8ff0d1aec4"
-					(reference "L3701")
+					(reference "LF3701")
 					(unit 1)
 				)
@@
 		)
 		(property "Value" "UMH2NTN"
-			(at 48.26 108.1277 0)
+			(at 46.99 107.95 0)
 			(show_name no)
 			(do_not_autoplace no)
@@
 			)
 		)
-		(property "Value" "Thermistor_PTC"
+		(property "Value" "!"
 			(at 189.5475 21.59 90)
 			(show_name no)
@@
 		(in_pos_files yes)
 		(dnp yes)
-		(property "Reference" "L3702"
+		(property "Reference" "LF3702"
 			(at 175.26 67.945 0)
 			(show_name no)
@@
 			(project "cok-001"
 				(path "/976eb78d-8215-4cc0-9d72-f9d535c7970b/a8d3d0f2-2567-4d70-a367-7d8ff0d1aec4"
-					(reference "L3702")
-					(unit 1)
-				)
+					(reference "LF3702")
+					(unit 1)
+				)
