File: cok-001/syscon.kicad_sch (KiCad schematic)
At the start: 80 parts, among them J4001 Conn_01x03_Pin, J4003 Conn_01x02_Pin, J4009 Conn_01x30_Socket, J4010 Conn_01x10_Socket, Q4014 DTC143ZUA, Y4001 Crystal, Y4002 Crystal

Commit message: sata
Parts:
- added C4031: 100u 16V, Capacitor_SMD:CP_Elec_5x3.9, symbol Device:C_Polarized_US
- added C4032, C4047, C4050, C4051, C4052, C4053, C4054, C4058, C4062: 0.001u 50V, Capacitor_SMD:C_0402_1005Metric, symbol Device:C
- added C4049: 1u 10V, Capacitor_SMD:C_0603_1608Metric, symbol Device:C
- added D4006: XX, LED_SMD:LED_0402_1005Metric, symbol Device:LED
- added D4010: EDZCTE616, Diode_SMD:D_SOD-923, symbol Device:D_Zener
- added FB4001: 0uH, Inductor_SMD:L_0603_1608Metric, symbol Device:FerriteBead_Small
- added JL4006, JL4007, TP9407: TestPoint, TestPoint:TestPoint_Pad_D1.5mm, symbol Connector:TestPoint
- added Q4011: DTC143ZUA, Package_TO_SOT_SMD:SOT-323_SC-70, symbol Transistor_BJT:DTC144E
- added R4114, R4138, R4139, R4140: 0, Resistor_SMD:R_0402_1005Metric, symbol Device:R_US
- added R4118, R4120: XX, Resistor_SMD:R_0402_1005Metric, symbol Device:R_US
- added RN4001, RN4002, RN4003: 10k, Resistor_SMD:R_Array_Convex_4x0402, symbol Device:R_Pack04
- added RN4004, RN4005, RN4006, RN4007: 22, Resistor_SMD:R_Array_Convex_4x0402, symbol Device:R_Pack04
- added TP4012, TP4084, TP4085, TP4087, TP4091, TP4092, TP4094, TP4099, TP4100, TP4101, TP4106, TP9408, TP9409: TestPoint, TestPoint:TestPoint_Pad_1.0x1.0mm, symbol Connector:TestPoint
- J4001: value Conn_01x03_Pin -> FAN; footprint (none) -> Connector_JST:JST_PH_B3B-PH-SM4-TB_1x03-1MP_P2.00mm_Vertical
- J4003: footprint Connector_JST:JST_ZH_B2B-ZR-SM4-TF_1x02-1MP_P1.50mm_Vertical -> Connector_PinHeader_1.27mm:PinHeader_1x02_P1.27mm_Vertical_SMD_Pin1Left
- J4010: value Conn_01x10_Socket -> BUTTONS; footprint Connector_Molex:Molex_Picoflex_90814-0010_2x05_P1.27mm_Vertical -> Connector_FFC-FPC:Hirose_FH26-13S-0.3SHW_2Rows-13Pins-1MP_P0.60mm_Horizontal
- Y4002: footprint Crystal:Crystal_SMD_5032-4Pin_5.0x3.2mm -> Crystal:Crystal_SMD_G8-2Pin_3.2x1.5mm
Connections:
- net GND: now also J4001.2 (Pin_2), J4010.2 (Pin_2), U4002.C2 (AvRef2), U4002.G6 (AVss), U4002.R4 (AVSUO), C4031.2, C4032.2, C4047.2, C4049.1, C4050.2, C4051.2, C4052.2, C4053.2, C4054.2, C4058.2, C4062.2, D4010.2 (A), Q4011.2 (E), RN4001.5 (R4.2), RN4001.6 (R3.2), RN4001.7 (R2.2), RN4001.8 (R1.2), RN4002.5 (R4.2), RN4002.6 (R3.2), RN4002.7 (R2.2), RN4002.8 (R1.2), RN4003.5 (R4.2), RN4003.6 (R3.2), RN4003.7 (R2.2), RN4003.8 (R1.2), TP9408.1
- net at J4009.17 (Pin_17), U4002.R10 (RMC_IN): now also R4120.1
- net at J4010.1 (Pin_1): now also C4049.2
- net at J4010.3 (Pin_3): now also C4054.1
- net at J4010.4 (Pin_4): now also U4002.N7 (STBY_LED), C4053.1
- net at J4010.5 (Pin_5): now also U4002.M7 (POW_LED), C4052.1
- net at J4010.6 (Pin_6): now also U4002.A12 (~{EJECT_SW}), C4051.1, JL4006.1
- net at J4010.7 (Pin_7): now also U4002.B12 (~{POW_SW}), C4050.1, JL4007.1
- net at J4010.8 (Pin_8): now also R4120.2
- net at J4010.9 (Pin_9): now also U4002.N9 (SW_PWM), C4062.1
- net at J4001.1 (Pin_1): now also FB4001.2
- net at J4001.3 (Pin_3): now also U4002.N8 (FANPWM0), D4010.1 (K), Q4011.1 (B), TP9407.1
- net at U4002.A14 (PE3): now also TP4094.1
- net at U4002.A3 (SW_0): now also RN4001.1 (R1.1)
- net SW_8_C: now reaches U4002.A4 (SW_8_C)
- net SW_8_C: now also RN4003.2 (R2.1)
- net at U4002.A6 (MC_RESERVED2): now also R4080.2
- net at U4002.B14 (VD_CECI1): now also TP4099.1
- net SW_8_B: now reaches U4002.B4 (SW_8_B)
- net SW_8_B: now also RN4003.3 (R3.1)
- net at U4002.B7 (MC_RESERVED1): no longer R4080.2
- net at U4002.C16 (OSCIN): now also C4027.1, Y4002.1
- net at U4002.D13 (SW_1A): now also R4138.1, RN4001.3 (R3.1)
- net at U4002.F13 (SW_5_B): now also RN4001.2 (R2.1)
- net at U4002.G12 (BEVRM_VID4): now also RN4004.3 (R3.1)
- net at U4002.G13 (BEVRM_VID5): now also RN4004.4 (R4.1)
- net at U4002.H1 (PN5): now also TP4084.1
- net at U4002.H12 (BEVRM_VID2): now also RN4004.2 (R2.1)
- net at U4002.H13 (BEVRM_VID3): now also RN4004.1 (R1.1)
- net at U4002.H2 (PN6): now also TP4012.1
- net at U4002.J11 (~{RST}): now also C4047.1, R4114.2
- net at U4002.J12 (BEVRM_VID0): now also RN4005.4 (R4.1)
- net at U4002.J13 (BEVRM_VID1): now also RN4005.3 (R3.1)
- net ~{RSX_INT}: now reaches U4002.J2 (~{RSX_INT})
- net ~{RSX_INT}: now also C4058.1
- net at U4002.K12 (I2CBUS_EN): now also TP4106.1
- net at U4002.K13 (PC7): now also TP4085.1
- net at U4002.L12 (RSXVRM_VID4): now also RN4006.3 (R3.1)
- net at U4002.L13 (RSXVRM_VID5): now also RN4006.4 (R4.1)
- net SW_PCI: now reaches U4002.L16 (SW_PCI)
- net SW_PCI: now also RN4002.3 (R3.1)
- net at U4002.M12 (RSXVRM_VID2): now also RN4007.3 (R3.1)
- net at U4002.M13 (RSXVRM_VID3): now also RN4006.2 (R2.1)
- net SW_2: now reaches U4002.M15 (SW_2)
- net SW_2: now also RN4002.4 (R4.1)
- net at U4002.M4 (PA0): now also TP4092.1
- net at U4002.M6 (PA4): now also TP4087.1
- net at U4002.N11 (SW_4_A): now also R4140.2, RN4003.4 (R4.1)
- net at U4002.N12 (RSXVRM_VID0): now also RN4007.4 (R4.1)
- net at U4002.N13 (RSXVRM_VID1): now also RN4006.1 (R1.1)
- net at U4002.N4 (SW_5_A): now also RN4007.1 (R1.1)
- net at U4002.R11 (VD_CECO0): now also TP4100.1
- net at U4002.R13 (SW_1_B): now also R4139.1, RN4001.4 (R4.1)
- net at U4002.R14 (SW_7_A): now also RN4005.2 (R2.1)
- net at U4002.R8 (RSX_FBVDD_SEL): now also RN4007.2 (R2.1)
- net at U4002.T12 (VD_CECO1): now also TP4101.1
- net SW_4_B: now reaches U4002.T13 (SW_4_B)
- net SW_4_B: now also RN4003.1 (R1.1)
- net SW_6: now reaches U4002.T14 (SW_6)
- net SW_6: now also RN4002.2 (R2.1)
- net SW_8_A: now reaches U4002.T15 (SW_8_A)
- net SW_8_A: now also RN4002.1 (R1.1)
- net BD_LED: now reaches R4080.1
- new net: D4006.1 (K), Q4011.3 (C)
- new net: D4006.2 (A), R4118.2
- new net +12V_MAIN: C4031.1, C4032.1, FB4001.1, TP9409.1
- new net BEVRM_VID0: RN4005.5 (R4.2)
- new net BEVRM_VID1: RN4005.6 (R3.2)
- new net BEVRM_VID2: RN4004.7 (R2.2)
- new net BEVRM_VID3: RN4004.8 (R1.2)
- new net BEVRM_VID4: RN4004.6 (R3.2)
- new net BEVRM_VID5: RN4004.5 (R4.2)
- new net RSX_FBVDD_SEL: RN4007.7 (R2.2)
- new net RXVRM_VID0: RN4007.5 (R4.2)
- new net RXVRM_VID1: RN4006.8 (R1.2)
- new net RXVRM_VID2: RN4007.6 (R3.2)
- new net RXVRM_VID3: RN4006.7 (R2.2)
- new net RXVRM_VID4: RN4006.6 (R3.2)
- new net RXVRM_VID5: RN4006.5 (R4.2)
- new net SW_1_A: R4138.2
- new net SW_1_B: R4139.2
- new net SW_4_A: R4140.1
- new net SW_5_A: RN4007.8 (R1.2)
- new net SW_7_A: RN4005.7 (R2.2)
- new net ~{SYSCON_RST}: R4114.1, TP4091.1
- no-connect marks 9 -> 11
Other:
- moved on the sheet: J4001, J4010

Commit message: southbridge
Connections:
- net ~{SB_SPI_CS}: now reaches R4002.2
- net SB_SPI_CLK: now reaches R4004.2
- net SB_SPI_DO: now reaches R4003.2
- net DVE_I2C_SDA: now reaches R4104.2
- net ACDC_STBY: now reaches U4002.A11 (ACDC_STBY)
- net SB_SPI_DI_M: now reaches U4002.A9 (SB_SPI_DI)
- net ~{DVE_RST}: now reaches U4002.B5 (~{DVE_RST})
- net at U4002.C16 (OSCIN): now also C4027.1, Y4002.1
- net XCG_EN: now reaches U4002.D5 (XCG_EN)
- net RSX_FLDO1: now reaches U4002.J1 (RSX_FLDO1)
- net DVE_I2C_SCL: now reaches R4105.2

Commit message: bridge sif
Parts:
- added R1101, R4037: 4700, Resistor_SMD:R_0402_1005Metric, symbol Device:R_US
- added TP9405, TP9406: TestPoint, TestPoint:TestPoint_Pad_D1.5mm, symbol Connector:TestPoint
- C4069: footprint Capacitor_SMD:C_0402_1005Metric -> Capacitor_SMD:C_0603_1608Metric
Connections:
- net at U4002.C16 (OSCIN): now also C4027.1, Y4002.1
- net at U4002.N15 (BACKUP_MODE): now also R1101.1, TP9406.1
- net at U4002.N16 (DIAG_MODE): now also R4037.1, TP9405.1
- new net: R1101.2, R4037.2

Commit message: update to 9
Connections:
- net at U4002.C16 (OSCIN): now also C4027.1, Y4002.1
Changed lines of the file:
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@@
 (kicad_sch
-	(version 20231120)
+	(version 20250114)
 	(generator "eeschema")
-	(generator_version "8.0")
+	(generator_version "9.0")
 	(paper "A4")
 	(junction

Commit message: temp sensor and clock
Parts:
- added Q4012, Q4013: UMH2NTN, Package_TO_SOT_SMD:SOT-363_SC-70-6, symbol Transistor_BJT:MUN5213DW1
- added Q4015: DTC143ZUA, Package_TO_SOT_SMD:SOT-323_SC-70, symbol Transistor_BJT:DTC144E
- added R4124: XX, Resistor_SMD:R_0402_1005Metric, symbol Device:R_US
- added R4129: 10k, Resistor_SMD:R_0402_1005Metric, symbol Device:R_US
- added U1: 74LVC1G34, Package_TO_SOT_SMD:SOT-353_SC-70-5, symbol 74xGxx:74LVC1G34
- added U4003, U4004, U4005: 74LVC2G34, Package_TO_SOT_SMD:SOT-363_SC-70-6, symbol 74xGxx:74LVC2G34
- D4006, R4118: now not fitted
- Y4001: value Crystal -> 16.9344MHz
- Y4002: value Crystal -> 32.768kHz; footprint Crystal:Crystal_SMD_G8-2Pin_3.2x1.5mm -> Crystal:Crystal_SMD_SeikoEpson_MC156-4Pin_7.1x2.5mm; symbol Device:Crystal -> Device:Crystal_GND23
Connections:
- net BD_LED: now also Q4015.1 (B)
- net GND: now also Q4012.1 (E1), Q4012.4 (E2), Q4013.4 (E2), Q4015.2 (E), R4129.2, U1.3 (GND), U4003.2 (GND), U4004.2 (GND), U4005.2 (GND)
- net +5V_EVER: now reaches BZ4001.2 (-), R4128.2
- net +5V_EVER: now also R4118.1
- net SW_4_A_M: now reaches R4140.2, RN4003.4 (R4.1), U4002.N11 (SW_4_A)
- net at C4054.1, J4010.3 (Pin_3): now also Q4013.3 (C2), Q4015.3 (C)
- net at U4002.C16 (OSCIN): now also C4027.1, Y4002.1
- net at U4002.D10 (~{MUL_TRG_OUT}): now also U1.2
- net ~{SB_INT}: now reaches U4002.D9 (~{SB_INT})
- net SW_ATA: now reaches U4002.M11 (SW_ATA)
- net SW_ATA: now also Q4013.2 (B1), R4129.1
- net SW_3: now reaches U4002.R12 (SW_3)
- new net: U1.4, U4003.3, U4003.6, U4004.3, U4004.6, U4005.3, U4005.6
- new net: Q4012.3 (C2), Q4012.6 (C1), Q4013.1 (E1), Q4013.5 (B2)
- new net: C4028.1, U4002.B16 (OSCOUT), Y4002.4
- new net: Q4013.6 (C1), R4124.2
- new net +1.2V_MC2_VDDIO: U4003.5 (VCC)
- new net +1.5V_RSX_VDDIO: U4004.5 (VCC)
- new net +3.3V_EVER: R4124.1, U1.5 (VCC), U4005.5 (VCC)
- new net BE_TRG_IN: U4003.4
- new net BE_TRG_OUT: U4003.1
- new net DISC_CHUCK: Q4012.5 (B2)
- new net MC_ALIVE: Q4012.2 (B1)
- new net SB_TRG_IN: U4005.4
- new net SB_TRG_OUT: U4005.1
- new net ~{RSX_TRG_IN}: U4004.4
- new net ~{RSX_TRG_OUT}: U4004.1
- now unconnected: U4002.B16 (OSCOUT), Y4002.2
- no-connect marks 11 -> 13
Other:
- moved on the sheet: R4140

Commit message: dumb numbers
Parts:
- added R4088, R4089: 0, Resistor_SMD:R_0402_1005Metric, symbol Device:R_US
- U4006: renamed from U1; now not fitted
Connections:
- net at U4002.C16 (OSCIN): now also C4027.1, Y4002.1
- net ~{SYS_THR_ALRT}: now reaches U4002.E9 (~{SYS_THR_ALRT})
- net ~{SYS_THR_ALRT}: now also R4088.2, R4089.2
- new net ~{THRBE_SEND_ALRT}: R4088.1
- new net ~{THRRSX_SENS_ALRT}: R4089.1

Commit message: qqq
Parts:
- added Q4008: DTC144E, Package_TO_SOT_SMD:SOT-323_SC-70, symbol Transistor_BJT:DTC144E
- D4006: value XX -> Thermal LED
Connections:
- net GND: now also Q4008.2 (E)
- net at U4002.C16 (OSCIN): now also C4027.1, Y4002.1
- net at U4002.M10 (~{XDR_FET_VREF}): now also Q4008.1 (B)
- new net XDR_RQ_VREF_FET: Q4008.3 (C)
Changed lines of the file:
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@@
 	(wire
 		(pts
+			(xy 247.65 82.55) (xy 247.65 -15.24)
+		)
+		(stroke
+			(width 0)
+			(type default)
+		)
+	)
+	(wire
+		(pts
 			(xy 424.18 121.92) (xy 424.18 90.17)
 		)
@@
 	(wire
 		(pts
+			(xy 247.65 -15.24) (xy 274.32 -15.24)
+		)
+		(stroke
+			(width 0)
+			(type default)
+		)
+	)
+	(wire
+		(pts
 			(xy 280.67 180.34) (xy 341.63 180.34)
 		)
@@
 		)
 	)
+	(global_label "XDR_RQ_VREF_FET"
+		(shape output)
+		(at 283.21 -20.32 0)
+		(fields_autoplaced yes)
+		(effects
+			(font
+				(size 1.27 1.27)
+			)
+			(justify left)
+		)
+		(property "Intersheetrefs" "${INTERSHEET_REFS}"
+			(at 303.2494 -20.32 0)
+			(effects
+				(font
+					(size 1.27 1.27)
+				)
+				(justify left)
+				(hide yes)
+			)
+		)
+	)
 	(global_label "ACDC_STBY"
 		(shape output)
@@
 	)
 	(symbol
+		(lib_id "power:GND")
+		(at 283.21 -10.16 0)
+		(unit 1)
+		(exclude_from_sim no)
+		(in_bom yes)
+		(on_board yes)
+		(dnp no)
+		(fields_autoplaced yes)
+		(property "Reference" "#PWR0327"
+			(at 283.21 -3.81 0)
+			(effects
+				(font
+					(size 1.27 1.27)
+				)
+				(hide yes)
+			)
+		)
+		(property "Value" "GND"
+			(at 283.21 -5.08 0)
+			(effects
+				(font
+					(size 1.27 1.27)
+				)
+			)
+		)
+		(property "Footprint" ""
+			(at 283.21 -10.16 0)
+			(effects
+				(font
+					(size 1.27 1.27)
+				)
+				(hide yes)
+			)
+		)
+		(property "Datasheet" ""
+			(at 283.21 -10.16 0)
+			(effects
+				(font
+					(size 1.27 1.27)
+				)
+				(hide yes)
+			)
+		)
+		(property "Description" "Power symbol creates a global label with name \"GND\" , ground"
+			(at 283.21 -10.16 0)
+			(effects
+				(font
+					(size 1.27 1.27)
+				)
+				(hide yes)
+			)
+		)
+		(pin "1"
+		)
+		(instances
+			(project "cok-001"
+				(path "/976eb78d-8215-4cc0-9d72-f9d535c7970b/c2fb6f44-7647-4597-badb-4e48fc7de398"
+					(reference "#PWR0327")
+					(unit 1)
+				)
+			)
+		)
+	)
+	(symbol
 		(lib_id "Device:R_US")
 		(at 133.35 72.39 180)
@@
 	)
 	(symbol
+		(lib_id "Transistor_BJT:DTC144E")
+		(at 280.67 -15.24 0)
+		(unit 1)
+		(exclude_from_sim no)
+		(in_bom yes)
+		(on_board yes)
+		(dnp no)
+		(property "Reference" "Q4008"
+			(at 285.75 -16.5101 0)
+			(effects
+				(font
+					(size 1.27 1.27)
+				)
+				(justify left)
+			)
+		)
+		(property "Value" "DTC144E"
+			(at 285.75 -13.9701 0)
+			(effects
+				(font
+					(size 1.27 1.27)
+				)
+				(justify left)
+			)
+		)
+		(property "Footprint" "Package_TO_SOT_SMD:SOT-323_SC-70"
+			(at 280.67 -15.24 0)
+			(effects
+				(font
+					(size 1.27 1.27)
+				)
+				(justify left)
+				(hide yes)
+			)
+		)
+		(property "Datasheet" ""
+			(at 280.67 -15.24 0)
+			(effects
+				(font
+					(size 1.27 1.27)
+				)
+				(justify left)
+				(hide yes)
+			)
+		)
+		(property "Description" "Digital NPN Transistor, 47k/47k, SOT-23"
+			(at 280.67 -15.24 0)
+			(effects
+				(font
+					(size 1.27 1.27)
+				)
+				(hide yes)
+			)
+		)
+		(pin "3"
+		)
+		(pin "1"
+		)
+		(pin "2"
+		)
+		(instances
+			(project "cok-001"
+				(path "/976eb78d-8215-4cc0-9d72-f9d535c7970b/c2fb6f44-7647-4597-badb-4e48fc7de398"
+					(reference "Q4008")
+					(unit 1)
+				)
+			)
+		)
+	)
+	(symbol
 		(lib_id "Connector:TestPoint")
 		(at 107.95 172.72 90)
@@
 			)
 		)
-		(property "Value" "XX"
+		(property "Value" "Thermal LED"
 			(at 326.39 32.0674 90)
 			(effects
