File: cok-001/syscon.kicad_sch (KiCad schematic)
At the start: 141 parts, among them J4001 FAN, J4003 Conn_01x02_Pin, J4009 Conn_01x30_Socket, J4010 BUTTONS, Q4008 DTC144E, Q4011 DTC143ZUA, Q4012 UMH2NTN, Q4013 UMH2NTN, Q4014 DTC143ZUA, Q4015 DTC143ZUA, U4003 74LVC2G34, U4004 74LVC2G34, U4005 74LVC2G34, U4006 74LVC1G34, Y4001 16.9344MHz, Y4002 32.768kHz

Commit message: update 10
Parts:
- U4002: value ~ -> (none)
Connections:
- net at U4002.C16 (OSCIN): now also C4027.1, Y4002.1

Commit message: lf
Parts:
- renumbered U4003 to IC4003, U4004 to IC4004, U4005 to IC4005, U4006 to IC4006
Connections:
- net ~{SS2_RESET}: now reaches U4002.A13 (~{SB_EBUS_RESET})
- net SS2_BRDY: now reaches U4002.B13 (SB_EBUS_BRDY)
- net at U4002.C16 (OSCIN): now also C4027.1, Y4002.1
- net ~{SB_RESET}: now reaches U4002.D11 (~{SB_RESET})
- net ~{SB_CGRST}: now reaches U4002.E11 (~{SB_CGRESET})
- net BT_WAKE: now reaches U4002.E12 (BT_WAKEON)
- net MK_EN: now reaches U4002.F12 (MK_EN)
- net BE_SPI_DI: now reaches U4002.M1 (BE_SPI_DI)
- net SC_BUZZER: now reaches Q4014.1 (B), U4002.M9 (BUZZER)
- net BE_INT: now reaches U4002.T2 (~{BE_INT})
