File: cok-001/sbmisc.kicad_sch (KiCad schematic)
At the start: 30 parts, among them X3001 ASCO

Commit message: sb
Parts:
- renumbered C1 to C3151
Changed lines of the file:
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@@
 		(on_board yes)
 		(dnp yes)
-		(property "Reference" "C1"
+		(property "Reference" "C3151"
 			(at 328.93 238.7599 0)
 			(effects
@@
 			(project "cok-001"
 				(path "/976eb78d-8215-4cc0-9d72-f9d535c7970b/f142be78-51ea-4b88-b7e4-d9b9ccfc7239"
-					(reference "C1")
+					(reference "C3151")
 					(unit 1)
 				)

Commit message: temp sensor and clock
Parts:
- added C3155: 0.1u 10V, Capacitor_SMD:C_0402_1005Metric, symbol Device:C
- added U3101: AD51/007Z, Package_SO:MSOP-8_3x3mm_P0.65mm, symbol Sensor_Temperature:MCP9804_MSOP
Connections:
- net GND: now also C3155.2, U3101.4 (GND), U3101.5 (A2), U3101.6 (A1)
- new net +3.3V_THERMAL: C3155.1, U3101.7 (A0), U3101.8 (V_{DD})
- new net THR_I2C_SCL: U3101.2 (SCL)
- new net THR_I2C_SDA: U3101.1 (SDA)
- no-connect marks 1 -> 2

Commit message: regulator
Parts:
- added Q3101: DTC143ZUA, Package_TO_SOT_SMD:SOT-323_SC-70, symbol Transistor_BJT:DTC144E
- added TP3031, TP3033, TP3034, TP3035, TP3036, TP3037, TP3038, TP3039, TP3040: TestPoint, TestPoint:TestPoint_Pad_1.0x1.0mm, symbol Connector:TestPoint
- X3001: footprint Oscillator:Oscillator_SMD_Abracon_ASCO-4Pin_1.6x1.2mm -> Oscillator:Oscillator_SMD_Abracon_ASE-4Pin_3.2x2.5mm
Connections:
- net GND: now also Q3101.2 (E)
- net SB_PIO10: now also TP3035.1
- net SB_PIO11: now also TP3036.1
- net SB_PIO12: now also TP3037.1
- net SB_PIO13: now also TP3038.1
- net SB_PIO14: now also TP3039.1
- net SB_PIO15: now also TP3040.1
- net SB_PIO8: now also TP3033.1
- net SB_PIO9: now also TP3034.1
- net SB_USB_CLK: now also TP3031.1
- new net SB_CHKSTP_IN: Q3101.3 (C)
- new net ~{BE_CHKSTP_OUT}: Q3101.1 (B)
Other:
- moved on the sheet: R3121

Commit message: msop
Parts:
- U3101: footprint Package_SO:MSOP-8_3x3mm_P0.65mm -> PS3:MSOP-8_2.9x4mm_P0.65mm
Changed lines of the file:
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@@
 			)
 		)
-		(property "Footprint" "Package_SO:MSOP-8_3x3mm_P0.65mm"
+		(property "Footprint" "PS3:MSOP-8_2.9x4mm_P0.65mm"
 			(at 195.58 252.73 0)
 			(effects
