File: cok-001/sbmisc.kicad_sch (KiCad schematic)
At the start: 42 parts, among them Q3101 DTC143ZUA, U3101 AD51/007Z, X3001 ASCO

Commit message: update 10
Parts:
- added R3092, R3096, R3162: 10k, Resistor_SMD:R_0402_1005Metric, symbol Device:R_US
Connections:
- net GND: now also R3092.2, R3096.2, R3162.2
- net SB_CHKSTP_OUT: now also R3092.1
- net SB_TRG_IN: now also R3162.1
- net SB_TRG_OUT: now also R3096.1
