File: cok-001/rsxvrm.kicad_sch (KiCad schematic)
At the start: 8 parts

Commit message: wireless
Parts:
- added R6206, R6208, R6209: 1500, Resistor_SMD:R_0402_1005Metric, symbol Device:R_US
- added U6204: TC7SG08FU, Package_TO_SOT_SMD:Texas_R-PDSO-N5_DRL-5, symbol 74xGxx:74LVC1G08
Connections:
- net +3.3V_MISC: now also R6206.1, R6208.1, R6209.1, U6204.5 (VCC)
- net GND: now also U6204.3 (GND)
- net RSXVRM_VID0: now also R6208.2
- net RSXVRM_VID1: now also R6206.2
- net SW_5_A: now also R6209.2, U6204.1
- net at U6201.8 (DRVON): now also U6204.2
- no-connect marks 0 -> 2
Other:
- moved on the sheet: R6200, R6201, R6202, R6203, R6204

Commit message: power
Parts:
- U6201: value ~ -> NCP5318FTR2G
- U6202, U6203: value ~ -> iP2003APbF
Other:
- moved on the sheet: U6202, U6203
Changed lines of the file:
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@@
 	(wire
 		(pts
-			(xy 171.45 111.76) (xy 173.99 111.76)
+			(xy 175.26 66.04) (xy 177.8 66.04)
 		)
 		(stroke
@@
 	(symbol
 		(lib_id "PS3:iP2003APbF")
-		(at 170.18 105.41 0)
+		(at 176.53 76.2 0)
 		(unit 1)
 		(exclude_from_sim no)
@@
 		(fields_autoplaced yes)
 		(property "Reference" "U6203"
-			(at 170.815 129.54 0)
-			(effects
-				(font
-					(size 1.27 1.27)
-				)
-			)
-		)
-		(property "Value" "~"
-			(at 170.815 130.81 0)
+			(at 176.53 86.36 0)
+			(effects
+				(font
+					(size 1.27 1.27)
+				)
+			)
+		)
+		(property "Value" "iP2003APbF"
+			(at 176.53 88.9 0)
 			(effects
 				(font
@@
 		)
 		(property "Footprint" "PS3:iP2003APbF"
-			(at 170.18 105.41 0)
+			(at 176.53 76.2 0)
+			(effects
+				(font
+					(size 1.27 1.27)
+				)
+				(hide yes)
+			)
+		)
+		(property "Datasheet" "https://mm.digikey.com/Volume0/opasdata/d220001/medias/docus/901/IP2003APbF.pdf"
+			(at 176.53 76.2 0)
+			(effects
+				(font
+					(size 1.27 1.27)
+				)
+				(hide yes)
+			)
+		)
+		(property "Description" ""
+			(at 176.53 76.2 0)
+			(effects
+				(font
+					(size 1.27 1.27)
+				)
+				(hide yes)
+			)
+		)
+		(pin "8"
+		)
+		(pin "4"
+		)
+		(pin "1"
+		)
+		(pin "6"
+		)
+		(pin "9"
+		)
+		(pin "5"
+		)
+		(pin "7"
+		)
+		(pin "2"
+		)
+		(pin "10"
+		)
+		(pin "3"
+		)
+		(instances
+			(project ""
+				(path "/976eb78d-8215-4cc0-9d72-f9d535c7970b/4d661cb0-b5d8-45b3-9841-d9751410231e"
+					(reference "U6203")
+					(unit 1)
+				)
+			)
+		)
+	)
+	(symbol
+		(lib_id "power:GND")
+		(at 186.69 157.48 90)
+		(unit 1)
+		(exclude_from_sim no)
+		(in_bom yes)
+		(on_board yes)
+		(dnp no)
+		(fields_autoplaced yes)
+		(property "Reference" "#PWR0212"
+			(at 193.04 157.48 0)
+			(effects
+				(font
+					(size 1.27 1.27)
+				)
+				(hide yes)
+			)
+		)
+		(property "Value" "GND"
+			(at 190.5 157.4799 90)
+			(effects
+				(font
+					(size 1.27 1.27)
+				)
+				(justify right)
+			)
+		)
+		(property "Footprint" ""
+			(at 186.69 157.48 0)
 			(effects
 				(font
@@
 		)
 		(property "Datasheet" ""
-			(at 170.18 105.41 0)
-			(effects
-				(font
-					(size 1.27 1.27)
-				)
-				(hide yes)
-			)
-		)
-		(property "Description" ""
-			(at 170.18 105.41 0)
-			(effects
-				(font
-					(size 1.27 1.27)
-				)
-				(hide yes)
-			)
-		)
-		(pin "8"
-		)
-		(pin "4"
-		)
-		(pin "1"
-		)
-		(pin "6"
-		)
-		(pin "9"
-		)
-		(pin "5"
-		)
-		(pin "7"
-		)
-		(pin "2"
-		)
-		(pin "10"
-		)
-		(pin "3"
-		)
-		(instances
-			(project ""
-				(path "/976eb78d-8215-4cc0-9d72-f9d535c7970b/4d661cb0-b5d8-45b3-9841-d9751410231e"
-					(reference "U6203")
-					(unit 1)
-				)
-			)
-		)
-	)
-	(symbol
-		(lib_id "power:GND")
-		(at 182.88 156.21 0)
-		(unit 1)
-		(exclude_from_sim no)
-		(in_bom yes)
-		(on_board yes)
-		(dnp no)
-		(fields_autoplaced yes)
-		(property "Reference" "#PWR0212"
-			(at 182.88 162.56 0)
-			(effects
-				(font
-					(size 1.27 1.27)
-				)
-				(hide yes)
-			)
-		)
-		(property "Value" "GND"
-			(at 182.88 161.29 0)
-			(effects
-				(font
-					(size 1.27 1.27)
-				)
-			)
-		)
-		(property "Footprint" ""
-			(at 182.88 156.21 0)
-			(effects
-				(font
-					(size 1.27 1.27)
-				)
-				(hide yes)
-			)
-		)
-		(property "Datasheet" ""
-			(at 182.88 156.21 0)
+			(at 186.69 157.48 0)
 			(effects
 				(font
@@
 		)
 		(property "Description" "Power symbol creates a global label with name \"GND\" , ground"
-			(at 182.88 156.21 0)
+			(at 186.69 157.48 0)
 			(effects
 				(font
@@
 	(symbol
 		(lib_id "power:GND")
-		(at 181.61 125.73 0)
+		(at 189.23 81.28 90)
 		(unit 1)
 		(exclude_from_sim no)
@@
 		(fields_autoplaced yes)
 		(property "Reference" "#PWR0211"
-			(at 181.61 132.08 0)
+			(at 195.58 81.28 0)
 			(effects
 				(font
@@
 		)
 		(property "Value" "GND"
-			(at 181.61 130.81 0)
-			(effects
-				(font
-					(size 1.27 1.27)
-				)
+			(at 193.04 81.2799 90)
+			(effects
+				(font
+					(size 1.27 1.27)
+				)
+				(justify right)
 			)
 		)
 		(property "Footprint" ""
-			(at 181.61 125.73 0)
+			(at 189.23 81.28 0)
 			(effects
 				(font
@@
 		)
 		(property "Datasheet" ""
-			(at 181.61 125.73 0)
+			(at 189.23 81.28 0)
 			(effects
 				(font
@@
 		)
 		(property "Description" "Power symbol creates a global label with name \"GND\" , ground"
-			(at 181.61 125.73 0)
+			(at 189.23 81.28 0)
 			(effects
 				(font
@@
 		(fields_autoplaced yes)
 		(property "Reference" "U6201"
-			(at 107.6041 96.52 0)
-			(effects
-				(font
-					(size 1.27 1.27)
-				)
-				(justify left)
-			)
-		)
-		(property "Value" "~"
-			(at 107.6041 99.06 0)
+			(at 107.5533 95.25 0)
+			(effects
+				(font
+					(size 1.27 1.27)
+				)
+				(justify left)
+			)
+		)
+		(property "Value" "NCP5318FTR2G"
+			(at 107.5533 97.79 0)
 			(effects
 				(font
@@
 	)
 	(symbol
+		(lib_name "iP2003APbF_1")
 		(lib_id "PS3:iP2003APbF")
-		(at 171.45 135.89 0)
+		(at 173.99 152.4 0)
 		(unit 1)
 		(exclude_from_sim no)
@@
 		(fields_autoplaced yes)
 		(property "Reference" "U6202"
-			(at 172.085 160.02 0)
-			(effects
-				(font
-					(size 1.27 1.27)
-				)
-			)
-		)
-		(property "Value" "~"
-			(at 172.085 161.29 0)
+			(at 173.99 162.56 0)
+			(effects
+				(font
+					(size 1.27 1.27)
+				)
+			)
+		)
+		(property "Value" "iP2003APbF"
+			(at 173.99 165.1 0)
 			(effects
 				(font
@@
 		)
 		(property "Footprint" "PS3:iP2003APbF"
-			(at 171.45 135.89 0)
-			(effects
-				(font
-					(size 1.27 1.27)
-				)
-				(hide yes)
-			)
-		)
-		(property "Datasheet" ""
-			(at 171.45 135.89 0)
+			(at 173.99 152.4 0)
+			(effects
+				(font
+					(size 1.27 1.27)
+				)
+				(hide yes)
+			)
+		)
+		(property "Datasheet" "https://mm.digikey.com/Volume0/opasdata/d220001/medias/docus/901/IP2003APbF.pdf"
+			(at 173.99 152.4 0)
 			(effects
 				(font
@@
 		)
 		(property "Description" ""
-			(at 171.45 135.89 0)
-			(effects
-				(font
+			(at 173.99 152.4 0)
+			(effects
+				(font

Commit message: rsx
Parts:
- added C6205: 1u 10V, Capacitor_SMD:C_0402_1005Metric, symbol Device:C
- added C6207: 0.022u 16V, Capacitor_SMD:C_0402_1005Metric, symbol Device:C
- added C6211: 0.1u 10V, Capacitor_SMD:C_0402_1005Metric, symbol Device:C
- added C6212: 22u 2.5V, Capacitor_SMD:C_0402_1005Metric, symbol Device:C_Polarized_US
- added FL6229, FL6230, FL6231, FL6232: 1200u, PS3:Proadlizer, symbol Device:Filter_EMI_CLC
- added L6201, L6202: 0.3uH, Inductor_SMD:L_Bourns_SRR1208_12.7x12.7mm, symbol Device:L
- added Q6200: SI4866DY, Package_SO:SSOP-8_3.9x5.05mm_P1.27mm, symbol Transistor_FET:IRF7607PBF
- added R6211: 220, Resistor_SMD:R_0402_1005Metric, symbol Device:R_US
- added R6214, R6216: XX, Resistor_SMD:R_0402_1005Metric, symbol Device:R_US
- added R6219, R6222: 0, Resistor_SMD:R_0402_1005Metric, symbol Device:R_US
- added R6248, R6249: 0.001, Resistor_SMD:R_2512_6332Metric, symbol Device:R_US
- added TP9651: TestPoint, TestPoint:TestPoint_Pad_D1.5mm, symbol Connector:TestPoint
- added U6200: BD3520FVM-TR, Package_SO:MSOP-8_3x3mm_P0.65mm, symbol PS3:BD35xxFVM-TR
Connections:
- net GND: now also C6205.2, C6207.2, C6211.2, C6212.2, FL6229.2, FL6230.2, FL6231.2, FL6232.2, R6214.1, R6216.1, U6200.2 (GND)
- net at U6203.6 (Vsw): now also L6202.1
- net at U6202.6 (Vsw): now also L6201.1
- new net: FL6229.1, FL6230.1, FL6231.1, FL6232.1, R6248.2, R6249.2
- new net: C6207.1, R6211.1
- new net: Q6200.4 (G), R6211.2, U6200.7 (G)
- new net: R6216.2, R6222.1, U6200.5 (VFB)
- new net: R6214.2, R6219.1, U6200.8 (VD)
- new net: L6202.2, R6249.1
- new net: L6201.2, R6248.1
- new net +1.2V_RSX_VDDA: C6211.1, C6212.1, Q6200.5 (D), Q6200.6 (D), Q6200.7 (D), Q6200.8 (D), R6222.2, TP9651.1, U6200.6 (VS)
- new net +1.2V_RSX_VDDC: FL6229.3, FL6230.3, FL6231.3, FL6232.3
- new net +1.7V_MISC: Q6200.1 (S), Q6200.2 (S), Q6200.3 (S), R6219.2
- new net +5V_MISC: C6205.1, U6200.4 (VCC)
- new net SW_5_B: U6200.3 (EN)
Other:
- moved on the sheet: U6202, U6203

Commit message: msop
Parts:
- U6200: footprint Package_SO:MSOP-8_3x3mm_P0.65mm -> PS3:MSOP-8_2.9x4mm_P0.65mm
Changed lines of the file:
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@@
 			)
 		)
-		(property "Footprint" "Package_SO:MSOP-8_3x3mm_P0.65mm"
+		(property "Footprint" "PS3:MSOP-8_2.9x4mm_P0.65mm"
 			(at 78.74 25.4 0)
 			(effects

Commit message: pid in
Parts:
- added R6228, R6233: 560, Resistor_SMD:R_0402_1005Metric, symbol Device:R_US
Connections:
- net at U6203.2 (ENABLE): now also U6202.2 (ENABLE), U6204.4
- net at U6203.3 (PWM): now also U6201.18 (GATE4)
- net at FL6229.1, FL6230.1, FL6231.1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: now also U6201.13 (CS4N), U6201.28 (CS2N)
- net at L6202.2, R6249.1: now also R6233.2
- net at L6201.2, R6248.1: now also R6228.2
- net at U6201.14 (CS4P): now also R6233.1
- net at U6201.20 (GATE2): now also U6202.3 (PWM)
- net at U6201.27 (CS2P): now also R6228.1
Other:
- moved on the sheet: FL6229, FL6230, FL6231, FL6232, R6200, R6201, R6202, R6203, R6204, R6206, R6208, U6201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
