File: cok-001/ethernet.kicad_sch (KiCad schematic)
At the start: 1 part, among them J3501 RJ45_Amphenol_RJMG1BD3B8K1ANR

Commit message: ethernet
Parts:
- added L3501, L3502, L3503, L3504: L_Iron_Coupled_Small_1243, Inductor_SMD:L_CommonModeChoke_Coilcraft_0805USB, symbol Device:L_Iron_Coupled_Small_1243
- added R3523: 22, Resistor_SMD:R_0402_1005Metric, symbol Device:R_US
- added R3524, R3525, R3526, R3527, R3528, R3529, R3530, R3531, R3532: 47, Resistor_SMD:R_0402_1005Metric, symbol Device:R_US
- added U3503: 88E6108, Package_QFP:LQFP-144_20x20mm_P0.5mm, symbol PS3:88E6108
Connections:
- net GND: now also U3503.107 (VSS), U3503.109 (VSS), U3503.121 (VSS), U3503.122 (P1_MDIN3), U3503.123 (P1_MDIP3), U3503.125 (P1_MDIN2), U3503.126 (P1_MDIP2), U3503.127 (P1_MDIN1), U3503.128 (P1_MDIP1), U3503.131 (P1_MDIN0), U3503.132 (P1_MDIP0), U3503.133 (VSS), U3503.134 (P0_MDIN3), U3503.135 (P0_MDIP3), U3503.137 (P0_MDIN2), U3503.138 (P0_MDIP2), U3503.139 (P0_MDIN1), U3503.140 (P0_MDIP1), U3503.143 (P0_MDIN0), U3503.144 (P0_MDIP0), U3503.39 (P7_VDDAH), U3503.42 (VSS), U3503.45 (P6_VDDAH), U3503.51 (P5_VDDAH), U3503.54 (VSS)
- new net: R3526.2, U3503.65 (P3_TXD6/MODE1)
- new net: R3524.2, U3503.63 (P3_TXEN/HALFDPX)
- new net: L3502.1, U3503.115 (P2_MDIN1)
- new net: L3502.4, U3503.116 (P2_MDIP1)
- new net: R3525.2, U3503.64 (P3_TXD7/MODE2)
- new net: L3501.1, U3503.119 (P2_MDIN0)
- new net: L3501.4, U3503.120 (P2_MDIP0)
- new net: L3503.1, U3503.113 (P2_MDIN2)
- new net: L3503.4, U3503.114 (P2_MDIP2)
- new net: R3523.2, U3503.62 (P3_CLK125n)
- new net: R3527.2, U3503.67 (P3_TXD5/MODE0)
- new net: R3529.2, U3503.70 (P3_TXD3/ADDR3)
- new net: L3504.1, U3503.110 (P2_MDIN3)
- new net: L3504.4, U3503.111 (P2_MDIP3)
- new net: R3530.2, U3503.71 (P3_TXD2/ADDR2)
- new net: R3528.2, U3503.68 (P3_TXD4/ADDR4)
- new net: R3532.2, U3503.73 (P3_TXD0/ADDR0)
- new net: R3531.2, U3503.72 (P3_TXD1/ADDR1)

Commit message: av
Parts:
- added C3567, C501, C502, C503: 0.01u, Capacitor_SMD:C_0402_1005Metric, symbol Device:C
- added R3570, R3573, R3576, R3579, R3582, R3585, R3588, R3591: 49.9, Resistor_SMD:R_0402_1005Metric, symbol Device:R_US
Connections:
- net GND: now also C3567.2, C501.2, C502.2, C503.2
- net at L3502.1, U3503.115 (P2_MDIN1): now also R3579.2
- net at L3502.4, U3503.116 (P2_MDIP1): now also R3576.2
- net at L3501.1, U3503.119 (P2_MDIN0): now also R3573.2
- net at L3501.4, U3503.120 (P2_MDIP0): now also R3570.2
- net at L3503.1, U3503.113 (P2_MDIN2): now also R3585.2
- net at L3503.4, U3503.114 (P2_MDIP2): now also R3582.2
- net at L3504.1, U3503.110 (P2_MDIN3): now also R3591.2
- net at L3504.4, U3503.111 (P2_MDIP3): now also R3588.2
- new net: C502.1, R3582.1, R3585.1
- new net: C3567.1, R3570.1, R3573.1
- new net: C503.1, R3588.1, R3591.1
- new net: C501.1, R3576.1, R3579.1
Other:
- moved on the sheet: L3501, L3502, L3503, L3504

Commit message: aj
Parts:
- added R3505, R3506, R3507, R3508, R3509, R3510, R3511, R3512, R3513, R3514, R3515: 33, Resistor_SMD:R_0402_1005Metric, symbol Device:R_US
- added TP3501, TP3502: TestPoint, TestPoint:TestPoint_Pad_1.0x1.0mm, symbol Connector:TestPoint
Connections:
- net at U3503.77 (P3_RXDV): now also R3505.2
- net at U3503.79 (P3_RXER): now also R3506.2
- net at U3503.80 (P3_RXD7): now also R3507.2
- net at U3503.81 (P3_RXD6): now also R3508.2
- net at U3503.82 (P3_RXD5): now also R3509.2
- net at U3503.83 (P3_RXD4): now also R3510.2
- net at U3503.85 (P3_RXD3): now also R3511.2
- net at U3503.87 (P3_RXD2): now also R3512.2
- net at U3503.88 (P3_RXD1): now also R3513.2
- net at U3503.89 (P3_RXD0): now also R3514.2
- net at U3503.90 (P3_RXCLK): now also R3515.2
- new net SB_GBE_ETOMOD: TP3502.1
- new net SB_GBE_GMIICLK: R3515.1
- new net SB_GBE_TXCLK: TP3501.1
- new net SB_GBE_TXD0: R3514.1
- new net SB_GBE_TXD1: R3513.1
- new net SB_GBE_TXD2: R3512.1
- new net SB_GBE_TXD3: R3511.1
- new net SB_GBE_TXD4: R3510.1
- new net SB_GBE_TXD5: R3509.1
- new net SB_GBE_TXD6: R3508.1
- new net SB_GBE_TXD7: R3507.1
- new net SB_GBE_TXEN: R3505.1
- new net SB_GBE_TXER: R3506.1

Commit message: update to 9
Changed lines of the file:
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@@
 (kicad_sch
-	(version 20231120)
+	(version 20250114)
 	(generator "eeschema")
-	(generator_version "8.0")
+	(generator_version "9.0")
 	(paper "A4")
 	(junction

Commit message: crystal
Parts:
- added C3502, C3503: 0.1u, Capacitor_SMD:C_0402_1005Metric, symbol Device:C
- added C3543, C3584: 15p 50V, Capacitor_SMD:C_0402_1005Metric, symbol Device:C
- added C3560: 0.1u 10V, Capacitor_SMD:C_0402_1005Metric, symbol Device:C
- added D351, D352, D353, D354, D355, D356, D357, D358: ESD5Zxx, Diode_SMD:D_SOD-923, symbol Diode:ESD5Zxx
- added R3561: 220, Resistor_SMD:R_0402_1005Metric, symbol Device:R_US
- added R3593: 0, Resistor_SMD:R_0402_1005Metric, symbol Device:R_US
- added U3501: BD3520FVM-TR, Package_SO:MSOP-8_3x3mm_P0.65mm, symbol PS3:BD35xxFVM-TR
- added U3502: MM1761KHBE, Package_SO:HTSOP-8-1EP_3.9x4.9mm_P1.27mm_EP2.4x3.2mm, symbol Regulator_Linear:BD15GA5WEFJ
- added Y3501: 25MHz, Crystal:Crystal_SMD_Abracon_ABM8G-4Pin_3.2x2.5mm, symbol Device:Crystal_GND24
- renumbered C501 to C3570, C502 to C3573, C503 to C3576
Connections:
- net GND: now also C3543.1, C3560.2, C3584.1, D351.2 (A), D352.2 (A), D353.2 (A), D354.2 (A), D355.2 (A), D356.2 (A), D357.2 (A), D358.2 (A), Y3501.2, Y3501.4
- net P2_LED2: now also C3560.1, R3561.2
- net SB_GBE_RXD6: now reaches R3526.1
- net at L3502.2: now also D353.1 (K)
- net at L3502.3: now also D354.1 (K)
- net SB_GBE_RXD7: now reaches R3525.1
- net at L3501.2: now also D351.1 (K)
- net at L3501.3: now also D352.1 (K)
- net at L3503.2: now also D355.1 (K)
- net at L3503.3: now also D356.1 (K)
- net SB_GBE_RXD5: now reaches R3527.1
- net SB_GBE_RXD3: now reaches R3529.1
- net at L3504.2: now also D357.1 (K)
- net at L3504.3: now also D358.1 (K)
- net SB_GBE_RXD2: now reaches R3530.1
- net SB_GBE_RXD4: now reaches R3528.1
- net SB_GBE_RXD0: now reaches R3532.1
- net at U3503.28 (P2_LED2): now also R3561.1
- net at U3503.55 (P4_RXN): now also C3502.2
- net at U3503.56 (P4_RXP): now also C3503.2
- net WLAN_TXN: now reaches U3503.58 (P4_TXN)
- net WLAN_TXP: now reaches U3503.59 (P4_TXP)
- net at U3503.7 (XTAL_IN): now also C3543.2, Y3501.3
- net at U3503.8 (XTAL_OUT): now also R3593.1
- net SB_GBE_RXD1: now reaches R3531.1
- new net: U3502.3 (GND), U3502.4 (GND), U3502.6 (GND), U3502.7 (GND), U3502.9 (GND)
- new net: C3584.2, R3593.2, Y3501.1
- new net WLAN_RXN: C3502.1
- new net WLAN_RXP: C3503.1
- no-connect marks 2 -> 3

Commit message: regulator
Parts:
- J3501: value RJ45_Amphenol_RJMG1BD3B8K1ANR -> RJ45; footprint Connector_RJ:RJ45_Amphenol_RJMG1BD3B8K1ANR -> PS3:RJ45; symbol Connector:RJ45_Amphenol_RJMG1BD3B8K1ANR -> Connector_Generic_MountingPin:Conn_01x13_MountingPin
Connections:
- net GND: now also J3501.6 (Pin_6), J3501.MP (MountPin), U3503.48 (VDD_CORE); no longer J3501.SH
- net P2_LED2: now also J3501.13 (Pin_13); no longer J3501.L3
- net at D352.1 (K), L3501.3: now also J3501.2 (Pin_2)
- net at D355.1 (K), L3503.2: now also J3501.8 (Pin_8)
- net at D354.1 (K), L3502.3: now also J3501.4 (Pin_4)
- net at D353.1 (K), L3502.2: now also J3501.5 (Pin_5)
- net at D356.1 (K), L3503.3: now also J3501.7 (Pin_7)
- net at D351.1 (K), L3501.2: now also J3501.3 (Pin_3)
- net at D357.1 (K), L3504.2: now also J3501.10 (Pin_10)
- net at D358.1 (K), L3504.3: now also J3501.9 (Pin_9)
- no-connect marks 3 -> 33

Commit message: msop
Parts:
- U3501: footprint Package_SO:MSOP-8_3x3mm_P0.65mm -> PS3:MSOP-8_2.9x4mm_P0.65mm
Changed lines of the file:
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@@
 			)
 		)
-		(property "Footprint" "Package_SO:MSOP-8_3x3mm_P0.65mm"
+		(property "Footprint" "PS3:MSOP-8_2.9x4mm_P0.65mm"
 			(at 96.52 210.82 0)
 			(effects

Commit message: voltage symbols
Parts:
- added Q3501: UMH2NTN, Package_TO_SOT_SMD:SOT-363_SC-70-6, symbol Transistor_BJT:MUN5213DW1
- added Q3502: DTC144E, Package_TO_SOT_SMD:SOT-323_SC-70, symbol Transistor_BJT:DTC144E
- added Q3503: SI3493, Package_SO:TSOP-6_1.65x3.05mm_P0.95mm, symbol Transistor_FET:PMN48XP
- added Q3504: Si3460DV, Package_SO:TSOP-6_1.65x3.05mm_P0.95mm, symbol Transistor_FET:Si3456DDV
- added R3520: 2200, Resistor_SMD:R_0402_1005Metric, symbol Device:R_US
- added R3521, R3522: 1500, Resistor_SMD:R_0402_1005Metric, symbol Device:R_US
- added R3536: 100k, Resistor_SMD:R_0402_1005Metric, symbol Device:R_US
- added R3537: 150k, Resistor_SMD:R_0402_1005Metric, symbol Device:R_US
- added R3538: XX, Resistor_SMD:R_0402_1005Metric, symbol Device:R_US
Connections:
- net GND: now also U3502.3 (GND), U3502.4 (GND), U3502.6 (GND), U3502.7 (GND), U3502.9 (GND), Q3501.1 (E1), Q3501.4 (E2), Q3502.2 (E)
- net at U3502.5 (EN): now also U3501.3 (EN), Q3501.6 (C1), Q3502.1 (B), R3522.1, R3538.2
- net at U3501.7 (G): now also Q3504.3 (G)
- new net: Q3502.3 (C), R3536.1, R3537.1
- new net: Q3503.3 (G), R3537.2
- new net: Q3501.5 (B2), R3520.2
- new net: Q3504.1 (D), Q3504.2 (D), Q3504.5 (D), Q3504.6 (D)
- new net: Q3501.2 (B1), Q3501.3 (C2), R3521.1
- new net +3.3V_ESW: Q3503.1 (D), Q3503.2 (D), Q3503.5 (D), Q3503.6 (D)
- new net +3.3V_EVER: R3521.2, R3522.2
- new net +3.3V_MISC: Q3503.4 (S), R3536.2
- new net SW_4_A: R3520.1, R3538.1
Other:
- moved on the sheet: U3501, U3502
