File: cok-001/rsxsetting.kicad_sch (KiCad schematic)
At the start: 30 parts, among them U2101 ADT7461A0002RMZR, U2105 TC7WP3125FK, U2108 ICS651MLFT, Y2101 24.576MHz

Commit message: pcb update
Connections:
- net ADAC_MCLK0 renamed ADAC_MCLKO0
- net RS_MCLK0 renamed RS_MCLKO0
Changed lines of the file:
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@@
 		)
 	)
-	(global_label "ADAC_MCLK0"
+	(global_label "ADAC_MCLKO0"
 		(shape output)
 		(at 107.95 171.45 180)
@@
 		)
 		(property "Intersheetrefs" "${INTERSHEET_REFS}"
-			(at 93.051 171.45 0)
+			(at 91.7205 171.45 0)
 			(effects
 				(font
@@
 		)
 	)
-	(global_label "RS_MCLK0"
+	(global_label "RS_MCLKO0"
 		(shape input)
 		(at 107.95 163.83 180)
@@
 		)
 		(property "Intersheetrefs" "${INTERSHEET_REFS}"
-			(at 95.2887 163.83 0)
+			(at 93.9582 163.83 0)
 			(effects
 				(font

Commit message: rsx
Parts:
- added C2124: 47u 6.3V, Capacitor_Tantalum_SMD:CP_EIA-3216-10_Kemet-I, symbol Device:C_Polarized_US
- added C2126, C2129: 0.1u 10V, Capacitor_SMD:C_0402_1005Metric, symbol Device:C
- added FB2101: 0uH, Resistor_SMD:R_0603_1608Metric, symbol Device:FerriteBead_Small
- added Q1: DTC144E, Package_TO_SOT_SMD:SOT-323_SC-70, symbol Transistor_BJT:DTC144E
- added R2131, R2132, R2133, R2134, R2135, R2136, R2137, R2139, R2140: 10k, Resistor_SMD:R_0402_1005Metric, symbol Device:R_US
- added R2173: 2012, Resistor_SMD:R_0603_1608Metric, symbol Device:R_US
- added R2180: 10k, Resistor_SMD:R_0603_1608Metric, symbol Device:R_US
Connections:
- net GND: now also C2124.2, C2126.2, C2129.2, Q1.2 (E), R2131.1, R2133.1, R2135.1, R2137.1, R2139.1
- net RSX_GPIO0: now reaches U2102.13 (SEL)
- net RSX_GPIO0: now also R2131.2
- net at U2102.18 (Vdd), U2102.19 (Vdd), U2102.2 (Vdd)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: now also FB2101.1
- net +3.3V_THERMAL: now reaches C2108.1, U2101.1 (Vdd)
- net +1.5V_AVCG_VDDIO: now reaches U2105.1 (VccA)
- net +1.5V_AVCG_VDDIO: now also C2129.1, R2180.2
- net at U2105.5 (~{OE}): now also Q1.3 (C), R2180.1
- net RSX_GPIO6: now reaches U2101.4 (~{THERM})
- net RSX_GPIO6: now also R2140.1
- new net: C2124.1, C2126.1, FB2101.2, R2173.1
- new net +1.5V_RSX_VDDIO: R2132.2, R2134.2, R2136.2, R2140.2
- new net +3.3V_ANA: R2173.2
- new net PCLKEN: Q1.1 (B)
- new net RSX_GPIO1: R2132.1, R2133.2
- new net RSX_GPIO2: R2134.1, R2135.2
- new net RSX_GPIO3: R2136.1, R2137.2
- new net RSX_GPIO5: R2139.2
Other:
- moved on the sheet: C2103, C2108, C2123, C2125, C2271, R2101, R2102, R2177, R2179, R2181, U2101, U2108

Commit message: dumb numbers
Parts:
- renumbered Q1 to Q2101
Changed lines of the file:
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@@
 		(on_board yes)
 		(dnp no)
-		(property "Reference" "Q1"
+		(property "Reference" "Q2101"
 			(at 142.24 133.3501 0)
 			(effects
@@
 			(project "cok-001"
 				(path "/976eb78d-8215-4cc0-9d72-f9d535c7970b/128112c3-c1d3-4d2b-b67e-431f0bf7f496"
-					(reference "Q1")
+					(reference "Q2101")
 					(unit 1)
 				)

Commit message: inductor
Parts:
- FB2101: footprint Resistor_SMD:R_0603_1608Metric -> Inductor_SMD:L_0603_1608Metric
Connections:
- net at C2124.1, C2126.1, R2173.1: now also FB2101.1; no longer FB2101.2
- net at U2102.18 (Vdd), U2102.19 (Vdd), U2102.2 (Vdd)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: now also FB2101.2; no longer FB2101.1
Other:
- moved on the sheet: FB2101
Changed lines of the file:
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@@
 	(symbol
 		(lib_id "Device:FerriteBead_Small")
-		(at 119.38 27.94 90)
+		(at 119.38 27.94 270)
 		(unit 1)
 		(exclude_from_sim no)
@@
 		(fields_autoplaced yes)
 		(property "Reference" "FB2101"
-			(at 119.3419 21.59 90)
+			(at 119.4181 21.59 90)
 			(effects
 				(font
@@
 		)
 		(property "Value" "0uH"
-			(at 119.3419 24.13 90)
+			(at 119.4181 24.13 90)
 			(effects
 				(font
@@
 			)
 		)
-		(property "Footprint" "Resistor_SMD:R_0603_1608Metric"
-			(at 119.38 29.718 90)
+		(property "Footprint" "Inductor_SMD:L_0603_1608Metric"
+			(at 119.38 26.162 90)
 			(effects
 				(font

Commit message: msop
Parts:
- U2101: footprint Package_SO:MSOP-8_3x3mm_P0.65mm -> PS3:MSOP-8_2.9x4mm_P0.65mm
Changed lines of the file:
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@@
 			)
 		)
-		(property "Footprint" "Package_SO:MSOP-8_3x3mm_P0.65mm"
+		(property "Footprint" "PS3:MSOP-8_2.9x4mm_P0.65mm"
 			(at 58.42 163.83 0)
 			(effects

Commit message: rsx pins
Parts:
- added R2145, R2146, R2147, R2148, R2149, R2150, R2151, R2152, R2153, R2154, R2155: 10k, Resistor_SMD:R_0402_1005Metric, symbol Device:R_US
- added TP2101, TP2102, TP2103, TP2104, TP2105, TP2106: TestPoint, TestPoint:TestPoint_Pad_1.0x1.0mm, symbol Connector:TestPoint
- U2102: value ~ -> ICS422A
Connections:
- net +1.5V_RSX_VDDIO: now also R2145.2, R2147.2, R2149.2, R2151.2, R2153.2, R2154.2, R2155.2
- net GND: now also R2146.1, R2148.1, R2150.1, R2152.1
- new net RS_TCK: TP2106.1
- new net RS_TDI: TP2103.1
- new net RS_TMS: TP2104.1
- new net TS_TDO: TP2102.1
- new net ~{RSX_CHKSTP_IN}: R2147.1, R2148.2
- new net ~{RSX_CHKSTP_OUT}: R2151.1, R2152.2
- new net ~{RSX_INT}: R2154.1
- new net ~{RSX_SPI_CS}: R2155.1
- new net ~{RSX_TRG_IN}: R2145.1, R2146.2
- new net ~{RSX_TRG_OUT}: R2149.1, R2150.2
- new net ~{RS_TRSTNEG}: R2153.1, TP2105.1
Other:
- moved on the sheet: C2109, C2112, R2107, R2131, R2132, R2133, R2134, R2135, R2136, R2137, R2139, R2140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

Commit message: voltage symbols
Parts:
- R2180: footprint Resistor_SMD:R_0603_1608Metric -> Resistor_SMD:R_0402_1005Metric
Changed lines of the file:
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@@
 			)
 		)
-		(property "Footprint" "Resistor_SMD:R_0603_1608Metric"
+		(property "Footprint" "Resistor_SMD:R_0402_1005Metric"
 			(at 140.716 141.224 90)
 			(effects
