File: cok-001/cok-001.kicad_pcb (KiCad board)
At the start: 2 copper layers, 313.2 x 237 mm, 1177 parts, among them J2401 AV OUT, J2501 HDMI_A, J3208 凸, J3209 ATA Power, J3221 IMSA-9637S-60Y801, J3301 USB_A_Stacked, J3302 USB_A_Stacked, J3401 Conn_01x22_Pin, J3501 RJ45_Amphenol_RJMG1BD3B8K1ANR, J3701 Conn_01x33_MountingPin, J4001 FAN, J4003 Conn_01x02_Pin, J4009 Conn_01x30_Socket, J4010 BUTTONS, J6004 +12V_MAIN, J6005 +5V_EVER, Q1101 DTC144E, Q1102 DTC144E, Q2401 DTC144E, Q2402 SI2303BDS, Q2502 DTA144E, Q2504 DTA144E, Q2507 DTC144E, Q3201 DTC144E, Q3401 DTC144E, Q3402 DTC144E, Q3403 DTC144E, Q3404 DTC144E, Q4011 DTC143ZUA, Q4014 DTC143ZUA, Q6001 FDQ7238AS, Q6002 FDQ7238AS, Q6003 DTC144E, Q6004 SI3493, Q6009 UMH2NTN, Q6010 SI4943, Q6301 FDQ7238AS, Q6302 SI4336, Q6303 SI4336, Q6304 SI4392, Q6305 SI4392, Q6306 SI4336, Q6307 SI4336, Q6308 IRF7607PBF, Q6309 SI4866DY, Q6310 SUD40N02, Q6311 UMH2NTN, Q6600 SUD40N02, U1101 ADT7461A0002RMZR, U1201 Y0_XDR0, U1202 Y0_XDR1, U1301 Y1_XDR0, U1302 Y1_XDR1, U2101 ADT7461A0002RMZR, U2105 TC7WP3125FK, U2108 ICS651MLFT, U2402 MC78M09, U2403 MC78M05, U2405 CX4351, U3001 CXD2973GB, U3302 BU9869W, U3501 BD3520FVM-TR, U3502 MM1761KHBE, U3503 88E6108, U3802 K9F1G08U0A, U3803 K9F1G08U0A, U6003 MB39A, U6005 NCP511SN33T1G, U6006 NCP511SN18T1, U6008 NCP511SN18T1, U6009 NCP511SN33T1G, U6011 NCP511, U6012 MM3141, U6013 MM1562, U6014 MM1591, U6019 NCP511SN18T1, U6021 MM1591, U6022 MM1593, U6103 NCP5318FTR2G, U6104 iP2003APbF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

Commit message: fix 1 rsx pin
Parts:
- removed IC1001: ~, PS3:CELL_multi
- added C2124: 47u 6.3V, Capacitor_Tantalum_SMD:CP_EIA-3216-10_Kemet-I, B.Cu at (331.0, 230.5)
- added C2126: 0.1u 10V, Capacitor_SMD:C_0402_1005Metric, B.Cu at (332.6, 230.9)
- added C2129: 0.1u 10V, Capacitor_SMD:C_0402_1005Metric, B.Cu at (346.5, 223.0)
- added C2469: 100u 10V, Capacitor_SMD:CP_Elec_6.3x5.4, F.Cu at (214.2, 304.4)
- added C3155: 0.1u 10V, Capacitor_SMD:C_0402_1005Metric, F.Cu at (208.2, 265.4)
- added C5105: 0.0027u 50V, Capacitor_SMD:C_0402_1005Metric, F.Cu at (184.9, 243.4)
- added C5106: 0.0027u 50V, Capacitor_SMD:C_0402_1005Metric, F.Cu at (184.9, 244.7)
- added C5155: XX 10V, Capacitor_SMD:C_0402_1005Metric, B.Cu at (156.4, 227.4)
- added C5156: XX 10V, Capacitor_SMD:C_0402_1005Metric, B.Cu at (158.3, 227.4)
- added C6002: 1u 16V, Capacitor_SMD:C_0603_1608Metric, B.Cu at (402.4, 93.6)
- added C6004: XX, Capacitor_SMD:C_0402_1005Metric, B.Cu at (406.3, 68.5)
- added C6022: 0.001u 50V, Capacitor_SMD:C_0402_1005Metric, B.Cu at (422.8, 75.9)
- added C6032: 0.022u 16V, Capacitor_SMD:C_0402_1005Metric, B.Cu at (422.8, 77.9)
- added C6050: 2.2u 10V, Capacitor_SMD:C_0805_2012Metric, F.Cu at (281.7, 53.8)
- added C6056: 2.2u 10V, Capacitor_SMD:C_0805_2012Metric, F.Cu at (281.7, 56.8)
- added C6057: 1u 10V, Capacitor_SMD:C_0402_1005Metric, F.Cu at (275.1, 53.2)
- added C6061: 0.1u 10V, Capacitor_SMD:C_0402_1005Metric, F.Cu at (275.1, 55.2)
- added C6062: 0.1u 10V, Capacitor_SMD:C_0402_1005Metric, F.Cu at (275.1, 57.2)
- added C6063: 0.1u 10V, Capacitor_SMD:C_0402_1005Metric, F.Cu at (275.1, 59.1)
- added C6073: 0.1u 10V, Capacitor_SMD:C_0402_1005Metric, F.Cu at (275.1, 61.1)
- added C6075: 2.2u 10V, Capacitor_SMD:C_0805_2012Metric, F.Cu at (295.2, 332.2)
- added C6076: 0.1u 10V, Capacitor_SMD:C_0402_1005Metric, F.Cu at (298.8, 331.7)
- added C6078: 1u 10V, Capacitor_SMD:C_0402_1005Metric, F.Cu at (298.8, 333.6)
- added C6079: XX 16V, Capacitor_SMD:C_0402_1005Metric, F.Cu at (265.4, 101.3)
- added C6080: 2.2u 10V, Capacitor_SMD:C_0805_2012Metric, B.Cu at (163.2, 256.9)
- added C6082: 2.2u 10V, Capacitor_SMD:C_0805_2012Metric, F.Cu at (295.2, 335.2)
- added C6084: 0.022u 16V, Capacitor_SMD:C_0402_1005Metric, F.Cu at (298.8, 335.6)
- added C6085: XX 25V, Capacitor_SMD:C_0402_1005Metric, F.Cu at (266.2, 98.2)
- added C6088: 470p, Capacitor_SMD:C_0402_1005Metric, B.Cu at (166.1, 248.1)
- added C6089: 10u 6.3V, Capacitor_SMD:C_0805_2012Metric, B.Cu at (162.9, 248.0)
- added C6090: 100p, Capacitor_SMD:C_0402_1005Metric, B.Cu at (166.2, 256.6)
- added C6091: 2.2u 10V, Capacitor_SMD:C_0805_2012Metric, F.Cu at (295.2, 338.2)
- added C6093: 0.022u 16V, Capacitor_SMD:C_0402_1005Metric, F.Cu at (336.5, 216.8)
- added C6095: 220u 2.5V, Capacitor_Tantalum_SMD:CP_EIA-3528-21_Kemet-B, F.Cu at (336.4, 212.7)
- added C6096: 100p, Capacitor_SMD:C_0402_1005Metric, F.Cu at (298.8, 339.5)
- added C6107: 0.1u 10V, Capacitor_SMD:C_0402_1005Metric, B.Cu at (192.7, 152.2)
- added C6136: 0.01u 25V, Capacitor_SMD:C_0402_1005Metric, F.Cu at (242.9, 134.7)
- added C6137: 0.01u 25V, Capacitor_SMD:C_0402_1005Metric, F.Cu at (222.9, 134.7)
- added C6138: 0.01u 25V, Capacitor_SMD:C_0402_1005Metric, F.Cu at (262.9, 134.7)
- added C6168: 0.1u 10V, Capacitor_SMD:C_0402_1005Metric, F.Cu at (271.4, 162.8)
- added C6184: 100p, Capacitor_SMD:C_0402_1005Metric, F.Cu at (227.0, 119.5)
- added C6185: 100p, Capacitor_SMD:C_0402_1005Metric, F.Cu at (227.0, 121.5)
- added C6186: 100p, Capacitor_SMD:C_0402_1005Metric, F.Cu at (227.0, 123.5)
- added C6187: 0.1u 16V, Capacitor_SMD:C_0402_1005Metric, F.Cu at (229.8, 119.5)
- added C6188: 0.1u 16V, Capacitor_SMD:C_0402_1005Metric, F.Cu at (229.8, 121.5)
- added C6189: 0.1u 16V, Capacitor_SMD:C_0402_1005Metric, F.Cu at (224.1, 124.3)
- added C6205: 1u 10V, Capacitor_SMD:C_0402_1005Metric, B.Cu at (290.9, 152.9)
- added C6207: 0.022u 16V, Capacitor_SMD:C_0402_1005Metric, B.Cu at (278.6, 153.1)
- added C6211: 0.1u 10V, Capacitor_SMD:C_0402_1005Metric, B.Cu at (278.6, 155.1)
- added C6212: 22u 2.5V, Capacitor_SMD:C_0402_1005Metric, B.Cu at (285.7, 158.3)
- added C6500: 100p, Capacitor_SMD:C_0402_1005Metric, F.Cu at (267.9, 99.4)
- added D2401: DAP202UT106, Package_TO_SOT_SMD:SOT-323_SC-70, B.Cu at (354.9, 296.4)
- added D3701: CL-197HG5-CD-T, Diode_SMD:D_0603_1608Metric, F.Cu at (250.1, 105.8)
- added FB2101: 0uH, Inductor_SMD:L_0603_1608Metric, B.Cu at (334.1, 231.6)
- added FL6229: 1200u, PS3:Proadlizer, F.Cu at (309.0, 157.3)
- added FL6230: 1200u, PS3:Proadlizer, B.Cu at (294.8, 157.3)
- added FL6231: 1200u, PS3:Proadlizer, F.Cu at (324.5, 157.3)
- added FL6232: 1200u, PS3:Proadlizer, B.Cu at (310.3, 157.3)
- added J3219: for Multi_Card_Board, Connector_FFC-FPC:Hirose_FH12-15S-0.5SH_1x15-1MP_P0.50mm_Horizontal, B.Cu at (272.6, 117.0)
- added L6201: 0.3uH, Inductor_SMD:L_Bourns_SRR1208_12.7x12.7mm, F.Cu at (306.7, 140.8)
- added L6202: 0.3uH, Inductor_SMD:L_Bourns_SRR1208_12.7x12.7mm, F.Cu at (326.8, 140.8)
- added L6305: 1.4uH, Inductor_SMD:L_TDK_SLF12555, F.Cu at (366.6, 147.0)
- added Q1201: RK7002, Package_TO_SOT_SMD:SOT-23, B.Cu at (162.4, 194.9)
- added Q1202: SST2222AT, Package_TO_SOT_SMD:SOT-23, B.Cu at (166.4, 224.2)
- added Q1301: RK7002, Package_TO_SOT_SMD:SOT-23, B.Cu at (162.4, 200.2)
- added Q1302: SST2222AT, Package_TO_SOT_SMD:SOT-23, B.Cu at (166.3, 190.7)
- added Q2101: DTC144E, Package_TO_SOT_SMD:SOT-323_SC-70, B.Cu at (351.1, 226.3)
- added Q2403: IMH20T108, Package_TO_SOT_SMD:ROHM_SOT-457_ClockwisePinNumbering, B.Cu at (353.6, 305.4)
- added Q2404: DTA144E, Package_TO_SOT_SMD:SOT-323_SC-70, B.Cu at (355.6, 300.1)
- added Q3101: DTC143ZUA, Package_TO_SOT_SMD:SOT-323_SC-70, B.Cu at (217.4, 258.4)
- added Q3501: UMH2NTN, Package_TO_SOT_SMD:SOT-363_SC-70-6, B.Cu at (329.4, 244.1)
- added Q3502: DTC144E, Package_TO_SOT_SMD:SOT-323_SC-70, B.Cu at (333.5, 243.7)
- added Q3503: SI3493, Package_SO:TSOP-6_1.65x3.05mm_P0.95mm, B.Cu at (332.7, 247.6)
- added Q3504: Si3460DV, Package_SO:TSOP-6_1.65x3.05mm_P0.95mm, F.Cu at (338.4, 252.8)
- added Q3701: UMH2NTN, Package_TO_SOT_SMD:SOT-363_SC-70-6, F.Cu at (255.1, 101.3)
- added Q4008: DTC144E, Package_TO_SOT_SMD:SOT-323_SC-70, B.Cu at (410.2, 105.6)
- added Q4012: UMH2NTN, Package_TO_SOT_SMD:SOT-363_SC-70-6, F.Cu at (388.4, 115.1)
- added Q4013: UMH2NTN, Package_TO_SOT_SMD:SOT-363_SC-70-6, F.Cu at (388.1, 109.8)
- added Q4015: DTC143ZUA, Package_TO_SOT_SMD:SOT-323_SC-70, F.Cu at (388.2, 107.2)
- added Q6006: UMH2NTN, Package_TO_SOT_SMD:SOT-363_SC-70-6, B.Cu at (332.1, 75.0)
- added Q6007: SI3493, Package_SO:TSOP-6_1.65x3.05mm_P0.95mm, F.Cu at (291.2, 103.9)
- added Q6008: SI3493, Package_SO:TSOP-6_1.65x3.05mm_P0.95mm, F.Cu at (291.2, 98.6)
- added Q6012: Si3460DV, Package_SO:TSOP-6_1.65x3.05mm_P0.95mm, F.Cu at (339.9, 210.3)
- added Q6200: SI4866DY, Package_SO:SSOP-8_3.9x5.05mm_P1.27mm, F.Cu at (287.6, 153.4)
- added R1001: 470k, Resistor_SMD:R_0402_1005Metric, B.Cu at (256.3, 171.1)
- added R1002: 470k, Resistor_SMD:R_0402_1005Metric, B.Cu at (258.3, 171.1)
- added R1003: 470k, Resistor_SMD:R_0402_1005Metric, B.Cu at (260.3, 171.1)
- added R1204: 10, Resistor_SMD:R_0805_2012Metric, B.Cu at (165.9, 194.1)
- added R1205: 22.1, Resistor_SMD:R_0805_2012Metric, B.Cu at (165.9, 195.8)
- added R1225: 43.2, Resistor_SMD:R_0402_1005Metric, B.Cu at (159.0, 173.8)
- added R1226: 43.2, Resistor_SMD:R_0402_1005Metric, B.Cu at (159.0, 175.8)
- added R1227: 43.2, Resistor_SMD:R_0402_1005Metric, B.Cu at (159.0, 177.8)
- added R1228: 43.2, Resistor_SMD:R_0402_1005Metric, B.Cu at (159.0, 179.8)
- added R1229: 43.2, Resistor_SMD:R_0402_1005Metric, B.Cu at (159.0, 181.8)
- added R1230: 43.2, Resistor_SMD:R_0402_1005Metric, B.Cu at (159.0, 183.8)
- added R1231: 43.2, Resistor_SMD:R_0402_1005Metric, B.Cu at (159.0, 185.8)
- added R1232: 43.2, Resistor_SMD:R_0402_1005Metric, B.Cu at (156.1, 173.8)
- added R1233: 43.2, Resistor_SMD:R_0402_1005Metric, B.Cu at (156.1, 175.8)
- added R1234: 43.2, Resistor_SMD:R_0402_1005Metric, B.Cu at (156.1, 177.8)
- added R1235: 43.2, Resistor_SMD:R_0402_1005Metric, B.Cu at (156.1, 179.8)
- added R1236: 43.2, Resistor_SMD:R_0402_1005Metric, B.Cu at (156.1, 181.8)
- added R1304: 10, Resistor_SMD:R_0805_2012Metric, B.Cu at (165.9, 199.3)
- added R1305: 22.1, Resistor_SMD:R_0805_2012Metric, B.Cu at (165.9, 201.2)
- added R1325: 43.2, Resistor_SMD:R_0402_1005Metric, B.Cu at (159.3, 219.1)
- added R1326: 43.2, Resistor_SMD:R_0402_1005Metric, B.Cu at (159.3, 221.1)
- added R1327: 43.2, Resistor_SMD:R_0402_1005Metric, B.Cu at (156.4, 209.1)
- added R1328: 43.2, Resistor_SMD:R_0402_1005Metric, B.Cu at (156.4, 211.1)
- added R1329: 43.2, Resistor_SMD:R_0402_1005Metric, F.Cu at (164.2, 210.8)
- added R1330: 43.2, Resistor_SMD:R_0402_1005Metric, B.Cu at (156.4, 215.1)
- added R1331: 43.2, Resistor_SMD:R_0402_1005Metric, B.Cu at (156.4, 217.1)
- added R1332: 43.2, Resistor_SMD:R_0402_1005Metric, B.Cu at (156.4, 219.1)
- added R1333: 43.2, Resistor_SMD:R_0402_1005Metric, B.Cu at (156.4, 221.1)
- added R1334: 43.2, Resistor_SMD:R_0402_1005Metric, B.Cu at (153.5, 209.1)
- added R1335: 43.2, Resistor_SMD:R_0402_1005Metric, B.Cu at (153.5, 211.1)
- added R1336: 43.2, Resistor_SMD:R_0402_1005Metric, B.Cu at (153.5, 213.1)
- added R2061: 240, Resistor_SMD:R_0402_1005Metric, B.Cu at (290.2, 174.0)
- added R2063: 22, Resistor_SMD:R_0402_1005Metric, F.Cu at (305.3, 218.1)
- added R2064: 22, Resistor_SMD:R_0402_1005Metric, F.Cu at (306.5, 215.6)
- added R2065: 22, Resistor_SMD:R_0402_1005Metric, F.Cu at (308.5, 215.6)
- added R2067: 60.4, Resistor_SMD:R_0402_1005Metric, F.Cu at (332.9, 181.0)
- added R2068: 39.2, Resistor_SMD:R_0402_1005Metric, B.Cu at (328.1, 179.6)
- added R2070: 39.2, Resistor_SMD:R_0402_1005Metric, B.Cu at (335.7, 181.5)
- added R2071: 240, Resistor_SMD:R_0603_1608Metric, B.Cu at (338.6, 182.1)
- added R2131: 10k, Resistor_SMD:R_0402_1005Metric, F.Cu at (303.1, 215.6)
- added R2132: 10k, Resistor_SMD:R_0402_1005Metric, B.Cu at (301.3, 216.2)
- added R2133: 10k, Resistor_SMD:R_0402_1005Metric, F.Cu at (301.3, 218.6)
- added R2134: 10k, Resistor_SMD:R_0402_1005Metric, B.Cu at (302.2, 216.2)
- added R2135: 10k, Resistor_SMD:R_0402_1005Metric, F.Cu at (302.2, 218.6)
- added R2136: 10k, Resistor_SMD:R_0402_1005Metric, B.Cu at (298.2, 216.2)
- added R2137: 10k, Resistor_SMD:R_0402_1005Metric, F.Cu at (298.2, 218.6)
- added R2139: 10k, Resistor_SMD:R_0402_1005Metric, F.Cu at (300.4, 218.6)
- added R2140: 10k, Resistor_SMD:R_0402_1005Metric, B.Cu at (300.0, 213.1)
- added R2145: 10k, Resistor_SMD:R_0402_1005Metric, B.Cu at (307.7, 218.2)
- added R2146: 10k, Resistor_SMD:R_0402_1005Metric, B.Cu at (307.7, 220.2)
- added R2147: 10k, Resistor_SMD:R_0402_1005Metric, B.Cu at (307.7, 222.2)
- added R2148: 10k, Resistor_SMD:R_0402_1005Metric, B.Cu at (307.7, 224.2)
- added R2149: 10k, Resistor_SMD:R_0402_1005Metric, B.Cu at (307.7, 226.2)
- added R2150: 10k, Resistor_SMD:R_0402_1005Metric, B.Cu at (307.7, 228.1)
- added R2151: 10k, Resistor_SMD:R_0402_1005Metric, B.Cu at (304.8, 218.2)
- added R2152: 10k, Resistor_SMD:R_0402_1005Metric, B.Cu at (304.8, 220.2)
- added R2153: 10k, Resistor_SMD:R_0402_1005Metric, B.Cu at (303.6, 211.1)
- added R2154: 10k, Resistor_SMD:R_0402_1005Metric, B.Cu at (304.8, 224.2)
- added R2155: 10k, Resistor_SMD:R_0402_1005Metric, B.Cu at (304.8, 226.2)
- added R2173: 2012, Resistor_SMD:R_0603_1608Metric, B.Cu at (328.5, 231.8)
- added R2180: 10k, Resistor_SMD:R_0402_1005Metric, B.Cu at (347.1, 223.9)
- added R2403: 0, Resistor_SMD:R_0402_1005Metric, F.Cu at (337.3, 203.8)
- added R2404: 0, Resistor_SMD:R_0402_1005Metric, F.Cu at (357.8, 199.8)
- added R2412: 0, Resistor_SMD:R_0603_1608Metric, F.Cu at (210.3, 308.5)
- added R2415: XX, Resistor_SMD:R_0402_1005Metric, F.Cu at (346.1, 309.4)
- added R2416: 4700, Resistor_SMD:R_0402_1005Metric, F.Cu at (347.0, 309.4)
- added R2417: 4700, Resistor_SMD:R_0402_1005Metric, B.Cu at (339.8, 305.1)
- added R2422: 0, Resistor_SMD:R_0805_2012Metric, F.Cu at (362.1, 326.1)
- added R2437: 10k, Resistor_SMD:R_0402_1005Metric, B.Cu at (353.8, 294.6)
- added R2465: 0, Resistor_SMD:R_0402_1005Metric, F.Cu at (357.8, 201.8)
- added R2466: 0, Resistor_SMD:R_0402_1005Metric, F.Cu at (357.8, 203.7)
- added R2467: 0, Resistor_SMD:R_0402_1005Metric, F.Cu at (338.1, 202.9)
- added R3303: 1k, Resistor_SMD:R_0402_1005Metric, F.Cu at (149.5, 132.8)
- added R3520: 2200, Resistor_SMD:R_0402_1005Metric, B.Cu at (337.0, 323.5)
- added R3521: 1500, Resistor_SMD:R_0402_1005Metric, B.Cu at (337.0, 325.5)
- added R3522: 1500, Resistor_SMD:R_0402_1005Metric, B.Cu at (337.0, 327.4)
- added R3536: 100k, Resistor_SMD:R_0402_1005Metric, B.Cu at (337.0, 329.4)
- added R3537: 150k, Resistor_SMD:R_0402_1005Metric, B.Cu at (337.0, 331.4)
- added R3538: XX, Resistor_SMD:R_0402_1005Metric, B.Cu at (337.0, 333.4)
- added R3701: 0, Resistor_SMD:R_0805_2012Metric, F.Cu at (249.4, 91.9)
- added R3723: 680, Resistor_SMD:R_0402_1005Metric, F.Cu at (254.3, 104.7)
- added R3724: XX, Resistor_SMD:R_0402_1005Metric, F.Cu at (255.8, 104.2)
- added R3725: 4700, Resistor_SMD:R_0402_1005Metric, F.Cu at (255.8, 103.2)
- added R3726: 0, Resistor_SMD:R_0402_1005Metric, F.Cu at (255.1, 99.4)
- added R4088: 0, Resistor_SMD:R_0402_1005Metric, F.Cu at (385.1, 100.3)
- added R4089: 0, Resistor_SMD:R_0402_1005Metric, F.Cu at (384.1, 100.3)
- added R4124: XX, Resistor_SMD:R_0402_1005Metric, F.Cu at (389.2, 111.7)
- added R4129: 10k, Resistor_SMD:R_0402_1005Metric, F.Cu at (368.3, 91.3)
- added R5065: 10k, Resistor_SMD:R_0402_1005Metric, F.Cu at (149.8, 231.7)
- added R5066: 10k, Resistor_SMD:R_0402_1005Metric, F.Cu at (150.8, 231.7)
- added R5077: 10k, Resistor_SMD:R_0402_1005Metric, F.Cu at (151.7, 231.7)
- added R5099: 2.2, Resistor_SMD:R_0603_1608Metric, F.Cu at (172.4, 239.7)
- added R5111: 49.9, Resistor_SMD:R_0402_1005Metric, F.Cu at (181.0, 247.9)
- added R5112: 49.9, Resistor_SMD:R_0402_1005Metric, F.Cu at (181.0, 249.6)
- added R5117: 33, Resistor_SMD:R_0402_1005Metric, F.Cu at (181.4, 243.6)
- added R5118: 22, Resistor_SMD:R_0402_1005Metric, F.Cu at (181.4, 244.5)
- added R5123: 33, Resistor_SMD:R_0402_1005Metric, F.Cu at (181.4, 242.7)
- added R5124: 33, Resistor_SMD:R_0402_1005Metric, F.Cu at (181.4, 245.4)
- added R5127: 17.4, Resistor_SMD:R_0402_1005Metric, F.Cu at (183.1, 243.6)
- added R5128: 17.4, Resistor_SMD:R_0402_1005Metric, F.Cu at (183.1, 244.5)
- added R6001: 3600, Resistor_SMD:R_0402_1005Metric, B.Cu at (400.1, 92.7)
- added R6002: 2700, Resistor_SMD:R_0402_1005Metric, B.Cu at (401.4, 93.6)
- added R6018: 200k, Resistor_SMD:R_0402_1005Metric, B.Cu at (405.9, 92.0)
- added R6019: 0, Resistor_SMD:R_0402_1005Metric, B.Cu at (407.0, 95.5)
- added R6020: 360k, Resistor_SMD:R_0402_1005Metric, B.Cu at (408.7, 95.5)
- added R6032: 10k, Resistor_SMD:R_0603_1608Metric, B.Cu at (422.2, 73.7)
- added R6039: XX, Resistor_SMD:R_0402_1005Metric, F.Cu at (278.0, 53.2)
- added R6043: XX, Resistor_SMD:R_0402_1005Metric, F.Cu at (280.0, 63.0)
- added R6060: 100k, Resistor_SMD:R_0603_1608Metric, B.Cu at (337.4, 79.1)
- added R6061: 100k, Resistor_SMD:R_0603_1608Metric, B.Cu at (334.9, 79.1)
- added R6063: 150k, Resistor_SMD:R_0603_1608Metric, B.Cu at (332.4, 79.1)
- added R6064: 150k, Resistor_SMD:R_0603_1608Metric, B.Cu at (329.9, 79.1)
- added R6079: 100k, Resistor_SMD:R_0402_1005Metric, F.Cu at (265.4, 102.2)
- added R6081: 150k, Resistor_SMD:R_0402_1005Metric, F.Cu at (265.4, 100.4)
- added R6083: 100k, Resistor_SMD:R_0402_1005Metric, F.Cu at (266.2, 97.2)
- added R6084: 220, Resistor_SMD:R_0402_1005Metric, F.Cu at (303.0, 326.9)
- added R6085: 150k, Resistor_SMD:R_0402_1005Metric, F.Cu at (266.2, 99.1)
- added R6098: 390, Resistor_SMD:R_0402_1005Metric, B.Cu at (162.8, 246.5)
- added R6100: 82, Resistor_SMD:R_0402_1005Metric, F.Cu at (303.0, 328.9)
- added R6103: 1500, Resistor_SMD:R_0402_1005Metric, B.Cu at (191.5, 152.7)
- added R6104: 1500, Resistor_SMD:R_0402_1005Metric, B.Cu at (200.4, 147.3)
- added R6105: 1500, Resistor_SMD:R_0402_1005Metric, B.Cu at (195.5, 152.2)
- added R6106: 1500, Resistor_SMD:R_0402_1005Metric, B.Cu at (196.6, 152.2)
- added R6107: 1500, Resistor_SMD:R_0402_1005Metric, B.Cu at (197.5, 152.2)
- added R6108: 1500, Resistor_SMD:R_0402_1005Metric, B.Cu at (200.4, 149.3)
- added R6109: 1500, Resistor_SMD:R_0402_1005Metric, B.Cu at (200.4, 148.3)
- added R6110: 1500, Resistor_SMD:R_0402_1005Metric, B.Cu at (200.4, 146.3)
- added R6111: 20k, Resistor_SMD:R_0402_1005Metric, B.Cu at (194.4, 153.1)
- added R6112: 15k, Resistor_SMD:R_0402_1005Metric, B.Cu at (194.0, 151.8)
- added R6113: 4700, Resistor_SMD:R_0402_1005Metric, B.Cu at (201.3, 125.8)
- added R6120: 10k, Resistor_SMD:R_0402_1005Metric, B.Cu at (201.9, 133.0)
- added R6124: 560, Resistor_SMD:R_0402_1005Metric, B.Cu at (200.7, 144.4)
- added R6126: 18k, Resistor_SMD:R_0402_1005Metric, B.Cu at (198.0, 141.0)
- added R6127: 0, Resistor_SMD:R_0402_1005Metric, B.Cu at (196.5, 140.4)
- added R6130: 560, Resistor_SMD:R_0402_1005Metric, B.Cu at (198.4, 127.8)
- added R6131: 10k, Resistor_SMD:R_0402_1005Metric, B.Cu at (198.9, 141.0)
- added R6132: 560, Resistor_SMD:R_0402_1005Metric, B.Cu at (188.2, 142.1)
- added R6135: 180, Resistor_SMD:R_0402_1005Metric, B.Cu at (198.9, 139.4)
- added R6154: 2.2, Resistor_SMD:R_0805_2012Metric, F.Cu at (240.8, 134.6)
- added R6155: 2.2, Resistor_SMD:R_0805_2012Metric, F.Cu at (220.8, 134.6)
- added R6156: 2.2, Resistor_SMD:R_0805_2012Metric, F.Cu at (260.8, 134.6)
- added R6158: 0.001, Resistor_SMD:R_2512_6332Metric, F.Cu at (240.3, 149.2)
- added R6159: 0.001, Resistor_SMD:R_2512_6332Metric, F.Cu at (220.3, 151.5)
- added R6160: 0.001, Resistor_SMD:R_2512_6332Metric, F.Cu at (260.3, 151.5)
- added R6211: 220, Resistor_SMD:R_0402_1005Metric, B.Cu at (287.4, 156.5)
- added R6214: XX, Resistor_SMD:R_0402_1005Metric, B.Cu at (281.5, 155.1)
- added R6216: XX, Resistor_SMD:R_0402_1005Metric, B.Cu at (290.9, 156.1)
- added R6219: 0, Resistor_SMD:R_0402_1005Metric, B.Cu at (286.4, 153.9)
- added R6222: 0, Resistor_SMD:R_0402_1005Metric, B.Cu at (289.2, 156.5)
- added R6228: 560, Resistor_SMD:R_0402_1005Metric, B.Cu at (345.9, 122.5)
- added R6233: 560, Resistor_SMD:R_0402_1005Metric, B.Cu at (332.6, 123.2)
- added R6248: 0.001, Resistor_SMD:R_2512_6332Metric, F.Cu at (296.8, 143.6)
- added R6249: 0.001, Resistor_SMD:R_2512_6332Metric, F.Cu at (316.8, 143.6)
- added R6524: 1k, Resistor_SMD:R_0603_1608Metric, B.Cu at (327.4, 79.1)
- added R6525: 1k, Resistor_SMD:R_0603_1608Metric, B.Cu at (324.9, 79.1)
- added R7010: XX, Resistor_SMD:R_0402_1005Metric, F.Cu at (366.5, 200.8)
- added R7012: XX, Resistor_SMD:R_0402_1005Metric, F.Cu at (365.0, 200.8)
- added R7038: 22, Resistor_SMD:R_0402_1005Metric, F.Cu at (425.4, 179.3)
- added RN7007: 22, Resistor_SMD:R_Array_Convex_4x0402, F.Cu at (373.6, 175.3)
- added RN7008: 22, Resistor_SMD:R_Array_Convex_4x0402, F.Cu at (373.6, 171.7)
- added RN7009: 22, Resistor_SMD:R_Array_Convex_4x0402, F.Cu at (373.6, 167.7)
- added RN7010: 22, Resistor_SMD:R_Array_Convex_4x0402, F.Cu at (377.6, 174.6)
- added RN7011: 22, Resistor_SMD:R_Array_Convex_4x0402, F.Cu at (377.6, 170.4)
- added RN7012: 22, Resistor_SMD:R_Array_Convex_4x0402, F.Cu at (377.6, 165.7)
- added TP1202: TestPoint, TestPoint:TestPoint_Pad_1.0x1.0mm, B.Cu at (160.2, 194.0)
- added TP1302: TestPoint, TestPoint:TestPoint_Pad_1.0x1.0mm, B.Cu at (160.2, 197.9)
- added TP2101: TestPoint, TestPoint:TestPoint_Pad_1.0x1.0mm, B.Cu at (311.1, 206.2)
- added TP2102: TestPoint, TestPoint:TestPoint_Pad_1.0x1.0mm, B.Cu at (305.1, 205.4)
- added TP2103: TestPoint, TestPoint:TestPoint_Pad_1.0x1.0mm, B.Cu at (304.1, 208.3)
- added TP2104: TestPoint, TestPoint:TestPoint_Pad_1.0x1.0mm, B.Cu at (301.1, 205.5)
- added TP2105: TestPoint, TestPoint:TestPoint_Pad_1.0x1.0mm, B.Cu at (302.4, 210.7)
- added TP2106: TestPoint, TestPoint:TestPoint_Pad_1.0x1.0mm, B.Cu at (300.2, 209.5)
- added TP3031: TestPoint, TestPoint:TestPoint_Pad_1.0x1.0mm, B.Cu at (251.7, 284.0)
- added TP3033: TestPoint, TestPoint:TestPoint_Pad_1.0x1.0mm, B.Cu at (203.6, 290.0)
- added TP3034: TestPoint, TestPoint:TestPoint_Pad_1.0x1.0mm, B.Cu at (202.2, 290.0)
- added TP3035: TestPoint, TestPoint:TestPoint_Pad_1.0x1.0mm, B.Cu at (203.6, 291.4)
- added TP3036: TestPoint, TestPoint:TestPoint_Pad_1.0x1.0mm, B.Cu at (202.2, 291.4)
- added TP3037: TestPoint, TestPoint:TestPoint_Pad_1.0x1.0mm, B.Cu at (215.8, 291.2)
- added TP3038: TestPoint, TestPoint:TestPoint_Pad_1.0x1.0mm, B.Cu at (214.4, 291.2)
- added TP3039: TestPoint, TestPoint:TestPoint_Pad_1.0x1.0mm, B.Cu at (217.2, 291.2)
- added TP3040: TestPoint, TestPoint:TestPoint_Pad_1.0x1.0mm, B.Cu at (218.6, 291.4)
- added TP4086: TestPoint, TestPoint:TestPoint_Pad_1.0x1.0mm, B.Cu at (397.9, 116.7)
- added TP6048: TestPoint, TestPoint:TestPoint_Pad_1.0x1.0mm, B.Cu at (327.2, 167.9)
- added TP6053: TestPoint, TestPoint:TestPoint_Pad_1.0x1.0mm, B.Cu at (160.4, 248.5)
- added TP6056: TestPoint, TestPoint:TestPoint_Pad_D1.0mm, B.Cu at (345.4, 223.0)
- added TP6109: TestPoint, TestPoint:TestPoint_Pad_D1.5mm, B.Cu at (241.6, 148.8)
- added TP6110: TestPoint, TestPoint:TestPoint_Pad_D1.5mm, B.Cu at (239.1, 149.8)
- added TP6111: TestPoint, TestPoint:TestPoint_Pad_D1.5mm, B.Cu at (221.6, 151.1)
- added TP6112: TestPoint, TestPoint:TestPoint_Pad_D1.5mm, B.Cu at (219.1, 151.9)
- added TP6113: TestPoint, TestPoint:TestPoint_Pad_D1.5mm, B.Cu at (261.6, 151.1)
- added TP6114: TestPoint, TestPoint:TestPoint_Pad_D1.5mm, B.Cu at (259.1, 151.9)
- added TP9623: TestPoint, TestPoint:TestPoint_Pad_D1.5mm, B.Cu at (156.9, 142.2)
- added TP9651: TestPoint, TestPoint:TestPoint_Pad_D1.5mm, B.Cu at (287.8, 148.1)
- added TP9656: TestPoint, TestPoint:TestPoint_Pad_1.0x1.0mm, F.Cu at (390.9, 79.5)
- added U1001: ~, PS3:CELL_multi, F.Cu at (240.7, 197.1)
- added U2001: ~, PS3:RSX, F.Cu at (309.6, 192.0)
- added U2409: LIGHT TRANSMITTER UNIT, OptoDevice:Vishay_MOLD-3Pin, F.Cu at (211.9, 312.8)
- added U3101: AD51/007Z, PS3:MSOP-8_2.9x4mm_P0.65mm, F.Cu at (208.0, 268.7)
- added U4003: 74LVC2G34, Package_TO_SOT_SMD:SOT-363_SC-70-6, F.Cu at (388.1, 100.0)
- added U4004: 74LVC2G34, Package_TO_SOT_SMD:SOT-363_SC-70-6, B.Cu at (387.9, 109.7)
- added U4005: 74LVC2G34, Package_TO_SOT_SMD:SOT-363_SC-70-6, F.Cu at (387.8, 95.7)
- added U4006: 74LVC1G34, Package_TO_SOT_SMD:SOT-353_SC-70-5, B.Cu at (393.8, 112.6)
- added U5006: PST36XX, Package_TO_SOT_SMD:SC-82AB, B.Cu at (156.9, 225.6)
- added U6004: PST3642UL, Package_TO_SOT_SMD:SC-82AB, B.Cu at (418.6, 97.0)
- added U6007: TPS73101DBV, Package_TO_SOT_SMD:SOT-23-5, B.Cu at (243.5, 227.8)
- added U6017: BD3521, PS3:MSOP-8_2.9x4mm_P0.65mm, B.Cu at (339.5, 208.9)
- added U6023: PST3642UL, Package_TO_SOT_SMD:SC-82AB, B.Cu at (405.9, 93.8)
- added U6108: AD51/007Z, PS3:MSOP-8_2.9x4mm_P0.65mm, F.Cu at (271.9, 166.1)
- added U6200: BD3520FVM-TR, PS3:MSOP-8_2.9x4mm_P0.65mm, B.Cu at (288.6, 153.1)
- added U6301: SN105233DBTR, Package_SO:TSSOP-30_4.4x7.8mm_P0.5mm, B.Cu at (362.1, 118.5)
- added U6302: TPS51117, Package_SO:TSSOP-14_4.4x5mm_P0.65mm, B.Cu at (179.1, 145.7)
- added U7001: ICS626BGLFT, Package_SO:TSSOP-24_4.4x7.8mm_P0.65mm, F.Cu at (363.0, 205.6)
- added Y3301: 12MHz, Crystal:Crystal_SMD_Abracon_ABM8G-4Pin_3.2x2.5mm, F.Cu at (151.8, 130.2)
- added Y7001: XX, Crystal:Crystal_SMD_FOX_FE-2Pin_7.5x5.0mm, F.Cu at (365.0, 197.7)
- C1136, C1137, C1152, C1153, C1154, C1155, C2271, C3560, C3570, C3573, C3576, C5001, C5002, C5004, C5005, C5013, C5045, C5046, Q3201, Q6003, R1108, R1109, R1112, R1113, R1114, R1115, R1118, R1119, R1120, R1121, R1150, R3105, R3121, R5001, R5006, R5008, TP1117, TP1118, U6012, U6019: moved to B.Cu
- C4032, Q3403, Q4011, R2106, R3099, R3102, R3103, R3131, R3144, R3145: moved to F.Cu
- D4006: value XX -> Thermal LED
- FB3401, FB3402: footprint Resistor_SMD:R_0603_1608Metric -> Inductor_SMD:L_0603_1608Metric
- FL2401, FL2402, FL2403: footprint Filter:Filter_Mini-Circuits_FV1206-7 -> PS3:FL_0805_2012Metric
- J3501: value RJ45_Amphenol_RJMG1BD3B8K1ANR -> RJ45; footprint Connector_RJ:RJ45_Amphenol_RJMG1BD3B8K1ANR -> PS3:RJ45
- J4010: footprint Connector_FFC-FPC:Hirose_FH26-13S-0.3SHW_2Rows-13Pins-1MP_P0.60mm_Horizontal -> PS3:ConnectorMicromatch-10
- R6022, R6029, R6030, R7044, R7045: footprint Resistor_SMD:R_0603_1608Metric -> Resistor_SMD:R_0402_1005Metric
- U1101, U2101, U3501, U6303, U6304, U6305, U6602: footprint Package_SO:MSOP-8_3x3mm_P0.65mm -> PS3:MSOP-8_2.9x4mm_P0.65mm
- U2102: value ~ -> ICS422A
- U5001: value ~ -> ICS1493G
- U5002, U5003: value ~ -> ICS9218
- U5004: value ~ -> ICS9214
- U6020: value ~ -> MM1593DFBEG
- X3001: footprint Oscillator:Oscillator_SMD_Abracon_ASCO-4Pin_1.6x1.2mm -> Oscillator:Oscillator_SMD_Abracon_ASE-4Pin_3.2x2.5mm; moved to B.Cu
- Y4001: value Crystal -> 16.9344MHz
- Y4002: value Crystal -> 32.768kHz; footprint Crystal:Crystal_SMD_G8-2Pin_3.2x1.5mm -> Crystal:Crystal_SMD_SeikoEpson_MC156-4Pin_7.1x2.5mm
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Connections:
- net Net-(RN4003-R4.1) renamed SW_4_A_M
- net Net-(U2407-Vout) renamed +3.3V_ANA
- BZ4001 pad 2: Net-(BZ4001--) -> +5V_EVER
- C2108 pad 1: Net-(U2101-Vdd) -> +3.3V_THERMAL
- C5064 pad 2: Net-(U5003-AVDD2.5) -> Net-(C5064-Pad2)
- FL6140 pad 1: Net-(FL6140-Pad1) -> Net-(U6103-CS1N)
- FL6141 pad 1: Net-(FL6140-Pad1) -> Net-(U6103-CS1N)
- FL6142 pad 1: Net-(FL6140-Pad1) -> Net-(U6103-CS1N)
- FL6143 pad 1: Net-(FL6140-Pad1) -> Net-(U6103-CS1N)
- J3701 pad 1: unconnected-(J3701-Pin_1-Pad1) -> Net-(J3701-Pin_1)
- J3701 pad 3: unconnected-(J3701-Pin_3-Pad3) -> Net-(J3701-Pin_3)
- J3701 pad 31: unconnected-(J3701-Pin_31-Pad31) -> Net-(J3701-Pin_31)
- J3701 pad 33: unconnected-(J3701-Pin_33-Pad33) -> Net-(J3701-Pin_33)
- J3701 pad 4: unconnected-(J3701-Pin_4-Pad4) -> Net-(J3701-Pin_3)
- J3701 pad 5: unconnected-(J3701-Pin_5-Pad5) -> Net-(J3701-Pin_3)
- J4010 pad 10: unconnected-(J4010-Pin_10-Pad10) -> GND
- L6104 pad 1: Net-(U6104-Vsw) -> Net-(L6104-Pad1)
- L6104 pad 2: Net-(FL6140-Pad1) -> Net-(U6104-Vsw)
- L6105 pad 1: Net-(U6105-Vsw) -> Net-(L6105-Pad1)
- L6105 pad 2: Net-(FL6140-Pad1) -> Net-(U6105-Vsw)
- L6106 pad 1: Net-(U6106-Vsw) -> Net-(L6106-Pad1)
- L6106 pad 2: Net-(FL6140-Pad1) -> Net-(U6106-Vsw)
- Q6009 pad 3: unconnected-(Q6009B-C2-Pad3) -> Net-(Q6009B-C2)
- Q6009 pad 6: unconnected-(Q6009A-C1-Pad6) -> Net-(Q6009A-C1)
- Q6010 pad 2: unconnected-(Q6010A-G1-Pad2) -> Net-(Q6010A-G1)
- Q6010 pad 4: unconnected-(Q6010B-G2-Pad4) -> Net-(Q6010B-G2)
- R2476 pad 1: unconnected-(R2476-Pad1) -> Net-(Q2403B-C2)
- R2477 pad 1: unconnected-(R2477-Pad1) -> Net-(Q2403A-C1)
- R4010 pad 1: unconnected-(R4010-Pad1) -> ~{RSX_SPI_CS}
- R4011 pad 1: unconnected-(R4011-Pad1) -> RSX_SPI_DO
- R4012 pad 1: unconnected-(R4012-Pad1) -> RSX_SPI_CLK
- R4030 pad 1: unconnected-(R4030-Pad1) -> THR_I2C_SDA
- R4031 pad 1: unconnected-(R4031-Pad1) -> THR_I2C_SCL
- R4107 pad 1: unconnected-(R4107-Pad1) -> BE_POWGOOD
- R4118 pad 1: unconnected-(R4118-Pad1) -> +5V_EVER
- R4128 pad 2: Net-(BZ4001--) -> +5V_EVER
- R5048 pad 1: Net-(U5003-AVDD2.5) -> Net-(C5064-Pad2)
- R5070 pad 1: Net-(U5003-AVDD2.5) -> Net-(C5064-Pad2)
- RN2401 pad 1: unconnected-(RN2401-R1.1-Pad1) -> RSX_VO71
- RN2401 pad 2: unconnected-(RN2401-R2.1-Pad2) -> RSX_VO68
- RN2401 pad 3: unconnected-(RN2401-R3.1-Pad3) -> RSX_VO66
- RN2401 pad 4: unconnected-(RN2401-R4.1-Pad4) -> RSX_VO64
- RN2402 pad 1: unconnected-(RN2402-R1.1-Pad1) -> RSX_VO65
- RN2402 pad 2: unconnected-(RN2402-R2.1-Pad2) -> RSX_VO67
- RN2402 pad 3: unconnected-(RN2402-R3.1-Pad3) -> RSX_VO69
- RN2402 pad 4: unconnected-(RN2402-R4.1-Pad4) -> RSX_VO70
- RN2403 pad 1: unconnected-(RN2403-R1.1-Pad1) -> RSX_VO62
- RN2403 pad 2: unconnected-(RN2403-R2.1-Pad2) -> RSX_VO61
- RN2403 pad 3: unconnected-(RN2403-R3.1-Pad3) -> RSX_VO60
- RN2403 pad 4: unconnected-(RN2403-R4.1-Pad4) -> RSX_VO58
- RN2404 pad 1: unconnected-(RN2404-R1.1-Pad1) -> RSX_VO56
- RN2404 pad 2: unconnected-(RN2404-R2.1-Pad2) -> RSX_VO57
- RN2404 pad 3: unconnected-(RN2404-R3.1-Pad3) -> RSX_VO59
- RN2404 pad 4: unconnected-(RN2404-R4.1-Pad4) -> RSX_VO63
- RN2405 pad 1: unconnected-(RN2405-R1.1-Pad1) -> RSX_VO55
- RN2405 pad 2: unconnected-(RN2405-R2.1-Pad2) -> RSX_VO53
- RN2405 pad 3: unconnected-(RN2405-R3.1-Pad3) -> RSX_VO51
- RN2405 pad 4: unconnected-(RN2405-R4.1-Pad4) -> RSX_VO49
- RN2406 pad 1: unconnected-(RN2406-R1.1-Pad1) -> RSX_VO48
- RN2406 pad 2: unconnected-(RN2406-R2.1-Pad2) -> RSX_VO50
- RN2406 pad 3: unconnected-(RN2406-R3.1-Pad3) -> RSX_VO54
- RN2406 pad 4: unconnected-(RN2406-R4.1-Pad4) -> RSX_VO52
- RN2406 pad 5: unconnected-(RN2406-R4.2-Pad5) -> Net-(RN2406-R4.2)
- RN2406 pad 6: unconnected-(RN2406-R3.2-Pad6) -> Net-(RN2406-R3.2)
- RN2406 pad 7: unconnected-(RN2406-R2.2-Pad7) -> Net-(RN2406-R2.2)
- RN2406 pad 8: unconnected-(RN2406-R1.2-Pad8) -> Net-(RN2406-R1.2)
- RN2407 pad 1: unconnected-(RN2407-R1.1-Pad1) -> RSX_VO46
- RN2407 pad 2: unconnected-(RN2407-R2.1-Pad2) -> RSX_VO44
- RN2407 pad 3: unconnected-(RN2407-R3.1-Pad3) -> RSX_VO42
- RN2407 pad 4: unconnected-(RN2407-R4.1-Pad4) -> RSX_VO40
- RN2408 pad 1: unconnected-(RN2408-R1.1-Pad1) -> RSX_VO41
- RN2408 pad 2: unconnected-(RN2408-R2.1-Pad2) -> RSX_VO43
- RN2408 pad 3: unconnected-(RN2408-R3.1-Pad3) -> RSX_VO45
- RN2408 pad 4: unconnected-(RN2408-R4.1-Pad4) -> RSX_VO47
- RN2408 pad 5: unconnected-(RN2408-R4.2-Pad5) -> Net-(RN2408-R4.2)
- RN2408 pad 6: unconnected-(RN2408-R3.2-Pad6) -> Net-(RN2408-R3.2)
- RN2408 pad 7: unconnected-(RN2408-R2.2-Pad7) -> Net-(RN2408-R2.2)
- RN2408 pad 8: unconnected-(RN2408-R1.2-Pad8) -> Net-(RN2408-R1.2)
- RN2409 pad 1: unconnected-(RN2409-R1.1-Pad1) -> RSX_VO39
- RN2409 pad 2: unconnected-(RN2409-R2.1-Pad2) -> RSX_VO38
- RN2409 pad 3: unconnected-(RN2409-R3.1-Pad3) -> RSX_VO37
- RN2409 pad 4: unconnected-(RN2409-R4.1-Pad4) -> RSX_VO36
- RN2409 pad 5: unconnected-(RN2409-R4.2-Pad5) -> Net-(RN2409-R4.2)
- RN2409 pad 6: unconnected-(RN2409-R3.2-Pad6) -> Net-(RN2409-R3.2)
- RN2409 pad 7: unconnected-(RN2409-R2.2-Pad7) -> Net-(RN2409-R2.2)
- RN2409 pad 8: unconnected-(RN2409-R1.2-Pad8) -> Net-(RN2409-R1.2)
- RN2502 pad 5: RSX_VO20 -> RSX_VO18
- RN2502 pad 6: RSX_VO23 -> RSX_VO16
- RN2502 pad 7: RSX_VO16 -> RSX_VO23
- RN2502 pad 8: RSX_VO18 -> RSX_VO20
- RN2504 pad 1: Net-(RN2504-R1.1) -> unconnected-(RN2504-R1.1-Pad1)
- RN2504 pad 5: RSX_VO5 -> RSX_VO0
- RN2504 pad 6: RSX_VO1 -> RSX_VO14
- RN2504 pad 7: RSX_VO14 -> RSX_VO1
- RN2504 pad 8: RSX_VO0 -> RSX_VO5
- RN2505 pad 5: RSX_VO11 -> RSX_VO7
- RN2505 pad 6: RSX_VO9 -> RSX_VO12
- RN2505 pad 7: RSX_VO12 -> RSX_VO9
- RN2505 pad 8: RSX_VO7 -> RSX_VO11
- RN7021 pad 3: unconnected-(RN7021-R3.1-Pad3) -> Net-(RN7021-R3.1)
- RN7021 pad 4: unconnected-(RN7021-R4.1-Pad4) -> Net-(RN7021-R4.1)
- U1201 pad C11: (no net) -> GND
- U1201 pad C6: (no net) -> +1.2V_YC_RC_VDDIO
- U1201 pad G3: unconnected-(U1201-CFM-PadG3) -> BE_Y0_RQ_CFM
- U1201 pad G4: unconnected-(U1201-CFMN-PadG4) -> BE_Y0_RQ_CFMN
- U1201 pad J11: (no net) -> GND
- U1201 pad J6: (no net) -> +1.2V_YC_RC_VDDIO
- U1202 pad C11: (no net) -> GND
- U1202 pad C6: (no net) -> +1.2V_YC_RC_VDDIO
- U1202 pad G3: unconnected-(U1202-CFM-PadG3) -> BE_Y0_RQ_CFM
- U1202 pad G4: unconnected-(U1202-CFMN-PadG4) -> BE_Y0_RQ_CFMN
- U1202 pad J11: (no net) -> GND
- U1202 pad J6: (no net) -> +1.2V_YC_RC_VDDIO
- U1301 pad C11: (no net) -> GND
- U1301 pad C6: (no net) -> +1.2V_YC_RC_VDDIO
- U1301 pad G3: unconnected-(U1301-CFM-PadG3) -> BE_Y1_RQ_CFM
- U1301 pad G4: unconnected-(U1301-CFMN-PadG4) -> BE_Y1_RQ_CFMN
- U1301 pad J11: (no net) -> GND
- U1301 pad J6: (no net) -> +1.2V_YC_RC_VDDIO
- U1302 pad C11: (no net) -> GND
- U1302 pad C6: (no net) -> +1.2V_YC_RC_VDDIO
- U1302 pad G3: unconnected-(U1302-CFM-PadG3) -> BE_Y1_RQ_CFM
- U1302 pad G4: unconnected-(U1302-CFMN-PadG4) -> BE_Y1_RQ_CFMN
- U1302 pad J11: (no net) -> GND
- U1302 pad J6: (no net) -> +1.2V_YC_RC_VDDIO
- U2101 pad 1: Net-(U2101-Vdd) -> +3.3V_THERMAL
- U2101 pad 4: unconnected-(U2101-~{THERM}-Pad4) -> RSX_GPIO6
- U2102 pad 13: unconnected-(U2102-SEL-Pad13) -> RSX_GPIO0
- U2105 pad 1: unconnected-(U2105-VccA-Pad1) -> +1.5V_AVCG_VDDIO
- U2105 pad 5: unconnected-(U2105-~{OE}-Pad5) -> Net-(Q2101-C)
- U2405 pad 10: unconnected-(U2405-~{RST}-Pad10) -> RSX_GPIO7
- U2405 pad 16: unconnected-(U2405-GND-Pad16) -> GND
- U2405 pad 5: unconnected-(U2405-VD-Pad5) -> Net-(U2405-VD)
- U2405 pad 6: unconnected-(U2405-GND-Pad6) -> GND
- U2405 pad 7: unconnected-(U2405-DIF1-Pad7) -> Net-(U2405-DIF1)
- U2405 pad 8: unconnected-(U2405-DIF0-Pad8) -> Net-(U2405-DIF0)
- U2405 pad 9: unconnected-(U2405-DEM-Pad9) -> Net-(U2405-DEM)
- U2406 pad 58: unconnected-(U2406-G6-Pad58) -> Net-(RN2406-R3.2)
- U2406 pad 61: unconnected-(U2406-G4-Pad61) -> Net-(RN2406-R4.2)
- U2406 pad 63: unconnected-(U2406-G2-Pad63) -> Net-(RN2406-R2.2)
- U2406 pad 65: unconnected-(U2406-G0-Pad65) -> Net-(RN2406-R1.2)
- U2406 pad 66: unconnected-(U2406-B11-Pad66) -> Net-(RN2408-R4.2)
- U2406 pad 68: unconnected-(U2406-B9-Pad68) -> Net-(RN2408-R3.2)
- U2406 pad 72: unconnected-(U2406-B7-Pad72) -> Net-(RN2408-R2.2)
- U2406 pad 74: unconnected-(U2406-B5-Pad74) -> Net-(RN2408-R1.2)
- U2406 pad 76: unconnected-(U2406-B3-Pad76) -> Net-(RN2409-R1.2)
- U2406 pad 77: unconnected-(U2406-B2-Pad77) -> Net-(RN2409-R2.2)
- U2406 pad 78: unconnected-(U2406-B1-Pad78) -> Net-(RN2409-R3.2)
- U2406 pad 79: unconnected-(U2406-B0-Pad79) -> Net-(RN2409-R4.2)
- U2406 pad 80: unconnected-(U2406-CSYNC-Pad80) -> Net-(U2406-CSYNC)
- U2406 pad 83: unconnected-(U2406-VSYNC-Pad83) -> Net-(U2406-VSYNC)
- U2406 pad 84: unconnected-(U2406-HSYNC-Pad84) -> Net-(U2406-HSYNC)
- U2406 pad 85: unconnected-(U2406-DEN-Pad85) -> Net-(U2406-DEN)
- U2406 pad 86: unconnected-(U2406-TMODE1-Pad86) -> GND
- U2406 pad 87: unconnected-(U2406-TMODE0-Pad87) -> GND
- U2406 pad 93: unconnected-(U2406-CLOCK-Pad93) -> Net-(U2406-CLOCK)
- U2502 pad K10: Net-(RN2504-R1.1) -> Net-(RN2504-R4.1)
- U2502 pad K11: Net-(RN2504-R3.1) -> Net-(RN2504-R2.1)
- U2502 pad K4: Net-(RN2502-R4.1) -> Net-(RN2502-R1.1)
- U2502 pad K8: Net-(RN2505-R4.1) -> Net-(RN2505-R1.1)
- U2502 pad L10: Net-(RN2505-R1.1) -> Net-(RN2505-R4.1)
- U2502 pad L11: Net-(RN2504-R4.1) -> unconnected-(U2502-SII0_D5-PadL11)
- U2502 pad L3: Net-(RN2502-R3.1) -> Net-(RN2502-R2.1)
- U2502 pad L5: Net-(RN2502-R1.1) -> Net-(RN2502-R4.1)
- U2502 pad L6: Net-(RN2502-R2.1) -> Net-(RN2502-R3.1)
- U2502 pad L7: Net-(RN2504-R2.1) -> Net-(RN2504-R3.1)
- U2502 pad L8: Net-(RN2505-R2.1) -> Net-(RN2505-R3.1)
- U2502 pad L9: Net-(RN2505-R3.1) -> Net-(RN2505-R2.1)
- U3001 pad AA30: 1.8_SB_VDD -> GND
- U3001 pad AA32: 1.8_SB_VDD -> GND
- U3001 pad AA33: 1.8_SB_VDD -> GND
- U3001 pad AA34: 1.8_SB_VDD -> GND
- U3001 pad AA36: 1.8_SB_VDD -> GND
- U3001 pad AA37: 1.8_SB_VDD -> GND
- U3001 pad AA38: 1.8_SB_VDD -> GND
- U3001 pad AA39: 1.8_SB_VDD -> GND
- U3001 pad AB30: 1.8_SB_VDD -> GND
- U3001 pad AB33: 1.8_SB_VDD -> GND
- U3001 pad AB34: 1.8_SB_VDD -> GND
- U3001 pad AB35: 1.8_SB_VDD -> GND
- U3001 pad AB36: 1.8_SB_VDD -> GND
- U3001 pad AB37: 1.8_SB_VDD -> GND
- U3001 pad AC30: 1.8_SB_VDD -> GND
- U3001 pad AC33: 1.8_SB_VDD -> GND
- U3001 pad AC34: 1.8_SB_VDD -> GND
- U3001 pad AC35: 1.8_SB_VDD -> GND
- U3001 pad AC36: 1.8_SB_VDD -> GND
- U3001 pad AC37: 1.8_SB_VDD -> GND
- U3001 pad AD30: 1.8_SB_VDD -> GND
- U3001 pad AD32: 1.8_SB_VDD -> GND
- U3001 pad AD33: 1.8_SB_VDD -> GND
- U3001 pad AD34: 1.8_SB_VDD -> GND
- U3001 pad AD36: 1.8_SB_VDD -> GND
- U3001 pad AD37: 1.8_SB_VDD -> GND
- U3001 pad AE30: 1.8_SB_VDD -> GND
- U3001 pad AE32: 1.8_SB_VDD -> GND
- U3001 pad AE33: 1.8_SB_VDD -> GND
- U3001 pad AE34: 1.8_SB_VDD -> GND
- U3001 pad AE36: 1.8_SB_VDD -> GND
- U3001 pad AE37: 1.8_SB_VDD -> GND
- U3001 pad AE38: 1.8_SB_VDD -> GND
- U3001 pad AE39: 1.8_SB_VDD -> GND
- U3001 pad AF30: 1.8_SB_VDD -> GND
- U3001 pad AF33: 1.8_SB_VDD -> GND
- U3001 pad AF34: 1.8_SB_VDD -> GND
- U3001 pad AF35: 1.8_SB_VDD -> GND
- U3001 pad AF36: 1.8_SB_VDD -> GND
- U3001 pad AF37: 1.8_SB_VDD -> GND
- U3001 pad AG30: 1.8_SB_VDD -> GND
- U3001 pad AG33: 1.8_SB_VDD -> GND
- U3001 pad AG34: 1.8_SB_VDD -> GND
- U3001 pad AG35: 1.8_SB_VDD -> GND
- U3001 pad AG36: 1.8_SB_VDD -> GND
- U3001 pad AG37: 1.8_SB_VDD -> GND
- U3001 pad AH30: 1.8_SB_VDD -> GND
- U3001 pad AH32: 1.8_SB_VDD -> GND
- U3001 pad AH33: 1.8_SB_VDD -> GND
- U3001 pad AH34: 1.8_SB_VDD -> GND
- U3001 pad AH36: 1.8_SB_VDD -> GND
- U3001 pad AH37: 1.8_SB_VDD -> GND
- U3001 pad AJ30: 1.8_SB_VDD -> GND
- U3001 pad AJ32: 1.8_SB_VDD -> GND
- U3001 pad AJ33: 1.8_SB_VDD -> GND
- U3001 pad AJ34: 1.8_SB_VDD -> GND
- U3001 pad AJ36: 1.8_SB_VDD -> GND
- U3001 pad AJ37: 1.8_SB_VDD -> GND
- U3001 pad AJ38: 1.8_SB_VDD -> GND
- U3001 pad AJ39: 1.8_SB_VDD -> GND
- U3001 pad AK30: 1.8_SB_VDD -> GND
- U3001 pad AK33: 1.8_SB_VDD -> GND
- U3001 pad AK34: 1.8_SB_VDD -> GND
- U3001 pad AK35: 1.8_SB_VDD -> GND
- U3001 pad AK36: 1.8_SB_VDD -> GND
- U3001 pad AK37: 1.8_SB_VDD -> GND
- U3001 pad AL33: 1.8_SB_VDD -> GND
- U3001 pad AL34: 1.8_SB_VDD -> GND
- U3001 pad AL35: 1.8_SB_VDD -> GND
- U3001 pad AL36: 1.8_SB_VDD -> GND
- U3001 pad AL37: 1.8_SB_VDD -> GND
- U3001 pad AM32: 1.8_SB_VDD -> GND
- U3001 pad AM33: 1.8_SB_VDD -> GND
- U3001 pad AM34: 1.8_SB_VDD -> GND
- U3001 pad AM36: 1.8_SB_VDD -> GND
- U3001 pad AM37: 1.8_SB_VDD -> GND
- U3001 pad AN32: 1.8_SB_VDD -> GND
- U3001 pad AN33: 1.8_SB_VDD -> GND
- U3001 pad AN34: 1.8_SB_VDD -> GND
- U3001 pad AN36: 1.8_SB_VDD -> GND
- U3001 pad AN37: 1.8_SB_VDD -> GND
- U3001 pad AN38: 1.8_SB_VDD -> GND
- U3001 pad AN39: 1.8_SB_VDD -> GND
- U3001 pad AP33: 1.8_SB_VDD -> GND
- U3001 pad AP34: 1.8_SB_VDD -> GND
- U3001 pad AP35: 1.8_SB_VDD -> GND
- U3001 pad AP36: 1.8_SB_VDD -> GND
- U3001 pad AP37: 1.8_SB_VDD -> GND
- U3001 pad AR33: 1.8_SB_VDD -> GND
- U3001 pad AR34: 1.8_SB_VDD -> GND
- U3001 pad AR35: 1.8_SB_VDD -> GND
- U3001 pad AR36: 1.8_SB_VDD -> GND
- U3001 pad AR37: 1.8_SB_VDD -> GND
- U3001 pad AU34: 1.8_SB_VDD -> GND
- U3001 pad AU35: 1.8_SB_VDD -> GND
- U3001 pad AU36: 1.8_SB_VDD -> GND
- U3001 pad AU37: 1.8_SB_VDD -> GND
- U3001 pad AU38: 1.8_SB_VDD -> GND
- U3001 pad AU39: 1.8_SB_VDD -> GND
- U3001 pad D33: 1.8_SB_VDD -> GND
- U3001 pad D34: 1.8_SB_VDD -> GND
- U3001 pad D35: 1.8_SB_VDD -> GND
- U3001 pad D36: 1.8_SB_VDD -> GND
- U3001 pad D37: 1.8_SB_VDD -> GND
- U3001 pad E38: 1.8_SB_VDD -> GND
- U3001 pad E39: 1.8_SB_VDD -> GND
- U3001 pad F33: 1.8_SB_VDD -> GND
- U3001 pad F34: 1.8_SB_VDD -> GND
- U3001 pad F35: 1.8_SB_VDD -> GND
- U3001 pad F36: 1.8_SB_VDD -> GND
- U3001 pad F37: 1.8_SB_VDD -> GND
- U3001 pad G33: 1.8_SB_VDD -> GND
- U3001 pad G34: 1.8_SB_VDD -> GND
- U3001 pad G35: 1.8_SB_VDD -> GND
- U3001 pad G36: 1.8_SB_VDD -> GND
- U3001 pad G37: 1.8_SB_VDD -> GND
- U3001 pad H32: 1.8_SB_VDD -> GND
- U3001 pad H33: 1.8_SB_VDD -> GND
- U3001 pad H34: 1.8_SB_VDD -> GND
- U3001 pad H36: 1.8_SB_VDD -> GND
- U3001 pad H37: 1.8_SB_VDD -> GND
- U3001 pad J32: 1.8_SB_VDD -> GND
- U3001 pad J33: 1.8_SB_VDD -> GND
- U3001 pad J34: 1.8_SB_VDD -> GND
- U3001 pad J36: 1.8_SB_VDD -> GND
- U3001 pad J37: 1.8_SB_VDD -> GND
- U3001 pad J38: 1.8_SB_VDD -> GND
- U3001 pad J39: 1.8_SB_VDD -> GND
- U3001 pad K33: 1.8_SB_VDD -> GND
- U3001 pad K34: 1.8_SB_VDD -> GND
- U3001 pad K35: 1.8_SB_VDD -> GND
- U3001 pad K36: 1.8_SB_VDD -> GND
- U3001 pad K37: 1.8_SB_VDD -> GND
- U3001 pad L33: 1.8_SB_VDD -> GND
- U3001 pad L34: 1.8_SB_VDD -> GND
- U3001 pad L35: 1.8_SB_VDD -> GND
- U3001 pad L36: 1.8_SB_VDD -> GND
- U3001 pad L37: 1.8_SB_VDD -> GND
- U3001 pad M30: 1.8_SB_VDD -> GND
- U3001 pad M32: 1.8_SB_VDD -> GND
- U3001 pad M33: 1.8_SB_VDD -> GND
- U3001 pad M34: 1.8_SB_VDD -> GND
- U3001 pad M36: 1.8_SB_VDD -> GND
- U3001 pad M37: 1.8_SB_VDD -> GND
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Routing:
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- added copper zone on F.Cu, net Net-(L6306-Pad1)
- removed copper zone on B.Cu, net 1.8_SB_VDD
Other:
- outline, holes or cut-outs redrawn
