File: cok-001/cok-001.kicad_pcb (KiCad board)
At the start: 2 copper layers, 313.2 x 237 mm, 1474 parts, among them J2401 AV OUT, J2501 HDMI_A, J3208 凸, J3209 ATA Power, J3219 for Multi_Card_Board, J3221 IMSA-9637S-60Y801, J3301 USB_A_Stacked, J3302 USB_A_Stacked, J3401 Conn_01x22_Pin, J3501 RJ45, J3701 Conn_01x33_MountingPin, J4001 FAN, J4003 Conn_01x02_Pin, J4009 Conn_01x30_Socket, J4010 BUTTONS, J6004 +12V_MAIN, J6005 +5V_EVER, Q1101 DTC144E, Q1102 DTC144E, Q1201 RK7002, Q1202 SST2222AT, Q1301 RK7002, Q1302 SST2222AT, Q2101 DTC144E, Q2401 DTC144E, Q2402 SI2303BDS, Q2403 IMH20T108, Q2404 DTA144E, Q2502 DTA144E, Q2504 DTA144E, Q2507 DTC144E, Q3101 DTC143ZUA, Q3201 DTC144E, Q3401 DTC144E, Q3402 DTC144E, Q3403 DTC144E, Q3404 DTC144E, Q3501 UMH2NTN, Q3502 DTC144E, Q3503 SI3493, Q3504 Si3460DV, Q3701 UMH2NTN, Q4008 DTC144E, Q4011 DTC143ZUA, Q4012 UMH2NTN, Q4013 UMH2NTN, Q4014 DTC143ZUA, Q4015 DTC143ZUA, Q6001 FDQ7238AS, Q6002 FDQ7238AS, Q6003 DTC144E, Q6004 SI3493, Q6006 UMH2NTN, Q6007 SI3493, Q6008 SI3493, Q6009 UMH2NTN, Q6010 SI4943, Q6012 Si3460DV, Q6200 SI4866DY, Q6301 FDQ7238AS, Q6302 SI4336, Q6303 SI4336, Q6304 SI4392, Q6305 SI4392, Q6306 SI4336, Q6307 SI4336, Q6308 IRF7607PBF, Q6309 SI4866DY, Q6310 SUD40N02, Q6311 UMH2NTN, Q6600 SUD40N02, U1101 ADT7461A0002RMZR, U1201 Y0_XDR0, U1202 Y0_XDR1, U1301 Y1_XDR0, U1302 Y1_XDR1, U2101 ADT7461A0002RMZR, U2102 ICS422A, U2105 TC7WP3125FK, U2108 ICS651MLFT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

Commit message: rdy
Parts:
- added C3324: 220u 10V, Capacitor_Tantalum_SMD:CP_EIA-6032-28_Kemet-C, F.Cu at (199.5, 96.7)
- added C3325: 220u 10V, Capacitor_Tantalum_SMD:CP_EIA-6032-28_Kemet-C, F.Cu at (213.7, 96.7)
- added D3316: EDZCTE616, Diode_SMD:D_SOD-923, F.Cu at (211.3, 120.9)
- added D3317: EDZCTE616, Diode_SMD:D_SOD-923, F.Cu at (211.3, 123.0)
- added D3318: EDZCTE616, Diode_SMD:D_SOD-923, F.Cu at (186.1, 120.5)
- added D3319: EDZCTE616, Diode_SMD:D_SOD-923, F.Cu at (186.1, 122.5)
- added D3320: EDZCTE616, Diode_SMD:D_SOD-923, B.Cu at (171.2, 128.8)
- added D3321: EDZCTE616, Diode_SMD:D_SOD-923, B.Cu at (171.2, 126.8)
- added D3322: EDZCTE616, Diode_SMD:D_SOD-923, B.Cu at (148.1, 126.8)
- added D3323: EDZCTE616, Diode_SMD:D_SOD-923, B.Cu at (150.2, 126.8)
- added R3342: 0, Resistor_SMD:R_0402_1005Metric, F.Cu at (154.6, 93.8)
- added R3343: XX, Resistor_SMD:R_0402_1005Metric, F.Cu at (155.9, 93.3)
- added R3345: 0, Resistor_SMD:R_0402_1005Metric, F.Cu at (201.2, 93.8)
- added R3346: XX, Resistor_SMD:R_0402_1005Metric, F.Cu at (207.3, 92.0)
- added R3350: 0, Resistor_SMD:R_0603_1608Metric, F.Cu at (162.9, 100.2)
- added R3356: 10k, Resistor_SMD:R_0402_1005Metric, F.Cu at (199.3, 92.8)
- added R3357: 10k, Resistor_SMD:R_0402_1005Metric, F.Cu at (199.3, 93.8)
- added R3358: 10k, Resistor_SMD:R_0402_1005Metric, F.Cu at (160.5, 91.5)
- added R3359: 10k, Resistor_SMD:R_0402_1005Metric, F.Cu at (159.2, 91.1)
- added R3459: 330, Resistor_SMD:R_0402_1005Metric, F.Cu at (237.8, 109.7)
- added R3462: 10k, Resistor_SMD:R_0402_1005Metric, F.Cu at (233.3, 108.2)
- added R7318: 56, Resistor_SMD:R_0402_1005Metric, B.Cu at (396.1, 230.3)
- added R7319: 56, Resistor_SMD:R_0402_1005Metric, F.Cu at (407.5, 244.7)
- added R7320: 56, Resistor_SMD:R_0402_1005Metric, F.Cu at (407.5, 245.6)
- added RN7305: 56, Resistor_SMD:R_Array_Convex_4x0402, B.Cu at (382.1, 249.9)
- added RN7310: 56, Resistor_SMD:R_Array_Convex_4x0402, B.Cu at (382.1, 253.8)
- D4006: footprint LED_SMD:LED_0402_1005Metric -> LED_SMD:LED_0603_1608Metric
- L3301, L3302, L3303, L3304: value L_Iron_Coupled_Small_1243 -> 0uH
- Q6004, R6039, R6043: moved to B.Cu
- R4118: footprint Resistor_SMD:R_0402_1005Metric -> Resistor_SMD:R_0603_1608Metric
- R6045: footprint Resistor_SMD:R_0603_1608Metric -> Resistor_SMD:R_0402_1005Metric; moved to B.Cu
- R6524, R6525: footprint Resistor_SMD:R_0603_1608Metric -> Resistor_SMD:R_0402_1005Metric; moved to F.Cu
- U3303, U3304: value ~ -> BD6517F
- moved R1101 226.3 mm to (183.2, 78.4), turned to 0 degrees
- moved Q6004 196.5 mm to (202.2, 266.3), turned to 90 degrees
- moved R6045 94.5 mm to (199.9, 266.9), turned to -90 degrees
- moved C6041 78.2 mm to (271.0, 77.6)
- moved Q6006 48.8 mm to (291.1, 101.5), turned to -90 degrees
- moved R6524 47.1 mm to (288.6, 105.8)
- moved R6039 43.7 mm to (261.3, 93.7), turned to -90 degrees
- moved R6525 39.8 mm to (289.0, 96.2), turned to 0 degrees
- moved R6043 34.1 mm to (265.1, 93.7), turned to 90 degrees
- moved C6186 33.7 mm to (260.1, 129.5), turned to 90 degrees
- moved C6184 16.5 mm to (240.1, 129.5), turned to 90 degrees
- moved C6073 11.4 mm to (283.2, 69.1)
- moved C6185 10.6 mm to (220.1, 129.5), turned to 90 degrees
- moved R2106 7.98 mm to (324.9, 222.8)
- moved TP9508 5.55 mm to (189.6, 120.6)
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- renumbered R5077 to R5067
Connections:
- net Net-(RN7301-R1.2) renamed BC_PCI_AD30
- net Net-(RN7301-R2.2) renamed BC_PCI_AD28
- net Net-(RN7301-R3.2) renamed BC_PCI_AD26
- net Net-(RN7301-R4.2) renamed BC_PCI_AD24
- net Net-(RN7302-R1.2) renamed BC_PCI_AD22
- net Net-(RN7302-R2.2) renamed BC_PCI_AD20
- net Net-(RN7302-R3.2) renamed BC_PCI_AD18
- net Net-(RN7302-R4.2) renamed BC_PCI_AD16
- net Net-(RN7303-R1.2) renamed BC_PCI_AD15
- net Net-(RN7303-R2.2) renamed BC_PCI_AD6
- net Net-(RN7303-R3.2) renamed BC_PCI_AD11
- net Net-(RN7303-R4.2) renamed BC_PCI_AD9
- net Net-(RN7304-R1.2) renamed BC_PCI_AD13
- net Net-(RN7304-R2.2) renamed BC_PCI_AD2
- net Net-(RN7304-R3.2) renamed BC_PCI_AD4
- net Net-(RN7306-R1.2) renamed BC_PCI_AD25
- net Net-(RN7306-R2.2) renamed BC_PCI_AD27
- net Net-(RN7306-R3.2) renamed BC_PCI_AD31
- net Net-(RN7306-R4.2) renamed BC_PCI_AD29
- net Net-(RN7307-R1.2) renamed BC_PCI_AD17
- net Net-(RN7307-R2.2) renamed BC_PCI_AD19
- net Net-(RN7307-R3.2) renamed BC_PCI_AD21
- net Net-(RN7307-R4.2) renamed BC_PCI_AD23
- net Net-(RN7308-R1.2) renamed BC_PCI_AD3
- net Net-(RN7308-R2.2) renamed BC_PCI_AD7
- net Net-(RN7308-R3.2) renamed BC_PCI_AD10
- net Net-(RN7308-R4.2) renamed BC_PCI_AD14
- net Net-(RN7309-R1.2) renamed BC_PCI_AD12
- net Net-(RN7309-R2.2) renamed BC_PCI_AD8
- net Net-(RN7309-R3.2) renamed BC_PCI_AD5
- net Net-(RN7309-R4.2) renamed BC_PCI_AD1
- net Net-(RN7312-R1.1) renamed SIF_BC_AD3
- net Net-(RN7312-R2.1) renamed SIF_BC_AD0
- net Net-(RN7312-R3.1) renamed SIF_BC_AD1
- net Net-(RN7312-R4.1) renamed SIF_BC_AD2
- net Net-(RN7313-R1.1) renamed SIF_BC_AD4
- net Net-(RN7313-R2.1) renamed SIF_BC_AD7
- net Net-(RN7313-R3.1) renamed SIF_BC_AD9
- net Net-(RN7313-R4.1) renamed SIF_BC_AD6
- net Net-(RN7314-R1.1) renamed SIF_BC_AD17
- net Net-(RN7314-R2.1) renamed SIF_BC_AD19
- net Net-(RN7314-R3.1) renamed SIF_BC_AD22
- net Net-(RN7314-R4.1) renamed SIF_BC_AD16
- net Net-(RN7315-R1.1) renamed SIF_BC_AD21
- net Net-(RN7315-R2.1) renamed SIF_BC_AD20
- net Net-(RN7315-R3.1) renamed SIF_BC_AD18
- net Net-(RN7315-R4.1) renamed SIF_BC_AD28
- net Net-(RN7316-R1.1) renamed SIF_BC_AD11
- net Net-(RN7316-R2.1) renamed SIF_BC_AD15
- net Net-(RN7316-R3.1) renamed SIF_BC_AD14
- net Net-(RN7316-R4.1) renamed SIF_BC_AD13
- net Net-(RN7317-R1.1) renamed SIF_BC_AD12
- net Net-(RN7317-R2.1) renamed SIF_BC_AD8
- net Net-(RN7317-R3.1) renamed SIF_BC_AD10
- net Net-(RN7317-R4.1) renamed SIF_BC_AD5
- net Net-(RN7318-R1.1) renamed SIF_BC_AD24
- net Net-(RN7318-R2.1) renamed SIF_BC_AD23
- net Net-(RN7318-R3.1) renamed SIF_BC_AD25
- net Net-(RN7318-R4.1) renamed SIF_BC_AD27
- net Net-(RN7319-R1.1) renamed SIF_BC_AD31
- net Net-(RN7319-R2.1) renamed SIF_BC_AD26
- net Net-(RN7319-R3.1) renamed SIF_BC_AD29
- net Net-(RN7319-R4.1) renamed SIF_BC_AD30
- net Net-(RN7321-R1.1) renamed ~{SIF_BE2_BC}
- net Net-(RN7321-R2.1) renamed ~{SIF_BE1_BC}
- net Net-(RN7321-R4.1) renamed ~{SIF_BE0_BC}
- net Net-(U7301-PCI_AD0) renamed BC_PCI_AD0
- net Net-(U7301-~{PCI_DEVSEL}) renamed BC_PCI_DEVSEL
- net Net-(U7301-~{PCI_FRAME}) renamed ~{BC_PCI_FRAME}
- net Net-(U7301-~{PCI_IADY}) renamed ~{BC_PCI_IRDY}
- net Net-(U7301-~{PCI_PERR}) renamed ~{BC_PCI_PERR}
- net Net-(U7301-~{PCI_REQ}) renamed ~{BC_PCI_REQ1}
- net Net-(U7301-~{PCI_SERR}) renamed ~{BC_PCI_SERR}
- net Net-(U7301-~{PCI_STOP}) renamed ~{BC_PCI_STOP}
- net Net-(U7301-~{PCI_TADY}) renamed ~{BC_PCI_TRDY}
- D3401 pad 2: unconnected-(D3401-A-Pad2) -> Net-(D3401-A)
- Q3402 pad 3: unconnected-(Q3402-C-Pad3) -> Net-(Q3402-C)
- Q3403 pad 1: unconnected-(Q3403-B-Pad1) -> Net-(Q3402-C)
- R5065 pad 1: Net-(R5065-Pad1) -> Net-(U5002-AVDD2.5)
- R5066 pad 1: Net-(R5065-Pad1) -> Net-(U5002-AVDD2.5)
- R5067 pad 1: Net-(R5065-Pad1) -> Net-(U5002-AVDD2.5)
- U1001 pad AF35: unconnected-(U1001AF-TX3_TXN1-PadAF35) -> BE_TX3_TXN1
- U1001 pad AF36: unconnected-(U1001AF-TX3_TXP1-PadAF36) -> BE_TX3_TXP1
- U1001 pad AF38: unconnected-(U1001AF-TX3_TXN2-PadAF38) -> BE_TX3_TXN2
- U1001 pad AF39: unconnected-(U1001AF-TX3_TXP2-PadAF39) -> BE_TX3_TXP2
- U1001 pad AF40: unconnected-(U1001AF-TX3_TXN0-PadAF40) -> BE_TX3_TXN0
- U1001 pad AF41: unconnected-(U1001AF-TX3_TXP0-PadAF41) -> BE_TX3_TXP0
- U1001 pad AT1: unconnected-(U1001AT-Y1_RQ10-PadAT1) -> BE_Y1_RQ10
- U1001 pad AT10: unconnected-(U1001AT-Y1_DQ3N_7-PadAT10) -> Y1_XDR1_DQN9
- U1001 pad AT26: unconnected-(U1001AT-RX4_RXN1-PadAT26) -> BE_RX4_RXN1
- U1001 pad AT27: unconnected-(U1001AT-RX4_RXN3-PadAT27) -> BE_RX4_RXN3
- U1001 pad AT28: unconnected-(U1001AT-RX4_RXN5-PadAT28) -> BE_RX4_RXN5
- U1001 pad AT29: unconnected-(U1001AT-RX4_RXN7-PadAT29) -> BE_RX4_RXN7
- U1001 pad AT3: unconnected-(U1001AT-Y1_RQ11-PadAT3) -> BE_Y1_RQ11
- U1001 pad AT30: unconnected-(U1001AT-TX6_TXP5-PadAT30) -> BE_TX6_TXP5
- U1001 pad AT31: unconnected-(U1001AT-TX6_TXP3-PadAT31) -> BE_TX6_TXP3
- U1001 pad AT32: unconnected-(U1001AT-TX6_TXP1-PadAT32) -> BE_TX6_TXP1
- U1001 pad AT7: unconnected-(U1001AT-Y1_DQ2N_2-PadAT7) -> Y1_XDR1_DQN1
- U1001 pad AT8: unconnected-(U1001AT-Y1_DQ2N_7-PadAT8) -> Y1_XDR1_DQN13
- U1001 pad AT9: unconnected-(U1001AT-Y1_DQ3N_0-PadAT9) -> Y1_XDR1_DQN5
- U1001 pad AU17: unconnected-(U1001AU-STI_THERMAL0-PadAU17) -> STI_THERMAL0
- U1001 pad AU34: unconnected-(U1001AU-RC_VOLGND1-PadAU34) -> BE_RC_VOLGND1
- U1001 pad AV1: unconnected-(U1001AV-Y1_DQ2_RLOAD-PadAV1) -> BE_Y1_DQ2_RLOAD
- U1001 pad AV13: unconnected-(U1001AV-SPI_SI-PadAV13) -> BE_SPI_DO
- U1001 pad AV14: unconnected-(U1001AV-/TRST-PadAV14) -> ~{BE_TRST}
- U1001 pad AV2: unconnected-(U1001AV-Y1_DQ2_1-PadAV2) -> Y1_XDR0_DQ1
- U1001 pad AV20: unconnected-(U1001AV-POWER_GOOD-PadAV20) -> BE_POWGOOD
- U1001 pad AV21: unconnected-(U1001AV-/CHECKSTOP_IN_B-PadAV21) -> ~{BE_CHKSTP_IN}
- U1001 pad AV22: unconnected-(U1001AV-SPI_CTL1-PadAV22) -> BE_SPI_CTL1
- U1001 pad AV26: unconnected-(U1001AV-RX4_RXP0-PadAV26) -> BE_RX4_RXP0
- U1001 pad AV27: unconnected-(U1001AV-RX4_RXCLKP-PadAV27) -> BE_RX4_RXCLKP
- U1001 pad AV28: unconnected-(U1001AV-RX4_RXP4-PadAV28) -> BE_RX4_RXP4
- U1001 pad AV3: unconnected-(U1001AV-Y1_DQ2_5-PadAV3) -> Y1_XDR0_DQ13
- U1001 pad AV31: unconnected-(U1001AV-TX6_TXCLKN-PadAV31) -> BE_TX6_TXCLKN
- U1001 pad AV4: unconnected-(U1001AV-Y1_DQ2_0-PadAV4) -> Y1_XDR0_DQ5
- U1001 pad AV5: unconnected-(U1001AV-Y1_DQ3_4-PadAV5) -> Y1_XDR0_DQ9
- U1001 pad AV7: unconnected-(U1001AV-Y1_DQ2_3-PadAV7) -> Y1_XDR1_DQ11
- U1001 pad AV8: unconnected-(U1001AV-Y1_DQ3_1-PadAV8) -> Y1_XDR1_DQ7
- U1001 pad AV9: unconnected-(U1001AV-Y1_DQ3_3-PadAV9) -> Y1_XDR1_DQ3
- U1001 pad AW26: unconnected-(U1001AW-RX4_RXN0-PadAW26) -> BE_RX4_RXN0
- U1001 pad AW27: unconnected-(U1001AW-RX4_RXCLKN-PadAW27) -> BE_RX4_RXCLKN
- U1001 pad AW28: unconnected-(U1001AW-RX4_RXN4-PadAW28) -> BE_RX4_RXN4
- U1001 pad AW31: unconnected-(U1001AW-TX6_TXCLKP-PadAW31) -> BE_TX6_TXCLKP
- U1001 pad AY26: unconnected-(U1001AY-RX4_RXP2-PadAY26) -> BE_RX4_RXP2
- U1001 pad AY28: unconnected-(U1001AY-RX4_RXP6-PadAY28) -> BE_RX4_RXP6
- U1001 pad AY30: unconnected-(U1001AY-TX6_TXN4-PadAY30) -> BE_TX6_TXN4
- U1001 pad AY32: unconnected-(U1001AY-TX6_TXN0-PadAY32) -> BE_TX6_TXN0
- U1001 pad BA26: unconnected-(U1001BA-RX4_RXN2-PadBA26) -> BE_RX4_RXN2
- U1001 pad BA28: unconnected-(U1001BA-RX4_RXN6-PadBA28) -> BE_RX4_RXN6
- U2001 pad AF6: unconnected-(U2001AF-TX2_TXN7-PadAF6) -> BE_RX2_RXN7
- U2001 pad AF7: unconnected-(U2001AF-TX2_TXP7-PadAF7) -> BE_RX2_RXP7
- U2001 pad AJ1: unconnected-(U2001AJ-TX2_TXN2-PadAJ1) -> BE_RX2_RXN2
- U2001 pad AJ2: unconnected-(U2001AJ-TX2_TXP2-PadAJ2) -> BE_RX2_RXP2
- U2001 pad AJ3: unconnected-(U2001AJ-TX2_TXN0-PadAJ3) -> BE_RX2_RXN0
- U2001 pad AJ4: unconnected-(U2001AJ-TX2_TXP0-PadAJ4) -> BE_RX2_RXP0
- U2001 pad AM1: unconnected-(U2001AM-RX3_RXP4-PadAM1) -> BE_TX3_TXP4
- U2001 pad AM2: unconnected-(U2001AM-RX3_RXN4-PadAM2) -> BE_TX3_TXN4
- U2001 pad AM3: unconnected-(U2001AM-RX3_RXP6-PadAM3) -> BE_TX3_TXP6
- U2001 pad AM4: unconnected-(U2001AM-RX3_RXN6-PadAM4) -> BE_TX3_TXN6
- U2001 pad AM6: unconnected-(U2001AM-RX3_RXP5-PadAM6) -> BE_TX3_TXP5
- U2001 pad AM7: unconnected-(U2001AM-RX3_RXN5-PadAM7) -> BE_TX3_TXN5
- U2001 pad AP1: unconnected-(U2001AP-REFCLKP-PadAP1) -> RSX_RC_REFCLK_P
- U2001 pad AP2: unconnected-(U2001AP-REFCLKN-PadAP2) -> RSX_RC_REFCLK_N
- U2001 pad U3: unconnected-(U2001U-RX1_RXCKP-PadU3) -> BE_TX1_TXCLKP
- U2001 pad U4: unconnected-(U2001U-RX1_RXCLN-PadU4) -> BE_TX1_TXCLKN
- U2001 pad U6: unconnected-(U2001U-RX1_RXP3-PadU6) -> BE_TX1_TXP3
- U2001 pad U7: unconnected-(U2001U-RX1_RXN3-PadU7) -> BE_TX1_TXN3
- U3001 pad AE1: unconnected-(U3001AE-IOIFRXDP0-PadAE1) -> BE_TX6_TXP0
- U3001 pad AE2: unconnected-(U3001AE-IOIFRXDN0-PadAE2) -> BE_TX6_TXN0
- U3001 pad AE3: unconnected-(U3001AE-IOIFRXDP2-PadAE3) -> BE_TX6_TXP2
- U3001 pad AE4: unconnected-(U3001AE-IOIFRXDN2-PadAE4) -> BE_TX6_TXN2
- U3001 pad AE6: unconnected-(U3001AE-IOIFRXDP1-PadAE6) -> BE_TX6_TXP1
- U3001 pad AE7: unconnected-(U3001AE-IOIFRXDN1-PadAE7) -> BE_TX6_TXN1
- U3001 pad AF3: unconnected-(U3001AF-IOIFRXCLKP-PadAF3) -> BE_TX6_TXCLKP
- U3001 pad AF4: unconnected-(U3001AF-IOIFRXCLKN-PadAF4) -> BE_TX6_TXCLKN
- U3001 pad AF6: unconnected-(U3001AF-IOIFRXDP3-PadAF6) -> BE_TX6_TXP3
- U3001 pad AF7: unconnected-(U3001AF-IOIFRXDN3-PadAF7) -> BE_TX6_TXN3
- U3303 pad 1: unconnected-(U3303-CTRLA-Pad1) -> Net-(U3303-CTRLA)
- U3303 pad 2: unconnected-(U3303-FLAGA-Pad2) -> Net-(U3303-FLAGA)
- U3303 pad 3: unconnected-(U3303-FLAGB-Pad3) -> Net-(U3303-FLAGB)
- U3304 pad 2: unconnected-(U3304-FLAGA-Pad2) -> Net-(U3304-FLAGA)
- U3304 pad 3: unconnected-(U3304-FLAGB-Pad3) -> Net-(U3304-FLAGB)
- U3304 pad 4: unconnected-(U3304-CTRLB-Pad4) -> Net-(U3304-CTRLB)
- U7301 pad A3: unconnected-(U7301-SIF_MSCLK-PadA3) -> MSCLK
- U7301 pad B5: unconnected-(U7301-~{SIF_BE3}-PadB5) -> ~{SIF_BE3_BC}
- U7301 pad K14: unconnected-(U7301-~{SIF_BREQ}-PadK14) -> ~{BREQ_BC}
- U7301 pad L13: unconnected-(U7301-~{SIF_BGNT}-PadL13) -> ~{BGNT_BC}
Routing:
- net ~{BGNT}: track 0.00 -> 108.9 mm
- net ~{BREQ}: track 0.00 -> 107.4 mm
- net unconnected-(U7301-SIF_MSCLK-PadA3): track 96.8 -> 0.00 mm
- net MSCLK: track 0.00 -> 96.8 mm
- net Y1_XDR1_DQN9: track 0.00 -> 85.7 mm, vias 0 -> 2
- net Y1_XDR1_DQN5: track 0.00 -> 83.2 mm, vias 0 -> 2
- net Y1_XDR1_DQ9: track 0.00 -> 82.7 mm, vias 0 -> 1
- net unconnected-(U1001AR-Y1_DQ3_0-PadAR9): track 0.00 -> 81.6 mm, vias 0 -> 1
- net Y1_XDR1_DQN13: track 0.00 -> 71.7 mm, vias 0 -> 2
- net Y1_XDR1_DQ13: track 0.00 -> 69.7 mm, vias 0 -> 1
- net Y1_XDR1_DQN1: track 0.00 -> 67.0 mm, vias 0 -> 2
- net unconnected-(U1001AR-Y1_DQ2_2-PadAR7): track 0.00 -> 64.0 mm, vias 0 -> 1
- net BE_TX6_TXN1: track 0.71 -> 60.1 mm, vias 1 -> 2
- net Y1_XDR1_DQ3: track 22.0 -> 80.9 mm
- net BE_TX6_TXP1: track 0.00 -> 57.8 mm, vias 0 -> 2
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