File: cok-001/cok-001.kicad_pcb (KiCad board)
At the start: 2 copper layers, 313.2 x 237 mm, 1500 parts, among them J2401 AV OUT, J2501 HDMI_A, J3208 凸, J3209 ATA Power, J3219 for Multi_Card_Board, J3221 IMSA-9637S-60Y801, J3301 USB_A_Stacked, J3302 USB_A_Stacked, J3401 Conn_01x22_Pin, J3501 RJ45, J3701 Conn_01x33_MountingPin, J4001 FAN, J4003 Conn_01x02_Pin, J4009 Conn_01x30_Socket, J4010 BUTTONS, J6004 +12V_MAIN, J6005 +5V_EVER, Q1101 DTC144E, Q1102 DTC144E, Q1201 RK7002, Q1202 SST2222AT, Q1301 RK7002, Q1302 SST2222AT, Q2101 DTC144E, Q2401 DTC144E, Q2402 SI2303BDS, Q2403 IMH20T108, Q2404 DTA144E, Q2502 DTA144E, Q2504 DTA144E, Q2507 DTC144E, Q3101 DTC143ZUA, Q3201 DTC144E, Q3401 DTC144E, Q3402 DTC144E, Q3403 DTC144E, Q3404 DTC144E, Q3501 UMH2NTN, Q3502 DTC144E, Q3503 SI3493, Q3504 Si3460DV, Q3701 UMH2NTN, Q4008 DTC144E, Q4011 DTC143ZUA, Q4012 UMH2NTN, Q4013 UMH2NTN, Q4014 DTC143ZUA, Q4015 DTC143ZUA, Q6001 FDQ7238AS, Q6002 FDQ7238AS, Q6003 DTC144E, Q6004 SI3493, Q6006 UMH2NTN, Q6007 SI3493, Q6008 SI3493, Q6009 UMH2NTN, Q6010 SI4943, Q6012 Si3460DV, Q6200 SI4866DY, Q6301 FDQ7238AS, Q6302 SI4336, Q6303 SI4336, Q6304 SI4392, Q6305 SI4392, Q6306 SI4336, Q6307 SI4336, Q6308 IRF7607PBF, Q6309 SI4866DY, Q6310 SUD40N02, Q6311 UMH2NTN, Q6600 SUD40N02, U1101 ADT7461A0002RMZR, U1201 Y0_XDR0, U1202 Y0_XDR1, U1301 Y1_XDR0, U1302 Y1_XDR1, U2101 ADT7461A0002RMZR, U2102 ICS422A, U2105 TC7WP3125FK, U2108 ICS651MLFT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

Commit message: update 10
Parts:
- added R2406: 100k, Resistor_SMD:R_0402_1005Metric, F.Cu at (246.9, 68.3)
- added R3092: 10k, Resistor_SMD:R_0402_1005Metric, F.Cu at (242.0, 63.7)
- added R3096: 10k, Resistor_SMD:R_0402_1005Metric, F.Cu at (242.0, 65.7)
- added R3162: 10k, Resistor_SMD:R_0402_1005Metric, F.Cu at (242.0, 67.7)
- added R3253: 0, Resistor_SMD:R_0603_1608Metric, F.Cu at (247.5, 64.0)
Connections:
- net Net-(U2403-OUT) renamed +5V_ANA
- J3219 pad 10: unconnected-(J3219-Pin_10-Pad10) -> Net-(J3219-Pin_10)
- J3219 pad 11: unconnected-(J3219-Pin_11-Pad11) -> Net-(J3219-Pin_10)
- J3219 pad 12: unconnected-(J3219-Pin_12-Pad12) -> Net-(J3219-Pin_10)
- J3219 pad 14: unconnected-(J3219-Pin_14-Pad14) -> ~{MC_DET}
- J3219 pad 3: unconnected-(J3219-Pin_3-Pad3) -> /External/SB_USB2_DP_32
- J3219 pad 4: unconnected-(J3219-Pin_4-Pad4) -> /External/SB_USB2_DM_32
- J3219 pad 7: unconnected-(J3219-Pin_7-Pad7) -> Net-(J3219-Pin_7)
- J3219 pad 9: unconnected-(J3219-Pin_9-Pad9) -> Net-(J3219-Pin_10)
- Q2401 pad 1: unconnected-(Q2401-B-Pad1) -> SW_8_B
- Q2402 pad 2: unconnected-(Q2402-S-Pad2) -> +12V_MAIN
- U1001 pad A40: unconnected-(U1001A-RC_VDDIO-PadA40) -> +1.2V_YC_RC_VDDIO
- U1001 pad AL1: Net-(U1001AL-NC_OPEN28) -> GND
- U1001 pad AL15: Net-(U1001AL-NC_OPEN28) -> GND
- U1001 pad AL19: Net-(U1001AL-NC_OPEN28) -> GND
- U1001 pad AL21: Net-(U1001AL-NC_OPEN28) -> GND
- U1001 pad AL23: Net-(U1001AL-NC_OPEN28) -> GND
- U1001 pad AL25: Net-(U1001AL-NC_OPEN28) -> GND
- U1001 pad AL27: Net-(U1001AL-NC_OPEN28) -> GND
- U1001 pad AL29: Net-(U1001AL-NC_OPEN28) -> GND
- U1001 pad AL3: Net-(U1001AL-NC_OPEN28) -> GND
- U1001 pad AL31: Net-(U1001AL-NC_OPEN28) -> GND
- U1001 pad AL33: Net-(U1001AL-NC_OPEN28) -> GND
- U1001 pad AL34: Net-(U1001AL-NC_OPEN28) -> GND
- U1001 pad AL37: Net-(U1001AL-NC_OPEN28) -> GND
- U1001 pad AL5: Net-(U1001AL-NC_OPEN28) -> GND
- U1001 pad AL6: Net-(U1001AL-NC_OPEN28) -> GND
- U1001 pad AN1: Net-(U1001AL-NC_OPEN28) -> GND
- U1001 pad AN3: Net-(U1001AL-NC_OPEN28) -> GND
- U1001 pad AN38: Net-(U1001AL-NC_OPEN28) -> GND
- U1001 pad AN5: Net-(U1001AL-NC_OPEN28) -> GND
- U1001 pad AP10: Net-(U1001AL-NC_OPEN28) -> GND
- U1001 pad AP11: Net-(U1001AL-NC_OPEN28) -> GND
- U1001 pad AP12: Net-(U1001AL-NC_OPEN28) -> GND
- U1001 pad AP14: Net-(U1001AL-NC_OPEN28) -> GND
- U1001 pad AP15: Net-(U1001AL-NC_OPEN28) -> GND
- U1001 pad AP18: Net-(U1001AL-NC_OPEN28) -> GND
- U1001 pad AP27: Net-(U1001AL-NC_OPEN28) -> GND
- U1001 pad AP32: Net-(U1001AL-NC_OPEN28) -> GND
- U1001 pad AP37: Net-(U1001AL-NC_OPEN28) -> GND
- U1001 pad AP4: Net-(U1001AL-NC_OPEN28) -> GND
- U1001 pad AP6: Net-(U1001AL-NC_OPEN28) -> GND
- U1001 pad AP7: Net-(U1001AL-NC_OPEN28) -> GND
- U1001 pad AP9: Net-(U1001AL-NC_OPEN28) -> GND
- U1001 pad AR14: Net-(U1001AL-NC_OPEN28) -> GND
- U1001 pad AR15: Net-(U1001AL-NC_OPEN28) -> GND
- U1001 pad AR16: Net-(U1001AL-NC_OPEN28) -> GND
- U1001 pad AR17: Net-(U1001AL-NC_OPEN28) -> GND
- U1001 pad AR18: Net-(U1001AL-NC_OPEN28) -> GND
- U1001 pad AR25: Net-(U1001AL-NC_OPEN28) -> GND
- U1001 pad AR3: Net-(U1001AL-NC_OPEN28) -> GND
- U1001 pad AR34: Net-(U1001AL-NC_OPEN28) -> GND
- U1001 pad AR37: Net-(U1001AL-NC_OPEN28) -> GND
- U1001 pad AR5: Net-(U1001AL-NC_OPEN28) -> GND
- U1001 pad C1: unconnected-(U1001C-GND-PadC1) -> GND
- U1001 pad C12: unconnected-(U1001C-VDD-PadC12) -> +1.0V_BE_VDDC
- U1001 pad D1: unconnected-(U1001D-GND-PadD1) -> GND
- U1001 pad E37: unconnected-(U1001E-RC_VDDIO-PadE37) -> +1.2V_YC_RC_VDDIO
- U1001 pad H37: unconnected-(U1001H-RC_VDDIO-PadH37) -> +1.2V_YC_RC_VDDIO
- U1001 pad H8: unconnected-(U1001H-Y0_DQ0_VDDA-PadH8) -> +1.2V_MC2_VDDIO
- U1001 pad J37: unconnected-(U1001J-RC_VDDIO-PadJ37) -> +1.2V_YC_RC_VDDIO
- U1001 pad J38: unconnected-(U1001J-RC_ROLREF0-PadJ38) -> +1.2V_YC_RC_VDDIO
- U1001 pad J8: unconnected-(U1001J-Y0_DQ1_VDDA-PadJ8) -> +1.2V_MC2_VDDIO
- U1001 pad L8: unconnected-(U1001L-Y0_RQ_VDDA-PadL8) -> +1.2V_MC2_VDDIO
- U2405 pad 17: unconnected-(U2405-VA_H-Pad17) -> Net-(U2402-OUT)
- U2407 pad 5: unconnected-(U2407-Cont-Pad5) -> SW_8_B
- U2408 pad 5: unconnected-(U2408-Cont-Pad5) -> SW_8_B
Routing:
- net SW_8_B: track 133.6 -> 195.2 mm, vias 4 -> 6
- net unconnected-(U2408-Cont-Pad5): track 61.0 -> 0.00 mm, vias 1 -> 0
- net GND: track 2643.1 -> 2644.5 mm
- net Net-(U1001AL-NC_OPEN28): track 1.41 -> 0.00 mm
- net +1.2V_YC_RC_VDDIO: track 0.00 -> 1.41 mm, vias 0 -> 2
- net unconnected-(U1001E-RC_VDDIO-PadE37): track 0.71 -> 0.00 mm, vias 1 -> 0
- net unconnected-(U1001A-RC_VDDIO-PadA40): track 0.71 -> 0.00 mm, vias 1 -> 0
- net unconnected-(Q2401-B-Pad1): track 0.54 -> 0.00 mm, vias 1 -> 0
