File: cok-001/sata.kicad_sch (KiCad schematic)
At the start: 56 parts, among them J3401 Conn_01x22_Pin, Q3401 DTC144E, Q3404 DTC144E

Commit message: southbridge
Connections:
- net SB_ATA1_DD12: now reaches R3425.1
- net SB_ATA1_DD10: now reaches R3429.1
- net SB_ATA1_DD13: now reaches R3423.1
- net SB_ATA1_DD11: now reaches R3427.1
- net SB_ATA1_DD0: now reaches R3420.1
- net SB_ATA1_DD7: now reaches R3434.1
- net SB_ATA1_DD3: now reaches R3426.1
- net SB_ATA1_DD1: now reaches R3422.1
- net SB_ATA1_DD14: now reaches R3421.1
- net SB_ATA1_DD5: now reaches R3430.1
- net SB_ATA1_DD15: now reaches R3419.1
- net SB_ATA1_DD8: now reaches R3433.1
- net SB_ATA1_DD2: now reaches R3424.1
- net SB_ATA1_DD9: now reaches R3431.1
- net SB_ATA1_DD6: now reaches R3432.1
- net SB_ATA1_DD4: now reaches R3428.1

Commit message: sc
Parts:
- added C3404: 0.1u 10V, Capacitor_SMD:C_0402_1005Metric, symbol Device:C
- added R3402, R3403, R3404, R3405, R3406, R3410: 33, Resistor_SMD:R_0402_1005Metric, symbol Device:R_US
- added R3407, R3408, R3409: 22, Resistor_SMD:R_0402_1005Metric, symbol Device:R_US
- added R3411, R3412: 10k, Resistor_SMD:R_0402_1005Metric, symbol Device:R_US
- added R3413: 5600, Resistor_SMD:R_0402_1005Metric, symbol Device:R_US
- added R3414, R3415, R3416: 82, Resistor_SMD:R_0402_1005Metric, symbol Device:R_US
- added R3417: 4700, Resistor_SMD:R_0402_1005Metric, symbol Device:R_US
- added TP3401, TP3402: TestPoint, TestPoint:TestPoint_Pad_D1.5mm, symbol Connector:TestPoint
Connections:
- net GND: now also C3404.2, R3411.2, R3412.2, R3413.2
- net SB_ATA1_DA2: now also R3404.1
- net SB_ATA1_DD7: now also R3411.1
- net at R3436.1: now also R3415.2, R3417.2
- net at C3421.1, R3466.1, R3467.2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: now also R3410.2
- net at R3437.1: now also R3413.1, R3416.2
- net at R3435.1: now also R3414.2
- net at C3408.1, U3401.41 (VDD), U3401.56 (VDD)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: now also C3404.1
- net ~{SB_RESET}: now reaches R3451.1, U3401.17 (RST_n)
- net at U3401.43 (UAI): now also TP3402.1
- net at U3401.45 (UAO): now also TP3401.1
- net at U3401.47 (H_CS1_n): now also R3402.2
- net at U3401.48 (H_CS0_n): now also R3403.2
- net at U3401.49 (H_DA2): now also R3404.2
- net at U3401.50 (H_DA0): now also R3405.2
- net at U3401.51 (H_DA1): now also R3406.2
- net at U3401.54 (H_DMACK_n): now also R3407.2
- net at U3401.58 (H_DIOR_n): now also R3408.2
- net at U3401.59 (H_DIOW_n): now also R3409.2
- new net SB_ATA1_DA0: R3405.1
- new net SB_ATA1_DA1: R3406.1
- new net SB_ATA1_DMARQ: R3416.1
- new net SB_ATA1_INTRQ: R3412.1, R3414.1
- new net SB_ATA1_IORDY: R3415.1
- new net ~{SB_ATA1_CS0}: R3403.1
- new net ~{SB_ATA1_CS1}: R3402.1
- new net ~{SB_ATA1_DIOR}: R3408.1
- new net ~{SB_ATA1_DIOW}: R3409.1
- new net ~{SB_ATA1_DMACK}: R3407.1
- new net ~{SB_ATA1_RESET}: R3410.1
- no-connect marks 0 -> 1
Other:
- moved on the sheet: R3423, R3424, R3425, R3426, R3427, R3428, R3429, R3430, R3431, R3432, R3433, R3434

Commit message: update to 9
Changed lines of the file:
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@@
 (kicad_sch
-	(version 20231120)
+	(version 20250114)
 	(generator "eeschema")
-	(generator_version "8.0")
+	(generator_version "9.0")
 	(paper "A4")
 	(junction

Commit message: sata crystal
Parts:
- added C3417: 0.1u 10V, Capacitor_SMD:C_0402_1005Metric, symbol Device:C
- added C3418, C3419: 15p 50V, Capacitor_SMD:C_0402_1005Metric, symbol Device:C
- added D3401: CL-196TLY-CD-T, Diode_SMD:D_0603_1608Metric, symbol Device:LED
- added FB3402: FerriteBead_Small, Resistor_SMD:R_0603_1608Metric, symbol Device:FerriteBead_Small
- added Q3402, Q3403: DTC144E, Package_TO_SOT_SMD:SOT-323_SC-70, symbol Transistor_BJT:DTC144E
- added R3460, R3468: XX, Resistor_SMD:R_0402_1005Metric, symbol Device:R_US
- added R3461: 220, Resistor_SMD:R_0402_1005Metric, symbol Device:R_US
- added TH3401: Polyfuse, Fuse:Fuse_1210_3225Metric, symbol Device:Polyfuse
- added Y3402: 25MHz, Crystal:Crystal_SMD_Abracon_ABM8G-4Pin_3.2x2.5mm, symbol Device:Crystal_GND24
Connections:
- net GND: now also C3417.2, C3418.1, C3419.1, Q3402.2 (E), Q3403.2 (E), Y3402.2
- net at C3405.1, FB3401.1, R3438.1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: now also R3468.2, Y3402.4
- net at J3401.P7 (5Vp), J3401.P8 (5V), J3401.P9 (5V): now also C3417.1, FB3402.2
- net at U3401.22 (XTALIN/OSC): now also C3419.2, R3460.2, R3468.1, Y3402.3
- net at U3401.23 (XTALOUT): now also R3460.1, R3461.1
- new net: D3401.1 (K), Q3403.3 (C)
- new net: C3418.2, R3461.2, Y3402.1
- new net: FB3402.1, TH3401.2
- new net +5V_HDD: TH3401.1
- no-connect marks 1 -> 7

Commit message: inductor
Parts:
- FB3401, FB3402: footprint Resistor_SMD:R_0603_1608Metric -> Inductor_SMD:L_0603_1608Metric
Changed lines of the file:
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@@
 			)
 		)
-		(property "Footprint" "Resistor_SMD:R_0603_1608Metric"
+		(property "Footprint" "Inductor_SMD:L_0603_1608Metric"
 			(at 162.56 27.178 90)
 			(effects
@@
 			)
 		)
-		(property "Footprint" "Resistor_SMD:R_0603_1608Metric"
+		(property "Footprint" "Inductor_SMD:L_0603_1608Metric"
 			(at 125.73 77.978 90)
 			(effects

Commit message: rdy
Parts:
- added R3459: 330, Resistor_SMD:R_0402_1005Metric, symbol Device:R_US
- added R3462: 10k, Resistor_SMD:R_0402_1005Metric, symbol Device:R_US
Connections:
- net at D3401.2 (A): now also R3459.1
- net at Q3403.1 (B): now also Q3402.3 (C), R3462.1
Other:
- moved on the sheet: D3401, Q3402, Q3403
Changed lines of the file:
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@@
 	)
 	(junction
+		(at 33.02 30.48)
+		(diameter 0)
+		(color 0 0 0 0)
+	)
+	(junction
 		(at 137.16 125.73)
 		(diameter 0)
@@
 	(symbol
 		(lib_id "power:GND")
-		(at 58.42 30.48 0)
+		(at 24.13 35.56 0)
 		(unit 1)
 		(exclude_from_sim no)
@@
 		(fields_autoplaced yes)
 		(property "Reference" "#PWR0302"
-			(at 58.42 36.83 0)
+			(at 24.13 41.91 0)
 			(effects
 				(font
@@
 		)
 		(property "Value" "GND"
-			(at 58.42 35.56 0)
+			(at 24.13 40.64 0)
 			(effects
 				(font
@@
 		)
 		(property "Footprint" ""
-			(at 58.42 30.48 0)
+			(at 24.13 35.56 0)
 			(effects
 				(font
@@
 		)
 		(property "Datasheet" ""
-			(at 58.42 30.48 0)
+			(at 24.13 35.56 0)
 			(effects
 				(font
@@
 		)
 		(property "Description" "Power symbol creates a global label with name \"GND\" , ground"
-			(at 58.42 30.48 0)
+			(at 24.13 35.56 0)
 			(effects
 				(font
@@
 	(symbol
 		(lib_id "Device:LED")
-		(at 58.42 16.51 270)
+		(at 24.13 21.59 270)
 		(mirror x)
 		(unit 1)
@@
 		(dnp no)
 		(property "Reference" "D3401"
-			(at 54.61 16.8274 90)
+			(at 20.32 21.9074 90)
 			(effects
 				(font
@@
 		)
 		(property "Value" "CL-196TLY-CD-T"
-			(at 54.61 19.3674 90)
+			(at 20.32 24.4474 90)
 			(effects
 				(font
@@
 		)
 		(property "Footprint" "Diode_SMD:D_0603_1608Metric"
-			(at 58.42 16.51 0)
+			(at 24.13 21.59 0)
 			(effects
 				(font
@@
 		)
 		(property "Datasheet" "~"
-			(at 58.42 16.51 0)
+			(at 24.13 21.59 0)
 			(effects
 				(font
@@
 		)
 		(property "Description" "Light emitting diode"
-			(at 58.42 16.51 0)
+			(at 24.13 21.59 0)
 			(effects
 				(font
@@
 		)
 		(property "Sim.Pins" "1=K 2=A"
-			(at 58.42 16.51 0)
+			(at 24.13 21.59 0)
 			(effects
 				(font
@@
 	(symbol
 		(lib_id "Device:R_US")
+		(at 24.13 13.97 180)
+		(unit 1)
+		(exclude_from_sim no)
+		(in_bom yes)
+		(on_board yes)
+		(dnp no)
+		(property "Reference" "R3459"
+			(at 26.67 12.6999 0)
+			(effects
+				(font
+					(size 1.27 1.27)
+				)
+				(justify right)
+			)
+		)
+		(property "Value" "330"
+			(at 26.67 15.2399 0)
+			(effects
+				(font
+					(size 1.27 1.27)
+				)
+				(justify right)
+			)
+		)
+		(property "Footprint" "Resistor_SMD:R_0402_1005Metric"
+			(at 23.114 13.716 90)
+			(effects
+				(font
+					(size 1.27 1.27)
+				)
+				(hide yes)
+			)
+		)
+		(property "Datasheet" "~"
+			(at 24.13 13.97 0)
+			(effects
+				(font
+					(size 1.27 1.27)
+				)
+				(hide yes)
+			)
+		)
+		(property "Description" "Resistor, US symbol"
+			(at 24.13 13.97 0)
+			(effects
+				(font
+					(size 1.27 1.27)
+				)
+				(hide yes)
+			)
+		)
+		(pin "2"
+		)
+		(pin "1"
+		)
+		(instances
+			(project "cok-001"
+				(path "/976eb78d-8215-4cc0-9d72-f9d535c7970b/f39dff98-fe81-4ce8-ac1c-e51ce9d90ef4"
+					(reference "R3459")
+					(unit 1)
+				)
+			)
+		)
+	)
+	(symbol
+		(lib_id "Device:R_US")
 		(at 50.8 100.33 90)
 		(unit 1)
@@
 	(symbol
 		(lib_id "power:GND")
-		(at 45.72 43.18 0)
+		(at 33.02 40.64 0)
 		(unit 1)
 		(exclude_from_sim no)
@@
 		(fields_autoplaced yes)
 		(property "Reference" "#PWR0301"
-			(at 45.72 49.53 0)
+			(at 33.02 46.99 0)
 			(effects
 				(font
@@
 		)
 		(property "Value" "GND"
-			(at 45.72 48.26 0)
+			(at 33.02 45.72 0)
 			(effects
 				(font
@@
 		)
 		(property "Footprint" ""
-			(at 45.72 43.18 0)
+			(at 33.02 40.64 0)
 			(effects
 				(font
@@
 		)
 		(property "Datasheet" ""
-			(at 45.72 43.18 0)
+			(at 33.02 40.64 0)
 			(effects
 				(font
@@
 		)
 		(property "Description" "Power symbol creates a global label with name \"GND\" , ground"
-			(at 45.72 43.18 0)
+			(at 33.02 40.64 0)
 			(effects
 				(font
@@
 	)
 	(symbol
+		(lib_id "Device:R_US")
+		(at 33.02 26.67 180)
+		(unit 1)
+		(exclude_from_sim no)
+		(in_bom yes)
+		(on_board yes)
+		(dnp no)
+		(property "Reference" "R3462"
+			(at 35.56 25.3999 0)
+			(effects
+				(font
+					(size 1.27 1.27)
+				)
+				(justify right)
+			)
+		)
+		(property "Value" "10k"
+			(at 35.56 27.9399 0)
+			(effects
+				(font
+					(size 1.27 1.27)
+				)
+				(justify right)
+			)
+		)
+		(property "Footprint" "Resistor_SMD:R_0402_1005Metric"
+			(at 32.004 26.416 90)
+			(effects
+				(font
+					(size 1.27 1.27)
+				)
+				(hide yes)
+			)
+		)
+		(property "Datasheet" "~"
+			(at 33.02 26.67 0)
+			(effects
+				(font
+					(size 1.27 1.27)
+				)
+				(hide yes)
+			)
+		)
+		(property "Description" "Resistor, US symbol"
+			(at 33.02 26.67 0)
+			(effects
+				(font
+					(size 1.27 1.27)
+				)
+				(hide yes)
+			)
+		)
+		(pin "2"
+		)
+		(pin "1"
+		)
+		(instances
+			(project "cok-001"
+				(path "/976eb78d-8215-4cc0-9d72-f9d535c7970b/f39dff98-fe81-4ce8-ac1c-e51ce9d90ef4"
+					(reference "R3462")
+					(unit 1)
+				)
+			)
+		)
+	)
+	(symbol
 		(lib_id "Device:Crystal_GND24")
 		(at 160.02 109.22 270)
@@
 	(symbol
 		(lib_id "Transistor_BJT:DTC144E")
-		(at 60.96 25.4 0)
+		(at 26.67 30.48 0)
 		(mirror y)
 		(unit 1)
@@
 		(fields_autoplaced yes)
 		(property "Reference" "Q3403"
-			(at 55.88 24.1299 0)
+			(at 21.59 29.2099 0)
 			(effects
 				(font
@@
 		)
 		(property "Value" "DTC144E"
-			(at 55.88 26.6699 0)
+			(at 21.59 31.7499 0)
 			(effects
 				(font
@@
 		)
 		(property "Footprint" "Package_TO_SOT_SMD:SOT-323_SC-70"
-			(at 60.96 25.4 0)
+			(at 26.67 30.48 0)
 			(effects
 				(font
@@
 		)
 		(property "Datasheet" ""
-			(at 60.96 25.4 0)
+			(at 26.67 30.48 0)
 			(effects
 				(font
@@
 		)
 		(property "Description" "Digital NPN Transistor, 47k/47k, SOT-23"
-			(at 60.96 25.4 0)
+			(at 26.67 30.48 0)
 			(effects
 				(font
@@
 	(symbol
 		(lib_id "Transistor_BJT:DTC144E")
-		(at 48.26 38.1 0)
+		(at 35.56 35.56 0)
 		(mirror y)
 		(unit 1)
@@
 		(fields_autoplaced yes)
 		(property "Reference" "Q3402"
-			(at 43.18 36.8299 0)
+			(at 30.48 34.2899 0)
 			(effects
 				(font
@@
 		)
 		(property "Value" "DTC144E"
-			(at 43.18 39.3699 0)
+			(at 30.48 36.8299 0)
 			(effects
 				(font
@@
 		)
 		(property "Footprint" "Package_TO_SOT_SMD:SOT-323_SC-70"
-			(at 48.26 38.1 0)
+			(at 35.56 35.56 0)
 			(effects
 				(font
@@
 		)
 		(property "Datasheet" ""
-			(at 48.26 38.1 0)
+			(at 35.56 35.56 0)
 			(effects
 				(font
@@
 		)
 		(property "Description" "Digital NPN Transistor, 47k/47k, SOT-23"
-			(at 48.26 38.1 0)
+			(at 35.56 35.56 0)
 			(effects
 				(font
