File: cok-001/usb.kicad_sch (KiCad schematic)
At the start: 37 parts, among them J3301 USB_A_Stacked, J3302 USB_A_Stacked, U3302 BU9869W

Commit message: seperate out
Parts:
- U3303, U3304: footprint Package_SO:SOIC-8_3.9x4.9mm_P1.27mm -> Package_SO:SSOP-8_3.9x5.05mm_P1.27mm
Changed lines of the file:
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@@
 			)
 		)
-		(property "Footprint" "Package_SO:SOIC-8_3.9x4.9mm_P1.27mm"
+		(property "Footprint" "Package_SO:SSOP-8_3.9x5.05mm_P1.27mm"
 			(at 181.61 48.26 0)
 			(effects
@@
 			)
 		)
-		(property "Footprint" "Package_SO:SOIC-8_3.9x4.9mm_P1.27mm"
+		(property "Footprint" "Package_SO:SSOP-8_3.9x5.05mm_P1.27mm"
 			(at 175.26 118.11 0)
 			(effects

Commit message: update to 9
Changed lines of the file:
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@@
 (kicad_sch
-	(version 20231120)
+	(version 20250114)
 	(generator "eeschema")
-	(generator_version "8.0")
+	(generator_version "9.0")
 	(paper "A4")
 	(junction

Commit message: led
Parts:
- added D3301, D3302, D3303, D3304, D3305: XX, Diode_SMD:D_0603_1608Metric, symbol Device:LED
- added L3303, L3304: L_Iron_Coupled_Small_1243, Inductor_SMD:L_CommonModeChoke_Coilcraft_0805USB, symbol Device:L_Iron_Coupled_Small_1243
- added R3306, R3307, R3308, R3309, R3310: XX, Resistor_SMD:R_0402_1005Metric, symbol Device:R_US
Connections:
- net GND: now also R3306.1, R3307.1, R3308.1, R3309.1, R3310.1
- net at J3301.2 (D1-), TP9508.1: now also L3303.4
- net at J3301.3 (D1+), TP9507.1: now also L3303.1
- net at J3301.6 (D2-), TP9506.1: now also L3304.4
- net at J3301.7 (D2+), TP9505.1: now also L3304.1
- net at R3363.2: now also L3303.2
- net at U3302.1 (CS), U3305.61 (AMBER1/EE_CS): now also D3304.2 (A)
- net at U3302.4 (DO), U3305.48 (GREEN2/EE_DO): now also D3303.2 (A)
- net at U3305.34 (GREEN4): now also D3301.2 (A)
- net at U3305.44 (GREEN3): now also D3302.2 (A)
- net at U3305.53 (PGANG/SUSPND): now also D3305.2 (A)
- net at R3362.2: now also L3303.3
- net at R3360.2: now also L3304.3
- net at R3361.2: now also L3304.2
- new net: D3304.1 (K), R3309.2
- new net: D3303.1 (K), R3308.2
- new net: D3302.1 (K), R3307.2
- new net: D3305.1 (K), R3310.2
- new net: D3301.1 (K), R3306.2
- no-connect marks 7 -> 9
Other:
- moved on the sheet: C3301, C3309, C3311, C3313, C3314, C3328, J3301, R3328, R3329, R3360, R3361, R3362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

Commit message: switching regulator
Parts:
- added R3303: 1k, Resistor_SMD:R_0402_1005Metric, symbol Device:R_US
- added Y3301: 12MHz, Crystal:Crystal_SMD_Abracon_ABM8G-4Pin_3.2x2.5mm, symbol Device:Crystal_GND24
Connections:
- net at U3305.20 (X1): now also Y3301.3
- net at U3305.21 (X2): now also R3303.2
- new net: R3303.1, Y3301.1
Changed lines of the file:
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@@
 	(wire
 		(pts
+			(xy 48.26 170.18) (xy 48.26 185.42)
+		)
+		(stroke
+			(width 0)
+			(type default)
+		)
+	)
+	(wire
+		(pts
 			(xy 254 92.71) (xy 232.41 92.71)
 		)
@@
 	(wire
 		(pts
+			(xy 45.72 170.18) (xy 48.26 170.18)
+		)
+		(stroke
+			(width 0)
+			(type default)
+		)
+	)
+	(wire
+		(pts
 			(xy 173.99 102.87) (xy 209.55 102.87)
 		)
@@
 	(wire
 		(pts
+			(xy 40.64 185.42) (xy 40.64 163.83)
+		)
+		(stroke
+			(width 0)
+			(type default)
+		)
+	)
+	(wire
+		(pts
 			(xy 173.99 171.45) (xy 173.99 102.87)
 		)
@@
 	(wire
 		(pts
+			(xy 45.72 152.4) (xy 45.72 162.56)
+		)
+		(stroke
+			(width 0)
+			(type default)
+		)
+	)
+	(wire
+		(pts
 			(xy 106.68 52.07) (xy 106.68 41.91)
 		)
@@
 	(wire
 		(pts
+			(xy 43.18 163.83) (xy 43.18 152.4)
+		)
+		(stroke
+			(width 0)
+			(type default)
+		)
+	)
+	(wire
+		(pts
 			(xy 93.98 82.55) (xy 68.58 82.55)
 		)
@@
 	(wire
 		(pts
+			(xy 40.64 163.83) (xy 43.18 163.83)
+		)
+		(stroke
+			(width 0)
+			(type default)
+		)
+	)
+	(wire
+		(pts
 			(xy 166.37 163.83) (xy 166.37 60.96)
 		)
@@
 	(symbol
 		(lib_id "Device:R_US")
+		(at 45.72 166.37 180)
+		(unit 1)
+		(exclude_from_sim no)
+		(in_bom yes)
+		(on_board yes)
+		(dnp no)
+		(property "Reference" "R3303"
+			(at 48.26 165.0999 0)
+			(effects
+				(font
+					(size 1.27 1.27)
+				)
+				(justify right)
+			)
+		)
+		(property "Value" "1k"
+			(at 48.26 167.6399 0)
+			(effects
+				(font
+					(size 1.27 1.27)
+				)
+				(justify right)
+			)
+		)
+		(property "Footprint" "Resistor_SMD:R_0402_1005Metric"
+			(at 44.704 166.116 90)
+			(effects
+				(font
+					(size 1.27 1.27)
+				)
+				(hide yes)
+			)
+		)
+		(property "Datasheet" "~"
+			(at 45.72 166.37 0)
+			(effects
+				(font
+					(size 1.27 1.27)
+				)
+				(hide yes)
+			)
+		)
+		(property "Description" "Resistor, US symbol"
+			(at 45.72 166.37 0)
+			(effects
+				(font
+					(size 1.27 1.27)
+				)
+				(hide yes)
+			)
+		)
+		(pin "1"
+		)
+		(pin "2"
+		)
+		(instances
+			(project "cok-001"
+				(path "/976eb78d-8215-4cc0-9d72-f9d535c7970b/9b5bec78-d40a-47da-955b-e0a66a63c4fa"
+					(reference "R3303")
+					(unit 1)
+				)
+			)
+		)
+	)
+	(symbol
+		(lib_id "Device:R_US")
 		(at 121.92 153.67 0)
 		(mirror x)
@@
 					(unit 1)
 				)
+			)
+		)
+	)
+	(symbol
+		(lib_id "Device:Crystal_GND24")
+		(at 44.45 185.42 180)
+		(unit 1)
+		(exclude_from_sim no)
+		(in_bom yes)
+		(on_board yes)
+		(dnp no)
+		(property "Reference" "Y3301"
+			(at 53.086 189.23 90)
+			(effects
+				(font
+					(size 1.27 1.27)
+				)
+			)
+		)
+		(property "Value" "12MHz"
+			(at 50.546 189.23 90)
+			(effects
+				(font
+					(size 1.27 1.27)
+				)
+			)
+		)
+		(property "Footprint" "Crystal:Crystal_SMD_Abracon_ABM8G-4Pin_3.2x2.5mm"
+			(at 44.45 185.42 0)
+			(effects
+				(font
+					(size 1.27 1.27)
+				)
+				(hide yes)
+			)
+		)
+		(property "Datasheet" "~"
+			(at 44.45 185.42 0)
+			(effects
+				(font
+					(size 1.27 1.27)
+				)
+				(hide yes)
+			)
+		)
+		(property "Description" "Four pin crystal, GND on pins 2 and 4"
+			(at 44.45 185.42 0)
+			(effects
+				(font
+					(size 1.27 1.27)
+				)
+				(hide yes)
+			)
+		)
+		(pin "4"
+		)
+		(pin "1"
+		)
+		(pin "2"
+		)
+		(pin "3"
+		)
+		(instances
+			(project "cok-001"
+				(path "/976eb78d-8215-4cc0-9d72-f9d535c7970b/9b5bec78-d40a-47da-955b-e0a66a63c4fa"
+					(reference "Y3301")
+					(unit 1)
+				)

Commit message: rdy
Parts:
- added C3324, C3325: 220u 10V, Capacitor_Tantalum_SMD:CP_EIA-6032-28_Kemet-C, symbol Device:C_Polarized_US
- added D3316, D3317, D3318, D3319, D3320, D3321, D3322, D3323: EDZCTE616, Diode_SMD:D_SOD-923, symbol Device:D_Zener
- added R3342, R3345: 0, Resistor_SMD:R_0402_1005Metric, symbol Device:R_US
- added R3343, R3346: XX, Resistor_SMD:R_0402_1005Metric, symbol Device:R_US
- added R3350: 0, Resistor_SMD:R_0603_1608Metric, symbol Device:R_US
- added R3356, R3357, R3358, R3359: 10k, Resistor_SMD:R_0402_1005Metric, symbol Device:R_US
- added TH3302: Thermistor, symbol Device:Thermistor
- L3301, L3302, L3303, L3304: value L_Iron_Coupled_Small_1243 -> 0uH
- U3303, U3304: value ~ -> BD6517F
Connections:
- net GND: now also C3324.2, C3325.2, D3316.2 (A), D3317.2 (A), D3318.2 (A), D3319.2 (A), D3320.2 (A), D3321.2 (A), D3322.2 (A), D3323.2 (A)
- net at J3302.2 (D1-), L3301.4, TP9512.1: now also D3322.1 (K)
- net at J3302.3 (D1+), L3301.1, TP9511.1: now also D3323.1 (K)
- net at J3302.6 (D2-), L3302.4, TP9510.1: now also D3321.1 (K)
- net at J3302.7 (D2+), L3302.1, TP9509.1: now also D3320.1 (K)
- net at J3301.1 (VBUS1), TP9520.1, U3303.5 (OUTB): now also C3324.1
- net at J3301.2 (D1-), L3303.4, TP9508.1: now also D3319.1 (K)
- net at J3301.3 (D1+), L3303.1, TP9507.1: now also D3318.1 (K)
- net at J3301.5 (VBUS2), TP9527.1, U3303.8 (OUTA): now also C3325.1
- net at J3301.6 (D2-), L3304.4, TP9506.1: now also D3317.1 (K)
- net at J3301.7 (D2+), L3304.1, TP9505.1: now also D3316.1 (K)
- net at U3304.2 (FLAGA): now also R3358.2
- net at U3304.3 (FLAGB): now also R3359.2
- net at U3304.4 (CTRLB): now also R3342.2, R3343.2
- net at C3316.1, U3304.7 (VDD): now also R3350.1
- net at U3303.1 (CTRLA): now also R3345.2, R3346.2
- net at U3303.2 (FLAGA): now also R3356.2
- net at U3303.3 (FLAGB): now also R3357.2
- new net: R3350.2, TH3302.2
- new net +5V_USB: TH3302.1
- new net H4_OVC1: R3356.1
- new net H4_OVC2: R3357.1
- new net H4_OVC3: R3358.1
- new net H4_OVC4: R3359.1
- new net H4_PWREN1: R3343.1, R3346.1
- new net H4_PWREN2: R3345.1
- new net H4_PWREN4: R3342.1
Other:
- moved on the sheet: C3316, L3301, L3303, L3304, TP9505, TP9511, TP9512, U3304
