File: cok-001/usb.kicad_sch (KiCad schematic)
At the start: 71 parts, among them J3301 USB_A_Stacked, J3302 USB_A_Stacked, U3302 BU9869W, U3303 BD6517F, U3304 BD6517F, Y3301 12MHz

Commit message: update 10
Parts:
- U3305: value ~ -> (none)

Commit message: lf
Parts:
- renumbered L3303 to LF3303, L3304 to LF3304
Changed lines of the file:
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@@
 		(in_pos_files yes)
 		(dnp no)
-		(property "Reference" "L3304"
+		(property "Reference" "LF3304"
 			(at 210.82 109.855 0)
 			(show_name no)
@@
 			(project "cok-001"
 				(path "/976eb78d-8215-4cc0-9d72-f9d535c7970b/9b5bec78-d40a-47da-955b-e0a66a63c4fa"
-					(reference "L3304")
+					(reference "LF3304")
 					(unit 1)
 				)
@@
 		(in_pos_files yes)
 		(dnp no)
-		(property "Reference" "L3303"
+		(property "Reference" "LF3303"
 			(at 210.82 100.965 0)
 			(show_name no)
@@
 			(project "cok-001"
 				(path "/976eb78d-8215-4cc0-9d72-f9d535c7970b/9b5bec78-d40a-47da-955b-e0a66a63c4fa"
-					(reference "L3303")
-					(unit 1)
-				)
+					(reference "LF3303")
+					(unit 1)
+				)
