File: cok-001/xcgclock.kicad_sch (KiCad schematic)
At the start: 83 parts, among them U5001 ICS1493G, U5002 ICS9218, U5003 ICS9218, U5004 ICS9214, U5006 PST36XX, Y5001 14.31818MHz

Commit message: update 10
Parts:
- U5005: value ~ -> (none)
