File: PCI_Breakout/PCI_Breakout.kicad_sch (KiCad schematic)
At the start: 2 parts, among them J1 凹

Commit message: pci
Parts:
- added J3: Conn_01x03_Pin, Connector_PinHeader_2.54mm:PinHeader_1x03_P2.54mm_Vertical, symbol Connector:Conn_01x03_Pin
- added J4: Conn_01x04_Pin, Connector_PinHeader_2.54mm:PinHeader_1x04_P2.54mm_Horizontal, symbol Connector:Conn_01x04_Pin
- added JP1: Jumper_3_Open, Jumper:SolderJumper-3_P2.0mm_Open_TrianglePad1.0x1.5mm, symbol Jumper:Jumper_3_Open
Connections:
- net +3.3V_BRIDGE is gone; now on net +3.3V: J1.2 (Pin_2)
- net +3.3V: now also JP1.3 (B)
- net +5V: now also J4.1 (Pin_1)
- net GND: now also J3.1 (Pin_1), J4.2 (Pin_2), J4.3 (Pin_3), JP1.1 (A)
- net SB_SIO0_RXD: now also J3.3 (Pin_3)
- net SB_SIO0_TXD: now also J3.2 (Pin_2)
- net SB_PCI_IDSEL: now reaches J1.34 (Pin_34)
- net SB_PCI_IDSEL: now also J2.48 (IDSEL)
- net at J2.104 (M66EN): now also JP1.2 (C)
- new net +12V: J4.4 (Pin_4)
