File: PCI_Breakout/PCI_Breakout.kicad_pcb (KiCad board)
At the start: 2 copper layers, 74 x 36 mm, 2 parts, among them J1 凹

Commit message: pci
Parts:
- added J3: Conn_01x03_Pin, Connector_PinHeader_2.54mm:PinHeader_1x03_P2.54mm_Vertical, F.Cu at (115.6, 97.8)
- added J4: Conn_01x04_Pin, Connector_PinHeader_2.54mm:PinHeader_1x04_P2.54mm_Horizontal, F.Cu at (151.2, 97.4)
- added JP1: Jumper_3_Open, Jumper:SolderJumper-3_P2.0mm_Open_TrianglePad1.0x1.5mm, F.Cu at (113.5, 117.5)
- moved J1 1.12 mm to (130.8, 106.7)
- moved J2 1.12 mm to (130.8, 106.7)
Connections:
- J1 pad 2: +3.3V_BRIDGE -> +3.3V
- J1 pad 34: unconnected-(J1-Pin_34-Pad34) -> SB_PCI_IDSEL
- J2 pad 104: unconnected-(J2-M66EN-Pad104) -> Net-(J2-M66EN)
- J2 pad 48: unconnected-(J2-IDSEL-Pad48) -> SB_PCI_IDSEL
Routing:
- net GND: track 0.00 -> 139.5 mm, vias 0 -> 19
- net +3.3V: track 0.00 -> 76.2 mm, vias 0 -> 1
- net +5V: track 0.00 -> 57.6 mm
- net SB_SIO0_RXD: track 0.00 -> 20.9 mm
- net SB_SIO0_TXD: track 0.00 -> 16.8 mm
- net SB_PCI_INTB: track 0.00 -> 16.7 mm, vias 0 -> 1
- net SB_PCI_INTA: track 0.00 -> 14.2 mm, vias 0 -> 1
- net SB_PCI0_CLK: track 0.00 -> 13.5 mm, vias 0 -> 1
- net SB_PCI_REQ0: track 0.00 -> 13.1 mm, vias 0 -> 1
- net SB_PCI_RST: track 0.00 -> 12.7 mm, vias 0 -> 1
- net SB_PCI_PAR: track 0.00 -> 12.2 mm, vias 0 -> 1
- net SB_PCI_AD31: track 0.00 -> 12.1 mm, vias 0 -> 1
- net SB_PCI_GNT0: track 0.00 -> 11.7 mm, vias 0 -> 1
- net SB_PCI_AD29: track 0.00 -> 11.6 mm, vias 0 -> 1
- net SB_PCI_PME: track 0.00 -> 11.4 mm, vias 0 -> 1
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Other:
- board size 74 x 36 mm -> 70 x 32 mm
- board text added: "5V"
- board text added: "GND"
- board text added: "RX"
- board text added: "TX"

Commit message: ide breakout prod
Parts:
- moved JP1 3.82 mm to (114.2, 121.2)
Routing:
- net Net-(J2-M66EN): track 7.10 -> 10.5 mm
- net +3.3V: track 76.2 -> 79.4 mm
Other:
- board text added: "PS3 PCI"
- board text added: "miniPCI"
Changed lines of the file:
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@@
 			(outputformat 1)
 			(mirror no)
-			(drillshape 1)
+			(drillshape 0)
 			(scaleselection 1)
-			(outputdirectory "")
+			(outputdirectory "production")
 		)
 	)
@@
 	(footprint "Jumper:SolderJumper-3_P2.0mm_Open_TrianglePad1.0x1.5mm"
 		(layer "F.Cu")
-		(at 113.5 117.5)
+		(at 114.25 121.25)
 		(descr "SMD Solder Jumper, 1x1.5mm Triangular Pads, 0.3mm gap, open")
 		(tags "solder jumper open")
@@
 	)
 	(gr_text "GND"
-		(at 114.5 95.5 0)
+		(at 117.2 95 180)
 		(layer "F.SilkS")
 		(effects
@@
 		)
 	)
+	(gr_text "miniPCI"
+		(at 121 120.5 0)
+		(layer "F.SilkS")
+		(effects
+			(font
+				(size 4 4)
+				(thickness 0.5)
+			)
+			(justify left bottom)
+		)
+	)
 	(gr_text "TX"
-		(at 112 95.5 0)
+		(at 113.8 95 180)
 		(layer "F.SilkS")
 		(effects
@@
 	)
 	(gr_text "RX"
-		(at 109 95.5 0)
+		(at 111.4 95 180)
 		(layer "F.SilkS")
 		(effects
@@
 		)
 	)
+	(gr_text "PS3 PCI"
+		(at 140.75 99 0)
+		(layer "B.SilkS")
+		(effects
+			(font
+				(size 3 3)
+				(thickness 0.5)
+				(bold yes)
+			)
+			(justify left bottom mirror)
+		)
+	)
 	(segment
 		(start 125.21 102.58)
@@
 	)
 	(segment
+		(start 115.21 113.79)
+		(end 115.21 110.78)
+		(width 0.2)
+		(layer "F.Cu")
+		(net 1)
+	)
+	(segment
 		(start 115.21 106.79)
 		(end 117 105)
@@
 	)
 	(segment
+		(start 115.75 114)
+		(end 115.42 114)
+		(width 0.2)
+		(layer "F.Cu")
+		(net 1)
+	)
+	(segment
 		(start 122.81 102.58)
 		(end 122.81 101.539943)
@@
 	)
 	(segment
-		(start 115.21 113.79)
-		(end 115 114)
+		(start 115.42 114)
+		(end 115.21 113.79)
 		(width 0.2)
 		(layer "F.Cu")
@@
 	)
 	(segment
-		(start 115.21 110.78)
-		(end 115.21 113.79)
-		(width 0.2)
-		(layer "F.Cu")
-		(net 1)
-	)
-	(segment
 		(start 136.01 110.78)
 		(end 136.01 109.01)
@@
 	)
 	(via
-		(at 115 114)
+		(at 115.75 114)
 		(size 0.6)
 		(drill 0.3)
@@
 	)
 	(segment
-		(start 114.255 110.935)
-		(end 114.41 110.78)
+		(start 114.25 121.25)
+		(end 114.4 121.1)
 		(width 0.2)
 		(layer "F.Cu")
@@
 	)
 	(segment
-		(start 113.5 117.5)
-		(end 114.255 116.745)
+		(start 114.4 121.1)
+		(end 114.4 110.79)
 		(width 0.2)
 		(layer "F.Cu")
@@
 	)
 	(segment
-		(start 114.255 116.745)
-		(end 114.255 110.935)
+		(start 114.4 110.79)
+		(end 114.41 110.78)
 		(width 0.2)
 		(layer "F.Cu")
@@
 	)
 	(segment
-		(start 115.5 117.5)
-		(end 116.12 117.5)
+		(start 140.01 109.89)
+		(end 140.01 110.78)
 		(width 0.2)
 		(layer "F.Cu")
@@
 	)
 	(segment
-		(start 140.01 109.89)
-		(end 140.01 110.78)
+		(start 116.25 121.25)
+		(end 116.12 121.12)
 		(width 0.2)
 		(layer "F.Cu")
@@
 	)
 	(segment
-		(start 116.12 117.5)
-		(end 120.81 112.81)
-		(width 0.2)
-		(layer "F.Cu")
-		(net 81)
-	)
-	(segment
 		(start 142 106)
 		(end 143 106)
@@
 	)
 	(segment
+		(start 116.12 121.12)
+		(end 116.12 117.5)
+		(width 0.2)
+		(layer "F.Cu")
+		(net 81)
+	)
+	(segment
 		(start 148.41 102.58)
 		(end 148.41 106.09)
@@
 		(width 0.2)
 		(layer "F.Cu")
+		(net 81)
+	)
+	(segment
+		(start 116.12 117.5)
+		(end 120.81 112.81)
+		(width 0.2)
+		(layer "F.Cu")
