File: IDE_Breakout/IDE_Breakout.kicad_pcb (KiCad board)
At the start: 2 copper layers, 83.8 x 36.8 mm, 48 parts, among them J1 Conn_02x20_Odd_Even, J2 Conn_01x15, J3209 ATA Power, J3221 ATA0 for BD, Q1 DTC144E, Q2 DTC144E, Q3 DTC144E, Q4 DTC144E, Q5 DTC144E, Q6 DTC144E, Q7 DTC144E, Q8 DTC144E, SW1 Eject, SW2 In

Commit message: ide breakout prod
Parts:
- moved D1 2.99 mm to (105.0, 111.9)
- moved D2 2.99 mm to (105.0, 113.4)
- moved D3 2.99 mm to (105.0, 114.9)
- moved D4 2.99 mm to (105.0, 116.4)
- moved D5 2.99 mm to (105.0, 117.9)
- moved D6 2.99 mm to (105.0, 119.4)
- moved D7 2.99 mm to (105.0, 120.9)
- moved D8 2.99 mm to (105.0, 122.4)
- moved Q1 2.99 mm to (108.5, 112.4)
- moved Q5 2.99 mm to (108.5, 117.9)
- moved Q8 2.99 mm to (108.5, 122.4)
- moved R1 2.99 mm to (102.0, 111.9)
- moved R2 2.99 mm to (102.0, 113.4)
- moved R3 2.99 mm to (102.0, 114.9)
- moved R4 2.99 mm to (102.0, 116.4)
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Routing:
- net DISC_IN: track 47.9 -> 44.8 mm
- net DISC_OUT12_SW: track 49.5 -> 46.4 mm
- net MECHA_INT: track 51.8 -> 49.4 mm
- net MC_ALIVE: track 48.8 -> 46.5 mm
- net DISC_CHUCK: track 52.5 -> 50.3 mm
- net DISC_OUT8_SW: track 57.1 -> 55.1 mm
- net BD_LED: track 87.8 -> 86.3 mm
- net GND: track 382.8 -> 381.9 mm, vias 13 -> 16
Other:
- board text added: "12V"
- board text added: "3.3V"
- board text added: "5V"
- board text added: "BD 3.3V D_IN D_CH DSC8 DSC12 MC_A MCH_I"
- board text added: "PS3 BD-ROM TO IDE"
- board text added: "SATA POWER"
